File: Boards/RP2040-Standard-Design/RP2040 Standard Design.kicad_pcb (KiCad board)
At the start: 4 copper layers, 60 x 22 mm, 37 parts, among them J1 BM03B-SRSS-TBLFSN, J3 USB_C, SW1 SW_Push, SW3 SW_Push, U1 ESD7L5.0DT5G, U2 ST1L05APU33R

Commit message: Atualização footprint RP2040
Parts:
- added CV1: 1uF, CAP_GCM155_MUR:CAP_GCM155_MUR, F.Cu at (193.7, 43.9)
- added CV10: 100nF, CAP_GCM155_MUR:CAP_GCM155_MUR, F.Cu at (200.5, 46.0)
- added CV11: 100nF, CAP_GCM155_MUR:CAP_GCM155_MUR, F.Cu at (200.5, 48.2)
- added CV12: 100nF, CAP_GCM155_MUR:CAP_GCM155_MUR, F.Cu at (200.5, 50.4)
- added CV2: 100nF, CAP_GCM155_MUR:CAP_GCM155_MUR, F.Cu at (193.7, 46.0)
- added CV3: 1uF, CAP_GCM155_MUR:CAP_GCM155_MUR, F.Cu at (193.7, 48.2)
- added CV31: 1uF, CAP_GCM155_MUR:CAP_GCM155_MUR, F.Cu at (203.8, 43.9)
- added CV32: 100nF, CAP_GCM155_MUR:CAP_GCM155_MUR, F.Cu at (203.8, 46.0)
- added CV33: 4.7uF, GRM15x:GRM15x, F.Cu at (200.6, 71.0)
- added CV34: 4.7uF, GRM15x:GRM15x, F.Cu at (200.6, 73.6)
- added CV35: 1uF, CAP_GCM155_MUR:CAP_GCM155_MUR, F.Cu at (203.8, 48.2)
- added CV36: 100nF, CAP_GCM155_MUR:CAP_GCM155_MUR, F.Cu at (203.8, 50.4)
- added CV4: 100nF, CAP_GCM155_MUR:CAP_GCM155_MUR, F.Cu at (193.7, 50.4)
- added CV5: 100nF, CAP_GCM155_MUR:CAP_GCM155_MUR, F.Cu at (197.1, 43.9)
- added CV6: 1uF, CAP_GCM155_MUR:CAP_GCM155_MUR, F.Cu at (197.1, 46.0)
- added CV7: 100nF, CAP_GCM155_MUR:CAP_GCM155_MUR, F.Cu at (197.1, 48.2)
- added CV8: 100nF, CAP_GCM155_MUR:CAP_GCM155_MUR, F.Cu at (197.1, 50.4)
- added CV9: 100nF, CAP_GCM155_MUR:CAP_GCM155_MUR, F.Cu at (200.5, 43.9)
- added D1: PMEG2010ER, PMEG2010ER:SODFL3517X110N, F.Cu at (202.1, 68.1)
- added J2: BM03B-SRSS-TBLFSN, SWD_Con:CONN_BM03B-SRSS-TBLFSN_JST, F.Cu at (194.4, 64.6)
- added J4: DX07S016JA1R1500, USBC-DX07S016JA1:JAE_DX07S016JA1R1500, F.Cu at (181.7, 46.0)
- added MCU1: RP2040, Package_DFN_QFN:QFN-56-1EP_7x7mm_P0.4mm_EP3.2x3.2mm, F.Cu at (195.0, 57.0)
- added R1: 1k, RC0402N_VIS:RC0402N_VIS, F.Cu at (177.8, 53.4)
- added R10: 1k, RC0402N_VIS:RC0402N_VIS, F.Cu at (177.8, 59.9)
- added R16: 10k, RC0402N_VIS:RC0402N_VIS, F.Cu at (177.8, 62.0)
- added R17: 1k, RC0402N_VIS:RC0402N_VIS, F.Cu at (177.8, 64.2)
- added R18: 5k1, ERA6AEB101V:ERA6AEB101V, F.Cu at (203.3, 54.5)
- added R6: 27, KTR03EZPF27R0:RES_R0603_ROM, F.Cu at (204.2, 71.0)
- added R7: 27, KTR03EZPF27R0:RES_R0603_ROM, F.Cu at (204.2, 73.5)
- added R8: 100, RC0402N_VIS:RC0402N_VIS, F.Cu at (177.8, 55.5)
- added R9: 100, RC0402N_VIS:RC0402N_VIS, F.Cu at (177.8, 57.7)
- added RC2: 5k1, ERA6AEB101V:ERA6AEB101V, F.Cu at (203.3, 58.8)
- added S1: TL3305CF160QG, E-Switch_7mm:SW_TL3305CF160QG, F.Cu at (185.2, 55.3)
- added S2: TL3305CF160QG, E-Switch_7mm:SW_TL3305CF160QG, F.Cu at (185.2, 61.4)
- added U1: ST1L05APU33R, LDO ST1L05A:DFN_5APU33R_STM, F.Cu at (202.4, 64.0)
- added U2: W25Q128JVSIQ TR, NOR Flash:SOIC_208MIL_WIN, F.Cu at (184.7, 67.9)
- added U3: ESD7L5.0DT5G, ESD7L5-Diode:SOT-723_0P85X1P25_ONS, F.Cu at (182.1, 73.1)
- added XTAL1: ASE-12.000MHZ-LC-T, AS12MHz:ASE-3.2X2.5_ABR, F.Cu at (194.8, 69.8)
