File: Boards/RP2040-Standard-Design/RP2040 Standard Design.kicad_pcb (KiCad board)
At the start: 4 copper layers, 60 x 22 mm, 75 parts, among them J1 BM03B-SRSS-TBLFSN, J2 BM03B-SRSS-TBLFSN, J3 USB_C, J4 DX07S016JA1R1500, SW1 SW_Push, SW3 SW_Push, U1 ESD7L5.0DT5G, U1 ST1L05APU33R, U2 ST1L05APU33R, U2 W25Q128JVSIQ TR, U3 ESD7L5.0DT5G

Commit message: Mudança de nome das footprints
Parts:
- CV1, CV10, CV11, CV12, CV2, CV3, CV31, CV32, CV35, CV36, CV4, CV5, CV6, CV7, CV8, CV9: footprint CAP_GCM155_MUR:CAP_GCM155_MUR -> Capacitor_0402:Capacitor_0402
- CV33, CV34: footprint GRM15x:GRM15x -> C_4uF7_0402:C_4uF7_0402
- R1, R10, R16, R17, R8, R9: footprint RC0402N_VIS:RC0402N_VIS -> RES_0402:RES_0402
- R18, RC2: footprint ERA6AEB101V:ERA6AEB101V -> R_0805_5K1:R_0805_5K1
- R6, R7: footprint KTR03EZPF27R0:RES_R0603_ROM -> RES_R0603_27:RES_R0603_27
Changed lines of the file:
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@@
 	(net 132 "unconnected-(U1-NC-Pad4)")
 	(net 133 "unconnected-(U1-NC-Pad1)")
-	(footprint "RC0402N_VIS:RC0402N_VIS"
+	(footprint "RES_0402:RES_0402"
 		(layer "F.Cu")
 		(at 177.760599 64.1781)
@@
 			)
 		)
-		(property "Footprint" "RC0402N_VIS:RC0402N_VIS"
+		(property "Footprint" "RES_0402:RES_0402"
 			(at 0 0 0)
 			(layer "F.Fab")
@@
 		)
 	)
-	(footprint "KTR03EZPF27R0:RES_R0603_ROM"
+	(footprint "RES_R0603_27:RES_R0603_27"
 		(layer "F.Cu")
 		(at 204.25 73.5)
@@
 			)
 		)
-		(property "Footprint" "KTR03EZPF27R0:RES_R0603_ROM"
+		(property "Footprint" "RES_R0603_27:RES_R0603_27"
 			(at 0 0 0)
 			(layer "F.Fab")
@@
 		)
 	)
-	(footprint "CAP_GCM155_MUR:CAP_GCM155_MUR"
+	(footprint "Capacitor_0402:Capacitor_0402"
 		(layer "F.Cu")
 		(at 197.0931 48.1969)
@@
 			)
 		)
-		(property "Footprint" "CAP_GCM155_MUR:CAP_GCM155_MUR"
+		(property "Footprint" "Capacitor_0402:Capacitor_0402"
 			(at 0 0 0)
 			(layer "F.Fab")
@@
 		)
 	)
-	(footprint "CAP_GCM155_MUR:CAP_GCM155_MUR"
+	(footprint "Capacitor_0402:Capacitor_0402"
 		(layer "F.Cu")
 		(at 197.0931 50.3653)
@@
 			)
 		)
-		(property "Footprint" "CAP_GCM155_MUR:CAP_GCM155_MUR"
+		(property "Footprint" "Capacitor_0402:Capacitor_0402"
 			(at 0 0 0)
 			(layer "F.Fab")
@@
 		)
 	)
-	(footprint "RC0402N_VIS:RC0402N_VIS"
+	(footprint "RES_0402:RES_0402"
 		(layer "F.Cu")
 		(at 177.760599 59.8573)
@@
 			)
 		)
-		(property "Footprint" "RC0402N_VIS:RC0402N_VIS"
+		(property "Footprint" "RES_0402:RES_0402"
 			(at 0 0 0)
 			(layer "F.Fab")
@@
 		)
 	)
-	(footprint "CAP_GCM155_MUR:CAP_GCM155_MUR"
+	(footprint "Capacitor_0402:Capacitor_0402"
 		(layer "F.Cu")
 		(at 197.0931 46.0285)
@@
 			)
 		)
-		(property "Footprint" "CAP_GCM155_MUR:CAP_GCM155_MUR"
+		(property "Footprint" "Capacitor_0402:Capacitor_0402"
 			(at 0 0 0)
 			(layer "F.Fab")
@@
 		)
 	)
-	(footprint "CAP_GCM155_MUR:CAP_GCM155_MUR"
+	(footprint "Capacitor_0402:Capacitor_0402"
 		(layer "F.Cu")
 		(at 193.7309 48.1969)
@@
 			)
 		)
-		(property "Footprint" "CAP_GCM155_MUR:CAP_GCM155_MUR"
+		(property "Footprint" "Capacitor_0402:Capacitor_0402"
 			(at 0 0 0)
 			(layer "F.Fab")
@@
 		)
 	)
-	(footprint "RC0402N_VIS:RC0402N_VIS"
+	(footprint "RES_0402:RES_0402"
 		(layer "F.Cu")
 		(at 177.760599 53.3761)
@@
 			)
 		)
-		(property "Footprint" "RC0402N_VIS:RC0402N_VIS"
+		(property "Footprint" "RES_0402:RES_0402"
 			(at 0 0 0)
 			(layer "F.Fab")
@@
 		)
 	)
-	(footprint "KTR03EZPF27R0:RES_R0603_ROM"
+	(footprint "RES_R0603_27:RES_R0603_27"
 		(layer "F.Cu")
 		(at 204.25 70.9506)
@@
 			)
 		)
-		(property "Footprint" "KTR03EZPF27R0:RES_R0603_ROM"
+		(property "Footprint" "RES_R0603_27:RES_R0603_27"
 			(at 0 0 0)
 			(layer "F.Fab")
@@
 		)
 	)
-	(footprint "CAP_GCM155_MUR:CAP_GCM155_MUR"
+	(footprint "Capacitor_0402:Capacitor_0402"
 		(layer "F.Cu")
 		(at 197.0931 43.8601)
@@
 			)
 		)
-		(property "Footprint" "CAP_GCM155_MUR:CAP_GCM155_MUR"
+		(property "Footprint" "Capacitor_0402:Capacitor_0402"
 			(at 0 0 0)
 			(layer "F.Fab")
@@
 		)
 	)
-	(footprint "ERA6AEB101V:ERA6AEB101V"
+	(footprint "R_0805_5K1:R_0805_5K1"
 		(layer "F.Cu")
 		(at 203.2998 54.4709)
@@
 			)
 		)
-		(property "Footprint" "ERA6AEB101V:ERA6AEB101V"
+		(property "Footprint" "R_0805_5K1:R_0805_5K1"
 			(at 0 0 0)
 			(layer "F.Fab")
@@
 		)
 	)
-	(footprint "RC0402N_VIS:RC0402N_VIS"
+	(footprint "RES_0402:RES_0402"
 		(layer "F.Cu")
 		(at 177.760599 62.0177)
@@
 			)
 		)
-		(property "Footprint" "RC0402N_VIS:RC0402N_VIS"
+		(property "Footprint" "RES_0402:RES_0402"
 			(at 0 0 0)
 			(layer "F.Fab")
@@
 		)
 	)
-	(footprint "GRM15x:GRM15x"
+	(footprint "C_4uF7_0402:C_4uF7_0402"
 		(layer "F.Cu")
 		(at 200.6198 73.5759)
@@
 			)
 		)
-		(property "Footprint" "GRM15x:GRM15x"
+		(property "Footprint" "C_4uF7_0402:C_4uF7_0402"
 			(at 0 0 0)
 			(layer "F.Fab")
@@
 		)
 	)
-	(footprint "ERA6AEB101V:ERA6AEB101V"
+	(footprint "R_0805_5K1:R_0805_5K1"
 		(layer "F.Cu")
 		(at 203.2998 58.8209)
@@
 			)
 		)
-		(property "Footprint" "ERA6AEB101V:ERA6AEB101V"
+		(property "Footprint" "R_0805_5K1:R_0805_5K1"
 			(at 0 0 0)
 			(layer "F.Fab")
@@
 		)
 	)
-	(footprint "CAP_GCM155_MUR:CAP_GCM155_MUR"
+	(footprint "Capacitor_0402:Capacitor_0402"
 		(layer "F.Cu")
 		(at 193.7309 50.3653)
@@
 			)
 		)
-		(property "Footprint" "CAP_GCM155_MUR:CAP_GCM155_MUR"
+		(property "Footprint" "Capacitor_0402:Capacitor_0402"
 			(at 0 0 0)
 			(layer "F.Fab")
@@
 		)
 	)
-	(footprint "CAP_GCM155_MUR:CAP_GCM155_MUR"
+	(footprint "Capacitor_0402:Capacitor_0402"
 		(layer "F.Cu")
 		(at 200.4553 46.0285)
@@
 			)
 		)
-		(property "Footprint" "CAP_GCM155_MUR:CAP_GCM155_MUR"
+		(property "Footprint" "Capacitor_0402:Capacitor_0402"
 			(at 0 0 0)
 			(layer "F.Fab")
@@
 		)
 	)
-	(footprint "CAP_GCM155_MUR:CAP_GCM155_MUR"
+	(footprint "Capacitor_0402:Capacitor_0402"
 		(layer "F.Cu")
 		(at 203.8175 48.1969)
@@
 			)
 		)
-		(property "Footprint" "CAP_GCM155_MUR:CAP_GCM155_MUR"
+		(property "Footprint" "Capacitor_0402:Capacitor_0402"
 			(at 0 0 0)
 			(layer "F.Fab")
@@
 		)
 	)
-	(footprint "CAP_GCM155_MUR:CAP_GCM155_MUR"
+	(footprint "Capacitor_0402:Capacitor_0402"
 		(layer "F.Cu")
 		(at 200.4553 43.8601)
@@
 			)
 		)
-		(property "Footprint" "CAP_GCM155_MUR:CAP_GCM155_MUR"
+		(property "Footprint" "Capacitor_0402:Capacitor_0402"
 			(at 0 0 0)
 			(layer "F.Fab")
@@
 		)
 	)
-	(footprint "GRM15x:GRM15x"
+	(footprint "C_4uF7_0402:C_4uF7_0402"
 		(layer "F.Cu")
 		(at 200.6198 70.9759)
@@
 			)
 		)
-		(property "Footprint" "GRM15x:GRM15x"
+		(property "Footprint" "C_4uF7_0402:C_4uF7_0402"
 			(at 0 0 0)
 			(layer "F.Fab")
@@
 		)
 	)
-	(footprint "CAP_GCM155_MUR:CAP_GCM155_MUR"
+	(footprint "Capacitor_0402:Capacitor_0402"
 		(layer "F.Cu")
 		(at 203.8175 43.8601)
@@
 			)
 		)
-		(property "Footprint" "CAP_GCM155_MUR:CAP_GCM155_MUR"
+		(property "Footprint" "Capacitor_0402:Capacitor_0402"
 			(at 0 0 0)
 			(layer "F.Fab")
@@
 		)
 	)
-	(footprint "RC0402N_VIS:RC0402N_VIS"
+	(footprint "RES_0402:RES_0402"
 		(layer "F.Cu")
 		(at 177.760599 57.6969)
@@
 			)
 		)
-		(property "Footprint" "RC0402N_VIS:RC0402N_VIS"
+		(property "Footprint" "RES_0402:RES_0402"
 			(at 0 0 0)
 			(layer "F.Fab")
@@
 		)
 	)
-	(footprint "CAP_GCM155_MUR:CAP_GCM155_MUR"
+	(footprint "Capacitor_0402:Capacitor_0402"
 		(layer "F.Cu")
 		(at 203.8175 50.3653)
@@
 			)
 		)
-		(property "Footprint" "CAP_GCM155_MUR:CAP_GCM155_MUR"
+		(property "Footprint" "Capacitor_0402:Capacitor_0402"
 			(at 0 0 0)
 			(layer "F.Fab")
@@
 		)
 	)
-	(footprint "RC0402N_VIS:RC0402N_VIS"
+	(footprint "RES_0402:RES_0402"
 		(layer "F.Cu")
 		(at 177.760599 55.5365)
@@
 			)
 		)
-		(property "Footprint" "RC0402N_VIS:RC0402N_VIS"
+		(property "Footprint" "RES_0402:RES_0402"
 			(at 0 0 0)
 			(layer "F.Fab")
@@
 		)
 	)
-	(footprint "CAP_GCM155_MUR:CAP_GCM155_MUR"
+	(footprint "Capacitor_0402:Capacitor_0402"
 		(layer "F.Cu")
 		(at 203.8175 46.0285)
@@
 			)
 		)
-		(property "Footprint" "CAP_GCM155_MUR:CAP_GCM155_MUR"
+		(property "Footprint" "Capacitor_0402:Capacitor_0402"
 			(at 0 0 0)
 			(layer "F.Fab")
@@
 		)
 	)
-	(footprint "CAP_GCM155_MUR:CAP_GCM155_MUR"
+	(footprint "Capacitor_0402:Capacitor_0402"
 		(layer "F.Cu")
 		(at 193.7309 46.0285)
@@
 			)
 		)
-		(property "Footprint" "CAP_GCM155_MUR:CAP_GCM155_MUR"
+		(property "Footprint" "Capacitor_0402:Capacitor_0402"
 			(at 0 0 0)
 			(layer "F.Fab")
@@
 		)
 	)
-	(footprint "CAP_GCM155_MUR:CAP_GCM155_MUR"
+	(footprint "Capacitor_0402:Capacitor_0402"
 		(layer "F.Cu")
 		(at 200.4553 50.3653)
@@
 			)
 		)
-		(property "Footprint" "CAP_GCM155_MUR:CAP_GCM155_MUR"
+		(property "Footprint" "Capacitor_0402:Capacitor_0402"
 			(at 0 0 0)
 			(layer "F.Fab")
@@
 		)
 	)
-	(footprint "CAP_GCM155_MUR:CAP_GCM155_MUR"
+	(footprint "Capacitor_0402:Capacitor_0402"
 		(layer "F.Cu")
 		(at 193.7309 43.8601)
@@
 			)
 		)
-		(property "Footprint" "CAP_GCM155_MUR:CAP_GCM155_MUR"
+		(property "Footprint" "Capacitor_0402:Capacitor_0402"
 			(at 0 0 0)
 			(layer "F.Fab")
@@
 		)
 	)
-	(footprint "CAP_GCM155_MUR:CAP_GCM155_MUR"
+	(footprint "Capacitor_0402:Capacitor_0402"
 		(layer "F.Cu")
 		(at 200.4553 48.1969)
@@
 			)
 		)
-		(property "Footprint" "CAP_GCM155_MUR:CAP_GCM155_MUR"
+		(property "Footprint" "Capacitor_0402:Capacitor_0402"
 			(at 0 0 0)
 			(layer "F.Fab")
