File: Boards/OBC board/OBC board.kicad_sch (KiCad schematic)
At the start: 55 parts, among them J3 Conn_01x01_Socket, J4 Conn_01x04_Socket, J5 Conn_01x04_Socket, J6 XT30UPB-M, J7 Conn_01x01_Socket, SW3 D2F-01-D, U10 IRLZ44NPBF, U3 MAX485CSA+T, U4 ASM330LHH, U5 TPS1120DR, U6 TPS1120DR, U7 TPS1120DR, U8 LPS22DFTR, U9 LIS2MDLTR

Commit message: parte 2
é isso
Parts:
- removed J4, J5: Conn_01x04_Socket, Connector_PinSocket_1.00mm:PinSocket_1x04_P1.00mm_Vertical_SMD_Pin1Right, symbol Connector:Conn_01x04_Socket
- added J4: 22022065, CONN_SA-4455_06_TE_MOL, symbol CONN Female Header 22022065:22022065
- added J5: XT60PW-M, XT60PW-M:AMASS_XT60PW-M, symbol XT60PW-M:XT60PW-M
Connections:
- net BMS_VIN: now also J5.1 (+)
- net Comms UART CTS: now also J4.3
- net Comms UART RTS: now also J4.4
- net Comms UART RX: now also J4.5
- net Comms UART TX: now also J4.6
- net GND: now also J4.1, J5.2 (-)
- new net: C1.1, C2.1, C3.1, C4.1, U9.5 (C1)

Commit message: Correção de erros ERC no OBC e correção de simbolos usados
Parts:
- removed BOSCH_AXL_GYRO1: BMI323, BMI323_BOS, symbol BMI323:BMI323
- removed BOSCH_BAR1: BMP581, QFN10_BMP581_BOS, symbol BMP581:BMP581
- removed C1, C10, C11, C12, C13, C18, C19, C2, C20, C24, C6: 100nF, Capacitor_SMD:C_0201_0603Metric, symbol c_mini:C_mini
- removed C3, C4: 10nF, Capacitor_SMD:C_0201_0603Metric, symbol c_mini:C_mini
- removed C5: 10uF, Capacitor_SMD:C_0201_0603Metric, symbol c_mini:C_mini
- removed J4: 22022065, CONN_SA-4455_06_TE_MOL, symbol CONN Female Header 22022065:22022065
- removed U3: MAX485CSA+T, 21-0041-3-M_90-0096-8L_MXM, symbol MAX485:MAX485CSA+T
- removed U4: ASM330LHH, LGA-14L_2P5X3X0P83_STM, symbol ST ASM330LHH:ASM330LHH
- added C1, C10, C11, C12, C13, C15, C16, C17, C5, C6, C9: 100nF, symbol Device:C_Small
- added C18: 10uF, symbol Device:C_Small
- added C2, C3: 10nF, symbol Device:C_Small
- added J8: 22022065, CONN_SA-4455_06_TE_MOL, symbol CONN_Female Header:22022065
- added U12: BMI323, BMI323_BOS, symbol IMU_BMI323:BMI323
- added U13: BMP581, QFN10_BMP581_BOS, symbol BARO_BMP581:BMP581
- added U3: MAX485CSA+T, 21-0041-3-M_90-0096-8L_MXM, symbol RS_Transceiver_MAX485:MAX485CSA+T
- added U4: ASM330LHHTR, LGA-14L_2P5X3X0P83_STM, symbol IMU_ASM330LHHTR:ASM330LHHTR
- U5: footprint Dual PMOS:D8 -> D8
Connections:
- net +3.3V: now also C10.1, C11.1, C12.1, C13.2, C15.1, C16.1, C17.1, C18.1, C6.1, C9.1, U12.5 (VDDIO), U12.8 (VDD), U13.1 (VDDIO), U13.10 (VDD), U4.2 (RES), U4.3 (RES), U4.5 (VDD_IO), U4.8 (VDD)
- net +5V: now also J8.5, U3.1 (RO)
- net BAR2 RDY: now also U13.7 (INT)
- net BAR2 SPI1_~{CS}: now also U13.6 (CSB)
- net Comms UART CTS: now also J8.4
- net Comms UART RTS: now also J8.3
- net Comms UART RX: now also J8.2
- net Comms UART TX: now also J8.1
- net GND: now also C1.2, C10.2, C11.2, C12.2, C13.1, C15.2, C16.2, C17.2, C18.2, C2.2, C3.2, C5.2, C6.2, C9.2, J8.6, U12.6 (GNDIO), U12.7 (GND), U13.3 (VSS), U13.8 (VSS), U13.9 (VSS), U3.4 (DI), U4.6 (GND), U4.7 (GND)
- net IMU1 RDY1: now also U12.4 (INT1)
- net IMU1 RDY2: now also U12.9 (INT2)
- net IMU1 SPI0_~{CS}: now also U12.12 (CSB)
- net IMU2 RDY: now also U4.9 (INT2)
- net IMU2 SPI1_~{CS}: now also U4.12 (CS)
- net RS_ENABLE: now also U3.6 (A), U3.7 (B)
- net RS_RX: now also U3.8 (VCC)
- net RS_TX: now also U3.5 (GND)
- net SPI0_MISO: now also U12.1 (SDO)
- net SPI0_MOSI: now also U12.14 (SDX)
- net SPI0_SCK: now also U12.13 (SCX); no longer U8.2 (SCL/SPC)
- net SPI1_MISO: now also U13.5 (SDO), U4.1 (SDO/SA0)
- net SPI1_MOSI: now also U13.4 (SDI), U4.14 (SDA)
- net SPI1_SCK: now also U13.2 (SCK), U4.13 (SCL)
- net at J3.1 (Pin_1), R13.1, R15.1: now also U3.2 (*RE)
- net at J7.1 (Pin_1), R13.2, R14.2: now also U3.3 (DE)
- net at U9.5 (C1): now also C1.1, C2.1, C3.1, C5.1
Other:
- note added: "Atribuir footprints Simbolos de connectores - Conectores RS"
- note added: "Este botão tem de ser trocado por um contacto. Este contacto vai estar a conectar o circuito a um botão ON-OFF armado por chave que se vai encontrar no painel de armação exterior do foguetão"
- note added: "Provavelmente este circuito vai sofrer alterações devido à não utilização de um ignitor e-match"
- note added: "Verificar necessidade de Heat-Sink no Mosfet"
- note removed: "Atribuir footprints Simbolos de connectores - Conectores dos 5V do OBC para BMS/Charger - Conectores RS - Pins para passar UART, 5V e GND para Comunication Board"
- note removed: "Botão mecânico normalmente aberto. É armado antes de lançamento."
- moved on the sheet: J5

Commit message: Atualizações footprints
Adicionei a Resistência de 27 ohms que faltava na biblioteca Symbols Lib;
Atualizei as footprints do OBC menos a componente J6;
Parts:
- C1, C10, C11, C12, C13, C15, C16, C17, C18, C2, C3, C5, C6, C9: footprint (none) -> CAP_GCM155_MUR:CAP_GCM155_MUR
- C14, C7, C8: footprint Capacitor_SMD:C_0201_0603Metric -> CAP_GCM155_MUR:CAP_GCM155_MUR
- J5: footprint XT60PW-M:AMASS_XT60PW-M -> Conn XT60PW-M:AMASS_XT60PW-M
- J6: footprint CONN_XT30UPB-M_AMA -> (none)
- J8: footprint CONN_SA-4455_06_TE_MOL -> CONN Female Header:CONN_SA-4455_06_TE_MOL
- LED1: footprint HSMHH191 -> MAG LIS2MDLTR:LGA-12_2X2X1_STM
- LED2, LED3, LED4, LED5, LED6, LED7: footprint HSMHH191 -> Red SMD LED:HSMHH191
- R10, R12, R13, R14, R15, R16, R17, R18, R19, R20, R21, R22, R23, R24, R25: footprint Resistor_SMD:R_0201_0603Metric -> RC0402N_VIS:RC0402N_VIS
- SW3: footprint D2F-01-D_OMR -> Switch D2F-01:D2F-01-D_OMR
- U10: footprint PG-TO220-3_INF -> NMOS IRLZ44:PG-TO220-3_INF
- U12: footprint BMI323_BOS -> IMU BMI323:BMI323_BOS
- U13: footprint QFN10_BMP581_BOS -> BARO BMP581:QFN10_BMP581_BOS
- U3: footprint 21-0041-3-M_90-0096-8L_MXM -> RS Transceiver:21-0041-3-M_90-0096-8L_MXM
- U4: footprint LGA-14L_2P5X3X0P83_STM -> IMU ASM330LHHTR:LGA-14L_2P5X3X0P83_STM
- U5, U6, U7: footprint D8 -> 2 PMOS:D8
- U8: footprint QFN_22DFTR_STM -> BARO LPS22DFTR:QFN_22DFTR_STM
- U9: footprint LGA-12_2X2X1_STM -> MAG LIS2MDLTR:LGA-12_2X2X1_STM
Changed lines of the file:
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@@
 			)
 		)
-		(property "Footprint" "Resistor_SMD:R_0201_0603Metric"
+		(property "Footprint" "RC0402N_VIS:RC0402N_VIS"
 			(at 405.638 55.245 90)
 			(effects
@@
 			)
 		)
-		(property "Footprint" "Resistor_SMD:R_0201_0603Metric"
+		(property "Footprint" "RC0402N_VIS:RC0402N_VIS"
 			(at 385.318 48.895 90)
 			(effects
@@
 			)
 		)
-		(property "Footprint" "BMI323_BOS"
+		(property "Footprint" "IMU BMI323:BMI323_BOS"
 			(at 220.98 49.53 0)
 			(effects
@@
 			)
 		)
-		(property "Footprint" "CONN_XT30UPB-M_AMA"
+		(property "Footprint" ""
 			(at 407.67 120.65 0)
 			(effects
@@
 			)
 		)
-		(property "Footprint" ""
+		(property "Footprint" "CAP_GCM155_MUR:CAP_GCM155_MUR"
 			(at 246.38 173.355 0)
 			(effects
@@
 			)
 		)
-		(property "Footprint" ""
+		(property "Footprint" "CAP_GCM155_MUR:CAP_GCM155_MUR"
 			(at 285.75 67.31 0)
 			(effects
@@
 			)
 		)
-		(property "Footprint" "QFN10_BMP581_BOS"
+		(property "Footprint" "BARO BMP581:QFN10_BMP581_BOS"
 			(at 276.86 160.02 0)
 			(effects
@@
 			)
 		)
-		(property "Footprint" ""
+		(property "Footprint" "CAP_GCM155_MUR:CAP_GCM155_MUR"
 			(at 182.88 224.155 0)
 			(effects
@@
 			)
 		)
-		(property "Footprint" "HSMHH191"
+		(property "Footprint" "Red SMD LED:HSMHH191"
 			(at 127 263.83 0)
 			(effects
@@
 			)
 		)
-		(property "Footprint" "CONN_SA-4455_06_TE_MOL"
+		(property "Footprint" "CONN Female Header:CONN_SA-4455_06_TE_MOL"
 			(at 35.56 44.45 0)
 			(effects
@@
 			)
 		)
-		(property "Footprint" "Resistor_SMD:R_0201_0603Metric"
+		(property "Footprint" "RC0402N_VIS:RC0402N_VIS"
 			(at 399.288 42.545 90)
 			(effects
@@
 			)
 		)
-		(property "Footprint" "HSMHH191"
+		(property "Footprint" "Red SMD LED:HSMHH191"
 			(at 127 310.82 0)
 			(effects
@@
 			)
 		)
-		(property "Footprint" "Resistor_SMD:R_0201_0603Metric"
+		(property "Footprint" "RC0402N_VIS:RC0402N_VIS"
 			(at 23.495 243.332 90)
 			(effects
@@
 			)
 		)
-		(property "Footprint" "Resistor_SMD:R_0201_0603Metric"
+		(property "Footprint" "RC0402N_VIS:RC0402N_VIS"
 			(at 457.962 38.735 90)
 			(effects
@@
 			)
 		)
-		(property "Footprint" ""
+		(property "Footprint" "CAP_GCM155_MUR:CAP_GCM155_MUR"
 			(at 207.01 224.155 0)
 			(effects
@@
 			)
 		)
-		(property "Footprint" "Resistor_SMD:R_0201_0603Metric"
+		(property "Footprint" "RC0402N_VIS:RC0402N_VIS"
 			(at 128.397 109.855 90)
 			(effects
@@
 			)
 		)
-		(property "Footprint" "Resistor_SMD:R_0201_0603Metric"
+		(property "Footprint" "RC0402N_VIS:RC0402N_VIS"
 			(at 23.495 169.672 90)
 			(effects
@@
 			)
 		)
-		(property "Footprint" "PG-TO220-3_INF"
+		(property "Footprint" "NMOS IRLZ44:PG-TO220-3_INF"
 			(at 379.349 124.968 0)
 			(effects
@@
 			)
 		)
-		(property "Footprint" "LGA-12_2X2X1_STM"
+		(property "Footprint" "MAG LIS2MDLTR:LGA-12_2X2X1_STM"
 			(at 213.36 208.28 0)
 			(effects
@@
 			)
 		)
-		(property "Footprint" "Resistor_SMD:R_0201_0603Metric"
+		(property "Footprint" "RC0402N_VIS:RC0402N_VIS"
 			(at 451.358 38.735 90)
 			(effects
@@
 			)
 		)
-		(property "Footprint" "Resistor_SMD:R_0201_0603Metric"
+		(property "Footprint" "RC0402N_VIS:RC0402N_VIS"
 			(at 23.495 214.122 90)
 			(effects
@@
 			)
 		)
-		(property "Footprint" "Resistor_SMD:R_0201_0603Metric"
+		(property "Footprint" "RC0402N_VIS:RC0402N_VIS"
 			(at 23.495 182.372 90)
 			(effects
@@
 			)
 		)
-		(property "Footprint" "Resistor_SMD:R_0201_0603Metric"
+		(property "Footprint" "RC0402N_VIS:RC0402N_VIS"
 			(at 23.495 201.422 90)
 			(effects
@@
 			)
 		)
-		(property "Footprint" ""
+		(property "Footprint" "CAP_GCM155_MUR:CAP_GCM155_MUR"
 			(at 188.595 224.155 0)
 			(effects
@@
 			)
 		)
-		(property "Footprint" "HSMHH191"
+		(property "Footprint" "MAG LIS2MDLTR:LGA-12_2X2X1_STM"
 			(at 223.825 116.205 0)
 			(effects
@@
 			)
 		)
-		(property "Footprint" ""
+		(property "Footprint" "CAP_GCM155_MUR:CAP_GCM155_MUR"
 			(at 299.085 207.645 0)
 			(effects
@@
 			)
 		)
-		(property "Footprint" ""
+		(property "Footprint" "CAP_GCM155_MUR:CAP_GCM155_MUR"
 			(at 241.3 173.355 0)
 			(effects
@@
 			)
 		)
-		(property "Footprint" "HSMHH191"
+		(property "Footprint" "Red SMD LED:HSMHH191"
 			(at 127 324.79 0)
 			(effects
@@
 			)
 		)
-		(property "Footprint" "Capacitor_SMD:C_0201_0603Metric"
+		(property "Footprint" "CAP_GCM155_MUR:CAP_GCM155_MUR"
 			(at 301.2948 93.345 0)
 			(effects
@@
 			)
 		)
-		(property "Footprint" "QFN_22DFTR_STM"
+		(property "Footprint" "BARO LPS22DFTR:QFN_22DFTR_STM"
 			(at 224.409 86.36 0)
 			(effects
@@
 			)
 		)
-		(property "Footprint" "Capacitor_SMD:C_0201_0603Metric"
+		(property "Footprint" "CAP_GCM155_MUR:CAP_GCM155_MUR"
 			(at 413.385 131.1148 0)
 			(effects
@@
 			)
 		)
-		(property "Footprint" "HSMHH191"
+		(property "Footprint" "Red SMD LED:HSMHH191"
 			(at 127 340.03 0)
 			(effects
@@
 			)
 		)
-		(property "Footprint" ""
+		(property "Footprint" "CAP_GCM155_MUR:CAP_GCM155_MUR"
 			(at 196.85 62.23 0)
 			(effects
@@
 			)
 		)
-		(property "Footprint" ""
+		(property "Footprint" "CAP_GCM155_MUR:CAP_GCM155_MUR"
 			(at 329.565 157.48 0)
 			(effects
@@
 			)
 		)
-		(property "Footprint" "LGA-14L_2P5X3X0P83_STM"
+		(property "Footprint" "IMU ASM330LHHTR:LGA-14L_2P5X3X0P83_STM"
 			(at 184.15 153.67 0)
 			(effects
@@
 			)
 		)
-		(property "Footprint" "Resistor_SMD:R_0201_0603Metric"
+		(property "Footprint" "RC0402N_VIS:RC0402N_VIS"
 			(at 456.438 38.735 90)
 			(effects
@@
 			)
 		)
-		(property "Footprint" "D2F-01-D_OMR"
+		(property "Footprint" "Switch D2F-01:D2F-01-D_OMR"
 			(at 426.72 120.65 0)
 			(effects
@@
 			)
 		)
-		(property "Footprint" "HSMHH191"
+		(property "Footprint" "Red SMD LED:HSMHH191"
 			(at 127 279.07 0)
 			(effects
@@
 			)
 		)
-		(property "Footprint" "Resistor_SMD:R_0201_0603Metric"
+		(property "Footprint" "RC0402N_VIS:RC0402N_VIS"
 			(at 443.23 133.858 90)
 			(effects
@@
 			)
 		)
-		(property "Footprint" "D8"
+		(property "Footprint" "2 PMOS:D8"
 			(at 46.99 173.99 0)
 			(effects
@@
 			)
 		)
-		(property "Footprint" "21-0041-3-M_90-0096-8L_MXM"
+		(property "Footprint" "RS Transceiver:21-0041-3-M_90-0096-8L_MXM"
 			(at 408.94 45.085 0)
 			(effects
@@
 			)
 		)
-		(property "Footprint" "Resistor_SMD:R_0201_0603Metric"
+		(property "Footprint" "RC0402N_VIS:RC0402N_VIS"
 			(at 23.495 230.632 90)
 			(effects
@@
 			)
 		)
-		(property "Footprint" ""
+		(property "Footprint" "CAP_GCM155_MUR:CAP_GCM155_MUR"
 			(at 197.485 224.155 0)
 			(effects
@@
 			)
 		)
-		(property "Footprint" ""
+		(property "Footprint" "CAP_GCM155_MUR:CAP_GCM155_MUR"
 			(at 290.83 207.645 0)
 			(effects
@@
 			)
 		)
-		(property "Footprint" ""
+		(property "Footprint" "CAP_GCM155_MUR:CAP_GCM155_MUR"
 			(at 171.45 167.64 0)
 			(effects
@@
 			)
 		)
-		(property "Footprint" "D8"
+		(property "Footprint" "2 PMOS:D8"
 			(at 46.99 234.95 0)
 			(effects
@@
 			)
 		)
-		(property "Footprint" "HSMHH191"
+		(property "Footprint" "Red SMD LED:HSMHH191"
 			(at 127 295.58 0)
 			(effects
@@
 			)
 		)
-		(property "Footprint" "Capacitor_SMD:C_0201_0603Metric"
+		(property "Footprint" "CAP_GCM155_MUR:CAP_GCM155_MUR"
 			(at 185.1152 92.71 0)
 			(effects
@@
 			)
 		)
-		(property "Footprint" ""
+		(property "Footprint" "CAP_GCM155_MUR:CAP_GCM155_MUR"
 			(at 267.335 156.21 0)
 			(effects
@@
 			)
 		)
-		(property "Footprint" "D8"
+		(property "Footprint" "2 PMOS:D8"
 			(at 46.99 205.74 0)
 			(effects
@@
 			)
 		)
-		(property "Footprint" ""
+		(property "Footprint" "CAP_GCM155_MUR:CAP_GCM155_MUR"
 			(at 309.245 207.645 0)
 			(effects
@@
 			)
 		)
-		(property "Footprint" "Resistor_SMD:R_0201_0603Metric"
+		(property "Footprint" "RC0402N_VIS:RC0402N_VIS"
 			(at 374.65 109.728 90)
 			(effects
@@
 			)
 		)
-		(property "Footprint" "XT60PW-M:AMASS_XT60PW-M"
+		(property "Footprint" "Conn XT60PW-M:AMASS_XT60PW-M"
 			(at 27.305 92.71 0)
 			(effects

Commit message: pequenas correções em algumas resistências e bugfix do simobolo do Barometro
Parts:
- removed R13: 120, RC0402N_VIS:RC0402N_VIS, symbol Device:R
- removed R14, R15: 20K, RC0402N_VIS:RC0402N_VIS, symbol Device:R
- removed R16, R17, R18: 10K, RC0402N_VIS:RC0402N_VIS, symbol Device:R
- removed SW3: D2F-01-D, Switch D2F-01:D2F-01-D_OMR, symbol Switch_D2F-01:D2F-01-D
- removed U3: MAX485CSA+T, RS Transceiver:21-0041-3-M_90-0096-8L_MXM, symbol RS_Transceiver_MAX485:MAX485CSA+T
- added J4, J9: Conn_01x01_Socket, Button_Switch_THT:SW_Lever_1P2T_NKK_GW12LxH, symbol Connector:Conn_01x01_Socket
- added R11: 120, RC0402N_VIS:RC0402N_VIS, symbol Device:R
- added R26, R27: 20K, RC0402N_VIS:RC0402N_VIS, symbol Device:R
- added R28, R29, R30: 10K, RC0402N_VIS:RC0402N_VIS, symbol Device:R
- added U14: MAX485CSA+T, RS Transceiver:21-0041-3-M_90-0096-8L_MXM, symbol RS_Transceiver_MAX485:MAX485CSA+T
- R19: value 130 -> 120
- U8: footprint BARO LPS22DFTR:QFN_22DFTR_STM -> QFN_22DFTR_STM
Connections:
- net +3.3V: now also R28.1, R29.1, R30.2
- net +5V: now also R26.1, U14.8 (VCC)
- net GND: now also R27.2, U14.5 (GND)
- net RS_ENABLE: now also R29.2, U14.2 (*RE), U14.3 (DE)
- net RS_RX: now also R28.2, U14.1 (RO)
- net RS_TX: now also R30.1, U14.4 (DI)
- net SPI0_SCK: now also U8.2 (SCK)
- net at J3.1 (Pin_1): now also C7.2, R12.1
- net at J7.1 (Pin_1): now also J6.2
- new net: J9.1 (Pin_1), R11.2, R26.2, U14.6 (A)
- new net: J4.1 (Pin_1), R11.1, R27.1, U14.7 (B)
- no-connect marks 7 -> 6
Other:
- note added: "Conectores alanvacados"
- note added: "Este contacto vai estar a conectar o circuito a um botão ON-OFF armado por chave que se vai encontrar no painel de armação exterior do foguetão"
- note added: "Simbolos de connectores - Conectores RS"
- note removed: "Atribuir footprints Simbolos de connectores - Conectores RS"
- note removed: "Este botão tem de ser trocado por um contacto. Este contacto vai estar a conectar o circuito a um botão ON-OFF armado por chave que se vai encontrar no painel de armação exterior do foguetão"
- note removed: "Ver simbolo de connectores alavancados para RS"
