File: Boards/Ground & Fill Station Systems/TVCS Fill/TVCS Fill.kicad_pcb (KiCad board)
At the start: 6 copper layers, 100 x 60 mm, 252 parts, among them J1 Conn_01x01_Socket, J10 Conn_01x01_Socket, J11 Conn_01x01_Socket, J12 Conn_01x01_Socket, J13 Conn_01x01_Socket, J14 Conn_01x01_Socket, J15 Conn_01x01_Socket, J16 DX07S016JA1R1500, J16 XT30UPB-M, J17 USB_C, J2 Conn_01x01_Socket, J3 XT30UPB-M, J4 XT30UPB-M, J5 Conn_01x01_Socket, J6 XT30UPB-M, J7 BM03B-SRSS-TBLFSN, J8 Conn_01x01_Socket, J9 Conn_01x01_Socket, SW2 SW_Push, SW3 SW_Push, U1 MAX31856, U1 MAX31856MUD+T, U10 MAX31856MUD+T, U10 TPS1120DR, U11 IRLZ44NPBF, U12 IRLZ44NPBF, U13 LM61460AASQRJRRQ1, U14 ADS1114IRUGR, U14 LM61460AASQRJRRQ1, U15 TPS1120DR, U16 TPS1120DR, U18 ST1L05APU33R, U2 ADS1114IDGS, U2 ESD7L5.0DT5G, U3 MAX31856, U3 MAX31856MUD+T, U4 MAX485CSA+T, U5 MAX31856, U5 MCP9808T-E/MC, U6 ESD7L5.0DT5G, U6 W25Q128JVSIQ TR, U7 ST1L05APU33R, U8 PCA9306DP_118, U9 LM61460AASQRJRRQ1, U9 TPS1120DR

Commit message: Tu viste o q eu fiz
Parts:
- removed the C1 at (99.5, 117.5)
- removed the C1 at (223.4, 32.8)
- removed the C10 at (153.9, 94.0)
- removed the C10 at (226.7, 34.9)
- removed the C11 at (226.7, 37.1)
- removed the C11 at (99.5, 115.0)
- removed C15, C16: 10nF, Capacitor_SMD:C_0201_0603Metric
- removed C17, C18, C20: 10nF, Capacitor_0402:Capacitor_0402
- removed C19, CV19, CV20, CV21, CV22, CV23, CV24, CV26, CV30: 100nF, Capacitor_0402:Capacitor_0402
- removed the C2 at (153.9, 80.0)
- removed the C2 at (223.4, 34.9)
- removed the C3 at (153.9, 81.8)
- removed the C3 at (223.4, 37.1)
- removed the C4 at (223.4, 39.3)
- removed the C4 at (153.9, 83.5)
- removed the C6 at (223.4, 41.4)
- removed the C6 at (153.9, 87.0)
- removed the C7 at (153.9, 88.8)
- removed the C7 at (223.4, 43.6)
- removed the C8 at (153.9, 90.5)
- removed the C8 at (223.4, 45.8)
- removed the C9 at (226.7, 32.8)
- removed the C9 at (153.9, 92.2)
- removed the CV13 at (102.4, 83.0)
- removed the CV13 at (228.5, 80.2)
- removed the CV14 at (228.5, 82.3)
- removed the CV14 at (102.4, 84.8)
- removed the CV15 at (102.4, 86.5)
- removed the CV15 at (228.5, 84.5)
- removed the CV16 at (228.5, 86.7)
- removed the CV16 at (102.4, 88.2)
- removed the CV17 at (102.4, 90.0)
- removed the CV17 at (231.9, 80.2)
- removed the CV18 at (231.9, 82.3)
- removed the CV18 at (102.4, 91.8)
- removed CV19, CV20, CV21, CV22, CV23, CV24, CV26, CV30: 100nF, Capacitor_SMD:C_0201_0603Metric
- removed CV25, CV29: 1uF, Capacitor_SMD:C_0201_0603Metric
- removed CV25, CV29: 1uF, Capacitor_0402:Capacitor_0402
- removed CV27, CV28: 4.7uF, Capacitor_SMD:C_0201_0603Metric
- removed CV27, CV28: 4.7uF, C_4uF7_0402:C_4uF7_0402
- removed the C_BT1 at (230.1, 32.8)
- removed the C_BT1 at (156.3, 90.5)
- removed the C_BT2 at (156.3, 92.2)
- removed the C_BT2 at (230.1, 34.9)
- removed C_FF2: C, Capacitor_0402:Capacitor_0402
- removed C_FF2, C_IN_HF1, C_IN_HF2: C, Capacitor_SMD:C_0201_0603Metric
- removed the C_IN-BLK1 at (230.1, 39.3)
- removed the C_IN-BLK1 at (158.8, 80.0)
- removed the C_IN-BLK2 at (158.8, 81.8)
- removed the C_IN-BLK2 at (230.1, 41.4)
- removed the C_IN_HFI1 at (158.8, 87.0)
- removed the C_IN_HFI1 at (230.1, 43.6)
- removed the C_IN_HFI2 at (158.8, 88.8)
- removed the C_IN_HFI2 at (230.1, 45.8)
- removed the C_OUT1 at (233.4, 37.1)
- removed the C_OUT1 at (158.8, 90.5)
- removed the C_OUT2 at (233.4, 39.3)
- removed the C_OUT2 at (158.8, 92.2)
- removed the C_VCC1 at (233.4, 41.4)
- removed the C_VCC1 at (158.8, 94.0)
- removed the C_VCC2 at (99.5, 110.1)
- removed the C_VCC2 at (233.4, 43.6)
- removed the D1 at (242.7, 49.0)
- removed the D1 at (117.0, 116.5)
- removed the D2 at (240.4, 76.0)
- removed the D2 at (121.8, 116.5)
- removed FlashM1: W25Q128JVSIQ_TR, NOR Flash:SOIC_208MIL_WIN
- removed J10, J11, J12, J9: Conn_01x01_Socket, Button_Switch_THT:SW_Lever_1P2T_NKK_GW12LxH
- removed the J16 at (218.3, 72.8)
- removed the J16 at (168.0, 116.0)
- removed the J7 at (232.7, 72.6)
- removed the J7 at (132.2, 82.9)
- removed the L1 at (225.9, 50.2)
- removed the L1 at (156.4, 99.4)
- removed L3: L, Inductor_SMD:L_Neosid_SM-PIC0512H
- removed LED1, LED2, LED3, LED4, LED5, LED6, LED7, LED8, LED9: HSMH-H191, Red SMD LED:HSMHH191
- removed MCU2 (x2): RP2040, Package_DFN_QFN:QFN-56-1EP_7x7mm_P0.4mm_EP3.2x3.2mm
- removed the R1 at (236.8, 32.8)
- removed the R1 at (161.2, 80.0)
- removed the R12 at (236.8, 43.6)
- removed the R12 at (163.7, 81.8)
- removed the R13 at (163.7, 83.5)
- removed the R13 at (236.8, 45.7)
- removed the R2 at (236.8, 34.9)
- removed the R2 at (161.2, 81.8)
- removed the R22 at (225.2, 82.3)
- removed the R22 at (107.3, 86.5)
- removed the R23 at (225.2, 84.5)
- removed the R23 at (107.3, 88.2)
- removed the R24 at (225.2, 86.7)
- removed the R24 at (107.3, 90.0)
- removed the R25 at (107.3, 91.8)
- removed the R25 at (225.2, 88.8)
- removed the R27 at (240.2, 41.4)
- removed the R27 at (163.7, 90.5)
- removed the R28 at (163.7, 92.2)
- removed the R28 at (240.2, 43.6)
- removed the R3 at (225.2, 80.2)
- removed the R3 at (161.2, 83.5)
- removed the R31 at (166.1, 80.0)
- removed the R31 at (240.2, 45.7)
- removed the R32 at (243.7, 32.8)
- removed the R32 at (166.1, 81.8)
- removed the R35 at (107.3, 93.5)
- removed the R35 at (225.2, 91.0)
- removed the R36 at (107.3, 95.2)
- removed the R36 at (225.2, 93.1)
- removed the R37 at (109.8, 83.0)
- removed the R37 at (225.2, 95.3)
- removed R38: 1k, RES_0402:RES_0402
- removed R38: 1k, Resistor_SMD:R_0201_0603Metric
- removed R39, RC1: 5k1, Resistor_SMD:R_0201_0603Metric
- removed the R5 at (236.8, 37.1)
- removed the R5 at (161.2, 87.0)
- removed the R6 at (236.8, 39.2)
- removed the R6 at (161.2, 88.8)
- removed the R7 at (236.8, 41.4)
- removed the R7 at (161.2, 90.5)
- removed RC1: 5k1, R_0805_5K1:R_0805_5K1
- removed the R_ENT1 at (166.1, 83.5)
- removed the R_ENT1 at (240.0, 63.1)
- removed the R_ENT2 at (240.0, 64.8)
- removed the R_ENT2 at (166.1, 85.2)
- removed the R_FBB1 at (166.1, 87.0)
- removed the R_FBB1 at (240.0, 66.6)
- removed the R_FBB2 at (166.1, 88.8)
- removed the R_FBB2 at (242.5, 63.1)
- removed the R_FBT1 at (243.7, 39.2)
- removed the R_FBT1 at (166.1, 90.5)
- removed the R_FBT2 at (166.1, 92.2)
- removed the R_FBT2 at (243.7, 41.4)
- removed R_FF2, R_pull1: R, Resistor_SMD:R_0201_0603Metric
- removed R_FF2, R_pull1, R_pull2: R, RES_0402:RES_0402
- removed the R_PG2 at (242.5, 66.6)
- removed the R_PG2 at (168.6, 81.8)
- removed the R_RT1 at (168.6, 83.5)
- removed the R_RT1 at (244.9, 63.1)
- removed the R_RT2 at (168.6, 85.2)
- removed the R_RT2 at (244.9, 64.8)
- removed S3, S4: TL3305CF160QG, E-Switch_7mm:SW_TL3305CF160QG
- removed SW2, SW3: SW_Push, Button_Switch_SMD:SW_Push_1P1T-MP_NO_Horizontal_Alps_SKRTLAE010
- removed the U1 at (217.0, 35.1)
- removed the U1 at (177.1, 81.8)
- removed the U10 at (165.0, 106.0)
- removed the U10 at (217.0, 48.6)
- removed U14: ADS1114IRUGR, ADS1114:RUG10
- removed U14: LM61460AASQRJRRQ1, DCDC_LM61460:VQFN-HR14_RJR_TEX
- removed U15: TPS1120DR, 2 PMOS:D8
- removed U18: ST1L05APU33R, LDO ST1L05A:DFN_5APU33R_STM
- removed the U2 at (94.0, 95.3)
- removed the U2 at (231.2, 76.9)
- removed the U3 at (177.1, 88.4)
- removed the U3 at (217.0, 41.8)
- removed the U4 at (243.1, 58.9)
- removed the U4 at (177.0, 101.6)
- removed the U5 at (177.1, 95.0)
- removed the U5 at (224.5, 62.2)
- removed the U6 at (217.8, 94.7)
- removed the U6 at (99.6, 77.9)
- removed the U9 at (233.3, 63.1)
- removed the U9 at (165.0, 99.3)
- removed the XTAL1 at (240.7, 90.3)
- removed the XTAL1 at (140.5, 101.0)
- added C1: 100nF, Capacitor-0402:Capacitor_0402, F.Cu at (186.5, 71.8)
- added C10: 10nF, Capacitor-0402:Capacitor_0402, F.Cu at (189.9, 78.3)
- added C11: 100 nF, Capacitor-0402:Capacitor_0402, F.Cu at (189.9, 80.5)
- added C2: 10nF, Capacitor-0402:Capacitor_0402, F.Cu at (186.5, 74.0)
- added C3: 100nF, Capacitor-0402:Capacitor_0402, F.Cu at (186.5, 76.2)
- added C4: 10nF, Capacitor-0402:Capacitor_0402, F.Cu at (186.5, 78.3)
- added C6: 10nF, Capacitor-0402:Capacitor_0402, F.Cu at (186.5, 82.7)
- added C7: 10nF, Capacitor-0402:Capacitor_0402, F.Cu at (189.9, 71.8)
- added C8: 10nF, Capacitor-0402:Capacitor_0402, F.Cu at (189.9, 74.0)
- added C9: 100nF, Capacitor-0402:Capacitor_0402, F.Cu at (189.9, 76.2)
- added CR1: VLMC3100-GS08, LED-Green_VLMC3100-GS08:LED_PLCC_VSMB, F.Cu at (154.1, 147.5)
- added CR2: VLMC3100-GS08, LED-Green_VLMC3100-GS08:LED_PLCC_VSMB, F.Cu at (189.0, 86.1)
- added CR3: VLMC3100-GS08, LED-Green_VLMC3100-GS08:LED_PLCC_VSMB, F.Cu at (189.0, 90.7)
- added CR4: VLMC3100-GS08, LED-Green_VLMC3100-GS08:LED_PLCC_VSMB, F.Cu at (189.0, 95.3)
- added CR5: VLMC3100-GS08, LED-Green_VLMC3100-GS08:LED_PLCC_VSMB, F.Cu at (189.0, 99.9)
- added CV1: 1uF, Capacitor-0402:Capacitor_0402, F.Cu at (130.8, 129.9)
- added CV10: 100nF, Capacitor-0402:Capacitor_0402, F.Cu at (134.2, 134.2)
- added CV11: 100nF, Capacitor-0402:Capacitor_0402, F.Cu at (134.2, 136.4)
- added CV12: 100nF, Capacitor-0402:Capacitor_0402, F.Cu at (134.2, 138.6)
- added CV13: 1uF, Capacitor-0402:Capacitor_0402, F.Cu at (134.2, 140.7)
- added CV14: 100nF, Capacitor-0402:Capacitor_0402, F.Cu at (134.2, 142.9)
- added CV15: 4.7uF, Capacitor-0402:Capacitor_0402, F.Cu at (137.5, 129.9)
- added CV16: 4.7uF, Capacitor-0402:Capacitor_0402, F.Cu at (137.5, 132.1)
- added CV17: 1uF, Capacitor-0402:Capacitor_0402, F.Cu at (137.5, 134.2)
- added CV18: 100nF, Capacitor-0402:Capacitor_0402, F.Cu at (137.5, 136.4)
- added CV2: 100nF, Capacitor-0402:Capacitor_0402, F.Cu at (130.8, 132.1)
- added CV3: 1uF, Capacitor-0402:Capacitor_0402, F.Cu at (130.8, 134.2)
- added CV4: 100nF, Capacitor-0402:Capacitor_0402, F.Cu at (130.8, 136.4)
- added CV5: 100nF, Capacitor-0402:Capacitor_0402, F.Cu at (130.8, 138.6)
- added CV6: 1uF, Capacitor-0402:Capacitor_0402, F.Cu at (130.8, 140.7)
- added CV7: 100nF, Capacitor-0402:Capacitor_0402, F.Cu at (130.8, 142.9)
- added CV8: 100nF, Capacitor-0402:Capacitor_0402, F.Cu at (134.2, 129.9)
- added CV9: 100nF, Capacitor-0402:Capacitor_0402, F.Cu at (134.2, 132.1)
- added C_BIAS1: 1u, Capacitor-0603:Capacitor_0603, F.Cu at (182.3, 96.4)
- added C_BT1: 100n, Capacitor-0402:Capacitor_0402, F.Cu at (193.2, 78.3)
- added C_BT2: 100n, Capacitor-0402:Capacitor_0402, F.Cu at (193.2, 80.5)
- added C_IN-BLK1: 10u, Capacitor-4mm:Capacitor_4mm, F.Cu at (196.9, 87.4)
- added C_IN-BLK2: 10u, Capacitor-4mm:Capacitor_4mm, F.Cu at (196.9, 94.8)
- added C_IN1: 4.7u, Capacitor-1206:Capacitor_1206, F.Cu at (187.4, 103.8)
- added C_IN2: 4.7u, Capacitor-1206:Capacitor_1206, F.Cu at (187.4, 106.9)
- added C_IN3: 4.7u, Capacitor-1206:Capacitor_1206, F.Cu at (187.4, 110.1)
- added C_IN4: 4.7u, Capacitor-1206:Capacitor_1206, F.Cu at (187.4, 113.3)
- added C_IN_HFI1: 100n, Capacitor-0402:Capacitor_0402, F.Cu at (196.6, 71.8)
- added C_IN_HFI2: 100n, Capacitor-0402:Capacitor_0402, F.Cu at (196.6, 74.0)
- added C_OUT1: 22u, Capacitor-0805:Capacitor_0805, F.Cu at (182.5, 72.3)
- added C_OUT10: 10u, Capacitor-0805:Capacitor_0805, F.Cu at (182.5, 93.6)
- added C_OUT11: 100u, Capacitor-6mm:Capacitor_6mm, F.Cu at (216.7, 99.1)
- added C_OUT2: 22u, Capacitor-0805:Capacitor_0805, F.Cu at (182.5, 75.3)
- added C_OUT3: 1u, Capacitor-0603:Capacitor_0603, F.Cu at (182.3, 98.9)
- added C_OUT4: 10u, Capacitor-0805:Capacitor_0805, F.Cu at (182.5, 78.4)
- added C_OUT5: 22u, Capacitor-0805:Capacitor_0805, F.Cu at (182.5, 81.4)
- added C_OUT6: 10u, Capacitor-0805:Capacitor_0805, F.Cu at (182.5, 84.5)
- added C_OUT7: 22u, Capacitor-0805:Capacitor_0805, F.Cu at (182.5, 87.5)
- added C_OUT8: 10u, Capacitor-0805:Capacitor_0805, F.Cu at (182.5, 90.6)
- added C_OUT9: 560u, Capacitor-8mm:Capacitor_8mm, F.Cu at (207.5, 89.0)
- added C_VCC1: 1u, Capacitor-0603:Capacitor_0603, F.Cu at (182.3, 101.5)
- added C_VCC2: 1u, Capacitor-0603:Capacitor_0603, F.Cu at (182.3, 104.0)
- added D1: RSX301L-30DDTE25, Diode-Schottky_RSX301L:DIOM5026X220N, F.Cu at (214.3, 106.1)
- added D2: PMEG2010ER, Diode-Schottky_PMEG2010ER:SODFL3517X110N, F.Cu at (155.4, 126.7)
- added D4: RSX301L-30DDTE25, Diode-Schottky_RSX301L:DIOM5026X220N, F.Cu at (214.3, 114.8)
- added IC1: NSVT30010MXV6T1G, 2 PNP:SOTFL50P160X60-6N, F.Cu at (182.0, 106.8)
- added IC2: NSVT30010MXV6T1G, 2 PNP:SOTFL50P160X60-6N, F.Cu at (182.0, 109.8)
- added IC3: ADS1115IRUGR, ADS1115:ADS1115IRUGR, F.Cu at (160.1, 114.5)
- added J16: DX07S016JA1R1500, USBC-DX07S016JA1:JAE_DX07S016JA1R1500, F.Cu at (134.8, 122.5)
- added J18: Conn_01x01_Socket, Pico_Conn1x1:Pico_01pin, F.Cu at (220.9, 86.9)
- added J19: Conn_01x01_Socket, Pico_Conn1x1:Pico_01pin, F.Cu at (225.0, 86.9)
- added J7: BM03B-SRSS-TBLFSN, SWD_Con:CONN_BM03B-SRSS-TBLFSN_JST, F.Cu at (156.2, 122.3)
- added L1: 15u, Inductor-10.1x10:Inductor_10.1x10, F.Cu at (219.4, 76.7)
- added MCU1: RP2040, Package_DFN_QFN:QFN-56-1EP_7x7mm_P0.4mm_EP3.2x3.2mm, F.Cu at (154.6, 140.5)
- added Q1: 2N7002H6327XTSA2, NMOS_2N7002:PG-SOT23-3-5_INF_MIN, F.Cu at (166.3, 114.5)
- added R1: 100, Resistor-0402:RES_0402, F.Cu at (145.4, 94.9)
- added R12: 10K, Resistor-0402:RES_0402, F.Cu at (148.9, 97.1)
- added R13: 10K, Resistor-0402:RES_0402, F.Cu at (148.9, 99.3)
- added R2: 100, Resistor-0402:RES_0402, F.Cu at (145.4, 97.1)
- added R22: 27, Resistor-0603:RES_0603, F.Cu at (137.2, 145.3)
- added R23: 27, Resistor-0603:RES_0603, F.Cu at (137.2, 147.8)
- added R24: 100, Resistor-0402:RES_0402, F.Cu at (140.9, 132.1)
- added R25: 100, Resistor-0402:RES_0402, F.Cu at (140.9, 134.2)
- added R27: 1k, Resistor-0402:RES_0402, F.Cu at (152.3, 99.3)
- added R28: 1k, Resistor-0402:RES_0402, F.Cu at (152.3, 101.4)
- added R3: 1k, Resistor-0402:RES_0402, F.Cu at (140.9, 129.9)
- added R31: 2k, Resistor-0402:RES_0402, F.Cu at (152.3, 103.6)
- added R32: 1k, Resistor-0402:RES_0402, F.Cu at (152.3, 105.7)
- added R33: 5k1, Resistor-0805:RES_0805, F.Cu at (148.8, 121.5)
- added R35: 1k, Resistor-0402:RES_0402, F.Cu at (140.9, 142.9)
- added R36: 5k1, Resistor-0805:RES_0805, F.Cu at (148.8, 125.8)
- added R37: 10k, Resistor-0402:RES_0402, F.Cu at (152.3, 110.1)
- added R5: 2k, Resistor-0402:RES_0402, F.Cu at (145.4, 101.4)
- added R6: 100, Resistor-0402:RES_0402, F.Cu at (145.4, 103.6)
- added R7: 100, Resistor-0402:RES_0402, F.Cu at (145.4, 105.7)
- added R_BIAS1: 10, Resistor-0402:RES_0402, F.Cu at (155.7, 94.9)
- added R_BT1: 100, Resistor-0402:RES_0402, F.Cu at (155.7, 97.1)
- added R_BT2: 50, Resistor-0402:RES_0402, F.Cu at (155.7, 99.3)
- added R_ENB1: 35k, Resistor-0402:RES_0402, F.Cu at (155.7, 101.4)
- added R_ENB2: 100k, Resistor-0603:RES_0603, F.Cu at (220.0, 105.2)
- added R_ENT1: 400k, Resistor-0805:RES_0805, F.Cu at (204.9, 114.9)
- added R_ENT2: 1.15M, Resistor-0603:RES_0603, F.Cu at (220.0, 107.8)
- added R_FBB1: 24k9, Resistor-0603:RES_0603, F.Cu at (220.0, 110.3)
- added R_FBB2: 9k09, Resistor-0603:RES_0603, F.Cu at (220.0, 112.9)
- added R_FBT1: 100K, Resistor-0603:RES_0603, F.Cu at (220.0, 115.4)
- added R_FBT2: 100K, Resistor-0603:RES_0603, F.Cu at (223.7, 105.2)
- added R_PG2: 100K, Resistor-0603:RES_0603, F.Cu at (223.7, 110.3)
- added R_RT1: 33k2, Resistor-0603:RES_0603, F.Cu at (223.7, 112.9)
- added R_RT2: 33k2, Resistor-0603:RES_0603, F.Cu at (223.7, 115.4)
- added S1: TL1017AABF160QG, E-Switch_Small:TL1017AABF160QG, F.Cu at (146.3, 131.6)
- added S2: TL1017AABF160QG, E-Switch_Small:TL1017AABF160QG, F.Cu at (146.3, 138.2)
- added U1: MAX31856MUD+T, Thermocouple:21-0066J_14_MXM, F.Cu at (175.6, 97.2)
- added U10: LM61460AASQRJRRQ1, Thermocouple:21-0066J_14_MXM, F.Cu at (175.6, 110.8)
- added U2: W25Q128JVSIQ TR, NOR Flash:SOIC_208MIL_WIN, F.Cu at (155.2, 132.3)
- added U3: MAX31856MUD+T, Thermocouple:21-0066J_14_MXM, F.Cu at (175.6, 104.0)
- added U4: PCA9306DP_118, I2C Voltage Translator:TSSOP8_SOT505-1_NXP, F.Cu at (204.9, 110.4)
- added U5: MAX485CSA+T, MCP9808-TempSensor:DFN8_2x3MC_MCH, F.Cu at (216.7, 91.8)
- added U6: ESD7L5.0DT5G, ESD7L5-Diode:SOT-723_0P85X1P25_ONS, F.Cu at (159.6, 146.8)
- added U9: MAX31856MUD+T, DCDC_LM61460:VQFN-HR14_RJR_TEX, F.Cu at (194.9, 107.2)
- added XTAL1: ASE-12.000MHZ-LC-T, AS12MHz:ASE-3.2X2.5_ABR, F.Cu at (147.1, 144.4)
- C12, C14: footprint Capacitor_SMD:C_0201_0603Metric -> Capacitor-0402:Capacitor_0402
- C13: value 100nF -> 10nF; footprint Capacitor_SMD:C_0201_0603Metric -> Capacitor-0402:Capacitor_0402
- C23: footprint Capacitor_0402:Capacitor_0402 -> Capacitor-0402:Capacitor_0402
- C5: value 100 nF -> 10nF; footprint Capacitor_SMD:C_0201_0603Metric -> Capacitor-0402:Capacitor_0402
- C_FF1: value C -> 22p; footprint Capacitor_0402:Capacitor_0402 -> Capacitor-0402:Capacitor_0402
- C_IN_HFI3, C_IN_HFI4: value C -> 100n; footprint Capacitor_0402:Capacitor_0402 -> Capacitor-0402:Capacitor_0402
- D3: footprint Schottky RSX301L:DIOM5026X220N -> Diode-Schottky_RSX301L:DIOM5026X220N
- J1, J13, J14, J5: value Conn_01x01_Socket -> 1190298; footprint Button_Switch_THT:SW_Lever_1P2T_NKK_GW12LxH -> LPT Conn 3 Entradas:1190298
- J15: footprint Button_Switch_THT:SW_Lever_1P2T_NKK_GW12LxH -> Pico_Conn1x1:Pico_01pin
- J17: value USB_C -> XT60PW-M; footprint Connector_USB:USB_C_Plug_JAE_DX07P024AJ1 -> Conn XT60PW-M:AMASS_XT60PW-M
- J2: value Conn_01x01_Socket -> 1190297; footprint Button_Switch_THT:SW_Lever_1P2T_NKK_GW12LxH -> LPT Conn 2 Entradas:1190297
- J3, J4: value XT30UPB-M -> XT60PW-M; footprint AMASS_XT30UPB-M:CONN_XT30UPB-M_AMA -> Conn XT60PW-M:AMASS_XT60PW-M
- J6: value XT30UPB-M -> 1190298; footprint AMASS_XT30UPB-M:CONN_XT30UPB-M_AMA -> LPT Conn 3 Entradas:1190298
- J8: value Conn_01x01_Socket -> XT60PW-M
- L2: value L -> 10u; footprint Inductor_SMD:L_Neosid_SM-PIC0512H -> Inductor-11.5x10:Inductor_11.5x10
- R10, R9: value 10K -> 20K; footprint RES_0402:RES_0402 -> Resistor-0402:RES_0402
- R11: value 20K -> 10K; footprint RES_0402:RES_0402 -> Resistor-0402:RES_0402
- R14, R17, R34, R4, R40: footprint RES_0402:RES_0402 -> Resistor-0402:RES_0402
- R15: value 20K -> 2k; footprint RES_0402:RES_0402 -> Resistor-0402:RES_0402
- R16: value 120 -> 100; footprint RES_0402:RES_0402 -> Resistor-0402:RES_0402
- R18: value 47 -> 100; footprint RES_0402:RES_0402 -> Resistor-0402:RES_0402
- R19, R20: value 47 -> 2k; footprint RES_0402:RES_0402 -> Resistor-0402:RES_0402
- R21: value 47 -> 1k; footprint RES_0402:RES_0402 -> Resistor-0402:RES_0402
- R26: value 130 -> 1k; footprint RES_0402:RES_0402 -> Resistor-0402:RES_0402
- R29: value 2k -> 10k; footprint Resistor_SMD:R_0201_0603Metric -> Resistor-0402:RES_0402
- R30: value 2k -> 665; footprint Resistor_SMD:R_0201_0603Metric -> Resistor-0402:RES_0402
- R8: value 10K -> 120; footprint RES_0402:RES_0402 -> Resistor-0402:RES_0402
- R_FF1: value R -> 1k; footprint RES_0402:RES_0402 -> Resistor-0402:RES_0402
- R_PG1: value R -> 100K; footprint RES_0402:RES_0402 -> Resistor-0603:RES_0603
- U16: value TPS1120DR -> IRLZ44NPBF; footprint 2 PMOS:D8 -> NMOS IRLZ44:PG-TO220-3_INF
- U8: value PCA9306DP_118 -> MCP9808T-E/MC; footprint I2C Voltage Translator:TSSOP8_SOT505-1_NXP -> DCDC_LM61460:VQFN-HR14_RJR_TEX
- moved R18 119.7 mm to (148.9, 110.1)
- moved R19 119.7 mm to (148.9, 112.2)
- moved R40 118.3 mm to (152.3, 112.2)
- moved R34 117.0 mm to (152.3, 107.9)
- moved R20 105.3 mm to (152.3, 94.9)
- moved R21 105.3 mm to (152.3, 97.1)
- moved U16 89.2 mm to (162.6, 109.6)
- moved J8 88.5 mm to (203.3, 95.8)
- moved J6 84.5 mm to (172.7, 54.3)
- moved U13 82.6 mm to (194.9, 112.9)
- moved J17 77.8 mm to (171.7, 81.9), turned to 0 degrees
- moved J15 73.6 mm to (216.8, 86.9)
- moved D3 63.8 mm to (214.3, 110.5)
- moved R_PG1 61.7 mm to (223.7, 107.8)
- moved L2 57.1 mm to (205.4, 76.7)
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Connections:
- C12 pad 1: Net-(U5-T+) -> GND
- C12 pad 2: GND -> +3.3V
- C13 pad 1: Net-(U5-T+) -> GND
- C13 pad 2: Net-(U5-T-) -> +3.3V
- C14 pad 1: Net-(U5-T-) -> +3.3V
- C23 pad 1: Net-(U8-EN) -> Net-(U4-EN)
- C5 pad 1: +5V -> GND
- C5 pad 2: GND -> +3.3V
- C_FF1 pad 2: GND -> Net-(U10-FB)
- C_IN_HFI3 pad 1: +12V -> +16V
- C_IN_HFI4 pad 1: +12V -> +16V
- J1 pad 2: (no net) -> /THERMO1 T+
- J1 pad 3: (no net) -> /THERMO1 T-
- J13 pad 2: (no net) -> +12V
- J13 pad 3: (no net) -> /ADC_AIN1
- J14 pad 1: /ADC_AIN0 -> +12V
- J14 pad 2: (no net) -> +12V
- J14 pad 3: (no net) -> /ADC_AIN2
- J15 pad 1: GND -> /RP2040 Standard/GP27_ADC1
- J17 pad S1: unconnected-(J17-SHIELD-PadS1)_2 -> (no net)
- J2 pad 1: Net-(J2-Pin_1) -> Net-(J2-1.1)
- J2 pad 2: (no net) -> Net-(J2-1.1)
- J2 pad 3: (no net) -> Net-(J2-2.1)
- J5 pad 1: Net-(J5-Pin_1) -> +12V
- J5 pad 2: (no net) -> +12V
- J5 pad 3: (no net) -> /ADC_AIN0
- J6 pad 1: GND -> /THERMO2 T-
- J6 pad 2: +16V -> /THERMO2 T-
- J8 pad 1: /THERMO1 T- -> GND
- J8 pad 2: (no net) -> +16V
- L2 pad 1: Net-(U14-SW) -> Net-(U13-SW)
- L2 pad 2: +5V -> +12V
- R10 pad 1: +3.3V -> Net-(J2-1.1)
- R10 pad 2: /RS_RX -> GND
- R11 pad 1: +5V -> +3.3V
- R11 pad 2: Net-(J5-Pin_1) -> /RS_RX
- R15 pad 1: Net-(J2-Pin_1) -> +3.3V
- R15 pad 2: GND -> /TEMP ALERT
- R16 pad 1: Net-(J2-Pin_1) -> Net-(U9-T+)
- R16 pad 2: Net-(J5-Pin_1) -> /THERMO3 T+
- R18 pad 2: +3.3V -> /THERMO3 T-
- R19 pad 1: Net-(U15-2SOURCE) -> +3.3V
- R19 pad 2: +3.3V -> /TEMP SDL I2C
- R20 pad 1: Net-(U16-1SOURCE) -> +3.3V
- R20 pad 2: +3.3V -> /TEMP SDA I2C
- R21 pad 1: Net-(U16-2SOURCE) -> Net-(IC1-E1)
- R21 pad 2: +3.3V -> Net-(CR2-Pad1)
- R26 pad 1: Net-(LED1-A) -> /RP2040 Standard/~{RST}
- R26 pad 2: /RP2040 Standard/GP25/PWM4 B -> Net-(MCU1-RUN)
- R29 pad 1: +5V -> Net-(XTAL1-TRI-STATE(STBY))
- R29 pad 2: Net-(U2-SDA) -> +3.3V
- R30 pad 1: +5V -> Net-(MCU1-GPIO25)
- R34 pad 2: Net-(U14-SCL) -> Net-(IC3-SCL)
- R4 pad 1: Net-(U8-EN) -> Net-(U4-EN)
- R40 pad 2: Net-(U14-SDA) -> Net-(IC3-SDA)
- R8 pad 1: /RS_TX -> Net-(J2-1.1)
- R8 pad 2: +3.3V -> Net-(J2-2.1)
- R9 pad 1: +3.3V -> +5V
- R9 pad 2: /RS_ENABLE -> Net-(J2-2.1)
- R_FF1 pad 1: +12V -> /5V REG
- R_PG1 pad 1: /DC.DC1 PGOOD -> /DC.DC2 PGOOD
- R_PG1 pad 2: +12V -> /5V REG
- U13 pad 13: Net-(U13-CBOOT) -> Net-(U13-RBOOT)
- U13 pad 2: Net-(U13-VCC) -> /DC.DC1 PGOOD
- U16 pad 1: Net-(U16-1SOURCE) -> /Valve Control 3
- U16 pad 2: /THERMO3_~{CS} -> Net-(D4-A)
- U16 pad 3: Net-(U16-2SOURCE) -> GND
- U7 pad 3: /5V REG -> /RP2040 Standard/+5V
- U8 pad 1: GND -> /TEMP SDA I2C
- U8 pad 2: +3.3V -> /TEMP SDL I2C
- U8 pad 3: /ADC SDL I2C -> /TEMP ALERT
- U8 pad 4: /ADC SDA I2C -> GND
- U8 pad 5: Net-(U14-SDA) -> GND
- U8 pad 6: Net-(U14-SCL) -> GND
- U8 pad 7: Net-(U8-EN) -> GND
- U8 pad 8: Net-(U8-EN) -> +3.3V
Other:
- board size 100 x 60 mm -> 100 x 100 mm
