File: Boards/Rocket Systems/RP2040 P/RP2040 P.kicad_sch (KiCad schematic)
At the start: 2 parts, among them J1 Conn_01x20_Pin, J3 Conn_01x18_Pin

Commit message: Repo Refactor and new systems update
Other:
- sheet RP2040 Standard renamed RP2040 Power
- sheet RP2040 Power: file RP2040 Standard.kicad_sch -> RP2040 Power Design.kicad_sch
- note added: "RP2040 Power"
- note removed: "RP2040 Standard"
- title: RP2040 Standard Design -> RP2040 Power
Changed lines of the file:
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@@
 	(paper "User" 160 160)
 	(title_block
-		(title "RP2040 Standard Design")
+		(title "RP2040 Power")
 		(date "2024-12-29")
 		(rev "V2")
@@
 		)
 	)
-	(text "RP2040 Standard\n"
+	(text "RP2040 Power\n"
 		(exclude_from_sim no)
 		(at 15.875 20.955 0)
@@
 			(color 0 0 0 0.0000)
 		)
-		(property "Sheetname" "RP2040 Standard"
+		(property "Sheetname" "RP2040 Power"
 			(at 54.61 37.3884 0)
 			(effects
@@
 			)
 		)
-		(property "Sheetfile" "RP2040 Standard.kicad_sch"
+		(property "Sheetfile" "RP2040 Power Design.kicad_sch"
 			(at 54.61 104.775 0)
 			(effects
@@
 		)
 		(instances
-			(project "RP2040 Standard Design"
+			(project "RP2040 P"
 				(path "/7712695e-3038-4da8-a54c-20dbd93db58d"
 					(page "2")

Commit message: Alterações RP2040 P
Other:
- moved on the sheet: J1, J3
