File: Boards/Development Boards/RP2040 P/RP2040 Power Design.kicad_sch (KiCad schematic)
At the start: 222 parts, among them J2 BM03B-SRSS-TBLFSN, U1 W25Q128JVSIQ TR, U3 ST1L05APU33R

Commit message: Atualização 2 RP2040 P
Parts:
- removed C?: 4.7u, symbol Device:C_Small
- removed C? (x4): 2.2u, Capacitor-0402:Capacitor_0402, symbol Device:C_Small
- removed C? (x8), C_BT? (x3), C_IN_HFI? (x6): 100n, Capacitor-0402:Capacitor_0402, symbol Device:C_Small
- removed C? (x3): 10n, Capacitor-0402:Capacitor_0402, symbol Device:C_Small
- removed C?: C, Capacitor-0402:Capacitor_0402, symbol Device:C_Small
- removed C? (x4): 1u, symbol Device:C_Small
- removed C? (x3): 1u, Capacitor-0402:Capacitor_0402, symbol Device:C_Small
- removed C? (x2): 470n, Capacitor-0402:Capacitor_0402, symbol Device:C_Small
- removed C? (x2): 100n, symbol Device:C_Small
- removed C?: 1n, symbol Device:C_Small
- removed CR? (x4): VLMC3100-GS08, LED_PLCC_VSMB, symbol GreenLED__VLMC3100-GS08:VLMC3100-GS08
- removed CR?: VLMC3100-GS08, LED-Green_VLMC3100-GS08:LED_PLCC_VSMB, symbol GreenLED__VLMC3100-GS08:VLMC3100-GS08
- removed CR? (x5): VLMT3100-GS08, LED_PLCC_VSMB, symbol VLMT3100-GS08:VLMT3100-GS08
- removed C_BIAS? (x2), C_OUT?, C_VCC? (x3): 1u, Capacitor-0603:Capacitor_0603, symbol Device:C_Small
- removed C_FF?: 22p, Capacitor-0402:Capacitor_0402, symbol Device:C_Small
- removed C_IN-BLK? (x3): 10u, Capacitor-4mm:Capacitor_4mm, symbol Device:C_Small
- removed C_IN? (x6): 4.7u, Capacitor-1206:Capacitor_1206, symbol Device:C_Small
- removed C_OUT? (x6): 22u, Capacitor-0805:Capacitor_0805, symbol Device:C_Small
- removed C_OUT?: 560u, Capacitor-8mm:Capacitor_8mm, symbol Device:C_Small
- removed C_OUT?: 100u, Capacitor-6mm:Capacitor_6mm, symbol Device:C_Small
- removed C_OUT? (x4): 10u, Capacitor-0805:Capacitor_0805, symbol Device:C_Small
- removed C_OUT?: 100u, Capacitor-8mm:Capacitor_8mm, symbol Device:C_Small
- removed C_OUT? (x2): 47u, Capacitor-0805:Capacitor_0805, symbol Device:C_Small
- removed D? (x2): RSX301L, DIOM5026X220N, symbol RSX301L-30DDTE25:RSX301L-30DDTE25
- removed D? (x2): RB095BGE, RD3P175SNFRATL, symbol RB095BGE-30TL:RB095BGE-30TL
- removed D?: SP3004-04XTG, SOTFL50P160X60-6N, symbol SP3004-04XTG:SP3004-04XTG
- removed IC?: CYPD3177-24LQXQT, QFN50P400X400X60-25N-D, symbol CYPD3177-24LQXQT:CYPD3177-24LQXQT
- removed IC?: INA2181A4IDSQR, SON40P200X200X80-11N, symbol INA2181A4IDSQR:INA2181A4IDSQR
- removed IC? (x2): NSVT30010MXV6T1G, 2 PNP:SOTFL50P160X60-6N, symbol NSVT30010MXV6T1G:NSVT30010MXV6T1G
- removed IC?: ADS1115IRUGR, ADS1115IRUGR, symbol ADS1115IRUGR:ADS1115IRUGR
- removed IC?: PCA9306GM,125, PCA9570GMH, symbol PCA9306GM_125:PCA9306GM,125
- removed IC?: INA181A4QDCKRQ1, SOT65P210X110-6N, symbol INA181A4QDCKRQ1:INA181A4QDCKRQ1
- removed J?: DX07S016JA1R1500, DX07S016JA1R1500:JAE_DX07S016JA1R1500, symbol DX07S016JA1R1500:DX07S016JA1R1500
- removed L?: 2.2u, Inductor-10.1x10:Inductor_10.1x10, symbol Device:L
- removed L_SW? (x2): 15u, Inductor-10.1x10:Inductor_10.1x10, symbol Device:L
- removed L_SW?: 10u, Inductor-11.5x10:Inductor_11.5x10, symbol Device:L
- removed Q? (x2): DMP3098LSD-13, SOIC127P600X175-8N, symbol DMP3098LSD-13:DMP3098LSD-13
- removed Q? (x3): 2N7002H6327XTSA2, NMOS_2N7002:PG-SOT23-3-5_INF_MIN, symbol NMOS_2N7002:2N7002H6327XTSA2
- removed R? (x12), R_FF?: 1k, Resistor-0402:RES_0402, symbol Device:R
- removed R?: DNP, Resistor-0402:RES_0402, symbol Device:R
- removed R? (x2): 54k2, Resistor-0402:RES_0402, symbol Device:R
- removed R? (x3): 20K, Resistor-0402:RES_0402, symbol Device:R
- removed R? (x3), R_BT?: 100, Resistor-0402:RES_0402, symbol Device:R
- removed R? (x3): 160, Resistor-0402:RES_0402, symbol Device:R
- removed R? (x11): 2k, Resistor-0402:RES_0402, symbol Device:R
- removed R?: 200k, Resistor-0402:RES_0402, symbol Device:R
- removed R? (x2): 50k, symbol Device:R
- removed R? (x3): 370, Resistor-0402:RES_0402, symbol Device:R
- removed R?: 120, Resistor-0402:RES_0402, symbol Device:R
- removed R? (x3): 10K, Resistor-0402:RES_0402, symbol Device:R
- removed R? (x2): 30k, Resistor-0402:RES_0402, symbol Device:R
- removed R? (x4): 500, Resistor-0402:RES_0402, symbol Device:R
- removed R?: 10k, symbol Device:R
- removed R?: PTS060301B100RP100, RESC1508X55N, symbol PTS060301B100RP100:PTS060301B100RP100
- removed R_BIAS? (x2): 5, Resistor-0402:RES_0402, symbol Device:R
- removed R_BT? (x2): 50, Resistor-0402:RES_0402, symbol Device:R
- removed R_ENB?: 63k4, Resistor-0402:RES_0402, symbol Device:R
- removed R_ENB?: 45k3, Resistor-0402:RES_0402, symbol Device:R
- removed R_ENB?: 100k, Resistor-0603:RES_0603, symbol Device:R
- removed R_ENT?: 931k, Resistor-0603:RES_0603, symbol Device:R
- removed R_ENT?: 422k, Resistor-0402:RES_0402, symbol Device:R
- removed R_ENT?: 590k, Resistor-0402:RES_0402, symbol Device:R
- removed R_FBB?: 8k66, Resistor-0603:RES_0603, symbol Device:R
- removed R_FBB?: 50, Resistor-0603:RES_0603, symbol Device:R
- removed R_FBB?: 30, Resistor-0603:RES_0603, symbol Device:R
- removed R_FBB?: 12k6, Resistor-0603:RES_0603, symbol Device:R
- removed R_FBB?: 120, Resistor-0603:RES_0603, symbol Device:R
- removed R_FBB?: 22k1, Resistor-0603:RES_0603, symbol Device:R
- removed R_FBT? (x3), R_PG? (x3): 100K, Resistor-0603:RES_0603, symbol Device:R
- removed R_RT? (x3): 33k2, Resistor-0603:RES_0603, symbol Device:R
- removed Rsense? (x2): 2.5m, symbol Device:R
- removed Rsense?: 7.5m, symbol Device:R
- removed U? (x3): LM61460AASQRJRRQ1, VQFN-HR14_RJR_TEX, symbol DCDC_LM61460:LM61460AASQRJRRQ1
- removed U?: MAX31856MUD+T, Thermocouple:21-0066J_14_MXM, symbol MAX31856MUD-T:MAX31856MUD+T
- removed U?: MAX485CSA+T, RS Transceiver:21-0041-3-M_90-0096-8L_MXM, symbol RS_Transceiver:MAX485CSA+T
Connections:
- no-connect marks 9 -> 5
Other:
- note removed: "4 Channel ESD Diode"
- note removed: ">15V to 12V Converter"
- note removed: ">15V to 5V Converter"
- note removed: ">15V to 8.4V Converter"
- note removed: "ADC + I2C Translator"
- note removed: "Anti-Aliasing Filter: Fs = 860Hz => Fc = 430Hz"
- note removed: "Buck Converters"
- note removed: "C_IN-BLK1 and C_OUT6 are electrolytic polarized capacitors! All others are ceramic X7R capacitors with appropriate voltage ratings."
- note removed: "C_IN-BLK2 and C_OUT10 are electrolytic polarized capacitors! All others are ceramic X7R capacitors with appropriate voltage ratings."
- note removed: "C_IN-BLK3 and C_OUT15 are electrolytic polarized capacitors! All others are ceramic X7R capacitors with appropriate voltage ratings."
- note removed: "Capacitor to adjust signal"
- note removed: "Current Sensor 1"
- note removed: "Current Sensor 2"
- note removed: "DC.DC1 VCC coloca PGOOD a 3.3V"
- note removed: "DC.DC2 VCC coloca PGOOD a 3.3V"
- note removed: "DC.DC3 VCC coloca PGOOD a 3.3V"
- note removed: "EMI Filter"
- note removed: "I2C ADDR is 0x08"
- note removed: "LEDs Drivers"
- note removed: "POWER (GREEN)"
- note removed: "RS Transceiver"
- note removed: "STATUS"
- note removed: "THERMO FAULT (RED) & RS ENABLED (GREEN)"
- note removed: "Temperature Sensor"
- note removed: "Thermocouple"
- note removed: "This ADC is to be set at max sampling rate (860Hz) With AIN0 and AIN1 on differential mode and AIN2 in single-ended mode. With ADDR to ground the ADC is configured for a 0x90 I2C address"
- note removed: "USB-C Power Delivery Controller (15V 5A)"
- note removed: "VBUS: 16V nominal when powered by battery VBUS: 15V nominal when powered through USB-C PD"
- note removed: "VMAX= 3V3/2 => 15V VMIN= 3V3/2 => 15V ICoarse = 3V3 => 5A Ifine = 0A"
- note removed: "Verificar valores de resistências nos PMOS"
- note removed: "Vout = 15V => to DC.DC Stage Iout.max = 4A"
- note removed: "Vout = 15V => to LDO Iout.max = 900mA"
- note removed: "Vout is set to 12.5V to compensate Diode and Rsense drops. The Schottky diode has a 425mV forward voltage drop."
- note removed: "Vout is set to 5.5V to compensate Diode and Rsense drops The Schottky diode has a 420mV forward voltage drop."
- note removed: "Vout is set to 5.5V to compensate Diode and Rsense drops. The Schottky diode has a 425mV forward voltage drop."
