File: Boards/Development Boards/RP2040 P/TVCS Dev.kicad_pcb (KiCad board)
At the start: 4 copper layers, 60 x 22 mm, 75 parts, among them J1 BM03B-SRSS-TBLFSN, J2 BM03B-SRSS-TBLFSN, J3 USB_C, J4 DX07S016JA1R1500, SW1 SW_Push, SW3 SW_Push, U1 ESD7L5.0DT5G, U1 ST1L05APU33R, U2 ST1L05APU33R, U2 W25Q128JVSIQ TR, U3 ESD7L5.0DT5G

Commit message: TVCS Dev
Copiei as footprints todas de uma vez
Parts:
- removed CV19, CV20, CV21, CV22, CV23, CV24, CV26, CV30: 100nF, Capacitor_SMD:C_0201_0603Metric
- removed CV25, CV29: 1uF, Capacitor_SMD:C_0201_0603Metric
- removed CV27, CV28: 4.7uF, Capacitor_SMD:C_0201_0603Metric
- removed CV31, CV35: 1uF, Capacitor_0402:Capacitor_0402
- removed CV32, CV36: 100nF, Capacitor_0402:Capacitor_0402
- removed CV33, CV34: 4.7uF, C_4uF7_0402:C_4uF7_0402
- removed FlashM1: W25Q128JVSIQ_TR, NOR Flash:SOIC_208MIL_WIN
- removed MCU2: RP2040, Package_DFN_QFN:QFN-56-1EP_7x7mm_P0.4mm_EP3.2x3.2mm
- removed RC1: 5k1, Resistor_SMD:R_0201_0603Metric
- removed RC2: 5k1, R_0805_5K1:R_0805_5K1
- removed SW1, SW3: SW_Push, Button_Switch_SMD:SW_Push_1P1T-MP_NO_Horizontal_Alps_SKRTLAE010
- removed the U1 at (164.9, 73.4)
- removed the U1 at (202.4, 64.0)
- removed the U2 at (184.7, 67.9)
- removed the U2 at (157.0, 74.0)
- removed the XTAL1 at (194.8, 69.8)
- removed the XTAL1 at (136.9, 67.8)
- added C1: 100n, Capacitor-0402:Capacitor_0402, F.Cu at (80.7, 86.1)
- added C10: 100n, Capacitor-0402:Capacitor_0402, F.Cu at (84.0, 86.1)
- added C11: 100n, Capacitor-0402:Capacitor_0402, F.Cu at (84.0, 88.2)
- added C12: 100n, Capacitor-0402:Capacitor_0402, F.Cu at (84.0, 90.4)
- added C13: 10u, Capacitor-0805:Capacitor_0805, F.Cu at (164.9, 76.3)
- added C17: 1u, Capacitor-0603:Capacitor_0603, F.Cu at (81.0, 105.8)
- added C18: 1u, Capacitor-0603:Capacitor_0603, F.Cu at (81.0, 108.3)
- added C19: 1u, Capacitor-0603:Capacitor_0603, F.Cu at (81.0, 110.8)
- added C2: 1u, Capacitor-0402:Capacitor_0402, F.Cu at (80.7, 88.2)
- added C20: 100n, Capacitor-0402:Capacitor_0402, F.Cu at (84.0, 92.6)
- added C21: 100n, Capacitor-0402:Capacitor_0402, F.Cu at (84.0, 94.7)
- added C22: 1u, Capacitor-0603:Capacitor_0603, F.Cu at (81.0, 113.3)
- added C23: 100n, Capacitor-0402:Capacitor_0402, F.Cu at (84.0, 96.9)
- added C24: 4.7u, Capacitor-1206:Capacitor_1206, F.Cu at (68.9, 90.4)
- added C25: 100n, Capacitor-0402:Capacitor_0402, F.Cu at (84.0, 99.1)
- added C3: 1u, Capacitor-0402:Capacitor_0402, F.Cu at (80.7, 90.4)
- added C30: C, Capacitor-0402:Capacitor_0402, F.Cu at (84.0, 101.2)
- added C31: 1n, Capacitor-0402:Capacitor_0402, F.Cu at (84.0, 103.4)
- added C32: 2.2u, Capacitor-0402:Capacitor_0402, F.Cu at (87.4, 86.1)
- added C33: 2.2u, Capacitor-0402:Capacitor_0402, F.Cu at (87.4, 88.2)
- added C34: 2.2u, Capacitor-0402:Capacitor_0402, F.Cu at (87.4, 90.4)
- added C35: 2.2u, Capacitor-0402:Capacitor_0402, F.Cu at (87.4, 92.6)
- added C36: 470n, Capacitor-0402:Capacitor_0402, F.Cu at (87.4, 94.7)
- added C37: 470n, Capacitor-0402:Capacitor_0402, F.Cu at (87.4, 96.9)
- added C4: 1u, Capacitor-0402:Capacitor_0402, F.Cu at (80.7, 92.6)
- added C5: 100n, Capacitor-0402:Capacitor_0402, F.Cu at (80.7, 94.7)
- added C6: 10n, Capacitor-0402:Capacitor_0402, F.Cu at (80.7, 96.9)
- added C7: 10n, Capacitor-0402:Capacitor_0402, F.Cu at (80.7, 99.1)
- added C8: 10n, Capacitor-0402:Capacitor_0402, F.Cu at (80.7, 101.2)
- added C9: 100n, Capacitor-0402:Capacitor_0402, F.Cu at (80.7, 103.4)
- added CR1: VLMY1300-GS08, LED-Yellow_VLMY1300-GS08:LED_VISHAY_VLMX1300_VIS, F.Cu at (89.6, 105.7)
- added CR2: VLMY1300-GS08, LED-Yellow_VLMY1300-GS08:LED_VISHAY_VLMX1300_VIS, F.Cu at (89.6, 108.2)
- added CR3: VLMY1300-GS08, LED-Yellow_VLMY1300-GS08:LED_VISHAY_VLMX1300_VIS, F.Cu at (89.6, 110.7)
- added CR4: VLMY1300-GS08, LED-Yellow_VLMY1300-GS08:LED_VISHAY_VLMX1300_VIS, F.Cu at (89.6, 113.1)
- added CR6: VLMT3100-GS08, LED-Red_VLMT3100-GS08:LED_PLCC_VSMB, F.Cu at (118.8, 125.0)
- added C_BIAS1: 1u, Capacitor-0603:Capacitor_0603, F.Cu at (81.0, 115.9)
- added C_BIAS2: 1u, Capacitor-0603:Capacitor_0603, F.Cu at (85.0, 105.8)
- added C_BT1: 100n, Capacitor-0402:Capacitor_0402, F.Cu at (87.4, 99.1)
- added C_BT2: 100n, Capacitor-0402:Capacitor_0402, F.Cu at (87.4, 101.2)
- added C_BT3: 100n, Capacitor-0402:Capacitor_0402, F.Cu at (87.4, 103.4)
- added C_FF1: 22p, Capacitor-0402:Capacitor_0402, F.Cu at (90.7, 86.1)
- added C_IN-BLK1: 10u, Capacitor-4mm:Capacitor_4mm, F.Cu at (108.0, 168.8)
- added C_IN-BLK2: 10u, Capacitor-4mm:Capacitor_4mm, F.Cu at (108.0, 176.2)
- added C_IN-BLK3: 10u, Capacitor-4mm:Capacitor_4mm, F.Cu at (108.0, 183.5)
- added C_IN1: 4.7u, Capacitor-1206:Capacitor_1206, F.Cu at (68.9, 93.5)
- added C_IN2: 4.7u, Capacitor-1206:Capacitor_1206, F.Cu at (68.9, 96.7)
- added C_IN3: 4.7u, Capacitor-1206:Capacitor_1206, F.Cu at (68.9, 99.9)
- added C_IN4: 4.7u, Capacitor-1206:Capacitor_1206, F.Cu at (68.9, 103.0)
- added C_IN5: 4.7u, Capacitor-1206:Capacitor_1206, F.Cu at (68.9, 106.2)
- added C_IN6: 4.7u, Capacitor-1206:Capacitor_1206, F.Cu at (68.9, 109.4)
- added C_IN_HFI1: 100n, Capacitor-0402:Capacitor_0402, F.Cu at (90.7, 88.2)
- added C_IN_HFI2: 100n, Capacitor-0402:Capacitor_0402, F.Cu at (90.7, 90.4)
- added C_IN_HFI3: 100n, Capacitor-0402:Capacitor_0402, F.Cu at (90.7, 92.6)
- added C_IN_HFI4: 100n, Capacitor-0402:Capacitor_0402, F.Cu at (90.7, 94.7)
- added C_IN_HFI5: 100n, Capacitor-0402:Capacitor_0402, F.Cu at (90.7, 96.9)
- added C_IN_HFI6: 100n, Capacitor-0402:Capacitor_0402, F.Cu at (90.7, 99.1)
- added C_OUT1: 1u, Capacitor-0603:Capacitor_0603, F.Cu at (85.0, 108.3)
- added C_OUT10: 22u, Capacitor-0805:Capacitor_0805, F.Cu at (169.4, 88.5)
- added C_OUT11: 10u, Capacitor-0805:Capacitor_0805, F.Cu at (174.0, 76.3)
- added C_OUT12: 47u, Capacitor-0805:Capacitor_0805, F.Cu at (174.0, 79.3)
- added C_OUT13: 22u, Capacitor-0805:Capacitor_0805, F.Cu at (174.0, 82.4)
- added C_OUT14: 100u, Capacitor-6mm:Capacitor_6mm, F.Cu at (146.0, 105.0)
- added C_OUT15: 100u, Capacitor-8mm:Capacitor_8mm, F.Cu at (31.4, 53.2)
- added C_OUT16: 560u, Capacitor-8mm:Capacitor_8mm, F.Cu at (31.4, 63.8)
- added C_OUT2: 10u, Capacitor-0805:Capacitor_0805, F.Cu at (164.9, 79.3)
- added C_OUT3: 22u, Capacitor-0805:Capacitor_0805, F.Cu at (164.9, 82.4)
- added C_OUT4: 22u, Capacitor-0805:Capacitor_0805, F.Cu at (164.9, 85.5)
- added C_OUT5: 10u, Capacitor-0805:Capacitor_0805, F.Cu at (164.9, 88.5)
- added C_OUT6: 22u, Capacitor-0805:Capacitor_0805, F.Cu at (169.4, 76.3)
- added C_OUT7: 22u, Capacitor-0805:Capacitor_0805, F.Cu at (169.4, 79.3)
- added C_OUT8: 10u, Capacitor-0805:Capacitor_0805, F.Cu at (169.4, 82.4)
- added C_OUT9: 47u, Capacitor-0805:Capacitor_0805, F.Cu at (169.4, 85.5)
- added C_VCC1: 1u, Capacitor-0603:Capacitor_0603, F.Cu at (85.0, 110.8)
- added C_VCC2: 1u, Capacitor-0603:Capacitor_0603, F.Cu at (85.0, 113.3)
- added C_VCC3: 1u, Capacitor-0603:Capacitor_0603, F.Cu at (85.0, 115.9)
- added D2: RSX301L, Diode-Schottky_RSX301L:DIOM5026X220N, F.Cu at (87.0, 148.7)
- added D4: SP3004-04XTG, TVS-SP3004:SOT563_LTF, F.Cu at (183.1, 72.2)
- added D5: RB095BGE, SchottkyDiode-RB095BGE:RD3P175SNFRATL, F.Cu at (100.3, 21.2)
- added D6: RB095BGE, SchottkyDiode-RB095BGE:RD3P175SNFRATL, F.Cu at (110.0, 21.2)
- added D7: RSX301L, Diode-Schottky_RSX301L:DIOM5026X220N, F.Cu at (87.0, 153.0)
- added IC1: INA2181A4IDSQR, INA2181A4IDSQR:SON40P200X200X80-11N, F.Cu at (178.6, 72.6)
- added IC10: NSVT30010MXV6T1G, 2 PNP:SOT-563_1P3X1P7_ONS, F.Cu at (76.5, 116.0)
- added IC2: CYPD3177-24LQXQT, USBC-PD_CYPD3177:QFN50P400X400X60-25N-D, F.Cu at (121.4, 61.8)
- added IC3: DMP2040USD-13, DMP2040USD-13:SOIC127P600X175-8N, F.Cu at (189.3, 44.6)
- added IC4: ADS1115IRUGR, ADS1115:ADS1115IRUGR, F.Cu at (158.9, 71.9)
- added IC5: INA181A4QDCKRQ1, INA181A4QDCKRQ1:SOT65P210X110-6N, F.Cu at (73.8, 108.9)
- added IC6: DMP2040USD-13, DMP2040USD-13:SOIC127P600X175-8N, F.Cu at (189.3, 51.1)
- added IC7: NCR420ZX, LED-Driver_NCR420ZX:SOT230P700X180-4N, F.Cu at (143.0, 124.5)
- added IC8: PCA9306GM,125, PCA9306GM,125:PCA9570GMH, F.Cu at (111.3, 65.7)
- added IC9: NSVT30010MXV6T1G, 2 PNP:SOT-563_1P3X1P7_ONS, F.Cu at (76.5, 112.6)
- added J10: Conn_01x01_Socket, Pico_Conn1x1:Pico_01pin, F.Cu at (143.0, 37.5)
- added J11: Conn_01x01_Socket, Pico_Conn1x1:Pico_01pin, F.Cu at (147.1, 37.5)
- added J13: Conn_01x01_Socket, Pico_Conn1x1:Pico_01pin, F.Cu at (126.6, 43.7)
- added J14: Conn_01x01_Socket, Pico_Conn1x1:Pico_01pin, F.Cu at (130.7, 43.7)
- added J15: Conn_01x01_Socket, Pico_Conn1x1:Pico_01pin, F.Cu at (134.8, 43.7)
- added J16: Conn_01x01_Socket, Pico_Conn1x1:Pico_01pin, F.Cu at (138.9, 43.7)
- added J17: Conn_01x01_Socket, Pico_Conn1x1:Pico_01pin, F.Cu at (143.0, 43.7)
- added J18: BM03B-SRSS-TBLFSN, SWD_Con:CONN_BM03B-SRSS-TBLFSN_JST, F.Cu at (52.1, 144.8)
- added J8: Conn_01x01_Socket, Pico_Conn1x1:Pico_01pin, F.Cu at (134.8, 37.5)
- added J9: Conn_01x01_Socket, Pico_Conn1x1:Pico_01pin, F.Cu at (138.9, 37.5)
- added L1: 2.2u, Inductor-10.1x10:Inductor_10.1x10, F.Cu at (32.0, 18.3)
- added LED1: VLMS1500-GS08, LED-Red_VLMS1500-GS08:LED_00-GS08_VIS_RED, F.Cu at (89.4, 115.5)
- added LED2: VLMS1500-GS08, LED-Red_VLMS1500-GS08:LED_00-GS08_VIS_RED, F.Cu at (89.4, 117.6)
- added LED3: APHB1608LG3R2C-AMT, APHB1608LG3R2C-AMT:APHB1608LG3R2CAMT, F.Cu at (164.0, 71.5)
- added L_SW1: 10u, Inductor-11.5x10:Inductor_11.5x10, F.Cu at (205.0, 59.0)
- added L_SW2: 15u, Inductor-10.1x10:Inductor_10.1x10, F.Cu at (32.0, 30.1)
- added L_SW3: 15u, Inductor-10.1x10:Inductor_10.1x10, F.Cu at (32.0, 42.0)
- added Q1: 2N7002H6327XTSA2, NMOS_2N7002:PG-SOT23-3-5_INF_MIN, F.Cu at (179.7, 77.2)
- added Q2: 2N7002H6327XTSA2, NMOS_2N7002:PG-SOT23-3-5_INF_MIN, F.Cu at (179.7, 82.1)
- added Q3: BC857CMB_315, PNP_BC857CMB_315:TRANS_PMZB550UNEYL, F.Cu at (168.2, 70.5)
- added Q4: BC857CMB_315, PNP_BC857CMB_315:TRANS_PMZB550UNEYL, F.Cu at (168.2, 72.8)
- added R19: 160, Resistor-0402:RES_0402, F.Cu at (73.1, 39.0)
- added R20: 160, Resistor-0402:RES_0402, F.Cu at (73.1, 41.2)
- added R21: 10k, Resistor-0402:RES_0402, F.Cu at (73.1, 43.3)
- added R22: 50k, Resistor-0402:RES_0402, F.Cu at (73.1, 45.5)
- added R23: 1k, Resistor-0402:RES_0402, F.Cu at (73.1, 47.7)
- added R24: 1k, Resistor-0402:RES_0402, F.Cu at (73.1, 49.8)
- added R25: 1k, Resistor-0402:RES_0402, F.Cu at (57.0, 122.7)
- added R26: 27, Resistor-0603:RES_0603, F.Cu at (60.6, 122.9)
- added R27: 10K, Resistor-0402:RES_0402, F.Cu at (73.1, 52.0)
- added R28: 2k, Resistor-0402:RES_0402, F.Cu at (73.1, 54.1)
- added R29: 2k, Resistor-0402:RES_0402, F.Cu at (73.1, 56.3)
- added R30: 50k, Resistor-0402:RES_0402, F.Cu at (76.6, 39.0)
- added R31: 10K, Resistor-0402:RES_0402, F.Cu at (76.6, 41.2)
- added R32: 10K, Resistor-0402:RES_0402, F.Cu at (76.6, 43.3)
- added R33: 54k2, Resistor-0402:RES_0402, F.Cu at (76.6, 45.5)
- added R34: 1k, Resistor-0402:RES_0402, F.Cu at (76.6, 47.7)
- added R35: 2k, Resistor-0402:RES_0402, F.Cu at (76.6, 49.8)
- added R36: 10k, Resistor-0402:RES_0402, F.Cu at (76.6, 52.0)
- added R37: 95, Resistor-0402:RES_0402, F.Cu at (76.6, 54.1)
- added R38: 1k, Resistor-0402:RES_0402, F.Cu at (76.6, 56.3)
- added R39: 1k, Resistor-0402:RES_0402, F.Cu at (80.0, 39.0)
- added R40: 2k, Resistor-0402:RES_0402, F.Cu at (80.0, 41.2)
- added R41: 160, Resistor-0402:RES_0402, F.Cu at (80.0, 43.3)
- added R42: 200k, Resistor-0402:RES_0402, F.Cu at (80.0, 45.5)
- added R43: 27, Resistor-0603:RES_0603, F.Cu at (60.6, 125.5)
- added R44: 100, Resistor-0402:RES_0402, F.Cu at (57.0, 124.9)
- added R45: 2k, Resistor-0402:RES_0402, F.Cu at (80.0, 47.7)
- added R46: 30k, Resistor-0402:RES_0402, F.Cu at (80.0, 49.8)
- added R47: 100, Resistor-0402:RES_0402, F.Cu at (80.0, 52.0)
- added R48: PTS060301B100RP100, PTS060301B100RP100:RESC1508X55N, F.Cu at (115.0, 65.2)
- added R49: 30k, Resistor-0402:RES_0402, F.Cu at (80.0, 54.1)
- added R50: 100, Resistor-0402:RES_0402, F.Cu at (57.0, 127.1)
- added R51: 1k, Resistor-0402:RES_0402, F.Cu at (57.0, 129.2)
- added R52: 1k, Resistor-0402:RES_0402, F.Cu at (57.0, 131.4)
- added R53: 10k, Resistor-0402:RES_0402, F.Cu at (57.0, 133.5)
- added R_BIAS1: 5, Resistor-0402:RES_0402, F.Cu at (80.0, 56.3)
- added R_BIAS2: 5, Resistor-0402:RES_0402, F.Cu at (83.4, 39.0)
- added R_BT1: 50, Resistor-0402:RES_0402, F.Cu at (83.4, 41.2)
- added R_BT2: 50, Resistor-0402:RES_0402, F.Cu at (83.4, 43.3)
- added R_BT3: 100, Resistor-0402:RES_0402, F.Cu at (83.4, 45.5)
- added R_ENB1: 100k, Resistor-0603:RES_0603, F.Cu at (148.2, 173.9)
- added R_ENB2: 63k4, Resistor-0402:RES_0402, F.Cu at (83.4, 47.7)
- added R_ENB3: 45k3, Resistor-0402:RES_0402, F.Cu at (83.4, 49.8)
- added R_ENT1: 931k, Resistor-0603:RES_0603, F.Cu at (148.2, 176.5)
- added R_ENT2: 590k, Resistor-0402:RES_0402, F.Cu at (83.4, 52.0)
- added R_ENT3: 422k, Resistor-0402:RES_0402, F.Cu at (83.4, 54.1)
- added R_FBB1: 8k66, Resistor-0603:RES_0603, F.Cu at (148.2, 179.0)
- added R_FBB2: 12k6, Resistor-0603:RES_0603, F.Cu at (148.2, 181.5)
- added R_FBB3: 22k1, Resistor-0603:RES_0603, F.Cu at (148.2, 184.1)
- added R_FBB4: 30, Resistor-0603:RES_0603, F.Cu at (148.2, 186.6)
- added R_FBB5: 50, Resistor-0603:RES_0603, F.Cu at (151.9, 173.9)
- added R_FBB6: 120, Resistor-0603:RES_0603, F.Cu at (151.9, 176.5)
- added R_FBT1: 100K, Resistor-0603:RES_0603, F.Cu at (151.9, 179.0)
- added R_FBT2: 100K, Resistor-0603:RES_0603, F.Cu at (151.9, 181.5)
- added R_FBT3: 100K, Resistor-0603:RES_0603, F.Cu at (151.9, 184.1)
- added R_FF1: 1k, Resistor-0402:RES_0402, F.Cu at (83.4, 56.3)
- added R_PG1: 100K, Resistor-0603:RES_0603, F.Cu at (151.9, 186.6)
- added R_PG2: 100K, Resistor-0603:RES_0603, F.Cu at (155.6, 173.9)
- added R_PG3: 100K, Resistor-0603:RES_0603, F.Cu at (155.6, 176.5)
- added R_RT1: 33k2, Resistor-0603:RES_0603, F.Cu at (155.6, 179.0)
- added R_RT2: 33k2, Resistor-0603:RES_0603, F.Cu at (155.6, 181.5)
- added R_RT3: 33k2, Resistor-0603:RES_0603, F.Cu at (155.6, 184.1)
- added Rsense1: 2.5m, Resistor-0805:RES_0805, F.Cu at (75.2, 100.6)
- added Rsense2: 7.5m, Resistor-2512:RES_WSLP2512, F.Cu at (113.7, 61.3)
- added Rsense3: 2.5m, Resistor-0805:RES_0805, F.Cu at (75.2, 104.9)
- added TP1: TestPoint, Test Hook:KEYSTONE_5277, F.Cu at (-32.2, 13.1)
- added TP10: TestPoint, Test Hook:KEYSTONE_5277, F.Cu at (-27.5, 13.1)
- added TP11: TestPoint, Test Hook:KEYSTONE_5277, F.Cu at (-27.5, 17.8)
- added TP12: TestPoint, Test Hook:KEYSTONE_5277, F.Cu at (-27.5, 22.5)
- added TP13: TestPoint, Test Hook:KEYSTONE_5277, F.Cu at (-27.5, 27.3)
- added TP14: TestPoint, Test Hook:KEYSTONE_5277, F.Cu at (-27.5, 32.0)
- added TP15: TestPoint, Test Hook:KEYSTONE_5277, F.Cu at (-27.5, 36.7)
- added TP16: TestPoint, Test Hook:KEYSTONE_5277, F.Cu at (-27.5, 41.5)
- added TP17: TestPoint, Test Hook:KEYSTONE_5277, F.Cu at (-27.5, 46.2)
- added TP18: TestPoint, Test Hook:KEYSTONE_5277, F.Cu at (-27.5, 50.9)
- added TP19: TestPoint, Test Hook:KEYSTONE_5277, F.Cu at (-22.7, 13.1)
- added TP2: TestPoint, Test Hook:KEYSTONE_5277, F.Cu at (-32.2, 17.8)
- added TP20: TestPoint, Test Hook:KEYSTONE_5277, F.Cu at (-22.7, 17.8)
- added TP21: TestPoint, Test Hook:KEYSTONE_5277, F.Cu at (-22.7, 22.5)
- added TP22: TestPoint, Test Hook:KEYSTONE_5277, F.Cu at (-22.7, 27.3)
- added TP23: TestPoint, Test Hook:KEYSTONE_5277, F.Cu at (-22.7, 32.0)
- added TP24: TestPoint, Test Hook:KEYSTONE_5277, F.Cu at (-22.7, 36.7)
- added TP25: TestPoint, Test Hook:KEYSTONE_5277, F.Cu at (-22.7, 41.5)
- added TP26: TestPoint, Test Hook:KEYSTONE_5277, F.Cu at (-22.7, 46.2)
- added TP27: TestPoint, Test Hook:KEYSTONE_5277, F.Cu at (-22.7, 50.9)
- added TP28: TestPoint, Test Hook:KEYSTONE_5277, F.Cu at (-18.0, 13.1)
- added TP29: TestPoint, Test Hook:KEYSTONE_5277, F.Cu at (-18.0, 17.8)
- added TP3: TestPoint, Test Hook:KEYSTONE_5277, F.Cu at (-32.2, 22.5)
- added TP30: TestPoint, Test Hook:KEYSTONE_5277, F.Cu at (-18.0, 22.5)
- added TP31: 5277, Test Hook:KEYSTONE_5277, F.Cu at (-18.0, 27.3)
- added TP32: 5277, Test Hook:KEYSTONE_5277, F.Cu at (-18.0, 32.0)
- added TP33: 5277, Test Hook:KEYSTONE_5277, F.Cu at (-18.0, 36.7)
- added TP34: 5277, Test Hook:KEYSTONE_5277, F.Cu at (-18.0, 41.5)
- added TP35: 5277, Test Hook:KEYSTONE_5277, F.Cu at (-18.0, 46.2)
- added TP36: 5277, Test Hook:KEYSTONE_5277, F.Cu at (-18.0, 50.9)
- added TP37: 5277, Test Hook:KEYSTONE_5277, F.Cu at (-13.3, 13.1)
- added TP38: 5277, Test Hook:KEYSTONE_5277, F.Cu at (-13.3, 17.8)
- added TP39: 5277, Test Hook:KEYSTONE_5277, F.Cu at (-13.3, 22.5)
- added TP4: TestPoint, Test Hook:KEYSTONE_5277, F.Cu at (-32.2, 27.3)
- added TP40: 5277, Test Hook:KEYSTONE_5277, F.Cu at (-13.3, 27.3)
- added TP41: 5277, Test Hook:KEYSTONE_5277, F.Cu at (-13.3, 32.0)
- added TP42: 5277, Test Hook:KEYSTONE_5277, F.Cu at (-13.3, 36.7)
- added TP43: 5277, Test Hook:KEYSTONE_5277, F.Cu at (-13.3, 41.5)
- added TP44: 5277, Test Hook:KEYSTONE_5277, F.Cu at (-13.3, 46.2)
- added TP45: TestPoint, Test Hook:KEYSTONE_5277, F.Cu at (-13.3, 50.9)
- added TP46: TestPoint, Test Hook:KEYSTONE_5277, F.Cu at (-8.54, 13.1)
- added TP47: TestPoint, Test Hook:KEYSTONE_5277, F.Cu at (-8.54, 17.8)
- added TP48: TestPoint, Test Hook:KEYSTONE_5277, F.Cu at (-8.54, 22.5)
- added TP49: TestPoint, Test Hook:KEYSTONE_5277, F.Cu at (-8.54, 27.3)
- added TP5: TestPoint, Test Hook:KEYSTONE_5277, F.Cu at (-32.2, 32.0)
- added TP50: 5277, Test Hook:KEYSTONE_5277, F.Cu at (-8.54, 32.0)
- added TP51: 5277, Test Hook:KEYSTONE_5277, F.Cu at (-8.54, 36.7)
- added TP6: TestPoint, Test Hook:KEYSTONE_5277, F.Cu at (-32.2, 36.7)
- added TP7: TestPoint, Test Hook:KEYSTONE_5277, F.Cu at (-32.2, 41.5)
- added TP8: TestPoint, Test Hook:KEYSTONE_5277, F.Cu at (-32.2, 46.2)
- added TP9: TestPoint, Test Hook:KEYSTONE_5277, F.Cu at (-32.2, 50.9)
- added U1: SQJA36EP-T1_GE3, SQJA36EP-T1-GE3:PowerPAK_SO-8L_3_VIS, F.Cu at (74.8, 93.2)
- added U10: VLMKG3400-GS08, VLMKG3400-GS08:SMT_00-GS08_VIS, F.Cu at (180.7, 86.9)
- added U2: MAX31856MUD+T, Thermocouple:21-0066J_14_MXM, F.Cu at (122.1, 137.3)
- added U4: W25Q128JVSIQ TR, NOR Flash:SOIC_208MIL_WIN, F.Cu at (53.3, 138.3)
- added U5: ST1L05APU33R, LDO ST1L05A:DFN_5APU33R_STM, F.Cu at (62.0, 137.1)
- added U7: LM61460AASQRJRRQ1, DCDC_LM61460:VQFN-HR14_RJR_TEX, F.Cu at (245.0, 88.8)
- added U8: LM61460AASQRJRRQ1, DCDC_LM61460:VQFN-HR14_RJR_TEX, F.Cu at (245.0, 94.5)
- added U9: LM61460AASQRJRRQ1, DCDC_LM61460:VQFN-HR14_RJR_TEX, F.Cu at (173.4, 71.9)
- added VR1: 3361P-1-102GLF, 1k Potenciometro:TRIM_3361P-1-102GLF, F.Cu at (-25.5, 83.0)
- added VR10: 3361P-1-102GLF, 1k Potenciometro:TRIM_3361P-1-102GLF, F.Cu at (-13.5, 116.0)
- added VR2: 3361P-1-102GLF, 1k Potenciometro:TRIM_3361P-1-102GLF, F.Cu at (-25.5, 91.2)
- added VR3: 3361P-1-102GLF, 1k Potenciometro:TRIM_3361P-1-102GLF, F.Cu at (-25.5, 99.5)
- added VR4: 3361P-1-102GLF, 1k Potenciometro:TRIM_3361P-1-102GLF, F.Cu at (-25.5, 107.8)
- added VR5: 3361P-1-102GLF, 1k Potenciometro:TRIM_3361P-1-102GLF, F.Cu at (-25.5, 116.0)
- added VR6: 3361P-1-102GLF, 1k Potenciometro:TRIM_3361P-1-102GLF, F.Cu at (-13.5, 83.0)
- added VR7: 3361P-1-102GLF, 1k Potenciometro:TRIM_3361P-1-102GLF, F.Cu at (-13.5, 91.2)
- added VR8: 3361P-1-102GLF, 1k Potenciometro:TRIM_3361P-1-102GLF, F.Cu at (-13.5, 99.5)
- added VR9: 3361P-1-102GLF, 1k Potenciometro:TRIM_3361P-1-102GLF, F.Cu at (-13.5, 107.8)
- added XTAL1: ASE-12.000MHZ-LC-T, AS12MHz:ASE-3.2X2.5_ABR, F.Cu at (61.0, 144.3)
- CV1, CV10, CV11, CV12, CV2, CV3, CV4, CV5, CV6, CV7, CV8, CV9: footprint Capacitor_0402:Capacitor_0402 -> Capacitor-0402:Capacitor_0402
- CV13, CV18: value 1uF -> 100nF; footprint Capacitor_SMD:C_0201_0603Metric -> Capacitor-0402:Capacitor_0402
- CV14: value 100nF -> 4.7uF; footprint Capacitor_SMD:C_0201_0603Metric -> Capacitor-0402:Capacitor_0402
- CV15: value 1uF -> 4.7uF; footprint Capacitor_SMD:C_0201_0603Metric -> Capacitor-0402:Capacitor_0402
- CV16, CV17: value 100nF -> 1uF; footprint Capacitor_SMD:C_0201_0603Metric -> Capacitor-0402:Capacitor_0402
- D1: value PMEG2010ER -> RB095BGE-30TL; footprint PMEG2010ER:SODFL3517X110N -> SchottkyDiode-RB095BGE:RD3P175SNFRATL
- J1: value BM03B-SRSS-TBLFSN -> DX07S016JA1R1500; footprint SWD_Con:CONN_BM03B-SRSS-TBLFSN_JST -> USBC-DX07S016JA1:JAE_DX07S016JA1R1500
- J2: value BM03B-SRSS-TBLFSN -> Conn_01x01_Socket; footprint SWD_Con:CONN_BM03B-SRSS-TBLFSN_JST -> Pico_Conn1x1:Pico_01pin
- J3: value USB_C -> Conn_01x01_Socket; footprint Connector_USB:USB_C_Plug_JAE_DX07P024AJ1 -> Pico_Conn1x1:Pico_01pin
- J4: value DX07S016JA1R1500 -> MEM2061-01-188-00-A_REVA; footprint USBC-DX07S016JA1:JAE_DX07S016JA1R1500 -> SD-CARD_MEM2061-01-188-00-A:GCT_MEM2061-01-188-00-A_REVA
- R1: value 1k -> 54k2; footprint RES_0402:RES_0402 -> Resistor-0402:RES_0402
- R10, R17: value 1k -> 2k; footprint RES_0402:RES_0402 -> Resistor-0402:RES_0402
- R11: value 100 -> 20K; footprint Resistor_SMD:R_0201_0603Metric -> Resistor-0402:RES_0402
- R12, R14: value 1k -> 370; footprint Resistor_SMD:R_0201_0603Metric -> Resistor-0402:RES_0402
- R13: value 10k -> 370; footprint Resistor_SMD:R_0201_0603Metric -> Resistor-0402:RES_0402
- R15: value 5k1 -> 100; footprint Resistor_SMD:R_0201_0603Metric -> Resistor-0402:RES_0402
- R16: value 10k -> 100; footprint RES_0402:RES_0402 -> Resistor-0402:RES_0402
- R18: value 5k1 -> 20K; footprint R_0805_5K1:R_0805_5K1 -> Resistor-0402:RES_0402
- R2: footprint Resistor_SMD:R_0201_0603Metric -> Resistor-0402:RES_0402
- R3, R4: value 27 -> 2k; footprint Resistor_SMD:R_0201_0603Metric -> Resistor-0402:RES_0402
- R5: value 100 -> DNP; footprint Resistor_SMD:R_0201_0603Metric -> Resistor-0402:RES_0402
- R6, R7: value 27 -> 2k; footprint RES_R0603_27:RES_R0603_27 -> Resistor-0402:RES_0402
- R8: value 100 -> 120; footprint RES_0402:RES_0402 -> Resistor-0402:RES_0402
- R9: value 100 -> 2k; footprint RES_0402:RES_0402 -> Resistor-0402:RES_0402
- S1, S2: value TL3305CF160QG -> TL1017AABF160QG; footprint E-Switch_7mm:SW_TL3305CF160QG -> E-Switch_Small:TL1017AABF160QG
- U3: value ESD7L5.0DT5G -> MAX485CSA+T; footprint ESD7L5-Diode:SOT-723_0P85X1P25_ONS -> RS Transceiver:21-0041-3-M_90-0096-8L_MXM
- moved CV5 180.2 mm to (39.6, 131.4)
- moved CV7 180.2 mm to (39.6, 135.8)
- moved CV6 180.2 mm to (39.6, 133.6)
- moved CV10 177.1 mm to (43.0, 127.1)
- moved CV11 177.1 mm to (43.0, 129.3)
- moved CV12 177.1 mm to (43.0, 131.4)
- moved CV9 177.1 mm to (43.0, 124.9)
- moved CV1 173.1 mm to (39.6, 122.7)
- moved CV2 173.1 mm to (39.6, 124.9)
- moved CV3 173.1 mm to (39.6, 127.1)
- moved CV4 173.1 mm to (39.6, 129.3)
- moved CV8 170.3 mm to (43.0, 122.7)
- moved J4 162.4 mm to (26.4, 93.3)
- moved S2 150.6 mm to (51.7, 131.0)
- moved S1 150.3 mm to (51.7, 124.5)
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Connections:
- CV13 pad 1: Net-(MCU2-RUN) -> +3.3V
- CV14 pad 2: Net-(MCU2-VREG_VOUT) -> +5V
- CV15 pad 1: Net-(MCU2-VREG_VOUT) -> GND
- CV15 pad 2: GND -> +3.3V
- CV16 pad 2: Net-(MCU2-VREG_VOUT) -> +5V
- J1 pad 1: Net-(J1-Pad1) -> GND
- J1 pad 2: GND -> /VBUS_IN
- J1 pad 3: Net-(J1-Pad3) -> Net-(D4-IO1)
- J1 pad 4: (no net) -> unconnected-(J1-SBU2-Pad4)
- J1 pad 5: (no net) -> USB_DM
- J2 pad 1: Net-(J2-Pad1) -> /THERMO1 T+
- J4 pad 1: GND -> unconnected-(J4-DAT2-Pad1)
- J4 pad 10: unconnected-(J4-SBU1-Pad10) -> GND
- J4 pad 11: Net-(D1-PadA) -> GND
- J4 pad 2: Net-(D1-PadA) -> /SD-Card ~{CS}
- J4 pad 3: Net-(J4-CC1) -> /SPI0_MOSI
- J4 pad 4: unconnected-(J4-SBU2-Pad4) -> +3.3V
- J4 pad 5: /RP2040 Standard/USB_DM -> /SPI0_SCK
- J4 pad 6: /RP2040 Standard/USB_DP -> GND
- J4 pad 7: /RP2040 Standard/USB_DP -> /SPI0_MISO
- J4 pad 8: /RP2040 Standard/USB_DM -> unconnected-(J4-DAT1-Pad8)
- J4 pad 9: Net-(J4-CC2) -> GND
- MCU1 pad 11: /RP2040 Standard/GP8/SPI1 MISO -> /SPI1_MISO
- MCU1 pad 12: /RP2040 Standard/GP9/SPI1 ~{CS} -> /THERMO1_~{CS}
- MCU1 pad 13: /RP2040 Standard/GP10/SPI1 SCK -> /SPI1_SCK
- MCU1 pad 14: /RP2040 Standard/GP11/SPI1 MOSI -> /SPI1_MOSI
- MCU1 pad 15: /RP2040 Standard/GP12/I2C0 SDA -> /THERMO1_~{FAULT}
- MCU1 pad 16: /RP2040 Standard/GP13/I2C0 SCL -> /LED Test1
- MCU1 pad 17: /RP2040 Standard/GP14/I2C1 SDA -> /SDA I2C
- MCU1 pad 18: /RP2040 Standard/GP15/I2C1 SCL -> /SCL I2C
- MCU1 pad 2: /RP2040 Standard/GP0/UART0 TX -> /DC.DC1 PGOOD
- MCU1 pad 20: CRYSTAL -> /RP2040 Standard1/Crystal
- MCU1 pad 27: /RP2040 Standard/GP16/SPI0 MISO -> /SPI0_MISO
- MCU1 pad 28: /RP2040 Standard/GP17/SPI0 ~{CS} -> /SD-Card ~{CS}
- MCU1 pad 29: /RP2040 Standard/GP18/SPI0 SCK -> /SPI0_SCK
- MCU1 pad 3: /RP2040 Standard/GP1/UART0 RX -> /DC.DC2 PGOOD
- MCU1 pad 30: /RP2040 Standard/GP19/SPI0 MOSI -> /SPI0_MOSI
- MCU1 pad 31: /RP2040 Standard/GP20/PWM2 A/CLKIN 0 -> /Solenoid Valve Enable
- MCU1 pad 32: /RP2040 Standard/GP21/PWM2 B/CLKOUT 0 -> /Status2 Green
- MCU1 pad 34: /RP2040 Standard/GP22/PWM3 A/CLKIN 1 -> /ADC RDY
- MCU1 pad 35: /RP2040 Standard/GP23/PWM3 B/CLKOUT 1 -> /USB-C PD ~{INT}
- MCU1 pad 36: /RP2040 Standard/GP24/PWM4 A -> /Status1 Red
- MCU1 pad 37: /RP2040 Standard/GP25/PWM4 B -> /Status1 Green
- MCU1 pad 38: /RP2040 Standard/GP26_ADC0 -> /12V_Sense
- MCU1 pad 39: /RP2040 Standard/GP27_ADC1 -> /8.4V_Sense
- MCU1 pad 4: /RP2040 Standard/GP2/UART0 CTS -> /DC.DC3 PGOOD
- MCU1 pad 40: /RP2040 Standard/GP28_ADC2 -> /5V_Sense
- MCU1 pad 41: /RP2040 Standard/GP29_ADC3 -> /Status2 Red
- MCU1 pad 5: /RP2040 Standard/GP3/UART0 RTS -> /Servo Valve PWM
- MCU1 pad 51: /RP2040 Standard/MCU QSPI_SD3 -> /RP2040 Standard1/MCU QSPI_SD3
- MCU1 pad 52: /RP2040 Standard/MCU QSPI_SCLK -> /RP2040 Standard1/MCU QSPI_SCLK
- MCU1 pad 53: /RP2040 Standard/MCU QSPI_SD0 -> /RP2040 Standard1/MCU QSPI_SD0
- MCU1 pad 54: /RP2040 Standard/MCU QSPI_SD2 -> /RP2040 Standard1/MCU QSPI_SD2
- MCU1 pad 55: /RP2040 Standard/MCU QSPI_SD1 -> /RP2040 Standard1/MCU QSPI_SD1
- MCU1 pad 56: /RP2040 Standard/MCU QSPI_SS -> /RP2040 Standard1/MCU QSPI_SS
- MCU1 pad 6: /RP2040 Standard/GP4/UART1 TX -> /RS_RX
- MCU1 pad 7: /RP2040 Standard/GP5/UART1 RX -> /RS_TX
- MCU1 pad 8: /RP2040 Standard/GP6/UART1 CTS -> /RS_ENABLE
- MCU1 pad 9: /RP2040 Standard/GP7/UART1 RTS -> /THERMO1_~{DRDY}
- R1 pad 1: +3.3V -> Net-(IC1-REF1)
- R1 pad 2: Net-(MCU1-RUN) -> +3.3V
- R10 pad 1: /RP2040 Standard/~{RST} -> GND
- R10 pad 2: Net-(MCU1-RUN) -> Net-(IC2-VBUS_MAX)
- R11 pad 1: Net-(J1-Pad3) -> +5V
- R11 pad 2: Net-(MCU2-SWD) -> /RS_A
- R12 pad 1: /~{RST} -> /TEMP SENSE +
- R12 pad 2: Net-(MCU2-RUN) -> /AIN0
- R13 pad 1: Net-(XTAL1-TRI-STATE(STBY)) -> /TEMP SENSE -
- R13 pad 2: +3.3V -> /AIN1
- R14 pad 1: /~{USB_BOOT} -> /PRESS_SENSE
- R14 pad 2: /MCU QSPI_SS -> /AIN2
- R15 pad 1: GND -> Net-(U2-T+)
- R15 pad 2: Net-(J3-CC1) -> /THERMO1 T+
- R16 pad 1: Net-(XTAL1-TRI-STATE(STBY)) -> Net-(U2-T-)
- R16 pad 2: +3.3V -> /THERMO1 T-
- R17 pad 1: /RP2040 Standard/~{USB_BOOT} -> Net-(IC2-ISNK_FINE)
- R17 pad 2: /RP2040 Standard/MCU QSPI_SS -> GND
- R18 pad 1: GND -> /RS_B
- R18 pad 2: Net-(J4-CC2) -> GND
- R2 pad 1: +3.3V -> GND
- R2 pad 2: Net-(MCU2-RUN) -> Net-(IC1-REF1)
- R3 pad 1: /USB_DP -> +3.3V
- R3 pad 2: Net-(MCU2-USB_DP) -> Net-(IC2-VBUS_MIN)
- R4 pad 1: /USB_DM -> +3.3V
- R4 pad 2: Net-(MCU2-USB_DM) -> Net-(IC2-VBUS_MAX)
- R5 pad 1: Net-(J1-Pad1) -> Net-(IC2-ISNK_FINE)
- R5 pad 2: Net-(MCU2-SWCLK) -> +3.3V
- R6 pad 1: /RP2040 Standard/USB_DP -> /SDL I2C
- R6 pad 2: Net-(MCU1-USB_DP) -> +3.3V
- R7 pad 1: /RP2040 Standard/USB_DM -> /SDA I2C
- R7 pad 2: Net-(MCU1-USB_DM) -> +3.3V
- R8 pad 1: Net-(J2-Pad3) -> /RS_B
- R8 pad 2: Net-(MCU1-SWCLK) -> /RS_A
- R9 pad 1: Net-(J2-Pad1) -> Net-(IC2-VBUS_MIN)
- R9 pad 2: Net-(MCU1-SWD) -> GND
- S1 pad 1: unconnected-(S1-Pad1) -> GND
- S1 pad 2: GND -> /RP2040 Standard1/~{RST}
- S2 pad 1: unconnected-(S2-Pad1) -> GND
- S2 pad 2: GND -> /RP2040 Standard1/~{USB_BOOT}
- U3 pad 1: /RP2040 Standard/USB_DM -> /RS_RX
- U3 pad 2: /RP2040 Standard/USB_DP -> /RS_ENABLE
- U3 pad 3: GND -> /RS_ENABLE
Other:
- board size 60 x 22 mm -> 0.9 x 0.6 mm
