File: Boards/Development Boards/RP2040 P/TVCS Dev.kicad_pcb (KiCad board)
At the start: 4 copper layers, 0.9 x 0.6 mm, 291 parts, among them IC1 INA2181A4IDSQR, IC10 NSVT30010MXV6T1G, IC2 CYPD3177-24LQXQT, IC3 DMP2040USD-13, IC4 ADS1115IRUGR, IC5 INA181A4QDCKRQ1, IC6 DMP2040USD-13, IC7 NCR420ZX, IC8 PCA9306GM,125, IC9 NSVT30010MXV6T1G, J1 DX07S016JA1R1500, J10 Conn_01x01_Socket, J11 Conn_01x01_Socket, J13 Conn_01x01_Socket, J14 Conn_01x01_Socket, J15 Conn_01x01_Socket, J16 Conn_01x01_Socket, J17 Conn_01x01_Socket, J18 BM03B-SRSS-TBLFSN, J2 Conn_01x01_Socket, J3 Conn_01x01_Socket, J4 MEM2061-01-188-00-A_REVA, J8 Conn_01x01_Socket, J9 Conn_01x01_Socket, Q1 2N7002H6327XTSA2, Q2 2N7002H6327XTSA2, Q3 BC857CMB_315, Q4 BC857CMB_315, U1 SQJA36EP-T1_GE3, U10 VLMKG3400-GS08, U2 MAX31856MUD+T, U3 MAX485CSA+T, U4 W25Q128JVSIQ TR, U5 ST1L05APU33R, U7 LM61460AASQRJRRQ1, U8 LM61460AASQRJRRQ1, U9 LM61460AASQRJRRQ1

Commit message: pcb
Parts:
- moved Q3 244.0 mm to (-75.2, 88.5)
- moved Q4 244.0 mm to (-75.2, 90.8)
- moved U10 209.1 mm to (-20.8, 142.8)
- moved LED3 185.4 mm to (-11.4, 131.7)
- moved CR1 132.7 mm to (-41.4, 126.6)
- moved CR2 132.7 mm to (-41.4, 129.1)
- moved CR3 132.7 mm to (-41.4, 131.5)
- moved CR4 132.7 mm to (-41.4, 134.0)
- moved TP19 129.3 mm to (-57.0, 137.8)
- moved TP20 129.3 mm to (-57.0, 142.5)
- moved CV18 120.6 mm to (155.0, 77.0)
- moved CV4 116.9 mm to (148.6, 87.0)
- moved TP3 114.1 mm to (-87.0, 122.6)
- moved TP5 114.1 mm to (-87.0, 132.1)
- moved TP6 114.1 mm to (-87.0, 136.8)
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Other:
- board size 0.9 x 0.6 mm -> 0.6 x 0.9 mm

Commit message: organizar a PCB
Parts:
- moved TP47 291.7 mm to (281.5, 48.5)
- moved TP51 268.7 mm to (259.5, 56.0)
- moved TP50 264.3 mm to (255.0, 52.5)
- moved TP49 238.6 mm to (230.0, 20.5)
- moved D2 222.7 mm to (271.5, 24.0)
- moved R5 214.6 mm to (280.6, 59.0)
- moved R29 208.1 mm to (280.9, 45.0)
- moved C19 207.5 mm to (275.5, 38.5)
- moved C18 206.7 mm to (267.2, 18.5)
- moved R36 206.4 mm to (281.9, 32.0)
- moved R3 200.7 mm to (266.9, 45.8)
- moved R4 200.7 mm to (266.9, 48.0)
- moved R9 200.1 mm to (265.4, 37.0)
- moved R6 200.0 mm to (265.4, 31.3)
- moved R7 200.0 mm to (265.4, 33.5)
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Other:
- copper layers 4 -> 6
