File: Boards/Development Boards/RP2040 P/TVCS Dev.kicad_sch (KiCad schematic)
At the start: 258 parts, among them IC1 INA2181A4IDSQR, IC10 NSVT30010MXV6T1G, IC2 CYPD3177-24LQXQT, IC3 DMP2040USD-13, IC4 ADS1115IRUGR, IC5 INA181A4QDCKRQ1, IC6 DMP2040USD-13, IC7 NCR420ZX, IC8 PCA9306GM,125, IC9 NSVT30010MXV6T1G, J1 DX07S016JA1R1500, J10 Conn_01x01_Socket, J11 Conn_01x01_Socket, J13 Conn_01x01_Socket, J14 Conn_01x01_Socket, J15 Conn_01x01_Socket, J16 Conn_01x01_Socket, J17 Conn_01x01_Socket, J2 Conn_01x01_Socket, J3 Conn_01x01_Socket, J4 MEM2061-01-188-00-A_REVA, J8 Conn_01x01_Socket, J9 Conn_01x01_Socket, Q1 2N7002H6327XTSA2, Q2 2N7002H6327XTSA2, Q3 BC857CMB_315, Q4 BC857CMB_315, U1 SQJA36EP-T1_GE3, U10 VLMKG3400-GS08, U2 MAX31856MUD+T, U3 MAX485CSA+T, U7 LM61460AASQRJRRQ1, U8 LM61460AASQRJRRQ1, U9 LM61460AASQRJRRQ1

Commit message: PCB Dev 2
Connections:
- net SDL I2C is gone; now on net SCL I2C: IC2.13 (HPI_SCL), R6.1
Changed lines of the file:
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@@
 		)
 	)
-	(label "SDL I2C"
+	(label "SCL I2C"
 		(at 25.4 433.07 0)
 		(effects

Commit message: continuação
Parts:
- CR1, CR2, CR3, CR4: footprint LED-Yellow_VLMY1300-GS08:LED_VISHAY_VLMX1300_VIS -> LED-Yellow_VLMY1300-GS08:LEDC1608X100N
- J4: Description_1 10 (8 + 2) Position Card Connector microSD Surface Mount, Right Angle Gold -> 10 (8 + 2) Position Card Connector microSD Surface Mount, Right Angle Gold
- TP31, TP32, TP33, TP34, TP35, TP36, TP37, TP38, TP39, TP40, TP41, TP42, TP43, TP44, TP50, TP51: Description_1 TEST POINT (BLUE) - COMPACT -> TEST POINT (BLUE) - COMPACT
Changed lines of the file:
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@@
 			)
 		)
-		(property "Description_1" "\n                        \n                            TEST POINT (BLUE) - COMPACT\n                        \n"
+		(property "Description_1" "TEST POINT (BLUE) - COMPACT"
 			(at 238.125 78.105 0)
 			(effects
@@
 			)
 		)
-		(property "Description_1" "\n                        \n                            TEST POINT (BLUE) - COMPACT\n                        \n"
+		(property "Description_1" "TEST POINT (BLUE) - COMPACT"
 			(at 338.455 57.785 0)
 			(effects
@@
 			)
 		)
-		(property "Description_1" "\n                        \n                            TEST POINT (BLUE) - COMPACT\n                        \n"
+		(property "Description_1" "TEST POINT (BLUE) - COMPACT"
 			(at 168.91 400.05 0)
 			(effects
@@
 			)
 		)
-		(property "Description_1" "\n                        \n                            TEST POINT (BLUE) - COMPACT\n                        \n"
+		(property "Description_1" "TEST POINT (BLUE) - COMPACT"
 			(at 134.62 312.42 0)
 			(effects
@@
 			)
 		)
-		(property "Description_1" "\n                        \n                            TEST POINT (BLUE) - COMPACT\n                        \n"
+		(property "Description_1" "TEST POINT (BLUE) - COMPACT"
 			(at 144.145 218.44 0)
 			(effects
@@
 			)
 		)
-		(property "Description_1" "\n                        \n                            TEST POINT (BLUE) - COMPACT\n                        \n"
+		(property "Description_1" "TEST POINT (BLUE) - COMPACT"
 			(at 338.455 62.865 0)
 			(effects
@@
 			)
 		)
-		(property "Description_1" "\n                        \n                            TEST POINT (BLUE) - COMPACT\n                        \n"
+		(property "Description_1" "TEST POINT (BLUE) - COMPACT"
 			(at 238.125 83.185 0)
 			(effects
@@
 			)
 		)
-		(property "Description_1" "\n                        \n                            TEST POINT (BLUE) - COMPACT\n                        \n"
+		(property "Description_1" "TEST POINT (BLUE) - COMPACT"
 			(at 159.385 397.51 0)
 			(effects
@@
 			)
 		)
-		(property "Footprint" "LED-Yellow_VLMY1300-GS08:LED_VISHAY_VLMX1300_VIS"
+		(property "Footprint" "LED-Yellow_VLMY1300-GS08:LEDC1608X100N"
 			(at 175.895 33.655 0)
 			(effects
@@
 			)
 		)
-		(property "Description_1" "\n                        \n                            TEST POINT (BLUE) - COMPACT\n                        \n"
+		(property "Description_1" "TEST POINT (BLUE) - COMPACT"
 			(at 144.145 231.14 0)
 			(effects
@@
 			)
 		)
-		(property "Description_1" "\n                        \n                            TEST POINT (BLUE) - COMPACT\n                        \n"
+		(property "Description_1" "TEST POINT (BLUE) - COMPACT"
 			(at 338.455 65.405 0)
 			(effects
@@
 			)
 		)
-		(property "Footprint" "LED-Yellow_VLMY1300-GS08:LED_VISHAY_VLMX1300_VIS"
+		(property "Footprint" "LED-Yellow_VLMY1300-GS08:LEDC1608X100N"
 			(at 114.3 33.655 0)
 			(effects
@@
 			)
 		)
-		(property "Footprint" "LED-Yellow_VLMY1300-GS08:LED_VISHAY_VLMX1300_VIS"
+		(property "Footprint" "LED-Yellow_VLMY1300-GS08:LEDC1608X100N"
 			(at 155.575 33.655 0)
 			(effects
@@
 			)
 		)
-		(property "Description_1" "\n                        \n                            TEST POINT (BLUE) - COMPACT\n                        \n"
+		(property "Description_1" "TEST POINT (BLUE) - COMPACT"
 			(at 338.455 60.325 0)
 			(effects
@@
 			)
 		)
-		(property "Description_1" "\n                        \n                            TEST POINT (BLUE) - COMPACT\n                        \n"
+		(property "Description_1" "TEST POINT (BLUE) - COMPACT"
 			(at 186.69 257.81 0)
 			(effects
@@
 			)
 		)
-		(property "Footprint" "LED-Yellow_VLMY1300-GS08:LED_VISHAY_VLMX1300_VIS"
+		(property "Footprint" "LED-Yellow_VLMY1300-GS08:LEDC1608X100N"
 			(at 135.89 33.655 0)
 			(effects
@@
 			)
 		)
-		(property "Description_1" "\n                        \n                            TEST POINT (BLUE) - COMPACT\n                        \n"
+		(property "Description_1" "TEST POINT (BLUE) - COMPACT"
 			(at 238.125 85.725 0)
 			(effects
@@
 			)
 		)
-		(property "Description_1" "\n                        \n                            TEST POINT (BLUE) - COMPACT\n                        \n"
+		(property "Description_1" "TEST POINT (BLUE) - COMPACT"
 			(at 128.27 257.81 0)
 			(effects
@@
 			)
 		)
-		(property "Description_1" "\n                        \n                            TEST POINT (BLUE) - COMPACT\n                        \n"
+		(property "Description_1" "TEST POINT (BLUE) - COMPACT"
 			(at 84.455 312.42 0)
 			(effects
@@
 			)
 		)
-		(property "Description_1" "\n                        \n                            TEST POINT (BLUE) - COMPACT\n                        \n"
+		(property "Description_1" "TEST POINT (BLUE) - COMPACT"
 			(at 238.125 75.565 0)
 			(effects
@@
 			)
 		)
-		(property "Description_1" "\n                        \n                            10 (8 + 2) Position Card Connector microSD Surface Mount, Right Angle Gold\n                        \n"
+		(property "Description_1" "10 (8 + 2) Position Card Connector microSD Surface Mount, Right Angle Gold"
 			(at 412.115 155.575 0)
 			(effects
