File: Boards/Development Boards/RP2040 P/TVCS Dev.kicad_sch (KiCad schematic)
At the start: 258 parts, among them IC1 INA2181A4IDSQR, IC10 NSVT30010MXV6T1G, IC2 CYPD3177-24LQXQT, IC3 DMP2040USD-13, IC4 ADS1115IRUGR, IC5 INA181A4QDCKRQ1, IC6 DMP2040USD-13, IC7 NCR420ZX, IC8 PCA9306GM,125, IC9 NSVT30010MXV6T1G, J1 DX07S016JA1R1500, J10 Conn_01x01_Socket, J11 Conn_01x01_Socket, J13 Conn_01x01_Socket, J14 Conn_01x01_Socket, J15 Conn_01x01_Socket, J16 Conn_01x01_Socket, J17 Conn_01x01_Socket, J2 Conn_01x01_Socket, J3 Conn_01x01_Socket, J4 MEM2061-01-188-00-A_REVA, J8 Conn_01x01_Socket, J9 Conn_01x01_Socket, Q1 2N7002H6327XTSA2, Q2 2N7002H6327XTSA2, Q3 BC857CMB_315, Q4 BC857CMB_315, U1 SQJA36EP-T1_GE3, U10 VLMKG3400-GS08, U2 MAX31856MUD+T, U3 MAX485CSA+T, U7 LM61460AASQRJRRQ1, U8 LM61460AASQRJRRQ1, U9 LM61460AASQRJRRQ1

Commit message: update RP DEV
Parts:
- removed J4: MEM2061-01-188-00-A_REVA, SD-CARD_MEM2061-01-188-00-A:GCT_MEM2061-01-188-00-A_REVA, symbol MEM2061-01-188-00-A_REVA:MEM2061-01-188-00-A_REVA
- removed R48: PTS060301B100RP100, PTS060301B100RP100:RESC1508X55N, symbol PTS060301B100RP100:PTS060301B100RP100
- removed R8: 120, Resistor-0402:RES_0402, symbol Device:R
- removed TP44: 5277, Test Hook:KEYSTONE_5277, symbol 5277:5277
- added C14: 100nF, Capacitor-0402:Capacitor_0402, symbol Device:C
- added C15, C28: 100n, Capacitor-0402:Capacitor_0402, symbol Device:C_Small
- added C16, C26, C27, C29, C38, C39: 10n, Capacitor-0402:Capacitor_0402, symbol Device:C_Small
- added H1, H2, H3, H4: MountingHole, MountingHole:MountingHole_3.2mm_M3_ISO7380_Pad_TopBottom, symbol Mechanical:MountingHole
- added J4, J5, J6, J7: Conn_01x01_Socket, Pico_Conn1x1:Pico_01pin, symbol Connector:Conn_01x01_Socket
- added R48, R54: 100, Resistor-0402:RES_0402, symbol Device:R
- added TP44: TestPoint, TestPoint:TestPoint_Pad_2.0x2.0mm, symbol Connector:TestPoint
- added U11: STLM20DD9F, STLM20DD9F:UDFN-4L_STM, symbol STLM20DD9F:STLM20DD9F
- added U12, U6: MAX31856MUD+T, Thermocouple:21-0066J_14_MXM, symbol MAX31856MUD-T:MAX31856MUD+T
- C13: value 10u -> 1u; footprint Capacitor-0805:Capacitor_0805 -> Capacitor-0402:Capacitor_0402
- R46: value 30k -> 370
- R49: value 30k -> 100
- TP1, TP10, TP11, TP12, TP13, TP14, TP15, TP16, TP17, TP18, TP19, TP2, TP20, TP21, TP22, TP23, TP24, TP25, TP26, TP27, TP28, TP29, TP3, TP30, TP4, TP5, TP6, TP7, TP8, TP9: footprint Test Hook:KEYSTONE_5277 -> TestPoint:TestPoint_Pad_2.0x2.0mm
Connections:
- net +3.3V: now also C14.1, C26.2, C27.2, C38.2, C39.2, U11.4 (VCC), U12.5 (AVDD), U12.8 (DVDD), U6.5 (AVDD), U6.8 (DVDD); no longer C13.1, R46.2, R49.1
- net DC.DC2 PGOOD: now also C_BIAS1.2
- net DC.DC3 PGOOD: now also C_BIAS2.2
- net GND: now also C14.2, C16.2, C26.1, C27.1, C29.2, C38.1, C39.1, U11.3 (GND), U12.1 (AGND), U12.14 (DGND), U6.1 (AGND), U6.14 (DGND); no longer C_BIAS1.2, C_BIAS2.2, IC4.7 (AIN3), R47.2
- net PRESS_SENSE: now also R13.1, R46.1
- net SPI1_MISO: now also U12.11 (SDO), U6.11 (SDO)
- net SPI1_MOSI: now also U12.12 (SDI), U6.12 (SDI)
- net SPI1_SCK: now also U12.10 (SCK), U6.10 (SCK)
- net THERMO1_~{CS}: now also TP21.1
- removed net TEMP SENSE +: R12.1, R49.2, TP22.1
- removed net TEMP SENSE -: R13.1, R46.1, R47.1, TP21.1
- new net: C15.2, C16.1, R48.1, U6.3 (T-)
- new net: C28.1, R49.1, U12.4 (T+)
- new net: C28.2, C29.1, R54.1, U12.3 (T-)
- new net: C15.1, R47.1, U6.4 (T+)
- new net AIN3: C13.1, IC4.7 (AIN3), R46.2
- new net THERMO2 T+: J7.1 (Pin_1), R47.2
- new net THERMO2 T-: J6.1 (Pin_1), R48.2, U6.2 (BIAS)
- new net THERMO2_~{CS}: TP44.1, U6.9 (~{CS})
- new net THERMO2_~{DRDY}: U6.7 (~{DRDY})
- new net THERMO3 T+: J5.1 (Pin_1), R49.2
- new net THERMO3 T-: J4.1 (Pin_1), R54.2, U12.2 (BIAS)
- new net THERMO3_~{CS}: TP22.1, U12.9 (~{CS})
- new net THERMO3_~{DRDY}: U12.7 (~{DRDY})
- new net Temp_Sense: R12.1, U11.1 (VOUT)
Other:
- sheet RP2040 Standard1 ports: added GP13/SPI1 ~{CS}, GP17, GP18, GP19, GP29/SPI1 ~{CS}, GPIO16; removed GP16/SPI0_MISO, GP17/SPI0 ~{CS}, GP18/SPI0 SCK, GP19/SPI0 MOSI, GPIO13, GPIO29
- note removed: "16G SD-Card"
- moved on the sheet: C1, C10, C11, C12, C17, C18, C19, C20, C22, C24, C25, C31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
