File: Boards/Rocket Systems/TVCS/TVCS.kicad_pcb (KiCad board)
At the start: 6 copper layers, 90 x 90 mm, 259 parts, among them IC1 NCR420ZX, IC2 NSVT30010MXV6T1G, IC3 CYPD3177-24LQXQT, IC4 ADS1115IRUGR, IC5 INA2181A4IDSQR, IC6 PCA9306GM,125, IC7 INA181A4QDCKRQ1, IC8 DMP2040USD-13, IC9 DMP2040USD-13, J1 Conn_01x01_Socket, J10 DX07S016JA1R1500, J11 Conn_01x01_Socket, J12 Conn_01x01_Socket, J13 Conn_01x01_Socket, J14 Conn_01x01_Socket, J15 Conn_01x01_Socket, J16 Conn_01x01_Socket, J17 Conn_01x01_Socket, J18 Conn_01x01_Socket, J2 Conn_01x01_Socket, J3 Conn_01x01_Socket, J4 Conn_01x01_Socket, J5 Conn_01x01_Socket, J6 Conn_01x01_Socket, J7 BM03B-SRSS-TBLFSN, J8 Conn_01x01_Socket, J9 Conn_01x01_Socket, Q1 2N7002H6327XTSA2, Q2 2N7002H6327XTSA2, Q5 BC857CMB_315, Q6 BC857CMB_315, Q7 BC857CMB_315, U1 MAX31856MUD+T, U11 MAX31856MUD+T, U13 LM61460AASQRJRRQ1, U14 LM61460AASQRJRRQ1, U2 W25Q128JVSIQ TR, U3 MAX31856MUD+T, U4 LM61460AASQRJRRQ1, U5 SQJA36EP-T1_GE3, U6 VLMKG3400-GS08, U7 ST1L05APU33R, U8 MAX485CSA+T, U9 SQJA36EP-T1_GE3

Commit message: organizar a PCB
Parts:
- CV13: value 1uF -> 100nF
- CV14: value 100nF -> 4.7uF
- CV16: value 4.7uF -> 1uF
- IC8, IC9: footprint DMP3098LSD-13:SOIC127P600X175-8N -> DMP2040USD-13:SOIC127P600X175-8N
- R26: value 10k -> 1k
- R33: value 1k -> 10k
Connections:
- CV14 pad 1: +3.3V -> GND
- CV14 pad 2: GND -> +5V
- CV15 pad 2: +5V -> +3.3V
- CV16 pad 2: +3.3V -> +5V
- CV17 pad 1: GND -> +3.3V
- CV17 pad 2: +5V -> GND
- R26 pad 1: Net-(XTAL1-TRI-STATE(STBY)) -> /RP2040 Standard/~{USB_BOOT}
- R26 pad 2: +3.3V -> /RP2040 Standard/MCU QSPI_SS
- R33 pad 1: /RP2040 Standard/~{USB_BOOT} -> Net-(XTAL1-TRI-STATE(STBY))
- R33 pad 2: /RP2040 Standard/MCU QSPI_SS -> +3.3V
