File: Boards/Rocket Systems/TVCS/TVCS.kicad_pcb (KiCad board)
At the start: 6 copper layers, 90 x 90 mm, 259 parts, among them IC1 NCR420ZX, IC2 NSVT30010MXV6T1G, IC3 CYPD3177-24LQXQT, IC4 ADS1115IRUGR, IC5 INA2181A4IDSQR, IC6 PCA9306GM,125, IC7 INA181A4QDCKRQ1, IC8 DMP2040USD-13, IC9 DMP2040USD-13, J1 Conn_01x01_Socket, J10 DX07S016JA1R1500, J11 Conn_01x01_Socket, J12 Conn_01x01_Socket, J13 Conn_01x01_Socket, J14 Conn_01x01_Socket, J15 Conn_01x01_Socket, J16 Conn_01x01_Socket, J17 Conn_01x01_Socket, J18 Conn_01x01_Socket, J2 Conn_01x01_Socket, J3 Conn_01x01_Socket, J4 Conn_01x01_Socket, J5 Conn_01x01_Socket, J6 Conn_01x01_Socket, J7 BM03B-SRSS-TBLFSN, J8 Conn_01x01_Socket, J9 Conn_01x01_Socket, Q1 2N7002H6327XTSA2, Q2 2N7002H6327XTSA2, Q5 BC857CMB_315, Q6 BC857CMB_315, Q7 BC857CMB_315, U1 MAX31856MUD+T, U11 MAX31856MUD+T, U13 LM61460AASQRJRRQ1, U14 LM61460AASQRJRRQ1, U2 W25Q128JVSIQ TR, U3 MAX31856MUD+T, U4 LM61460AASQRJRRQ1, U5 SQJA36EP-T1_GE3, U6 VLMKG3400-GS08, U7 ST1L05APU33R, U8 MAX485CSA+T, U9 SQJA36EP-T1_GE3

Commit message: mudei cores
Other:
- copper layers 6 -> 4
Changed lines of the file:
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@@
 		(4 "In1.Cu" signal)
 		(6 "In2.Cu" signal)
-		(8 "In3.Cu" signal)
-		(10 "In4.Cu" signal)
 		(2 "B.Cu" signal)
 		(9 "F.Adhes" user "F.Adhesive")
@@
 			)
 			(layer "dielectric 2"
-				(type "prepreg")
-				(thickness 0.535)
+				(type "core")
+				(thickness 1.24)
 				(material "FR4")
 				(epsilon_r 4.5)
@@
 				(type "prepreg")
 				(thickness 0.1)
-				(material "FR4")
-				(epsilon_r 4.5)
-				(loss_tangent 0.02)
-			)
-			(layer "In3.Cu"
-				(type "copper")
-				(thickness 0.035)
-			)
-			(layer "dielectric 4"
-				(type "core")
-				(thickness 0.535)
-				(material "FR4")
-				(epsilon_r 4.5)
-				(loss_tangent 0.02)
-			)
-			(layer "In4.Cu"
-				(type "copper")
-				(thickness 0.035)
-			)
-			(layer "dielectric 5"
-				(type "prepreg")
-				(thickness 0.1)
