File: Boards/Rocket Systems/TVCS/TVCS.kicad_sch (KiCad schematic)
At the start: 226 parts, among them IC1 NCR420ZX, IC2 NSVT30010MXV6T1G, IC3 CYPD3177-24LQXQT, IC4 ADS1115IRUGR, IC5 INA2181A4IDSQR, IC6 PCA9306GM,125, IC7 INA181A4QDCKRQ1, IC8 DMP2040USD-13, IC9 DMP2040USD-13, J1 Conn_01x01_Socket, J10 DX07S016JA1R1500, J11 Conn_01x01_Socket, J12 Conn_01x01_Socket, J13 Conn_01x01_Socket, J14 Conn_01x01_Socket, J15 Conn_01x01_Socket, J16 Conn_01x01_Socket, J17 Conn_01x01_Socket, J18 Conn_01x01_Socket, J2 Conn_01x01_Socket, J3 Conn_01x01_Socket, J4 Conn_01x01_Socket, J5 Conn_01x01_Socket, J6 Conn_01x01_Socket, J8 Conn_01x01_Socket, J9 Conn_01x01_Socket, Q1 2N7002H6327XTSA2, Q2 2N7002H6327XTSA2, Q5 BC857CMB_315, Q6 BC857CMB_315, Q7 BC857CMB_315, U1 MAX31856MUD+T, U11 MAX31856MUD+T, U13 LM61460AASQRJRRQ1, U14 LM61460AASQRJRRQ1, U3 MAX31856MUD+T, U4 LM61460AASQRJRRQ1, U5 SQJA36EP-T1_GE3, U6 VLMKG3400-GS08, U8 MAX485CSA+T, U9 SQJA36EP-T1_GE3

Commit message: Development board update
Changed lines of the file:
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@@
 	(polyline
 		(pts
-			(xy 11.43 184.15) (xy 230.505 184.15)
+			(xy 12.065 184.15) (xy 230.505 184.15)
 		)
 		(stroke
@@
 	(polyline
 		(pts
-			(xy 12.7 454.025) (xy 231.775 454.025)
+			(xy 12.065 454.025) (xy 231.775 454.025)
 		)
 		(stroke
@@
 	(text "Tem de se escolher contactos apropriados para os termocouples!"
 		(exclude_from_sim no)
-		(at 80.645 117.475 0)
+		(at 351.79 114.935 0)
 		(effects
 			(font
@@
 		)
 		(instances
-			(project "TVCS Top"
+			(project "TVCS"
 				(path "/2cb205da-01dc-4dd5-90f3-3844dc2f7334"
 					(page "2")

Commit message: organizar a PCB
Parts:
- IC8, IC9: footprint DMP3098LSD-13:SOIC127P600X175-8N -> DMP2040USD-13:SOIC127P600X175-8N
- U5, U9: footprint PowerPAK_SO-8L_3_VIS -> SQJA36EP-T1-GE3:PowerPAK_SO-8L_3_VIS
