File: Boards/Rocket Systems/TVCS/TVCS.kicad_sch (KiCad schematic)
At the start: 226 parts, among them IC1 NCR420ZX, IC2 NSVT30010MXV6T1G, IC3 CYPD3177-24LQXQT, IC4 ADS1115IRUGR, IC5 INA2181A4IDSQR, IC6 PCA9306GM,125, IC7 INA181A4QDCKRQ1, IC8 DMP2040USD-13, IC9 DMP2040USD-13, J1 Conn_01x01_Socket, J10 DX07S016JA1R1500, J11 Conn_01x01_Socket, J12 Conn_01x01_Socket, J13 Conn_01x01_Socket, J14 Conn_01x01_Socket, J15 Conn_01x01_Socket, J16 Conn_01x01_Socket, J17 Conn_01x01_Socket, J18 Conn_01x01_Socket, J2 Conn_01x01_Socket, J3 Conn_01x01_Socket, J4 Conn_01x01_Socket, J5 Conn_01x01_Socket, J6 Conn_01x01_Socket, J8 Conn_01x01_Socket, J9 Conn_01x01_Socket, Q1 2N7002H6327XTSA2, Q2 2N7002H6327XTSA2, Q5 BC857CMB_315, Q6 BC857CMB_315, Q7 BC857CMB_315, U1 MAX31856MUD+T, U11 MAX31856MUD+T, U13 LM61460AASQRJRRQ1, U14 LM61460AASQRJRRQ1, U3 MAX31856MUD+T, U4 LM61460AASQRJRRQ1, U5 SQJA36EP-T1_GE3, U6 VLMKG3400-GS08, U8 MAX485CSA+T, U9 SQJA36EP-T1_GE3

Commit message: TVCS refactor
Muitas alterações e correções na placa TVCSO:
Novo ADC, filtros passa baixo, novo RS transceiver, reformulação de
conexões
Parts:
- removed C1, C11, C15, C17, C18, C26, C27, C35, C36, C37, C5, C7, C_BT1, C_BT2, C_BT3, C_IN_HFI1, C_IN_HFI2, C_IN_HFI3, C_IN_HFI4, C_IN_HFI5, C_IN_HFI6: 100n, Capacitor-0402:Capacitor_0402, symbol Device:C_Small
- removed C10, C24, C25, C28: 2.2u, Capacitor-0402:Capacitor_0402, symbol Device:C_Small
- removed C12, C13, C14, C2, C3, C4, C6, C8, C9: 10n, Capacitor-0402:Capacitor_0402, symbol Device:C_Small
- removed C16, C19, C20, C21, C_BIAS1, C_BIAS2, C_OUT1, C_VCC1, C_VCC2, C_VCC3: 1u, Capacitor-0603:Capacitor_0603, symbol Device:C_Small
- removed C22, C_IN1, C_IN2, C_IN3, C_IN4, C_IN5, C_IN6: 4.7u, Capacitor-1206:Capacitor_1206, symbol Device:C_Small
- removed C23: 1n, Capacitor-0402:Capacitor_0402, symbol Device:C_Small
- removed C29, C30: 470n, Capacitor-0402:Capacitor_0402, symbol Device:C_Small
- removed C31, C32, C33: 1u, Capacitor-0402:Capacitor_0402, symbol Device:C_Small
- removed C34: C, Capacitor-0402:Capacitor_0402, symbol Device:C_Small
- removed C_FF1: 22p, Capacitor-0402:Capacitor_0402, symbol Device:C_Small
- removed C_IN-BLK1, C_IN-BLK2, C_IN-BLK3: 10u, Capacitor-4mm:Capacitor_4mm, symbol Device:C_Small
- removed C_OUT10, C_OUT9: 47u, Capacitor-0805:Capacitor_0805, symbol Device:C_Small
- removed C_OUT11, C_OUT12, C_OUT13, C_OUT14, C_OUT7, C_OUT8: 22u, Capacitor-0805:Capacitor_0805, symbol Device:C_Small
- removed C_OUT15: 560u, Capacitor-8mm:Capacitor_8mm, symbol Device:C_Small
- removed C_OUT16: 100u, Capacitor-8mm:Capacitor_8mm, symbol Device:C_Small
- removed C_OUT2, C_OUT3, C_OUT4, C_OUT5: 10u, Capacitor-0805:Capacitor_0805, symbol Device:C_Small
- removed C_OUT6: 100u, Capacitor-6mm:Capacitor_6mm, symbol Device:C_Small
- removed D1, D6: RB095BGE, SchottkyDiode-RB095BGE:RD3P175SNFRATL, symbol RB095BGE-30TL:RB095BGE-30TL
- removed D2, D5: RSX301L, Diode-Schottky_RSX301L:DIOM5026X220N, symbol RSX301L-30DDTE25:RSX301L-30DDTE25
- removed D3: SP3004-04XTG, TVS-SP3004:SOT563_LTF, symbol SP3004-04XTG:SP3004-04XTG
- removed IC1: NCR420ZX, LED-Driver_NCR420ZX:SOT230P700X180-4N, symbol NCR420ZX:NCR420ZX
- removed IC3: CYPD3177-24LQXQT, USBC-PD_CYPD3177:QFN50P400X400X60-25N-D, symbol CYPD3177-24LQXQT:CYPD3177-24LQXQT
- removed IC4: ADS1115IRUGR, ADS1115:ADS1115IRUGR, symbol ADS1115IRUGR:ADS1115IRUGR
- removed IC5: INA2181A4IDSQR, INA2181A4IDSQR:SON40P200X200X80-11N, symbol INA2181A4IDSQR:INA2181A4IDSQR
- removed IC6: PCA9306GM,125, PCA9306GM,125:PCA9570GMH, symbol PCA9306GM_125:PCA9306GM,125
- removed IC7: INA181A4QDCKRQ1, INA181A4QDCKRQ1:SOT65P210X110-6N, symbol INA181A4QDCKRQ1:INA181A4QDCKRQ1
- removed IC8, IC9: DMP2040USD-13, DMP2040USD-13:SOIC127P600X175-8N, symbol DMP2040USD-13:DMP2040USD-13
- removed J10: DX07S016JA1R1500, USBC-DX07S016JA1:JAE_DX07S016JA1R1500, symbol DX07S016JA1R1500:DX07S016JA1R1500
- removed L1: 2.2u, Inductor-10.1x10:Inductor_10.1x10, symbol Device:L
- removed LED4: VLMS1500-GS08, LED-Red_VLMS1500-GS08:LED_00-GS08_VIS_RED, symbol VLMS1500-GS08:VLMS1500-GS08
- removed L_SW1: 10u, Inductor-11.5x10:Inductor_11.5x10, symbol Device:L
- removed L_SW2, L_SW3: 15u, Inductor-10.1x10:Inductor_10.1x10, symbol Device:L
- removed Q1: 2N7002H6327XTSA2, NMOS_2N7002:PG-SOT23-3-5_INF_MIN, symbol NMOS_2N7002:2N7002H6327XTSA2
- removed R1, R19, R2, R20, R4, R5, R59, R_BT3: 100, Resistor-0402:RES_0402, symbol Device:R
- removed R10, R11, R15: 370, Resistor-0402:RES_0402, symbol Device:R
- removed R12, R13, R16: 10K, Resistor-0402:RES_0402, symbol Device:R
- removed R14, R28, R36, R38, R39, R40, R41, R44, R45, R46: 2k, Resistor-0402:RES_0402, symbol Device:R
- removed R18, R21, R66: 160, Resistor-0402:RES_0402, symbol Device:R
- removed R27: 54k2, Resistor-0402:RES_0402, symbol Device:R
- removed R37: 95, Resistor-0402:RES_0402, symbol Device:R
- removed R47: DNP, Resistor-0402:RES_0402, symbol Device:R
- removed R49, R50: 50k, Resistor-0402:RES_0402, symbol Device:R
- removed R51: 10k, Resistor-0402:RES_0402, symbol Device:R
- removed R52, R53, R61, R62, R65, R_FF1: 1k, Resistor-0402:RES_0402, symbol Device:R
- removed R60: 200k, Resistor-0402:RES_0402, symbol Device:R
- removed R63: PTS060301B100RP100, PTS060301B100RP100:RESC1508X55N, symbol PTS060301B100RP100:PTS060301B100RP100
- removed R7: 120, Resistor-0402:RES_0402, symbol Device:R
- removed R8, R9: 20K, Resistor-0402:RES_0402, symbol Device:R
- removed R_BIAS1, R_BIAS2: 5, Resistor-0402:RES_0402, symbol Device:R
- removed R_BT1, R_BT2: 50, Resistor-0402:RES_0402, symbol Device:R
- removed R_ENB1: 100k, Resistor-0603:RES_0603, symbol Device:R
- removed R_ENB2: 63k4, Resistor-0402:RES_0402, symbol Device:R
- removed R_ENB3: 45k3, Resistor-0402:RES_0402, symbol Device:R
- removed R_ENT1: 931k, Resistor-0603:RES_0603, symbol Device:R
- removed R_ENT2: 590k, Resistor-0402:RES_0402, symbol Device:R
- removed R_ENT3: 422k, Resistor-0402:RES_0402, symbol Device:R
- removed R_FBB1: 8k66, Resistor-0603:RES_0603, symbol Device:R
- removed R_FBB2: 30, Resistor-0603:RES_0603, symbol Device:R
- removed R_FBB3: 12k6, Resistor-0603:RES_0603, symbol Device:R
- removed R_FBB4: 50, Resistor-0603:RES_0603, symbol Device:R
- removed R_FBB5: 22k1, Resistor-0603:RES_0603, symbol Device:R
- removed R_FBB6: 120, Resistor-0603:RES_0603, symbol Device:R
- removed R_FBT1, R_FBT2, R_FBT3, R_PG1, R_PG2, R_PG3: 100K, Resistor-0603:RES_0603, symbol Device:R
- removed R_RT1, R_RT2, R_RT3: 33k2, Resistor-0603:RES_0603, symbol Device:R
- removed Rsense1, Rsense2: 2.5m, Resistor-0805:RES_0805, symbol Device:R
- removed Rsense3: 7.5m, Resistor-2512:RES_WSLP2512, symbol Device:R
- removed U1, U11, U3: MAX31856MUD+T, Thermocouple:21-0066J_14_MXM, symbol MAX31856MUD-T:MAX31856MUD+T
- removed U13, U14, U4: LM61460AASQRJRRQ1, DCDC_LM61460:VQFN-HR14_RJR_TEX, symbol DCDC_LM61460:LM61460AASQRJRRQ1
- removed U8: MAX485CSA+T, RS Transceiver:21-0041-3-M_90-0096-8L_MXM, symbol RS_Transceiver:MAX485CSA+T
- added C40, C42: 100n, Capacitor-0402:Capacitor_0402, symbol Device:C_Small
- added Q3: 2N7002H6327XTSA2, NMOS_2N7002:PG-SOT23-3-5_INF_MIN, symbol NMOS_2N7002:2N7002H6327XTSA2
- added R55: 120, Resistor-0603:RES_0603, symbol Device:R
- added SW1: D2F-01-D, D2F-01-D_OMR, symbol Switch_D2F-01:D2F-01-D
- added U12: THVD2410VDRCR, VSON10_DRC_TEX, symbol THVD2410VDRCR:THVD2410VDRCR
- added VD1, VD2: SMAJ30CA, symbol SMAJ30CA:SMAJ30CA
- R30: value 1k -> 10k
- R48: value 54k2 -> 10k
- R57, R58: value 30k -> 2k
Connections:
- net TEMP SENSE - is gone; now on net +5V: R57.1
- net +3.3V: now also R48.1, C42.2, Q3.1 (G), U12.1 (VIO); no longer R48.2, R57.2
- net +5V: now also C40.1, SW1.2, U12.10 (VCC)
- net GND: now also R30.2, C40.2, C42.1, SW1.1, U12.11 (EPAD), U12.6 (GND), VD1.A, VD2.A; no longer R30.1
- net Main Servo Valve renamed Servo_OUT1 PWM
- net PRESS_SENSE: no longer names the net of J16.1 (Pin_1)
- net Purge Valve Drive renamed Purge Solenoid Valve
- net RS_A renamed RS_DP
- net RS_DP: now also R55.2, U12.8 (A), VD2.K
- net RS_B renamed RS_DN
- net RS_DN: now also R55.1, U12.9 (B), VD1.K
- net Servo Valve PWM renamed Servo_IN1 PWM
- net Status Green renamed Green Status
- net Status Red renamed Red Status
- net TEMP SENSE + renamed Servo_IN2 PWM
- net Servo_IN2 PWM: now also Q3.2 (S)
- net THERMO1 T+ renamed THERMO1 DP
- net THERMO1 T- renamed THERMO1 DN
- net THERMO1_~{FAULT} renamed 1~{FAULT} THERMO
- net THERMO2 T+ renamed THERMO2 DP
- net THERMO2 T- renamed THERMO2 DN
- net THERMO2_~{FAULT} renamed 2~{FAULT} THERMO
- net THERMO3 T+ renamed THERMO3 DP
- net THERMO3 T- renamed THERMO3 DN
- net THERMO3_~{FAULT} renamed 3~{FAULT} THERMO
- new net: SW1.3, U12.7 (SLR)
- new net ENABLE_RS: R30.1, U12.3 (DE), U12.4 (~{RE})
- new net READ_RS: R48.2, U12.2 (R)
- new net Servo_OUT2 PWM: Q3.3 (D), R57.2
- new net WRITE_RS: U12.5 (D)
- no-connect marks 4 -> 0
Other:
- added sheet Power Unit (Power Unit.kicad_sch)
- added sheet Sensor Unit (Sensor Unit.kicad_sch)
- sheet RP2040 Standard ports: added USB DN, USB DP; removed none
- note added: "SLR LOW = 1Mpbs SLR HIGH = 250kbps"
- note added: "Servo Valve Driver"
- note added: "TODO LIST: LEDs PGOOD Power Multiplexer na USB-C Novo LED Driver USB-C Atualizar Pinout Recalcular Current Sense Resistors Buffer a criar Vref nos sensores de corrente Buzzer"
- note removed: "4 Channel ESD Diode"
- note removed: ">15V to 12V Converter"
- note removed: ">15V to 5V Converter"
- note removed: ">15V to 8.4V Converter"
- note removed: "ADC + I2C Translator"
- note removed: "Anti-Aliasing Filter: Fs = 860Hz => Fc = 430Hz"
- note removed: "Buck Converters"
- note removed: "C_IN-BLK1 and C_OUT6 are electrolytic polarized capacitors! All others are ceramic X7R capacitors with appropriate voltage ratings."
- note removed: "C_IN-BLK2 and C_OUT10 are electrolytic polarized capacitors! All others are ceramic X7R capacitors with appropriate voltage ratings."
- note removed: "C_IN-BLK3 and C_OUT15 are electrolytic polarized capacitors! All others are ceramic X7R capacitors with appropriate voltage ratings."
- note removed: "Capacitor to adjust signal"
- note removed: "Current Sensor"
- note removed: "DC.DC1 VCC coloca PGOOD a 3.3V"
- note removed: "DC.DC2 VCC coloca PGOOD a 3.3V"
- note removed: "DC.DC3 VCC coloca PGOOD a 3.3V"
- note removed: "EMI Filter"
- note removed: "I2C ADDR is 0x08"
- note removed: "Implementar Power Multiplexing para desarmar a USB-C caso a bateria seja conectada"
- note removed: "Main Valve Driver - Servo Motor"
- note removed: "Não Prioritário:"
- note removed: "Temperature Sensor"
- note removed: "Thermocouples"
- note removed: "This ADC is to be set at max sampling rate (860Hz) With AIN0 and AIN1 on differential mode and AIN2 in single-ended mode. With ADDR to ground the ADC is configured for a 0x90 I2C address"
- note removed: "USB-C Power Delivery Controller (15V 5A)"
- note removed: "VBUS: 16V nominal when powered by battery VBUS: 15V nominal when powered through USB-C PD"
- note removed: "VMAX= 3V3/2 => 15V VMIN= 3V3/2 => 15V ICoarse = 3V3 => 5A Ifine = 0A"
- note removed: "Vout = 15V => to DC.DC Stage Iout.max = 4A"
- note removed: "Vout = 15V => to LDO Iout.max = 900mA"
- note removed: "Vout is set to 12.5V to compensate Diode and Rsense drops. The Schottky diode has a 425mV forward voltage drop."
- note removed: "Vout is set to 5.5V to compensate Diode and Rsense drops The Schottky diode has a 420mV forward voltage drop."
- note removed: "Vout is set to 5.5V to compensate Diode and Rsense drops. The Schottky diode has a 425mV forward voltage drop."
- note removed: "differential routing"
- moved on the sheet: CR1, CR2, CR3, CR4, D4, D7, IC2, J1, J11, J12, J13, J14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

Commit message: TVCS fixes and required additions
Parts:
- added IC1: BC846BLT1G, BJT NPN:SOT96P237X111-3N, symbol BC846BLT1G:BC846BLT1G
- added LS1: PKLCS1212E20A0-R1, PKLCS1212E20A0-R1:PKLCS1212E20A0-R1, symbol PKLCS1212E20A0-R1:PKLCS1212E20A0-R1
- added R18, R19: 1k, Resistor-0402:RES_0402, symbol Device:R
Connections:
- net +5V: now also LS1.P, R19.1
- net GND: now also IC1.2 (E)
- new net: IC1.3 (C), LS1.N, R19.2
- new net: IC1.1 (B), R18.1
- new net Buzzer: R18.2
Other:
- note added: "TODO LIST: Power Multiplexer na USB-C Buffer a criar Vref nos sensores de corrente Meter isto mais apresentavel Atualizar Pinout"
- note removed: "TODO LIST: LEDs PGOOD Power Multiplexer na USB-C Novo LED Driver USB-C Atualizar Pinout Recalcular Current Sense Resistors Buffer a criar Vref nos sensores de corrente Buzzer"

Commit message: small pinout update
Other:
- sheet Sensor Unit ports: added 1~{DRDY} THERMO, 1~{FAULT} THERMO, 2~{DRDY} THERMO, 2~{FAULT} THERMO, 3~{DRDY} THERMO, 3~{FAULT} THERMO, MISO SPI, MOSI SPI, SCK SPI, THERMO1 DN, THERMO1 DP, THERMO2 DN, THERMO2 DP, THERMO3 DN, THERMO3 DP, Temp_Sense, ~{CS} THERMO1 SPI, ~{CS} THERMO2 SPI, ~{CS} THERMO3 SPI; removed Temp Sense
- moved on the sheet: IC1, LS1, R18, R19
