File: Boards/Rocket Systems/TVCS/TVCS.kicad_sch (KiCad schematic)
At the start: 62 parts, among them IC1 BC846BLT1G, IC2 NSVT30010MXV6T1G, J1 Conn_01x01_Socket, J11 Conn_01x01_Socket, J12 Conn_01x01_Socket, J13 Conn_01x01_Socket, J14 Conn_01x01_Socket, J15 Conn_01x01_Socket, J16 Conn_01x01_Socket, J17 Conn_01x01_Socket, J18 Conn_01x01_Socket, J2 Conn_01x01_Socket, J3 Conn_01x01_Socket, J4 Conn_01x01_Socket, J5 Conn_01x01_Socket, J6 Conn_01x01_Socket, J8 Conn_01x01_Socket, J9 Conn_01x01_Socket, Q2 2N7002H6327XTSA2, Q3 2N7002H6327XTSA2, Q5 BC857CMB_315, Q6 BC857CMB_315, Q7 BC857CMB_315, SW1 D2F-01-D, U12 THVD2410VDRCR, U5 SQJA36EP-T1_GE3, U6 VLMKG3400-GS08, U9 SQJA36EP-T1_GE3

Commit message: Gnd update
Other:
- note added: "TODO LIST: REVER GROUNDs -> Analog, Digital, Supply LDO AGND? , USB-C PD Split AGND?, Shields nos DC.DC? Power Ground, star connection? Power Multiplexer na USB-C Buffer a criar Vref nos sensores de corrente Meter isto mais apresentavel Atualizar Pinout"
- note removed: "TODO LIST: Power Multiplexer na USB-C Buffer a criar Vref nos sensores de corrente Meter isto mais apresentavel Atualizar Pinout"
Changed lines of the file:
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@@
 		)
 	)
-	(text "TODO LIST:\n\nPower Multiplexer na USB-C\nBuffer a criar Vref nos sensores de corrente\nMeter isto  mais apresentavel \nAtualizar Pinout"
+	(text "TODO LIST:\n\nREVER GROUNDs -> Analog, Digital, Supply\nLDO AGND? , USB-C PD Split AGND?, Shields nos DC.DC?\nPower Ground, star connection?\n\nPower Multiplexer na USB-C\nBuffer a criar Vref nos sensores de corrente\nMeter isto  mais apresentavel \nAtualizar Pinout"
 		(exclude_from_sim no)
-		(at 115.316 193.04 0)
+		(at 111.125 213.995 0)
 		(effects
 			(font
