File: Boards/Rocket Systems/TVCS/Sensor Unit.kicad_sch (KiCad schematic)
At the start: 79 parts, among them IC5 INA2181A4IDSQR, IC6 PCA9306GM,125, IC7 INA181A4QDCKRQ1, U1 MAX31856MUD+T, U10 STLM20DD9F, U11 MAX31856MUD+T, U15 AD8040ARUZ, U16 AD8040ARUZ, U3 MAX31856MUD+T, U8 max11614eee+

Commit message: TVCS fixes and required additions
Connections:
- net 2~{DRDY} THERMO: now also U11.7 (~{DRDY}); no longer U3.7 (~{DRDY})
- net 2~{FAULT} THERMO: now also U11.13 (~{FAULT}); no longer U3.13 (~{FAULT})
- net 3~{DRDY} THERMO: now also U3.7 (~{DRDY}); no longer U11.7 (~{DRDY})
- net 3~{FAULT} THERMO: now also U3.13 (~{FAULT}); no longer U11.13 (~{FAULT})
- net THERMO2 DN: now also R11.2, U11.2 (BIAS); no longer R5.2, U3.2 (BIAS)
- net THERMO2 DP: now also R10.2; no longer R4.2
- net THERMO3 DN: now also R4.2; no longer R11.2, U11.2 (BIAS)
- net THERMO3 DP: now also R5.2, U3.2 (BIAS); no longer R10.2
- net ~{CS} THERMO2 SPI: now also U11.9 (~{CS}); no longer U3.9 (~{CS})
- net ~{CS} THERMO3 SPI: now also U3.9 (~{CS}); no longer U11.9 (~{CS})
Other:
- note removed: "FALTA METER PINOS NOS TERMOCOUPLES"
- moved on the sheet: C1, C11, C12, C2, C27, C3, C31, C32, C35, C4, C41, C43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

Commit message: small pinout update
Connections:
- net 12V_Sense: now also R63.1; no longer R70.1
- net 5V_Sense: now also R70.1; no longer R63.1
- net LoadCell2 Sense: now also R77.1; no longer R76.1
- net LoadCell3 Sense: now also R76.1; no longer R77.1
Other:
- moved on the sheet: C45, C46, C47, C48, C49, C50, C51, C52, C53, C54, C55, C56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

Commit message: Gnd update
Parts:
- removed C43: 100n, Capacitor-0402:Capacitor_0402, symbol Device:C_Small
- added C67: 4.7u, Capacitor-1206:Capacitor_1206, symbol Device:C_Small
Connections:
- net +5V: now also C67.1
- net GND: no longer C27.2, C36.2, C38.2, C44.2, C45.2, C46.2, C47.1, C48.2, C51.2, C53.2, C55.2, C60.2, C61.2, C62.2, C63.2, C64.1, C65.2, C66.2, IC5.11 (GND_2), IC5.4 (GND_1), IC5.5 (REF1), IC5.6 (REF2), IC7.1 (REF), IC7.2 (GND), U1.1 (AGND), U10.3 (GND), U11.1 (AGND), U15.11 (-VS), U16.11 (-VS), U3.1 (AGND), U8.15 (GND)
- new net GNDA: C27.2, C36.2, C38.2, C44.2, C45.2, C46.2, C47.1, C48.2, C51.2, C53.2, C55.2, C60.2, C61.2, C62.2, C63.2, C64.1, C65.2, C66.2, C67.2, IC5.11 (GND_2), IC5.4 (GND_1), IC5.5 (REF1), IC5.6 (REF2), IC7.1 (REF), IC7.2 (GND), U1.1 (AGND), U10.3 (GND), U11.1 (AGND), U15.11 (-VS), U16.11 (-VS), U3.1 (AGND), U8.15 (GND)
Other:
- moved on the sheet: C44
