File: Boards/Rocket Systems/TVCS/_autosave-TVCS.kicad_sch (KiCad schematic)
At the start: 63 parts, among them IC1 BC846BLT1G, IC2 NSVT30010MXV6T1G, J1 Conn_01x01_Socket, J11 Conn_01x01_Socket, J12 Conn_01x01_Socket, J13 Conn_01x01_Socket, J14 Conn_01x01_Socket, J15 Conn_01x01_Socket, J16 Conn_01x01_Socket, J17 Conn_01x01_Socket, J18 Conn_01x01_Socket, J2 Conn_01x01_Socket, J3 Conn_01x01_Socket, J4 Conn_01x01_Socket, J5 Conn_01x01_Socket, J6 Conn_01x01_Socket, J8 Conn_01x01_Socket, J9 Conn_01x01_Socket, Q2 2N7002H6327XTSA2, Q3 2N7002H6327XTSA2, Q5 BC857CMB_315, Q6 BC857CMB_315, Q7 BC857CMB_315, SW1 D2F-01-D, U12 THVD2410VDRCR, U18 SC0915, U5 SQJA36EP-T1_GE3, U6 VLMKG3400-GS08, U9 SQJA36EP-T1_GE3

Commit message: Design da Hydra Breakout (Part 1)
Inclui algumas adições à biblioteca.
Parts:
- removed U18: SC0915, SC0915 (RP2040):MODULE_SC0915, symbol SC0915:SC0915
Other:
- sheet Power Unit ports: added GNDPWR; removed none
- moved on the sheet: C42, CR2, CR3, CR4, D4, IC1, IC2, J1, J11, J12, J13, J14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
