File: Boards/Rocket Systems/R COMMS/R COMMS.kicad_pcb (KiCad board)
At the start: 4 copper layers, 100 x 35 mm, 112 parts, among them IC1 BC846BLT1G, IC2 NSVT30010MXV6T1G, IC3 THVD2412VDR, J1 BM03B-SRSS-TBLFSN, J2 22285061, J3 DX07S016JA1R1500, J4 MEM2061-01-188-00-A_REVA, J5 5023520600, J6 SMARA_CONNECTOR, U1 W25Q128JVSIQ TR, U10 IP4220CZ6, U2 IP4220CZ6, U3 SX1280IMLTRT, U4 NRF21540-QDAA-R, U5 ST1L05APU33R, U6 IP4220CZ6, U7 IP4220CZ6, U8 STLM20DD9F, U9 VLMKG3400-GS08

Commit message: OBC a Navigator Updates
Parts:
- removed C40: 4.7u, Capacitor-0402:Capacitor_0402
- removed C41, C42, CV10, CV11, CV12, CV14, CV18, CV2, CV4, CV5, CV7, CV8, CV9: 100nF, Capacitor-0402:Capacitor_0402
- removed CR3: VLMY1300-GS08, LED-Yellow_VLMY1300-GS08:LEDC1608X100N
- removed CV1, CV13, CV17, CV3, CV6: 1uF, Capacitor-0402:Capacitor_0402
- removed CV15, CV16: 4.7uF, Capacitor-0402:Capacitor_0402
- removed IC3: THVD2412VDR, THVD2412VDR:SOIC127P600X175-14N
- removed R23, R30: 10k, Resistor-0402:RES_0402
- removed R24, R25: 120, Resistor-0402:RES_0402
- removed R26, R27, R28, R29: 523, Resistor-0402:RES_0402
- removed U10: IP4220CZ6, IP4220CZ6:SOT457_NEX
- removed U8: STLM20DD9F, STLM20DD9F:UDFN-4L_STM
- removed U9: VLMKG3400-GS08, VLMKG3400-GS08:SMT_00-GS08_VIS
- added C10: 1.2pF, Capacitor-0402:Capacitor_0402, F.Cu at (46.1, 68.4)
- added C11: 10u, Capacitor-0805:Capacitor_0805, F.Cu at (53.4, 66.6)
- added C12: 0.5pF, Capacitor-0402:Capacitor_0402, F.Cu at (46.1, 70.5)
- added C13: 1.2pF, Capacitor-0402:Capacitor_0402, F.Cu at (46.1, 72.7)
- added C14: 1p, Capacitor-0402:Capacitor_0402, F.Cu at (46.1, 74.9)
- added C15: 100n, Capacitor-0402:Capacitor_0402, F.Cu at (46.1, 77.0)
- added C16: 100n, Capacitor-0402:Capacitor_0402, F.Cu at (49.5, 66.2)
- added C17: 100n, Capacitor-0402:Capacitor_0402, F.Cu at (49.5, 68.4)
- added C18: 0.9p, Capacitor-0402:Capacitor_0402, F.Cu at (49.5, 70.5)
- added C3: 4.7u, Capacitor-0402:Capacitor_0402, F.Cu at (42.7, 66.2)
- added C4: 100nF, Capacitor-0402:Capacitor_0402, F.Cu at (42.7, 68.4)
- added C5: 4.7u, Capacitor-0402:Capacitor_0402, F.Cu at (42.7, 70.5)
- added C6: 470nF, Capacitor-0402:Capacitor_0402, F.Cu at (42.7, 72.7)
- added C7: 0.8pF, Capacitor-0402:Capacitor_0402, F.Cu at (42.7, 74.9)
- added C8: 100nF, Capacitor-0402:Capacitor_0402, F.Cu at (42.7, 77.0)
- added C9: 100nF, Capacitor-0402:Capacitor_0402, F.Cu at (46.1, 66.2)
- added CR1: VLMY1300-GS08, LED-Yellow_VLMY1300-GS08:LEDC1608X100N, F.Cu at (53.4, 69.7)
- added D2: SP3004-04XTG, TVS-SP3004:SOT563_LTF, F.Cu at (53.5, 72.8)
- added D3: SP3004-04XTG, TVS-SP3004:SOT563_LTF, F.Cu at (218.6, 48.2)
- added D4: RSX301L-30DDTE25, Diode-Schottky_RSX301L:DIOM5026X220N, F.Cu at (223.0, 59.1)
- added R12: 150, Resistor-0402:RES_0402, F.Cu at (42.8, 79.2)
- added R14: 27, Resistor-0402:RES_0402, F.Cu at (46.1, 50.1)
- added R20: 5k1, Resistor-0402:RES_0402, F.Cu at (46.1, 52.2)
- added SW1: D2F-01-D, Switch D2F-01:D2F-01-D_OMR, F.Cu at (219.4, 42.8)
- C1: value 10u -> 10nF; footprint Capacitor-0805:Capacitor_0805 -> Capacitor-0402:Capacitor_0402; moved to F.Cu
- C19: value 10nF -> 100n
- C2: value 100nF -> 10nF
- C20: value 10nF -> 0.3p
- C21: value 100nF -> 1uF
- C22: value 470nF -> 100nF
- C23: value 0.8pF -> 1uF
- C25, C27: value 1.2pF -> 100nF
- C26: value 0.5pF -> 1uF
- C28: value 1p -> 100nF
- C29: value 4.7u -> 100nF
- C30, C31, C39: moved to F.Cu
- C32: value 100n -> 100nF
- C33: value 100n -> 1uF
- C34: value 0.9p -> 100nF
- C35: value 0.3p -> 4.7uF
- C37: value 100nF -> 4.7uF; moved to F.Cu
- C38: value 100nF -> 1uF; moved to F.Cu
- D1: value RSX301L-30DDTE25 -> SP3004-04XTG; footprint Diode-Schottky_RSX301L:DIOM5026X220N -> TVS-SP3004:SOT563_LTF
- IC1: value BC846BLT1G -> NSVT30010MXV6T1G; footprint BJT NPN:SOT96P237X111-3N -> 2 PNP:SOT-563_1P3X1P7_ONS
- IC2: value NSVT30010MXV6T1G -> BC846BLT1G; footprint 2 PNP:SOT-563_1P3X1P7_ONS -> BJT NPN:SOT96P237X111-3N
- J1: value BM03B-SRSS-TBLFSN -> 22285061; footprint SWD_Con:CONN_BM03B-SRSS-TBLFSN_JST -> CONN Male Header:CONN_SD-42375-001_M320_06_MOL
- J2: value 22285061 -> 5023520200; footprint CONN Male Header:CONN_SD-42375-001_M320_06_MOL -> Molex 2 Conn:CONN02_502352_MOL; moved to F.Cu
- J3: value DX07S016JA1R1500 -> MEM2061-01-188-00-A_REVA; footprint USBC-DX07S016JA1:JAE_DX07S016JA1R1500 -> SD-CARD_MEM2061-01-188-00-A:GCT_MEM2061-01-188-00-A_REVA
- J4: value MEM2061-01-188-00-A_REVA -> SMARA_CONNECTOR; footprint SD-CARD_MEM2061-01-188-00-A:GCT_MEM2061-01-188-00-A_REVA -> Side Angle SMA:SMARACONNECTOR
- J5: value 5023520600 -> BM03B-SRSS-TBLFSN; footprint 5023520600:CONN06_502352_MOL -> SWD_Con:CONN_BM03B-SRSS-TBLFSN_JST
- J6: value SMARA_CONNECTOR -> DX07S016JA1R1500; footprint Side Angle SMA:SMARACONNECTOR -> USBC-DX07S016JA1:JAE_DX07S016JA1R1500
- JP1, JP2, JP3: value Jumper_2_Bridged -> Jumper_2_Open; moved to F.Cu
- R10: value 65 -> 523
- R11: value 150 -> 65
- R15: value 100 -> 27
- R16, R17: value 1k -> 100
- R19: value 5k1 -> 10k
- R2, R3: value 27 -> 10k
- R21: value 10k -> 5k1; moved to F.Cu
- R22: value 10k -> 1k; moved to F.Cu
- R7: value 10k -> 1k
- R8: value 100 -> 523
- R9: value 5k1 -> 120; footprint Resistor-0402:RES_0402 -> Resistor-0603:RES_0603
- U1: value W25Q128JVSIQ TR -> SX1280IMLTRT; footprint NOR Flash:SOIC_208MIL_WIN -> SX1280:QFN24_4X4_SEM
- U2: value IP4220CZ6 -> STLM20DD9F; footprint IP4220CZ6:SOT457_NEX -> STLM20DD9F:UDFN-4L_STM
- U3: value SX1280IMLTRT -> NRF21540-QDAA-R; footprint SX1280:QFN24_4X4_SEM -> RF FEM:QFN16_4X4_NOR
- U4: value NRF21540-QDAA-R -> THVD2410VDRCR; footprint RF FEM:QFN16_4X4_NOR -> THVD2410VDRCR:VSON10_DRC_TEX
- U5: value ST1L05APU33R -> VLMKG3400-GS08; footprint LDO ST1L05A:DFN_5APU33R_STM -> VLMKG3400-GS08:SMT_00-GS08_VIS
- U6: value IP4220CZ6 -> W25Q128JVSIQ TR; footprint IP4220CZ6:SOT457_NEX -> NOR Flash:SOIC_208MIL_WIN; moved to F.Cu
- U7: value IP4220CZ6 -> ST1L05APU33R; footprint IP4220CZ6:SOT457_NEX -> LDO ST1L05A:DFN_5APU33R_STM
- XTAL1: value ASE-12.000MHZ-LC-T -> NX2016SA-52MHZ-EXS00A-CS07103; footprint AS12MHz:ASE24576MHZLCT -> NX2016SA_52MHZ:OSCCC200X160X50N
- XTAL2: value NX2016SA-52MHZ-EXS00A-CS07103 -> ASE-12.000MHZ-LC-T; footprint NX2016SA_52MHZ:OSCCC200X160X50N -> AS12MHz:ASE24576MHZLCT
- moved J4 172.3 mm to (1.93, 39.8)
- moved C2 137.5 mm to (267.7, 79.2)
- moved J1 137.5 mm to (263.6, 88.0)
- moved R13 137.5 mm to (261.4, 60.5)
- moved R19 137.5 mm to (273.8, 63.9)
- moved R3 137.5 mm to (271.1, 71.0)
- moved R4 137.5 mm to (259.3, 86.6)
- moved R5 137.5 mm to (262.0, 84.8)
- moved R6 137.5 mm to (267.9, 86.6)
- moved R7 137.5 mm to (251.7, 84.8)
- moved R9 137.5 mm to (273.8, 65.1)
- moved MCU1 137.5 mm to (261.1, 75.0)
- moved R1 137.5 mm to (269.8, 86.0)
- moved R2 137.5 mm to (271.1, 69.8)
- moved XTAL1 137.5 mm to (254.1, 82.4)
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Connections:
- C1 pad 1: +3.3V -> Net-(U1-VR_PA)
- C19 pad 1: Net-(U3-VR_PA) -> +5V
- C2 pad 1: +3.3V -> Net-(U1-DCC_FB)
- C20 pad 1: Net-(U3-DCC_FB) -> Net-(C18-Pad1)
- C21 pad 1: +3.3V -> Net-(MCU1-RUN)
- C22 pad 1: Net-(U3-DCC_FB) -> GND
- C22 pad 2: GND -> Net-(MCU1-VREG_VOUT)
- C23 pad 1: Net-(U3-RFIO) -> Net-(MCU1-VREG_VOUT)
- C24 pad 1: +3.3V -> GND
- C24 pad 2: GND -> Net-(MCU1-VREG_VOUT)
- C25 pad 1: Net-(C25-Pad1) -> +3.3V
- C26 pad 1: Net-(C26-Pad1) -> +3.3V
- C26 pad 2: Net-(C25-Pad1) -> GND
- C27 pad 1: Net-(C26-Pad1) -> +3.3V
- C28 pad 1: Net-(C26-Pad1) -> +3.3V
- C28 pad 2: Net-(U4-TRX) -> GND
- C29 pad 1: GND -> +3.3V
- C29 pad 2: +5V -> GND
- C31 pad 1: GND -> +3.3V
- C31 pad 2: +5V -> GND
- C34 pad 1: Net-(C34-Pad1) -> +3.3V
- C35 pad 1: Net-(C34-Pad1) -> GND
- C35 pad 2: GND -> +5V
- C37 pad 1: +3.3V -> GND
- C37 pad 2: GND -> +3.3V
- C39 pad 1: +5V -> +3.3V
- CR2 pad 2: +3.3V -> +5V
- D1 pad 1: +5V -> /Nav RX UART
- D1 pad 2: VBUS -> GND
- IC1 pad 1: Net-(IC1-B) -> Net-(IC1-E2)
- IC1 pad 2: GND -> /Green Status
- IC1 pad 3: Net-(IC1-C) -> GND
- IC2 pad 1: Net-(IC2-E2) -> Net-(IC2-B)
- IC2 pad 2: /Status1 Green -> GND
- IC2 pad 3: GND -> Net-(IC2-C)
- J1 pad 1: Net-(J1-Pad1) -> +5V
- J1 pad 3: Net-(J1-Pad3) -> /Nav RX UART
- J1 pad 4: (no net) -> /Nav TX UART
- J1 pad 5: (no net) -> /Nav RTS UART
- J2 pad 1: +5V -> /RS_DN
- J2 pad 2: GND -> /RS_DP
- J2 pad 3: /OBC UART TX -> (no net)
- J2 pad 4: /OBC UART RX -> (no net)
- J3 pad 1: GND -> unconnected-(J3-DAT2-Pad1)
- J3 pad 10: unconnected-(J3-SBU1-Pad10) -> GND
- J3 pad 11: VBUS -> GND
- J3 pad 2: VBUS -> /SD-Card  ~{CS} SPI
- J3 pad 3: Net-(J3-CC1) -> /SD-Card MOSI SPI
- J3 pad 4: unconnected-(J3-SBU2-Pad4) -> +3.3V
- J3 pad 5: /RP2040/USB_DN -> /SD-Card SCK SPI
- J3 pad 6: /RP2040/USB_DP -> GND
- J3 pad 7: /RP2040/USB_DP -> /SD-Card MISO SPI
- J3 pad 8: /RP2040/USB_DN -> unconnected-(J3-DAT1-Pad8)
- J3 pad 9: Net-(J3-CC2) -> GND
- J4 pad 1: unconnected-(J4-DAT2-Pad1) -> Net-(C18-Pad1)
- J4 pad 2: /SD-Card SPI ~{CS} -> GND
- J4 pad 3: /SD-Card SPI MOSI -> GND
- J4 pad 4: +3.3V -> GND
- J4 pad 5: /SD-Card SPI SCK -> GND
- J5 pad 1: /Pyro Main Chute -> /RP2040/CLK SWD
- J5 pad 2: /Pyro Drogue -> GND
- J5 pad 3: /RS-TX_DP -> /RP2040/SWD
- J5 pad 4: /RS-TX_DN -> (no net)
- J5 pad 5: /RS-RX_DN -> (no net)
- J6 pad 1: Net-(C34-Pad1) -> GND
- J6 pad 2: GND -> VBUS
- J6 pad 3: GND -> Net-(J6-CC1)
- J6 pad 4: GND -> unconnected-(J6-SBU2-Pad4)
- J6 pad 5: GND -> /RP2040/USB_DN
- L1 pad 1: Net-(U3-DCC_FB) -> Net-(U1-DCC_FB)
- L1 pad 2: Net-(U3-DCC_SW) -> Net-(U1-DCC_SW)
- L2 pad 1: Net-(U3-RFIO) -> Net-(U1-RFIO)
- L2 pad 2: Net-(C25-Pad1) -> Net-(C10-Pad1)
- L3 pad 1: Net-(C25-Pad1) -> Net-(C10-Pad1)
- L3 pad 2: Net-(C26-Pad1) -> Net-(C12-Pad1)
- L4 pad 1: Net-(U4-ANT1) -> Net-(U3-ANT1)
- L4 pad 2: Net-(C34-Pad1) -> Net-(C18-Pad1)
- LS1 pad N: Net-(IC1-C) -> Net-(IC2-C)
- MCU1 pad 11: /RADIO SPI MISO -> /RADIO SCK SPI
- MCU1 pad 12: /NRF21540 SPI ~{CS} -> /NRF21540 ~{CS} SPI
- MCU1 pad 13: /RADIO SPI SCK -> /RADIO MOSI SPI
- MCU1 pad 14: /RADIO SPI MOSI -> /RADIO MISO SPI
- MCU1 pad 15: /NRF21540 MODE -> /MODE NRF21540
- MCU1 pad 16: /SX1280 SPI ~{CS} -> /SX1280 ~{CS} SPI
- MCU1 pad 17: /NRF21540 RX_EN -> /RX_EN NRF21540
- MCU1 pad 18: /NRF21540 TX_EN -> /TX_EN NRF21540
- MCU1 pad 2: /OBC UART RX -> /Nav RX UART
- MCU1 pad 27: /SD-Card SPI MISO -> /SD-Card MISO SPI
- MCU1 pad 28: /SD-Card SPI ~{CS} -> /SD-Card  ~{CS} SPI
- MCU1 pad 29: /SD-Card SPI SCK -> /SD-Card SCK SPI
- MCU1 pad 3: /OBC UART TX -> /Nav TX UART
- MCU1 pad 30: /SD-Card SPI MOSI -> /SD-Card MOSI SPI
- MCU1 pad 31: /SX1280 BUSY -> /BUSY SX1280
- MCU1 pad 32: /SX1280 DIO1 -> /DIO1 SX1280
- MCU1 pad 34: /SX1280 DIO2 -> /DIO2 SX1280
- MCU1 pad 35: /SX1280 DIO3 -> /DIO3 SX1280
- MCU1 pad 36: /SX1280 ~{RST} -> /~{RST} SX1280
- MCU1 pad 37: /Status1 Green -> /Buzzer
- MCU1 pad 38: /Status1 Red -> /Temp_Sense
- MCU1 pad 39: /Temp_Sense -> /Green Status
- MCU1 pad 4: /OBC UART RTS -> /Nav RTS UART
- MCU1 pad 40: /Pyro Main Chute -> /Red Status
- MCU1 pad 41: /Pyro Drogue -> /RP2040/GPIO29
- MCU1 pad 5: /OBC UART CTS -> /Nav CTS UART
- MCU1 pad 51: /RP2040/MCU QSPI_SD3 -> /RP2040/MCU SD3 SPI
- MCU1 pad 52: /RP2040/MCU QSPI_SCLK -> /RP2040/MCU SCLK SPI
- MCU1 pad 53: /RP2040/MCU QSPI_SD0 -> /RP2040/MCU SD0 SPI
- MCU1 pad 54: /RP2040/MCU QSPI_SD2 -> /RP2040/MCU SD2 SPI
- MCU1 pad 55: /RP2040/MCU QSPI_SD1 -> /RP2040/MCU SD1 SPI
- MCU1 pad 56: /RP2040/MCU QSPI_SS -> /RP2040/MCU ~{CS} SPI
- MCU1 pad 6: /RS_TX -> /WRITE_RS
- MCU1 pad 7: /RS_RX -> /READ_RS
- MCU1 pad 8: /Buzzer -> /ENABLE_RS
- MCU1 pad 9: /NRF21540 ~{PDN} -> /~{PDN} NRF21540
- R1 pad 1: +3.3V -> Net-(JP1-B)
- R1 pad 2: Net-(MCU1-RUN) -> /~{RST} SX1280
- R10 pad 1: GND -> /RS_DP
- R10 pad 2: Net-(CR2-Pad1) -> GND
- R13 pad 1: /RP2040/~{USB_BOOT} -> +3.3V
- R13 pad 2: /RP2040/MCU QSPI_SS -> Net-(MCU1-RUN)
- R15 pad 1: Net-(IC2-E1) -> /RP2040/USB_DN
- R15 pad 2: Net-(U9-A_Red) -> /RP2040/USB_D-
- R16 pad 1: Net-(JP1-B) -> /RP2040/CLK SWD
- R16 pad 2: /SX1280 ~{RST} -> Net-(MCU1-SWCLK)
- R17 pad 1: Net-(IC1-B) -> /RP2040/SWD
- R17 pad 2: /Buzzer -> Net-(MCU1-SWD)
- R18 pad 1: +5V -> /RP2040/~{RST}
- R18 pad 2: Net-(IC1-C) -> Net-(MCU1-RUN)
- R19 pad 1: Net-(J3-CC2) -> Net-(XTAL2-TRI-STATE(STBY))
- R19 pad 2: GND -> +3.3V
- R2 pad 1: /RP2040/USB_DP -> +3.3V
- R2 pad 2: /RP2040/USB_D+ -> /READ_RS
- R21 pad 1: +3.3V -> Net-(J6-CC2)
- R21 pad 2: /RS_RX -> GND
- R22 pad 1: Net-(IC3-SLR) -> /RP2040/~{USB_BOOT}
- R22 pad 2: GND -> /RP2040/MCU ~{CS} SPI
- R3 pad 1: /RP2040/USB_DN -> /ENABLE_RS
- R3 pad 2: /RP2040/USB_D- -> GND
- R4 pad 1: Net-(J1-Pad1) -> Net-(U5-A_Green)
- R4 pad 2: Net-(MCU1-SWCLK) -> Net-(IC1-E2)
- R5 pad 1: Net-(J1-Pad3) -> Net-(IC1-E1)
- R5 pad 2: Net-(MCU1-SWD) -> Net-(U5-A_Red)
- R6 pad 1: /RP2040/~{RST} -> Net-(IC2-B)
- R6 pad 2: Net-(MCU1-RUN) -> /Buzzer
- R7 pad 1: Net-(XTAL1-TRI-STATE(STBY)) -> +5V
- R7 pad 2: +3.3V -> Net-(IC2-C)
- R8 pad 1: Net-(U9-A_Green) -> +5V
- R8 pad 2: Net-(IC2-E2) -> /RS_DN
- R9 pad 1: GND -> /RS_DN
- R9 pad 2: Net-(J3-CC1) -> /RS_DP
- U1 pad 1: /RP2040/MCU QSPI_SS -> Net-(U1-VR_PA)
- U1 pad 2: /RP2040/MCU QSPI_SD1 -> Net-(U1-DCC_FB)
- U1 pad 3: /RP2040/MCU QSPI_SD2 -> /~{RST} SX1280
- U1 pad 4: GND -> /SX1280 XTA -
- U1 pad 5: /RP2040/MCU QSPI_SD0 -> GND
- U1 pad 6: /RP2040/MCU QSPI_SCLK -> /SX1280 XTB +
- U1 pad 7: /RP2040/MCU QSPI_SD3 -> /BUSY SX1280
- U1 pad 8: +3.3V -> /DIO1 SX1280
- U2 pad 1: /RP2040/USB_DP -> /Temp_Sense
- U2 pad 2: GND -> unconnected-(U2-NC-Pad2)
- U2 pad 3: /RP2040/USB_DN -> GND
- U2 pad 4: /RP2040/USB_DN -> +3.3V
- U3 pad 1: Net-(U3-VR_PA) -> GND
- U3 pad 10: /SX1280 DIO3 -> Net-(U3-TRX)
- U3 pad 11: +3.3V -> /~{PDN} NRF21540
- U3 pad 12: Net-(U3-DCC_FB) -> /RADIO SCK SPI
- U3 pad 13: GND -> /RADIO MOSI SPI
- U3 pad 14: Net-(U3-DCC_SW) -> /RADIO MISO SPI
- U3 pad 15: +3.3V -> /NRF21540 ~{CS} SPI
- U3 pad 16: /RADIO SPI MISO -> GND
- U3 pad 17: /RADIO SPI MOSI -> GND
- U3 pad 2: Net-(U3-DCC_FB) -> Net-(U3-ANT1)
- U3 pad 3: /SX1280 ~{RST} -> unconnected-(U3-ANT2-Pad3)
- U3 pad 4: /SX1280 XTA -> /MODE NRF21540
- U3 pad 5: GND -> +3.3V
- U3 pad 6: /SX1280 XTB -> +3.3V
- U3 pad 7: /SX1280 BUSY -> /RX_EN NRF21540
- U3 pad 8: /SX1280 DIO1 -> GND
- U3 pad 9: /SX1280 DIO2 -> /TX_EN NRF21540
- U4 pad 1: GND -> +3.3V
- U4 pad 10: Net-(U4-TRX) -> +5V
- U4 pad 11: /NRF21540 ~{PDN} -> GND
- U4 pad 2: Net-(U4-ANT1) -> /READ_RS
- U4 pad 3: unconnected-(U4-ANT2-Pad3) -> /ENABLE_RS
- U4 pad 4: /NRF21540 MODE -> /ENABLE_RS
- U4 pad 5: +3.3V -> /WRITE_RS
- U4 pad 6: +3.3V -> GND
- U4 pad 7: /NRF21540 RX_EN -> Net-(U4-SLR)
- U4 pad 8: GND -> /RS_DP
- U4 pad 9: /NRF21540 TX_EN -> /RS_DN
- U5 pad 1: unconnected-(U5-NC-Pad1) -> +5V
- U5 pad 2: +3.3V -> Net-(U5-A_Green)
- U5 pad 4: unconnected-(U5-NC-Pad4) -> Net-(U5-A_Red)
- U6 pad 1: /RS-TX_DN -> /RP2040/MCU ~{CS} SPI
- U6 pad 2: GND -> /RP2040/MCU SD1 SPI
- U6 pad 3: /RS-TX_DP -> /RP2040/MCU SD2 SPI
- U6 pad 4: /RS-RX_DN -> GND
- U6 pad 5: +5V -> /RP2040/MCU SD0 SPI
- U6 pad 6: /RS-RX_DP -> /RP2040/MCU SCLK SPI
- U7 pad 1: /OBC UART TX -> unconnected-(U7-NC-Pad1)
- U7 pad 2: GND -> +3.3V
- U7 pad 3: /OBC UART RX -> +5V
- U7 pad 4: /OBC UART RTS -> unconnected-(U7-NC-Pad4)
- U7 pad 5: +3.3V -> unconnected-(U7-NC-Pad5)
- U7 pad 6: /OBC UART CTS -> GND
- XTAL1 pad 1: Net-(XTAL1-TRI-STATE(STBY)) -> /SX1280 XTB +
- XTAL1 pad 3: /RP2040/Crystal -> /SX1280 XTA -
- XTAL1 pad 4: +3.3V -> GND
- XTAL2 pad 1: /SX1280 XTB -> Net-(XTAL2-TRI-STATE(STBY))
- XTAL2 pad 3: /SX1280 XTA -> /RP2040/Crystal
- XTAL2 pad 4: GND -> +3.3V
Routing:
- net /Nav CTS UART: track 0.00 -> 24.2 mm
- net /Nav TX UART: track 0.00 -> 20.7 mm
- net +3.3V: track 0.26 -> 20.3 mm
- net /OBC UART CTS: track 19.9 -> 0.00 mm
- net /OBC UART TX: track 18.8 -> 0.00 mm
- net /ENABLE_RS: track 0.00 -> 17.7 mm
- net /RP2040/USB_DN: track 17.7 -> 2.15 mm
- net /RP2040/USB_DP: track 15.0 -> 0.00 mm
- net /OBC UART RX: track 14.6 -> 0.00 mm
- net /Nav RX UART: track 0.00 -> 11.5 mm
- net /RADIO SCK SPI: track 0.00 -> 5.41 mm
- net (no net): track 0.18 -> 5.50 mm
- net Net-(C26-Pad1): track 5.08 -> 0.00 mm
- net /OBC UART RTS: track 4.32 -> 0.00 mm
- net /~{RST} SX1280: track 0.00 -> 4.04 mm
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Other:
- board size 100 x 35 mm -> 0.9 x 0.6 mm
- board text added: "Power and Ground Planes - pesquisar como fazer grounds para RF Guard Rings e como fazer routing com eles Fazer routing 1- RF 2- Differential pairs + length tunning 3- Digital 4- Analógico Via Stitching Silk Screen Solder Mask"
- board text removed: "Fazer sinal de corrente para o Pyro Channel Rever placement de alguns condensadores -> Passar para B.Cu Stack up Criar Nets Power and Ground Planes - pesquisar como fazer grounds para RF Ver questão de Vias on pad Guard Rings e como fazer routing com eles Fazer routing 1- RF 2- Differential pairs + length tunning 3- Digital 4- Analógico Via Stitching Silk Screen Solder Mask"
