File: Boards/Rocket Systems/OBC/OBC.kicad_sch (KiCad schematic)
At the start: 91 parts, among them IC1 HDC3022QDEJRQ1, IC2 NSVT30010MXV6T1G, IC3 INA181A4QDCKRQ1, J1 22285061, J3 SMARA_CONNECTOR, SW1 D2F-01-D, U10 BMP581, U12 BMI323, U4 ASM330LHHTR, U5 CD-PA1616, U6 VLMKG3400-GS08, U7 LM61460AASQRJRRQ1, U8 LPS22DFTR, U9 LIS2MDLTR

Commit message: commit to fix merge (1)
Parts:
- removed C19, C_BT2, C_IN_HFI3, C_IN_HFI4: 100n, Capacitor-0402:Capacitor_0402, symbol Device:C_Small
- removed C20, C21, C22, C23: 2.2u, Capacitor-0402:Capacitor_0402, symbol Device:C_Small
- removed C24, C25: 470n, Capacitor-0402:Capacitor_0402, symbol Device:C_Small
- removed C_BIAS2, C_VCC2: 1u, Capacitor-0603:Capacitor_0603, symbol Device:C_Small
- removed C_FF2: 22p, Capacitor-0402:Capacitor_0402, symbol Device:C_Small
- removed C_IN-BLK2: 10u, Capacitor-4mm:Capacitor_4mm, symbol Device:C_Small
- removed C_IN3, C_IN4: 4.7u, Capacitor-1206:Capacitor_1206, symbol Device:C_Small
- removed C_LP1: 10n, Capacitor-0603:Capacitor_0603, symbol Device:C_Small
- removed C_OUT10: 560u, Capacitor-8mm:Capacitor_8mm, symbol Device:C_Small
- removed C_OUT6, C_OUT7, C_OUT8, C_OUT9: 22u, Capacitor-0805:Capacitor_0805, symbol Device:C_Small
- removed D4: RSX301L, Diode-Schottky_RSX301L:DIOM5026X220N, symbol RSX301L-30DDTE25:RSX301L-30DDTE25
- removed IC3: INA181A4QDCKRQ1, INA181A4QDCKRQ1:SOT65P210X110-6N, symbol INA181A4QDCKRQ1:INA181A4QDCKRQ1
- removed L1: 2.2u, Inductor-10.1x10:Inductor_10.1x10, symbol Device:L
- removed L_SW1: 15u, Inductor-10.1x10:Inductor_10.1x10, symbol Device:L
- removed R_BIAS2: 5, Resistor-0402:RES_0402, symbol Device:R
- removed R_BT2: 100, Resistor-0402:RES_0402, symbol Device:R
- removed R_ENB2: 45k3, Resistor-0402:RES_0402, symbol Device:R
- removed R_ENT2: 422k, Resistor-0402:RES_0402, symbol Device:R
- removed R_FBB2: 22k1, Resistor-0603:RES_0603, symbol Device:R
- removed R_FBB3: 120, Resistor-0603:RES_0603, symbol Device:R
- removed R_FBT2, R_PG1: 100K, Resistor-0603:RES_0603, symbol Device:R
- removed R_FF2, R_REF2: 1k, Resistor-0402:RES_0402, symbol Device:R
- removed R_LP1: 160, Resistor-0402:RES_0402, symbol Device:R
- removed R_REF1: 54k2, Resistor-0402:RES_0402, symbol Device:R
- removed R_RT2: 33k2, Resistor-0603:RES_0603, symbol Device:R
- removed Rsense1: 7.5m, Resistor-2512:RES_WSLP2512, symbol Device:R
- removed U7: LM61460AASQRJRRQ1, DCDC_LM61460:VQFN-HR14_RJR_TEX, symbol DCDC_LM61460:LM61460AASQRJRRQ1
Other:
- note removed: ">15V to 5V Converter"
- note removed: "C_IN-BLK3 and C_OUT15 are electrolytic polarized capacitors! All others are ceramic X7R capacitors with appropriate voltage ratings."
- note removed: "DC.DC2 VCC coloca PGOOD a 3.3V"
- note removed: "EMI Filter"
- note removed: "VBUS: 16V nominal when powered by battery VBUS: 15V nominal when powered through USB-C PD"
- note removed: "Voltage divider for 60mV to improve reading accuracies"
- note removed: "Vout is set to 5.5V to compensate Diode and Rsense drops The Schottky diode has a 420mV forward voltage drop."
- note removed: "differential routing"
- moved on the sheet: C27, CR3, CR4, IC1, IC2, R15, R16, R17, R18, R19, R20, R8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

Commit message: OBC layout update
Parts:
- removed J1: 22285061, CONN Male Header:CONN_SD-42375-001_M320_06_MOL, symbol PinCon_22285061:22285061
- added J1: 22022065, CONN Female Header:CONN_SA-4455_06_TE_MOL, symbol CONN_SA-4455_06_TE_MOL:22022065
- BT1: Description_1 Holder; SMT; Vibra-Fit; Cells 2025 & 2032; Tape & Reel | Keystone Electronics 1060TR -> Holder; SMT; Vibra-Fit; Cells 2025 & 2032; Tape & Reel | Keystone Electronics 1060TR
- CR3, CR4: footprint LED-Yellow_VLMY1300-GS08:LED_VISHAY_VLMX1300_VIS -> LED-Yellow_VLMY1300-GS08:LEDC1608X100N
- D2: Description_1 Rectifier Diode Schottky 1A Automotive 2-Pin SOD-123W T/R -> Rectifier Diode Schottky 1A Automotive 2-Pin SOD-123W T/R
- U10: footprint QFN10_BMP581_BOS -> BARO BMP581:QFN10_BMP581_BOS
- U8: footprint QFN_22DFTR_STM -> BARO LPS22DFTR:QFN_22DFTR_STM
Connections:
- net +5V: now also J1.6
- net Comms UART CTS: now also J1.2
- net Comms UART RTS: now also J1.3
- net Comms UART RX: now also J1.5
- net Comms UART TX: now also J1.4
- net GND: now also J1.1
- no-connect marks 4 -> 6
Other:
- moved on the sheet: BT1, C1, C11, C12, C13, C15, C16, C17, C18, C2, C27, C3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

Commit message: organizei umas coisas, condensadores e jumper pads
Parts:
- removed S3: TL1017AABF160QG, E-Switch_Small:TL1017AABF160QG, symbol TL1017AABF160QG:TL1017AABF160QG
- added JP3: Jumper_2_Bridged, Jumper:SolderJumper-2_P1.3mm_Open_RoundedPad1.0x1.5mm, symbol Jumper:Jumper_2_Bridged
Connections:
- net GND: now also JP3.1 (A)
- net at R10.1: now also JP3.2 (B)
Changed lines of the file:
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@@
 	)
 	(junction
-		(at 372.11 62.865)
-		(diameter 0)
-		(color 0 0 0 0)
-	)
-	(junction
 		(at 195.58 52.07)
 		(diameter 0)
@@
 	(wire
 		(pts
-			(xy 372.11 62.865) (xy 363.855 62.865)
-		)
-		(stroke
-			(width 0)
-			(type default)
-		)
-	)
-	(wire
-		(pts
 			(xy 121.92 59.69) (xy 143.51 59.69)
 		)
@@
 	(wire
 		(pts
-			(xy 379.73 59.055) (xy 380.365 59.055)
-		)
-		(stroke
-			(width 0)
-			(type default)
-		)
-	)
-	(wire
-		(pts
 			(xy 195.58 50.8) (xy 195.58 52.07)
 		)
@@
 	(wire
 		(pts
-			(xy 363.855 59.055) (xy 364.49 59.055)
+			(xy 363.855 59.055) (xy 367.03 59.055)
 		)
 		(stroke
@@
 	(wire
 		(pts
+			(xy 377.19 59.055) (xy 380.365 59.055)
+		)
+		(stroke
+			(width 0)
+			(type default)
+		)
+	)
+	(wire
+		(pts
 			(xy 81.915 239.395) (xy 81.915 242.57)
 		)
@@
 	(wire
 		(pts
-			(xy 377.19 62.865) (xy 372.11 62.865)
+			(xy 363.855 62.865) (xy 377.19 62.865)
 		)
 		(stroke
@@
 	)
 	(symbol
-		(lib_id "TL1017AABF160QG:TL1017AABF160QG")
-		(at 381 62.865 0)
-		(mirror y)
-		(unit 1)
-		(exclude_from_sim no)
-		(in_bom yes)
-		(on_board yes)
-		(dnp no)
-		(property "Reference" "S3"
-			(at 372.11 51.435 0)
-			(effects
-				(font
-					(size 1.27 1.27)
-				)
-			)
-		)
-		(property "Value" "TL1017AABF160QG"
-			(at 371.475 53.975 0)
-			(effects
-				(font
-					(size 1.27 1.27)
-				)
-			)
-		)
-		(property "Footprint" "E-Switch_Small:TL1017AABF160QG"
-			(at 359.41 157.785 0)
-			(effects
-				(font
-					(size 1.27 1.27)
-				)
-				(justify left top)
-				(hide yes)
-			)
-		)
-		(property "Datasheet" "https://configured-product-images.s3.amazonaws.com/2D/specs/TL1017AABF160QG.pdf"
-			(at 359.41 257.785 0)
-			(effects
-				(font
-					(size 1.27 1.27)
-				)
-				(justify left top)
-				(hide yes)
-			)
-		)
-		(property "Description" "TACT, Surface Mount"
-			(at 381 62.865 0)
-			(effects
-				(font
-					(size 1.27 1.27)
-				)
-				(hide yes)
-			)
-		)
-		(property "Height" "1.7"
-			(at 359.41 457.785 0)
-			(effects
-				(font
-					(size 1.27 1.27)
-				)
-				(justify left top)
-				(hide yes)
-			)
-		)
-		(property "Mouser Part Number" "612-TL1017AABF160QG"
-			(at 359.41 557.785 0)
-			(effects
-				(font
-					(size 1.27 1.27)
-				)
-				(justify left top)
-				(hide yes)
-			)
-		)
-		(property "Mouser Price/Stock" "https://www.mouser.co.uk/ProductDetail/E-Switch/TL1017AABF160QG?qs=9vOqFld9vZWEDSBQD0ZM5A%3D%3D"
-			(at 359.41 657.785 0)
-			(effects
-				(font
-					(size 1.27 1.27)
-				)
-				(justify left top)
-				(hide yes)
-			)
-		)
-		(property "Manufacturer_Name" "E-Switch"
-			(at 359.41 757.785 0)
-			(effects
-				(font
-					(size 1.27 1.27)
-				)
-				(justify left top)
-				(hide yes)
-			)
-		)
-		(property "Manufacturer_Part_Number" "TL1017AABF160QG"
-			(at 359.41 857.785 0)
-			(effects
-				(font
-					(size 1.27 1.27)
-				)
-				(justify left top)
-				(hide yes)
-			)
-		)
-		(pin "G1"
-		)
-		(pin "1"
-		)
-		(pin "2"
-		)
-		(instances
-			(project "OBC"
-				(path "/1ff41ee6-31ba-481b-ae3a-c725064eb5fe"
-					(reference "S3")
-					(unit 1)
-				)
-			)
-		)
-	)
-	(symbol
 		(lib_id "Device:R")
 		(at 36.195 184.785 0)
@@
 					(unit 1)
 				)
+			)
+		)
+	)
+	(symbol
+		(lib_id "Jumper:Jumper_2_Bridged")
+		(at 372.11 59.055 0)
+		(unit 1)
+		(exclude_from_sim yes)
+		(in_bom yes)
+		(on_board yes)
+		(dnp no)
+		(fields_autoplaced yes)
+		(property "Reference" "JP3"
+			(at 372.11 53.975 0)
+			(effects
+				(font
+					(size 1.27 1.27)
+				)
+			)
+		)
+		(property "Value" "Jumper_2_Bridged"
+			(at 372.11 56.515 0)
+			(effects
+				(font
+					(size 1.27 1.27)
+				)
+			)
+		)
+		(property "Footprint" "Jumper:SolderJumper-2_P1.3mm_Open_RoundedPad1.0x1.5mm"
+			(at 372.11 59.055 0)
+			(effects
+				(font
+					(size 1.27 1.27)
+				)
+				(hide yes)
+			)
+		)
+		(property "Datasheet" "~"
+			(at 372.11 59.055 0)
+			(effects
+				(font
+					(size 1.27 1.27)
+				)
+				(hide yes)
+			)
+		)
+		(property "Description" "Jumper, 2-pole, closed/bridged"
+			(at 372.11 59.055 0)
+			(effects
+				(font
+					(size 1.27 1.27)
+				)
+				(hide yes)
+			)
+		)
+		(pin "2"
+		)
+		(pin "1"
+		)
+		(instances
+			(project "OBC"
+				(path "/1ff41ee6-31ba-481b-ae3a-c725064eb5fe"
+					(reference "JP3")
+					(unit 1)
+				)

Commit message: Navigator update
Parts:
- removed BT1: 1060TR, BAT Holder 1060TR:BAT_1060TR, symbol 1060TR:1060TR
- removed C11, C12: 100nF, Capacitor-0402:Capacitor_0402, symbol Device:C_Small
- removed C14, C7, C8: 100nF, Capacitor-0402:Capacitor_0402, symbol Device:C
- removed C27: 100n, Capacitor-0402:Capacitor_0402, symbol Device:C_Small
- removed C4: 1uF, Capacitor-0402:Capacitor_0402, symbol Device:C
- removed CR2: VLMC3100-GS08, LED-Green_VLMC3100-GS08:LED_PLCC_VSMB, symbol GreenLED__VLMC3100-GS08:VLMC3100-GS08
- removed D2: PMEG2010ER, Diode-Schottky_PMEG2010ER:SODFL3517X110N, symbol PMEG2010ER:PMEG2010ER
- removed FB1: FerriteBead, Ferrite:Ferrite_0603, symbol Device:FerriteBead
- removed IC1: HDC3022QDEJRQ1, HDC3022QDEJRQ1:HDC3022QDEJRQ1, symbol HDC3022QDEJRQ1:HDC3022QDEJRQ1
- removed J1: 22022065, CONN Female Header:CONN_SA-4455_06_TE_MOL, symbol CONN_SA-4455_06_TE_MOL:22022065
- removed JP3: Jumper_2_Bridged, Jumper:SolderJumper-2_P1.3mm_Open_RoundedPad1.0x1.5mm, symbol Jumper:Jumper_2_Bridged
- removed R12, R20: 10k, Resistor-0402:RES_0402, symbol Device:R
- removed R24: 470, Resistor-0402:RES_0402, symbol Device:R
- removed SW1: D2F-01-D, Switch D2F-01:D2F-01-D_OMR, symbol Switch_D2F-01:D2F-01-D
- removed U10: BMP581, BARO BMP581:QFN10_BMP581_BOS, symbol BARO_BMP581:BMP581
- removed U4: ASM330LHHTR, IMU ASM330LHHTR:LGA-14L_2P5X3X0P83_STM, symbol IMU_ASM330LHHTR:ASM330LHHTR
- removed U5: CD-PA1616, GPS_adafruit:CD-PA1616D_ADA, symbol GPS_adafruit:5186
- removed U8: LPS22DFTR, BARO LPS22DFTR:QFN_22DFTR_STM, symbol BARO_LPS22DFTR:LPS22DFTR
- added BT1: BAT-HLD-012-SMT-TR, BAT_HLD_012:BAT_BAT-HLD-012-SMT-TR, symbol BAT-HLD-012-SMT-TR:BAT-HLD-012-SMT-TR
- added C11, C12: 100nF, Capacitor-0402:Capacitor_0402, symbol Device:C
- added C14, C4: 4.7u, Capacitor-0402:Capacitor_0402, symbol Device:C_Small
- added C21, C22, C23, C24: 100n, Capacitor-0402:Capacitor_0402, symbol Device:C_Small
- added C7: 1u, Capacitor-0402:Capacitor_0402, symbol Device:C_Small
- added C8: 100nF, Capacitor-0402:Capacitor_0402, symbol Device:C_Small
- added CR1: VLMC3100-GS08, LED-Green_VLMC3100-GS08:LED_PLCC_VSMB, symbol GreenLED__VLMC3100-GS08:VLMC3100-GS08
- added D2: SP3004-04XTG, TVS-SP3004:SOT563_LTF, symbol SP3004-04XTG:SP3004-04XTG
- added D3: PMEG2010ER, Diode-Schottky_PMEG2010ER:SODFL3517X110N, symbol PMEG2010ER:PMEG2010ER
- added FL1: FTCap0603, FTCap_0603:FTCap_0603, symbol FTCap0603:FTCap0603
- added H1, H2, H3, H4: MountingHole, MountingHole:MountingHole_3.2mm_M3_ISO7380_Pad_TopBottom, symbol Mechanical:MountingHole
- added HM1: BME280, BME280:BME280, symbol BME280:BME280
- added IC1: NEO-M8Q-0, NEO-M8Q-0:NEO-M8_UBL, symbol NEO-M8Q-0:NEO-M8Q-0
- added IC3: BC846BLT1G, BJT NPN:SOT96P237X111-3N, symbol BC846BLT1G:BC846BLT1G
- added J1: 22027063, 6 Female Conn:CONN6X1_22027063_MOL, symbol 022027063:22027063
- added J4: 5023520200, Molex 2 Conn:CONN02_502352_MOL, symbol DuraClick_2Conn:5023520200
- added JP6, JP8: Jumper_2_Open, Jumper:SolderJumper-2_P1.3mm_Open_RoundedPad1.0x1.5mm, symbol Jumper:Jumper_2_Open
- added L1: 27n, Inductor-0402:Inductor_0402, symbol Device:L
- added LS1: PKLCS1212E20A0-R1, PKLCS1212E20A0-R1:PKLCS1212E20A0-R1, symbol PKLCS1212E20A0-R1:PKLCS1212E20A0-R1
- added Q1: BC857CMB_315, PNP_BC857CMB_315:TRANS_PMZB550UNEYL, symbol BC857CMB_315:BC857CMB_315
- added R22, R30: 1k, Resistor-0402:RES_0402, symbol Device:R
- added R23, R28, R29: 2k, Resistor-0402:RES_0402, symbol Device:R
- added R4: 10, Resistor-0402:RES_0402, symbol Device:R
- added U4: LPS22DFTR, BARO LPS22DFTR:QFN_22DFTR_STM, symbol BARO_LPS22DFTR:LPS22DFTR
- added U7: BMP581, BARO BMP581:QFN10_BMP581_BOS, symbol BARO_BMP581:BMP581
- added U8: LSM6DSOTR, LSM6DSOTR:LGA-14L_2P5X3X0P86_STM, symbol LSM6DSOTR:LSM6DSOTR
- C15, C16: value 100nF -> 100n
- R11: value 470 -> 1k
- R17, R18: value 2k -> 5k1
- R25: value 470 -> 10k
Connections:
- net SCL I2C is gone; now on net +3.3V: R18.2
- net SDA I2C is gone; now on net +3.3V: R17.2
- net SPI1_MISO is gone; now on net MISO SPI: U9.7 (INT/DRDY/SDO)
- net SPI1_MOSI is gone; now on net MOSI SPI: U9.4 (SDA/SDI/SDO)
- net SPI1_SCK is gone; now on net SCK SPI: U9.1 (SCL/SPC)
- net +3.3V: now also R25.2, C11.2, C12.2, C21.2, C22.2, C23.2, C24.2, C8.1, HM1.6 (VDDIO), HM1.8 (VDD), IC1.23 (VCC), R28.1, R29.1, R30.1, U4.1 (Vdd_IO), U4.10 (VDD), U4.6 (CS), U7.1 (VDDIO), U7.10 (VDD), U8.5 (VDDIO), U8.8 (VDD); no longer C15.1, R17.1, R18.1
- net +5V: now also R11.1, C4.2, C7.2, CR1.2, D2.5 (VCC), J1.1, LS1.P
- net BAR2 RDY: now also U7.7 (INT)
- net GND: now also BT1.N, C11.1, C12.1, C14.2, C21.1, C22.1, C23.1, C24.1, C4.1, C7.1, C8.2, D2.2 (GND), FL1.2, FL1.4, HM1.1 (GND), HM1.7 (GND), IC1.10 (GND_1), IC1.12 (GND_2), IC1.13 (GND_3), IC1.24 (GND_4), IC1.7 (VDD_USB), IC3.2 (E), J1.2, JP8.2 (B), Q1.3, U4.3 (RES), U4.5 (SDO/SA0), U4.8 (GND_IO), U4.9 (GND), U7.3 (VSS), U7.5 (SDO), U7.8 (VSS), U7.9 (VSS), U8.1 (SDO/SA0), U8.2 (SDx), U8.3 (SCx), U8.6 (GND), U8.7 (GND)
- net GPS VBACKUP: now also C15.1, C14.1, D3.C, IC1.22 (V_BCKP)
- net at R11.2: now also IC3.3 (C), LS1.N
- net at R10.1: now also IC3.1 (B)
- net Buzzer: now reaches R10.2
- net RF: now reaches J3.1
- net RF: now also IC1.11 (RF_IN), L1.2
- net GPS RX renamed GPS ~{BOOT}
- net GPS ~{BOOT}: now also IC1.8 (RESET_N), JP8.1 (A)
- net IMU1 RDY1 renamed INT1 BOSH IMU
- net IMU1 RDY2 renamed INT2 BOSH IMU
- net IMU1 SPI0_~{CS} renamed IMU1 ~{CS} SPI
- net MAG SPI1_~{CS} renamed MAG ~{CS} SPI
- net SPI0_MISO renamed MISO SPI
- net MISO SPI: now also HM1.5 (SDO)
- net SPI0_MOSI renamed MOSI SPI
- net MOSI SPI: now also HM1.3 (SDI)
- net SPI0_SCK renamed SCK SPI
- net SCK SPI: now also HM1.4 (SCK)
- net Status Green renamed Green Status
- net Status Red renamed Red Status
- new net: CR1.1, R22.1, R23.1
- new net: Q1.2, R22.2, R23.2
- new net: D3.A, JP6.1 (A)
- new net: FL1.1, R4.2
- new net: FL1.3, L1.1
- new net: IC1.9 (VCC_RF), R4.1
- new net: R30.2, U8.12 (CS)
- new net BAR1 RDY: U4.7 (INT_DRDY)
- new net Droge ENABLE: J4.1
- new net GPS RX UART: IC1.21 (RXD/SPI_MOSI)
- new net GPS TX UART: IC1.20 (TXD/SPI_MISO)
- new net HUM ~{CS} SPI: HM1.2 (~{CS})
- new net INT GPS: IC1.4 (EXTINT)
- new net INT1 ST IMU: U8.4 (INT1)
- new net INT2 ST IMU: U8.9 (INT2)
- new net OBC CTS UART: D2.4 (IO3), J1.5
- new net OBC RTS UART: D2.6 (IO4), J1.6
- new net OBC RX UART: D2.3 (IO2), J1.4
- new net OBC TX UART: D2.1 (IO1), J1.3
- new net Parachute ENABLE: J4.2
- new net SCL0 I2C: R28.2, U4.2 (SCK), U7.2 (SCK)
- new net SCL1 I2C: R18.1, U8.13 (SCL)
- new net SDA0 I2C: R29.2, U4.4 (SDA/SDI/SDISDO), U7.4 (SDI)
- new net SDA1 I2C: R17.1, U8.14 (SDA)
- new net TIMER GPS: IC1.3 (TIMEPULSE), Q1.1
- new net VBAT: BT1.P1, BT1.P2, JP6.2 (B)
- no-connect marks 6 -> 15
Other:
- sheet RP2040 Standard ports: added GP20/I2C SDA, GP21/I2C SDL, GP24/UART1 TX, GP25/UART1 RX, GPIO16, GPIO17, GPIO26, GPIO4, GPIO5; removed GP16/SPI0 MISO, GP17/SPI0 ~{CS}, GP21/SPI0 ~{CS}, GP26_ADC0, GP4/UART1 TX, GP5/UART1 RX, GPIO20, GPIO24, GPIO25
- note added: "4 Channel ESD Diode"
- note added: "BMI323: 6.4KHz, SPI 10MHz LIS2MDL: 100Hz, SPI 10MHz BME280: 1Hz, SPI 10MHz"
- note added: "LSM6DSO: 6.4KHz, I2C Fast Mode 400kHz, ADDR 0x6A BMP581: 400Hz, I2C Fast Mode Plus 1MHz, ADDR 0x46 LPS22DF: 200Hz, I2C Fast Mode Plus 1MHz, ADDR 0x5C"
- note added: "Sensor Unit 1: BOSH AXL&GYRO + ST MAGNETOMETER + BOSH HUMIDITY"
- note added: "Sensor Unit 2: ST AXL&GYRO + BOSH BAROMETER + ST MAGNETOMETER"
- note added: "ublox NEO-M8Q-0: 10Hz with -167dBm"
- note removed: "ASM339LHH: 6.4KHz BMP581: 400Hz LIS2MDL: 100Hz"
- note removed: "BMI323: 6.4KHz LPS22DF 200Hz"
- note removed: "CD-PA1616D: 1Hz to 10Hz with -165dBm"
- note removed: "Humidity Sensor"
- note removed: "PA1616 GPS L1 Band"
- note removed: "Sensor Unit 1: BOSH AXL&GYRO + ST BARO"
- note removed: "Sensor Unit 2: ST AXL&GYRO + BOSH BARO + ST MAG"
- note removed: "Texas: HDC3022 Humidity 1Hz I2C ADDR 0x47"
- title: On Board Computer -> Navigator
- moved on the sheet: C1, C10, C17, C18, C2, C3, C5, C6, C9, CR3, CR4, IC2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
