File: Boards/Rocket Systems/OBC/OBC.kicad_sch (KiCad schematic)
At the start: 68 parts, among them IC1 NSVT30010MXV6T1G, IC2 BC846BLT1G, J1 1718560006, J2 5023520200, J3 MEM2061-01-188-00-A_REVA, J4 SMARA_CONNECTOR, U1 SX1280IMLTRT, U2 STLM20DD9F, U3 NRF21540-QDAA-R, U4 THVD2410VDRCR, U5 VLMKG3400-GS08

Commit message: New OBC PCB project
Parts:
- R13, R14, R4, R5, R6, R7: footprint Resistor-0402:RES_0402 -> Resistor-0603:RES_0603
Connections:
- net SD-Card  ~{CS} SPI: now also D2.6 (IO4); no longer D2.3 (IO2)
- net SD-Card MISO SPI: now also D2.4 (IO3); no longer D2.1 (IO1)
- net SD-Card MOSI SPI: now also D2.1 (IO1); no longer D2.4 (IO3)
- net SD-Card SCK SPI: now also D2.3 (IO2); no longer D2.6 (IO4)
Other:
- moved on the sheet: D2

Commit message: Nav & OBC update
Changed lines of the file:
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@@
 	(text "16G SD-Card"
 		(exclude_from_sim no)
-		(at 127.635 19.685 0)
+		(at 182.245 20.32 0)
 		(effects
 			(font
@@
 		(fields_autoplaced yes)
 		(property "Reference" "U3"
-			(at 260.985 153.035 0)
+			(at 260.985 153.67 0)
 			(effects
 				(font
@@
 		)
 		(property "Value" "NRF21540-QDAA-R"
-			(at 260.985 155.575 0)
+			(at 260.985 156.21 0)
 			(effects
 				(font

Commit message: Finished OBC
Parts:
- removed J4: SMARA_CONNECTOR, Side Angle SMA:SMARACONNECTOR, symbol SMARA_CONNECTOR:SMARA_CONNECTOR
- added J4: RFPC-SMA27-F, RFPC-SMA27-F:GRADCONN_RFPC-SMA27-F, symbol RFPC-SMA27-F:RFPC-SMA27-F
- H1, H2, H3, H4: footprint MountingHole:MountingHole_3.2mm_M3_ISO7380_Pad_TopBottom -> MountingHole:MountingHole_3.2mm_M3_ISO7380
Connections:
- net GND: now also J4.G1, J4.G2, J4.G3, J4.G4
- net at C19.1, C21.1, L4.2: now also J4.1
Other:
- sheet RP2040 ports: added GP23/UART1 RTS, GP24/UART1 TX, GP25/UART1 RX, GP29/PWM6 B, GPIO4, GPIO5, GPIO6; removed GP25/PWM4 B, GP4/UART1 TX, GP5/UART1 RX, GP6/UART1 CTS, GPIO23, GPIO24, GPIO29

Commit message: Silkcreen and Logos
Parts:
- added S1: RFI Shield 20x25, RFI Shield:RFI Shield, symbol RFI Shield:RFI_Shield
Changed lines of the file:
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@@
+	)
+	(symbol
+		(lib_id "RFI Shield:RFI_Shield")
+		(at 262.89 212.725 0)
+		(unit 1)
+		(exclude_from_sim no)
+		(in_bom yes)
+		(on_board yes)
+		(dnp no)
+		(property "Reference" "S1"
+			(at 261.62 207.645 0)
+			(effects
+				(font
+					(size 1.27 1.27)
+				)
+				(justify left)
+			)
+		)
+		(property "Value" "RFI Shield 20x25"
+			(at 255.27 210.185 0)
+			(effects
+				(font
+					(size 1.27 1.27)
+				)
+				(justify left)
+			)
+		)
+		(property "Footprint" "RFI Shield:RFI Shield"
+			(at 262.89 212.725 0)
+			(effects
+				(font
+					(size 1.27 1.27)
+				)
+				(hide yes)
+			)
+		)
+		(property "Datasheet" ""
+			(at 262.89 212.725 0)
+			(effects
+				(font
+					(size 1.27 1.27)
+				)
+				(hide yes)
+			)
+		)
+		(property "Description" "Harwin Shield"
+			(at 262.89 212.725 0)
+			(effects
+				(font
+					(size 1.27 1.27)
+				)
+				(hide yes)
+			)
+		)
+		(instances
+			(project ""
+				(path "/169b1789-9bea-4709-830d-1c7983087293"
+					(reference "S1")
+					(unit 1)
+				)
+			)
+		)
 	)
 	(symbol

Commit message: small nav and OBC updates - DFM corrections
Parts:
- J2: footprint Molex 2 Conn:CONN02_502352_MOL -> CONN02_502352_MOL
Connections:
- net GND: now also J2.3 (EP), J2.4 (EP)
Changed lines of the file:
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@@
 			)
 		)
-		(property "Footprint" "Molex 2 Conn:CONN02_502352_MOL"
+		(property "Footprint" "CONN02_502352_MOL"
 			(at 110.49 108.585 0)
 			(effects
@@
 		(pin "2"
 		)
+		(pin "3"
+		)
+		(pin "4"
+		)
 		(instances
 			(project ""
@@
 					(unit 1)
 				)
+			)
+		)
+	)
+	(symbol
+		(lib_id "power:GND")
+		(at 111.76 113.665 0)
+		(unit 1)
+		(exclude_from_sim no)
+		(in_bom yes)
+		(on_board yes)
+		(dnp no)
+		(property "Reference" "#PWR070"
+			(at 111.76 120.015 0)
+			(effects
+				(font
+					(size 1.27 1.27)
+				)
+				(hide yes)
+			)
+		)
+		(property "Value" "GND"
+			(at 111.76 117.475 0)
+			(effects
+				(font
+					(size 1.27 1.27)
+				)
+			)
+		)
+		(property "Footprint" ""
+			(at 111.76 113.665 0)
+			(effects
+				(font
+					(size 1.27 1.27)
+				)
+				(hide yes)
+			)
+		)
+		(property "Datasheet" ""
+			(at 111.76 113.665 0)
+			(effects
+				(font
+					(size 1.27 1.27)
+				)
+				(hide yes)
+			)
+		)
+		(property "Description" "Power symbol creates a global label with name \"GND\" , ground"
+			(at 111.76 113.665 0)
+			(effects
+				(font
+					(size 1.27 1.27)
+				)
+				(hide yes)
+			)
+		)
+		(pin "1"
+		)
+		(instances
+			(project "OBC"
+				(path "/169b1789-9bea-4709-830d-1c7983087293"
+					(reference "#PWR070")
+					(unit 1)
+				)

Commit message: obc schematic
Parts:
- R10, R12: value 523 -> 510
- R13: value 65 -> 62
Changed lines of the file:
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@@
 			)
 		)
-		(property "Value" "523"
+		(property "Value" "510"
 			(at 335.28 113.03 90)
 			(effects
@@
 			)
 		)
-		(property "Value" "65"
+		(property "Value" "62"
 			(at 337.82 57.15 90)
 			(effects
@@
 			)
 		)
-		(property "Value" "523"
+		(property "Value" "510"
 			(at 330.835 93.345 90)
 			(effects

Commit message: OBC final BOM and Fabfiles
Parts:
- removed J4: RFPC-SMA27-F, RFPC-SMA27-F:GRADCONN_RFPC-SMA27-F, symbol RFPC-SMA27-F:RFPC-SMA27-F
- added J4: PCB.RPSMAFRA.HT, PCBRPSMAFRAHT, symbol PCB_RPSMAFRA_HT:PCB.RPSMAFRA.HT
- C2: footprint Capacitor-0402:Capacitor_0402 -> Capacitor-0603:Capacitor_0603
- C41: value 220n -> 470n
- R25: value 6k8 -> 3k6
- R8, R9: footprint Resistor-0402:RES_0402 -> Resistor-0603:RES_0603
Connections:
- net GND: now also J4.2, J4.3, J4.4, J4.5
- net at C19.1, C21.1, L4.2: now also J4.1
Changed lines of the file:
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@@
 	)
 	(junction
+		(at 311.785 173.355)
+		(diameter 0)
+		(color 0 0 0 0)
+	)
+	(junction
 		(at 309.245 119.38)
 		(diameter 0)
@@
 	)
 	(junction
-		(at 311.785 173.355)
-		(diameter 0)
-		(color 0 0 0 0)
-	)
-	(junction
 		(at 298.45 114.3)
 		(diameter 0)
@@
 	(wire
 		(pts
-			(xy 311.785 173.355) (xy 321.945 173.355)
-		)
-		(stroke
-			(width 0)
-			(type default)
-		)
-	)
-	(wire
-		(pts
 			(xy 256.54 110.49) (xy 257.175 110.49)
 		)
@@
 	(wire
 		(pts
+			(xy 311.785 173.355) (xy 315.595 173.355)
+		)
+		(stroke
+			(width 0)
+			(type default)
+		)
+	)
+	(wire
+		(pts
 			(xy 80.01 108.585) (xy 80.01 103.505)
 		)
@@
 			)
 		)
-		(property "Footprint" "Resistor-0402:RES_0402"
+		(property "Footprint" "Resistor-0603:RES_0603"
 			(at 302.26 116.078 90)
 			(effects
@@
 			)
 		)
-		(property "Value" "220n"
+		(property "Value" "470n"
 			(at 147.955 109.855 0)
 			(effects
@@
 			)
 		)
-		(property "Footprint" "Capacitor-0402:Capacitor_0402"
+		(property "Footprint" "Capacitor-0603:Capacitor_0603"
 			(at 59.69 106.045 0)
 			(effects
@@
 	)
 	(symbol
-		(lib_id "RFPC-SMA27-F:RFPC-SMA27-F")
-		(at 324.485 173.355 0)
-		(mirror y)
-		(unit 1)
-		(exclude_from_sim no)
-		(in_bom yes)
-		(on_board yes)
-		(dnp no)
-		(property "Reference" "J4"
-			(at 324.8279 167.005 0)
-			(effects
-				(font
-					(size 1.27 1.27)
-				)
-			)
-		)
-		(property "Value" "RFPC-SMA27-F"
-			(at 324.8279 169.545 0)
-			(effects
-				(font
-					(size 1.27 1.27)
-				)
-			)
-		)
-		(property "Footprint" "RFPC-SMA27-F:GRADCONN_RFPC-SMA27-F"
-			(at 324.485 173.355 0)
-			(effects
-				(font
-					(size 1.27 1.27)
-				)
-				(justify bottom)
-				(hide yes)
-			)
-		)
-		(property "Datasheet" ""
-			(at 324.485 173.355 0)
-			(effects
-				(font
-					(size 1.27 1.27)
-				)
-				(hide yes)
-			)
-		)
-		(property "Description" ""
-			(at 324.485 173.355 0)
-			(effects
-				(font
-					(size 1.27 1.27)
-				)
-				(hide yes)
-			)
-		)
-		(property "MF" "GradConn"
-			(at 324.485 173.355 0)
-			(effects
-				(font
-					(size 1.27 1.27)
-				)
-				(justify bottom)
-				(hide yes)
-			)
-		)
-		(property "MAXIMUM_PACKAGE_HEIGHT" "10.3mm"
-			(at 324.485 173.355 0)
-			(effects
-				(font
-					(size 1.27 1.27)
-				)
-				(justify bottom)
-				(hide yes)
-			)
-		)
-		(property "Package" "None"
-			(at 324.485 173.355 0)
-			(effects
-				(font
-					(size 1.27 1.27)
-				)
-				(justify bottom)
-				(hide yes)
-			)
-		)
-		(property "Price" "None"
-			(at 324.485 173.355 0)
-			(effects
-				(font
-					(size 1.27 1.27)
-				)
-				(justify bottom)
-				(hide yes)
-			)
-		)
-		(property "Check_prices" "https://www.snapeda.com/parts/RFPC-SMA27-F/GradConn/view-part/?ref=eda"
-			(at 324.485 173.355 0)
-			(effects
-				(font
-					(size 1.27 1.27)
-				)
-				(justify bottom)
-				(hide yes)
-			)
-		)
-		(property "STANDARD" "Manufacturer Recommendations"
-			(at 324.485 173.355 0)
-			(effects
-				(font
-					(size 1.27 1.27)
-				)
-				(justify bottom)
-				(hide yes)
-			)
-		)
-		(property "PARTREV" "1.0"
-			(at 324.485 173.355 0)
-			(effects
-				(font
-					(size 1.27 1.27)
-				)
-				(justify bottom)
-				(hide yes)
-			)
-		)
-		(property "SnapEDA_Link" "https://www.snapeda.com/parts/RFPC-SMA27-F/GradConn/view-part/?ref=snap"
-			(at 324.485 173.355 0)
-			(effects
-				(font
-					(size 1.27 1.27)
-				)
-				(justify bottom)
-				(hide yes)
-			)
-		)
-		(property "MP" "RFPC-SMA27-F"
-			(at 324.485 173.355 0)
-			(effects
-				(font
-					(size 1.27 1.27)
-				)
-				(justify bottom)
-				(hide yes)
-			)
-		)
-		(property "Description_1" "SMA Connector Jack, Female Socket 50 Ohms Panel Mount, Through Hole, Right Angle Solder"
-			(at 324.485 173.355 0)
-			(effects
-				(font
-					(size 1.27 1.27)
-				)
-				(justify bottom)
-				(hide yes)
-			)
-		)
-		(property "Availability" "In Stock"
-			(at 324.485 173.355 0)
-			(effects
-				(font
-					(size 1.27 1.27)
-				)
-				(justify bottom)
-				(hide yes)
-			)
-		)
-		(property "MANUFACTURER" "GradConn"
-			(at 324.485 173.355 0)
-			(effects
-				(font
-					(size 1.27 1.27)
-				)
-				(justify bottom)
-				(hide yes)
-			)
-		)
-		(pin "1"
-		)
-		(pin "G1"
-		)
-		(pin "G2"
-		)
-		(pin "G3"
-		)
-		(pin "G4"
-		)
-		(instances
-			(project ""
-				(path "/169b1789-9bea-4709-830d-1c7983087293"
-					(reference "J4")
-					(unit 1)
-				)
-			)
-		)
-	)
-	(symbol
 		(lib_id "Device:C")
 		(at 300.355 177.165 0)
@@
 	)
 	(symbol
+		(lib_id "PCB_RPSMAFRA_HT:PCB.RPSMAFRA.HT")
+		(at 321.945 173.355 0)
+		(unit 1)
+		(exclude_from_sim no)
+		(in_bom yes)
+		(on_board yes)
+		(dnp no)
+		(fields_autoplaced yes)
+		(property "Reference" "J4"
+			(at 332.105 166.37 0)
+			(effects
+				(font
+					(size 1.27 1.27)
+				)
+			)
+		)
+		(property "Value" "PCB.RPSMAFRA.HT"
+			(at 332.105 168.91 0)
+			(effects
+				(font
+					(size 1.27 1.27)
+				)
+			)
+		)
+		(property "Footprint" "PCBRPSMAFRAHT"
+			(at 338.455 268.275 0)
+			(effects
+				(font
+					(size 1.27 1.27)
+				)
+				(justify left top)
+				(hide yes)
+			)
+		)
+		(property "Datasheet" "https://www.taoglas.com/datasheets/PCB.RPSMAFRA.HT.pdf"
+			(at 338.455 368.275 0)
+			(effects
+				(font
+					(size 1.27 1.27)
+				)
+				(justify left top)
+				(hide yes)
+			)
+		)
+		(property "Description" "RF Connectors / Coaxial Connectors SMA RA Reverse Polarity PCB Mount, Jack, Gold, 50 , Through Hole Pin"
+			(at 321.945 173.355 0)
+			(effects
+				(font
+					(size 1.27 1.27)
+				)
+				(hide yes)
+			)
+		)
+		(property "Height" "9.5"
+			(at 338.455 568.275 0)
+			(effects
+				(font
+					(size 1.27 1.27)
+				)
+				(justify left top)
+				(hide yes)
+			)
+		)
+		(property "Mouser Part Number" "960-PCB.RPSMAFRA.HT"
+			(at 338.455 668.275 0)
+			(effects
+				(font
+					(size 1.27 1.27)
+				)
+				(justify left top)
+				(hide yes)
+			)
+		)
+		(property "Mouser Price/Stock" "https://www.mouser.co.uk/ProductDetail/Taoglas/PCB.RPSMAFRA.HT?qs=RuW%2Fu%252BNMQmvVc2WiXpnkVw%3D%3D"
+			(at 338.455 768.275 0)
+			(effects
+				(font
+					(size 1.27 1.27)
+				)
+				(justify left top)
+				(hide yes)
+			)
+		)
+		(property "Manufacturer_Name" "Taoglas"
+			(at 338.455 868.275 0)
+			(effects
+				(font
+					(size 1.27 1.27)
+				)
+				(justify left top)
+				(hide yes)
+			)
+		)
+		(property "Manufacturer_Part_Number" "PCB.RPSMAFRA.HT"
+			(at 338.455 968.275 0)
+			(effects
+				(font
+					(size 1.27 1.27)
+				)
+				(justify left top)
+				(hide yes)
+			)
+		)
+		(pin "4"
+		)
+		(pin "5"
+		)
+		(pin "3"
+		)
+		(pin "1"
+		)
+		(pin "2"
+		)
+		(instances
+			(project ""
+				(path "/169b1789-9bea-4709-830d-1c7983087293"
+					(reference "J4")
+					(unit 1)
+				)
+			)
+		)
+	)
+	(symbol
 		(lib_id "Device:C_Small")
 		(at 247.65 95.25 0)
@@
 			)
 		)
-		(property "Value" "6k8"
+		(property "Value" "3k6"
 			(at 154.94 107.95 90)
 			(effects
@@
 			)
 		)
-		(property "Footprint" "Resistor-0402:RES_0402"
+		(property "Footprint" "Resistor-0603:RES_0603"
 			(at 302.26 121.158 90)
 			(effects
