File: Boards/Rocket Systems/Elyra/Elytra.kicad_sch (KiCad schematic)
At the start: 7 parts, among them J1 XT30UPB-M, J2 Conn_01x01_Socket, J3 Conn_01x01_Socket, U1 IRLZ44NPBF

Commit message: Elytra update
ok
Parts:
- removed C1: C, Capacitor-0402:Capacitor_0402, symbol Device:C
- removed J1: XT30UPB-M, AMASS_XT30UPB-M:CONN_XT30UPB-M_AMA, symbol AMASS_XT30UPB-M:XT30UPB-M
- removed J2, J3: Conn_01x01_Socket, Button_Switch_THT:SW_Lever_1P2T_NKK_GW12LxH, symbol Connector:Conn_01x01_Socket
- removed R2: R, Resistor-0402:RES_0402, symbol Device:R
- removed U1: IRLZ44NPBF, NMOS IRLZ44:PG-TO220-3_INF, symbol NMOS IRLZ44:IRLZ44NPBF
- R1: value 100k -> R; footprint Resistor-0402:RES_0402 -> Resistor-0603:RES_0603
Connections:
- net E-Match Activation: no longer names the net of R1.2
- net GND: no longer names the net of R1.1
- no-connect marks 0 -> 1
Other:
- note removed: "Conectores alanvacados"
- note removed: "E-Match Circuit"
- note removed: "Este contacto vai estar a conectar o circuito a um botão ON-OFF armado por chave que se vai encontrar no painel de armação exterior do foguetão"
- note removed: "Provavelmente este circuito vai sofrer alterações devido à não utilização de um ignitor e-match"
- note removed: "To E-Match"
- note removed: "Verificar necessidade de Heat-Sink no Mosfet"
- note removed: "Verificar os valores de R12 e C7, para uma constante tempo apropriada"
