File: Boards/Breakout Boards/Hydra Breakout/ALL NEW ALL DIFFERENT Hydra Breakout/Hydra Breakout.kicad_sch (KiCad schematic)
At the start: 40 parts, among them J1 Conn_01x01_Socket, J11 Conn_01x01_Socket, J12 Conn_01x01_Socket, J13 Conn_01x01_Socket, J14 Conn_01x01_Socket, J15 Conn_01x01_Socket, J16 Conn_01x01_Socket, J17 Conn_01x01_Socket, J18 Conn_01x01_Socket, J2 Conn_01x01_Socket, J3 Conn_01x01_Socket, J4 Conn_01x01_Socket, J5 Conn_01x01_Socket, J6 Conn_01x01_Socket, J7 BM03B-SRSS-TBLFSN, J8 Conn_01x01_Socket, J9 Conn_01x01_Socket, SW1 D2F-01-D, U1 SC0915, U12 THVD2410VDRCR

Commit message: Design da Hydra Breakout (Part 1)
Inclui algumas adições à biblioteca.
Parts:
- removed C40, C42: 100n, Capacitor-0402:Capacitor_0402, symbol Device:C_Small
- removed R30, R48: 10k, Resistor-0402:RES_0402, symbol Device:R
- removed R55: 120, Resistor-0603:RES_0603, symbol Device:R
- removed SW1: D2F-01-D, D2F-01-D_OMR, symbol Switch_D2F-01:D2F-01-D
- removed U12: THVD2410VDRCR, VSON10_DRC_TEX, symbol THVD2410VDRCR:THVD2410VDRCR
- removed VD1, VD2: SMAJ30CA, symbol SMAJ30CA:SMAJ30CA
- added C16, C20: 100n, Capacitor-0603:Capacitor_0603, symbol Device:C_Small
- added CR5: SP712-02HTG, 2Channel ESD RS485 - P712-02HTG:SOT23-3_LTF, symbol SP712-02HTG:SP712-02HTG
- added D4, D7: RB095BGE-30TL, SchottkyDiode-RB095BGE:RD3P175SNFRATL, symbol RB095BGE-30TL:RB095BGE-30TL
- added Q2, Q3: 2N7002H6327XTSA2, NMOS_2N7002:PG-SOT23-3-5_INF_MIN, symbol NMOS_2N7002:2N7002H6327XTSA2
- added R17, R18, R19, R68: 10k, Capacitor-0603:Capacitor_0603, symbol Device:R
- added R20, R21: 0, Resistor-0603:RES_0603, symbol Device:R
- added R35, R43, R57, R58: 2k, Capacitor-0603:Capacitor_0603, symbol Device:R
- added U5, U9: SQJA36EP-T1_GE3, SQJA36EP-T1-GE3:PowerPAK_SO-8L_3_VIS, symbol SQJA36EP-T1-GE3:SQJA36EP-T1_GE3
- added U6: THVD2410VDRCR, THVD2410VDRCR:VSON10_DRC_TEX, symbol THVD2410VDRCR:THVD2410VDRCR
- CV1: footprint Capacitor-0402:Capacitor_0402 -> Capacitor-0603:Capacitor_0603
- R23, R24, R25, R3: footprint Resistor-0402:RES_0402 -> Capacitor-0603:Capacitor_0603
Connections:
- net +12V: now also D4.2, D7.2
- net +3.3V: now also C16.2, Q2.1 (G), Q3.1 (G), R18.1, R43.1, R58.1, U6.1 (VIO)
- net +5V: now also C20.1, R20.2, R35.1, R57.1, U6.10 (VCC)
- net ENABLE_RS: now also R19.1, U6.3 (DE), U6.4 (~{RE})
- net GND: now also C16.1, C20.2, CR5.3, R17.2, R19.2, R21.2, R68.2, U5.1 (S), U5.2 (S), U5.3 (S), U6.11 (EPAD), U6.6 (GND), U9.1 (S), U9.2 (S), U9.3 (S)
- net Main Solenoid Valve: now also D7.1, D7.3, U9.5 (D)
- net Purge Solenoid Valve: now also D4.1, D4.3, U5.5 (D)
- net Purge Valve Enable: now also R17.1, U5.4 (G)
- net READ_RS: now also R18.2, U6.2 (R)
- net RS_DN: now also CR5.1, U6.9 (B)
- net RS_DP: now also CR5.2, U6.8 (A)
- net Servo_IN1 PWM: now also Q2.2 (S), R43.2
- net Servo_IN2 PWM: now also Q3.2 (S), R58.2
- net Servo_OUT1 PWM: now also Q2.3 (D), R35.2
- net Solenoid Valve Enable: now also R68.1, U9.4 (G)
- net WRITE_RS: now also U6.5 (D)
- net Sensor Unit/SCL I2C: now reaches U1.19 (GP14)
- net Sensor Unit/SDA I2C: now reaches U1.20 (GP15)
- net Sensor Unit/Temp_Sense: now reaches U1.32 (GP27)
- new net: R20.1, R21.1, U6.7 (SLR)
- new net Servo_OUT2 PWM: Q3.3 (D), R57.2
Other:
- sheet Sensor Unit ports: added LoadCell1 Sense, LoadCell2 Sense, LoadCell3 Sense, Pressure1 Sense, Pressure2 Sense, SCL I2C, SDA I2C, Temp_Sense; removed none
- note added: "Main Valve Driver - Solenoid"
- note added: "Purge Valve Driver - Solenoid"
- note added: "Servo Valve Driver"
- note added: "Valve Drivers"
- moved on the sheet: C10, C24, C25, C28, C29, C30, L1

Commit message: Design da Hydra Breakout (Part 3)
Other:
- added sheet Thermo 1 (Thermo1.kicad_sch)
- added sheet Thermo 2 (Thermo1.kicad_sch)
- added sheet Thermo 3 (Thermo1.kicad_sch)
- sheet Sensor Unit ports: added none; removed 1~{DRDY} THERMO, 1~{FAULT} THERMO, 2~{DRDY} THERMO, 2~{FAULT} THERMO, 3~{DRDY} THERMO, 3~{FAULT} THERMO, MISO SPI, MOSI SPI, SCK SPI, THERMO1 DN, THERMO1 DP, THERMO2 DN, THERMO2 DP, THERMO3 DN, THERMO3 DP, ~{CS} THERMO1 SPI, ~{CS} THERMO2 SPI, ~{CS} THERMO3 SPI
