File: Boards/Breakout Boards/Hydra Breakout/ALL NEW ALL DIFFERENT Hydra Breakout/Hydra Breakout.kicad_pcb (KiCad board)
At the start: 2 copper layers, 85.4 x 92.2 mm, 1 part, among them U1 SC0915

Commit message: Design da Hydra Breakout (Part 1)
Inclui algumas adições à biblioteca.
Parts:
- added C1: 100n, Capacitor-0603:Capacitor_0603, F.Cu at (29.6, 159.2)
- added C10: 2.2u, Capacitor-1206:Capacitor_1206, F.Cu at (244.7, 52.8)
- added C11: 100n, Capacitor-0603:Capacitor_0603, F.Cu at (239.8, 73.3)
- added C12: 10n, Capacitor-0603:Capacitor_0603, F.Cu at (239.8, 75.4)
- added C13: 100n, Capacitor-0603:Capacitor_0603, F.Cu at (239.8, 77.6)
- added C14: 100n, Capacitor-0603:Capacitor_0603, F.Cu at (239.8, 79.8)
- added C16: 100n, Capacitor-0603:Capacitor_0603, F.Cu at (213.5, 89.0)
- added C2: 10n, Capacitor-0603:Capacitor_0603, F.Cu at (24.6, 159.2)
- added C20: 100n, Capacitor-0603:Capacitor_0603, F.Cu at (213.5, 91.2)
- added C24: 2.2u, Capacitor-1206:Capacitor_1206, F.Cu at (244.7, 55.9)
- added C25: 2.2u, Capacitor-1206:Capacitor_1206, F.Cu at (244.7, 59.1)
- added C28: 2.2u, Capacitor-1206:Capacitor_1206, F.Cu at (244.7, 62.3)
- added C29: 470n, Capacitor-1206:Capacitor_1206, F.Cu at (244.7, 65.4)
- added C3: 100n, Capacitor-0603:Capacitor_0603, F.Cu at (40.8, 161.0)
- added C30: 470n, Capacitor-1206:Capacitor_1206, F.Cu at (244.7, 68.6)
- added C31: 10n, Capacitor-0603:Capacitor_0603, F.Cu at (24.6, 160.8)
- added C32: 10n, Capacitor-0603:Capacitor_0603, F.Cu at (239.8, 84.1)
- added C33: 100n, Capacitor-0603:Capacitor_0603, F.Cu at (239.8, 86.3)
- added C35: 100n, Capacitor-0603:Capacitor_0603, F.Cu at (123.0, 166.4)
- added C36: 100n, Capacitor-0603:Capacitor_0603, F.Cu at (243.2, 73.3)
- added C37: 100n, Capacitor-0603:Capacitor_0603, F.Cu at (243.2, 75.4)
- added C38: 100n, Capacitor-0603:Capacitor_0603, F.Cu at (243.2, 77.6)
- added C39: 10n, Capacitor-0603:Capacitor_0603, F.Cu at (243.2, 79.8)
- added C4: 100n, Capacitor-0603:Capacitor_0603, F.Cu at (30.4, 162.0)
- added C40: 100n, Capacitor-0402:Capacitor_0402, F.Cu at (237.6, 51.4)
- added C41: 100n, Capacitor-0603:Capacitor_0603, F.Cu at (243.2, 82.0)
- added C42: 100n, Capacitor-0402:Capacitor_0402, F.Cu at (237.6, 53.6)
- added C43: 100n, Capacitor-0603:Capacitor_0603, F.Cu at (243.2, 84.1)
- added C44: 10n, Capacitor-0603:Capacitor_0603, F.Cu at (243.2, 86.3)
- added C45: 10n, Capacitor-0603:Capacitor_0603, F.Cu at (243.2, 88.5)
- added C46: 10n, Capacitor-0603:Capacitor_0603, F.Cu at (246.6, 73.3)
- added C47: 100n, Capacitor-0603:Capacitor_0603, F.Cu at (246.6, 75.4)
- added C48: 100nF, Capacitor-0603:Capacitor_0603, F.Cu at (246.6, 77.6)
- added C49: 100n, Capacitor-0603:Capacitor_0603, F.Cu at (246.6, 79.8)
- added C5: 100n, Capacitor-0603:Capacitor_0603, F.Cu at (236.5, 82.0)
- added C50: 1u, Capacitor-0603:Capacitor_0603, F.Cu at (114.8, 166.4)
- added C51: 100n, Capacitor-0603:Capacitor_0603, F.Cu at (123.6, 171.6)
- added C6: 10n, Capacitor-0603:Capacitor_0603, F.Cu at (236.5, 84.1)
- added C67: 4.7u, Capacitor-1206:Capacitor_1206, F.Cu at (116.8, 165.8)
- added C8: 100n, Capacitor-0603:Capacitor_0603, F.Cu at (236.5, 86.3)
- added C9: 100n, Capacitor-0603:Capacitor_0603, F.Cu at (236.5, 88.5)
- added CR5: SP712-02HTG, 2Channel ESD RS485 - P712-02HTG:SOT23-3_LTF, F.Cu at (209.4, 85.7)
- added CV1: 1uF, Capacitor-0603:Capacitor_0603, F.Cu at (237.6, 55.7)
- added C_BIAS1: 1u, Capacitor-0603:Capacitor_0603, F.Cu at (220.9, 66.4)
- added C_BIAS2: 1u, Capacitor-0603:Capacitor_0603, F.Cu at (220.9, 68.9)
- added C_BT1: 100n, Capacitor-0603:Capacitor_0603, F.Cu at (214.6, 26.6)
- added C_BT2: 100n, Capacitor-0603:Capacitor_0603, F.Cu at (214.6, 28.8)
- added C_BT3: 100n, Capacitor-0603:Capacitor_0603, F.Cu at (214.6, 30.9)
- added C_FF1: 22p, Capacitor-0603:Capacitor_0603, F.Cu at (214.6, 33.1)
- added C_IN-BLK1: 10u, Capacitor-4mm:Capacitor_4mm, F.Cu at (200.9, 43.3)
- added C_IN-BLK2: 10u, Capacitor-4mm:Capacitor_4mm, F.Cu at (200.9, 50.6)
- added C_IN-BLK3: 10u, Capacitor-4mm:Capacitor_4mm, F.Cu at (200.9, 58.0)
- added C_IN1: 4.7u, Capacitor-1206:Capacitor_1206, F.Cu at (178.1, 60.5)
- added C_IN2: 4.7u, Capacitor-1206:Capacitor_1206, F.Cu at (178.1, 63.6)
- added C_IN3: 4.7u, Capacitor-1206:Capacitor_1206, F.Cu at (178.1, 66.8)
- added C_IN4: 4.7u, Capacitor-1206:Capacitor_1206, F.Cu at (178.1, 70.0)
- added C_IN5: 4.7u, Capacitor-1206:Capacitor_1206, F.Cu at (178.1, 73.1)
- added C_IN6: 4.7u, Capacitor-1206:Capacitor_1206, F.Cu at (178.1, 76.3)
- added C_IN_HFI1: 100n, Capacitor-0603:Capacitor_0603, F.Cu at (214.6, 35.3)
- added C_IN_HFI2: 100n, Capacitor-0603:Capacitor_0603, F.Cu at (218.0, 26.6)
- added C_IN_HFI3: 100n, Capacitor-0603:Capacitor_0603, F.Cu at (218.0, 28.8)
- added C_IN_HFI4: 100n, Capacitor-0603:Capacitor_0603, F.Cu at (218.0, 30.9)
- added C_IN_HFI5: 100n, Capacitor-0603:Capacitor_0603, F.Cu at (218.0, 33.1)
- added C_IN_HFI6: 100n, Capacitor-0603:Capacitor_0603, F.Cu at (218.0, 35.3)
- added C_OUT1: 1u, Capacitor-0603:Capacitor_0603, F.Cu at (220.9, 71.5)
- added C_OUT10: 47u, Capacitor-0805:Capacitor_0805, F.Cu at (212.1, 75.8)
- added C_OUT11: 22u, Capacitor-0805:Capacitor_0805, F.Cu at (216.7, 66.7)
- added C_OUT12: 22u, Capacitor-0805:Capacitor_0805, F.Cu at (216.7, 69.7)
- added C_OUT13: 22u, Capacitor-0805:Capacitor_0805, F.Cu at (216.7, 72.8)
- added C_OUT14: 22u, Capacitor-0805:Capacitor_0805, F.Cu at (216.7, 75.8)
- added C_OUT15: 560u, Capacitor-8mm:Capacitor_8mm, F.Cu at (189.6, 44.9)
- added C_OUT16: 100u, Capacitor-8mm:Capacitor_8mm, F.Cu at (189.6, 55.5)
- added C_OUT2: 10u, Capacitor-0805:Capacitor_0805, F.Cu at (207.6, 66.7)
- added C_OUT3: 10u, Capacitor-0805:Capacitor_0805, F.Cu at (207.6, 69.7)
- added C_OUT4: 10u, Capacitor-0805:Capacitor_0805, F.Cu at (207.6, 72.8)
- added C_OUT5: 10u, Capacitor-0805:Capacitor_0805, F.Cu at (207.6, 75.8)
- added C_OUT6: 100u, Capacitor-6mm:Capacitor_6mm, F.Cu at (175.8, 54.0)
- added C_OUT7: 22u, Capacitor-0805:Capacitor_0805, F.Cu at (212.1, 66.7)
- added C_OUT8: 22u, Capacitor-0805:Capacitor_0805, F.Cu at (212.1, 69.7)
- added C_OUT9: 47u, Capacitor-0805:Capacitor_0805, F.Cu at (212.1, 72.8)
- added C_VCC1: 1u, Capacitor-0603:Capacitor_0603, F.Cu at (220.9, 74.0)
- added C_VCC2: 1u, Capacitor-0603:Capacitor_0603, F.Cu at (220.9, 76.5)
- added C_VCC3: 1u, Capacitor-0603:Capacitor_0603, F.Cu at (220.9, 79.0)
- added D1: RB095BGE, SchottkyDiode-RB095BGE:RD3P175SNFRATL, F.Cu at (188.1, 32.3)
- added D4: RB095BGE-30TL, SchottkyDiode-RB095BGE:RD3P175SNFRATL, F.Cu at (247.0, 32.3)
- added D5: RSX301L, Diode-Schottky_RSX301L:DIOM5026X220N, F.Cu at (199.8, 77.9)
- added D6: RB095BGE, SchottkyDiode-RB095BGE:RD3P175SNFRATL, F.Cu at (197.8, 32.3)
- added D7: RB095BGE-30TL, SchottkyDiode-RB095BGE:RD3P175SNFRATL, F.Cu at (256.7, 32.3)
- added IC1: BC846BLT1G, BJT NPN:SOT96P237X111-3N, F.Cu at (185.7, 75.8)
- added IC6: INA2181A4IDSQR, INA2181A4IDSQR:SON40P200X200X80-11N, F.Cu at (227.9, 101.5)
- added IC7: INA181A4QDCKRQ1, INA181A4QDCKRQ1:SOT65P210X110-6N, F.Cu at (228.0, 97.5)
- added IC8: PCA9306GM,125, PCA9306GM,125:PCA9570GMH, F.Cu at (120.8, 170.7)
- added J1: Conn_01x01_Socket, Pico_Conn1x1:Pico_01pin, F.Cu at (228.6, 28.6)
- added J11: Conn_01x01_Socket, Pico_Conn1x1:Pico_01pin, F.Cu at (228.6, 41.0)
- added J12: Conn_01x01_Socket, Pico_Conn1x1:Pico_01pin, F.Cu at (232.7, 41.0)
- added J13: Conn_01x01_Socket, Pico_Conn1x1:Pico_01pin, F.Cu at (236.8, 41.0)
- added J14: Conn_01x01_Socket, Pico_Conn1x1:Pico_01pin, F.Cu at (240.9, 41.0)
- added J15: Conn_01x01_Socket, Pico_Conn1x1:Pico_01pin, F.Cu at (228.6, 47.2)
- added J16: Conn_01x01_Socket, Pico_Conn1x1:Pico_01pin, F.Cu at (232.7, 47.2)
- added J17: Conn_01x01_Socket, Pico_Conn1x1:Pico_01pin, F.Cu at (236.8, 47.2)
- added J18: Conn_01x01_Socket, Pico_Conn1x1:Pico_01pin, F.Cu at (240.9, 47.2)
- added J2: Conn_01x01_Socket, Pico_Conn1x1:Pico_01pin, F.Cu at (232.7, 28.6)
- added J3: Conn_01x01_Socket, Pico_Conn1x1:Pico_01pin, F.Cu at (236.8, 28.6)
- added J4: Conn_01x01_Socket, Pico_Conn1x1:Pico_01pin, F.Cu at (240.9, 28.6)
- added J5: Conn_01x01_Socket, Pico_Conn1x1:Pico_01pin, F.Cu at (228.6, 34.8)
- added J6: Conn_01x01_Socket, Pico_Conn1x1:Pico_01pin, F.Cu at (232.7, 34.8)
- added J7: BM03B-SRSS-TBLFSN, SWD_Con:CONN_BM03B-SRSS-TBLFSN_JST, F.Cu at (235.6, 62.0)
- added J8: Conn_01x01_Socket, Pico_Conn1x1:Pico_01pin, F.Cu at (236.8, 34.8)
- added J9: Conn_01x01_Socket, Pico_Conn1x1:Pico_01pin, F.Cu at (240.9, 34.8)
- added L1: 2.2u, Inductor-2.2uH_SPM10065VT:IND_SPM10065VT-2R2M-D, F.Cu at (248.9, 45.4)
- added LED1: VLMS1500-GS08, LED-Red_VLMS1500-GS08:LED_00-GS08_VIS_RED, F.Cu at (46.3, 157.6)
- added LED2: VLMS1500-GS08, LED-Red_VLMS1500-GS08:LED_00-GS08_VIS_RED, F.Cu at (247.4, 99.5)
- added LED3: VLMS1500-GS08, LED-Red_VLMS1500-GS08:LED_00-GS08_VIS_RED, F.Cu at (247.4, 101.7)
- added LS1: PKLCS1212E20A0-R1, PKLCS1212E20A0-R1:PKLCS1212E20A0-R1, F.Cu at (212.2, 46.4)
- added L_SW1: 10u, Inductor-11.5x10:Inductor_11.5x10, F.Cu at (212.4, 59.1)
- added L_SW2: 15u, Inductor-10.1x10:Inductor_10.1x10, F.Cu at (176.4, 31.4)
- added L_SW3: 15u, Inductor-10.1x10:Inductor_10.1x10, F.Cu at (176.4, 43.3)
- added Q2: 2N7002H6327XTSA2, NMOS_2N7002:PG-SOT23-3-5_INF_MIN, F.Cu at (229.2, 61.4)
- added Q3: 2N7002H6327XTSA2, NMOS_2N7002:PG-SOT23-3-5_INF_MIN, F.Cu at (229.2, 66.3)
- added Q5: BC857CMB_315, PNP_BC857CMB_315:TRANS_PMZB550UNEYL, F.Cu at (40.8, 157.2)
- added Q6: BC857CMB_315, PNP_BC857CMB_315:TRANS_PMZB550UNEYL, F.Cu at (246.9, 92.9)
- added Q7: BC857CMB_315, PNP_BC857CMB_315:TRANS_PMZB550UNEYL, F.Cu at (246.9, 95.2)
- added R1: 100, Capacitor-0603:Capacitor_0603, F.Cu at (27.2, 161.6)
- added R10: 100, Capacitor-0603:Capacitor_0603, F.Cu at (239.9, 92.8)
- added R11: 100, Capacitor-0603:Capacitor_0603, F.Cu at (239.9, 94.9)
- added R12: 3.9k, Capacitor-0603:Capacitor_0603, F.Cu at (239.9, 97.1)
- added R13: 3.9k, Capacitor-0603:Capacitor_0603, F.Cu at (239.9, 99.3)
- added R14: 3.9k, Capacitor-0603:Capacitor_0603, F.Cu at (239.9, 101.4)
- added R15: 1.5k, Capacitor-0603:Capacitor_0603, F.Cu at (239.9, 103.6)
- added R16: 180k, Capacitor-0603:Capacitor_0603, F.Cu at (243.4, 90.6)
- added R17: 10k, Capacitor-0603:Capacitor_0603, F.Cu at (227.4, 53.6)
- added R18: 1k, Resistor-0402:RES_0402, F.Cu at (204.4, 26.6)
- added R18: 10k, Capacitor-0603:Capacitor_0603, F.Cu at (216.8, 89.0)
- added R19: 10k, Capacitor-0603:Capacitor_0603, F.Cu at (216.8, 91.2)
- added R19: 1k, Resistor-0402:RES_0402, F.Cu at (204.4, 28.8)
- added R2: 100, Capacitor-0603:Capacitor_0603, F.Cu at (27.2, 158.4)
- added R20: 0, Resistor-0603:RES_0603, F.Cu at (208.9, 89.7)
- added R21: 0, Resistor-0603:RES_0603, F.Cu at (208.9, 92.3)
- added R23: 100, Capacitor-0603:Capacitor_0603, F.Cu at (227.4, 55.7)
- added R24: 100, Capacitor-0603:Capacitor_0603, F.Cu at (227.4, 57.9)
- added R25: 1k, Capacitor-0603:Capacitor_0603, F.Cu at (230.8, 51.4)
- added R29: 100, Capacitor-0603:Capacitor_0603, F.Cu at (43.2, 157.6)
- added R3: 1k, Capacitor-0603:Capacitor_0603, F.Cu at (227.4, 51.4)
- added R30: 10k, Resistor-0402:RES_0402, F.Cu at (230.8, 53.6)
- added R31: 150, Capacitor-0603:Capacitor_0603, F.Cu at (204.4, 30.9)
- added R32: 100, Capacitor-0603:Capacitor_0603, F.Cu at (243.4, 94.9)
- added R34: 100, Capacitor-0603:Capacitor_0603, F.Cu at (243.4, 97.1)
- added R35: 2k, Capacitor-0603:Capacitor_0603, F.Cu at (230.8, 55.7)
- added R4: 100, Capacitor-0603:Capacitor_0603, F.Cu at (236.5, 94.9)
- added R42: 65, Capacitor-0603:Capacitor_0603, F.Cu at (204.4, 33.1)
- added R43: 2k, Capacitor-0603:Capacitor_0603, F.Cu at (230.8, 57.9)
- added R48: 10k, Resistor-0402:RES_0402, F.Cu at (234.3, 51.4)
- added R5: 100, Capacitor-0603:Capacitor_0603, F.Cu at (236.5, 97.1)
- added R54: 320, Capacitor-0603:Capacitor_0603, F.Cu at (204.4, 35.2)
- added R55: 120, Resistor-0603:RES_0603, F.Cu at (233.3, 65.9)
- added R56: 500, Capacitor-0603:Capacitor_0603, F.Cu at (204.4, 37.4)
- added R57: 2k, Capacitor-0603:Capacitor_0603, F.Cu at (234.3, 53.6)
- added R58: 2k, Capacitor-0603:Capacitor_0603, F.Cu at (234.3, 55.7)
- added R6: 1.5k, Capacitor-0603:Capacitor_0603, F.Cu at (236.5, 99.3)
- added R60: 200k, Capacitor-0603:Capacitor_0603, F.Cu at (119.8, 167.2)
- added R61: 1k, Capacitor-0603:Capacitor_0603, F.Cu at (117.0, 173.0)
- added R62: 1k, Capacitor-0603:Capacitor_0603, F.Cu at (117.0, 169.6)
- added R68: 10k, Capacitor-0603:Capacitor_0603, F.Cu at (234.3, 57.9)
- added R7: 1.5k, Capacitor-0603:Capacitor_0603, F.Cu at (236.5, 101.4)
- added R8: 1.5k, Capacitor-0603:Capacitor_0603, F.Cu at (236.5, 103.6)
- added R9: 1.5k, Capacitor-0603:Capacitor_0603, F.Cu at (239.9, 90.6)
- added REF**: Pico_01pin, Pico_Conn1x1:Pico_01pin, F.Cu at (112.6, 175.0)
- added REF**: Pico_01pin, Pico_Conn1x1:Pico_01pin, F.Cu at (114.8, 175.0)
- added REF**: Pico_01pin, Pico_Conn1x1:Pico_01pin, F.Cu at (102.5, 172.2)
- added REF**: Pico_01pin, Pico_Conn1x1:Pico_01pin, F.Cu at (108.2, 175.0)
- added REF**: Pico_01pin, Pico_Conn1x1:Pico_01pin, F.Cu at (110.4, 175.0)
- added REF**: Pico_01pin, Pico_Conn1x1:Pico_01pin, F.Cu at (126.0, 167.8)
- added REF**: Pico_01pin, Pico_Conn1x1:Pico_01pin, F.Cu at (102.5, 174.4)
- added REF**: Pico_01pin, Pico_Conn1x1:Pico_01pin, F.Cu at (114.0, 162.6)
- added REF**: Pico_01pin, Pico_Conn1x1:Pico_01pin, F.Cu at (116.2, 162.6)
- added REF**: Pico_01pin, Pico_Conn1x1:Pico_01pin, F.Cu at (109.0, 162.6)
- added REF**: Pico_01pin, Pico_Conn1x1:Pico_01pin, F.Cu at (102.5, 170.0)
- added REF**: Pico_01pin, Pico_Conn1x1:Pico_01pin, F.Cu at (126.0, 170.0)
- added REF**: Pico_01pin, Pico_Conn1x1:Pico_01pin, F.Cu at (102.5, 167.8)
- added R_BIAS1: 5, Capacitor-0603:Capacitor_0603, F.Cu at (207.8, 26.6)
- added R_BIAS2: 5, Capacitor-0603:Capacitor_0603, F.Cu at (207.8, 28.8)
- added R_BT1: 50, Capacitor-0603:Capacitor_0603, F.Cu at (207.8, 30.9)
- added R_BT2: 50, Capacitor-0603:Capacitor_0603, F.Cu at (207.8, 33.1)
- added R_BT3: 100, Capacitor-0603:Capacitor_0603, F.Cu at (207.8, 35.2)
- added R_ENB1: 100k, Resistor-0603:RES_0603, F.Cu at (185.1, 62.0)
- added R_ENB2: 63k4, Capacitor-0603:Capacitor_0603, F.Cu at (207.8, 37.4)
- added R_ENB3: 45k3, Capacitor-0603:Capacitor_0603, F.Cu at (211.2, 26.6)
- added R_ENT1: 931k, Resistor-0603:RES_0603, F.Cu at (185.1, 64.5)
- added R_ENT2: 590k, Capacitor-0603:Capacitor_0603, F.Cu at (211.2, 28.8)
- added R_ENT3: 422k, Capacitor-0603:Capacitor_0603, F.Cu at (211.2, 30.9)
- added R_FBB1: 8k66, Resistor-0603:RES_0603, F.Cu at (185.1, 67.1)
- added R_FBB3: 12k7, Resistor-0603:RES_0603, F.Cu at (185.1, 69.6)
- added R_FBB5: 22k1, Resistor-0603:RES_0603, F.Cu at (185.1, 72.2)
- added R_FBT1: 100K, Resistor-0603:RES_0603, F.Cu at (188.8, 62.0)
- added R_FBT2: 100K, Resistor-0603:RES_0603, F.Cu at (188.8, 64.5)
- added R_FBT3: 100K, Resistor-0603:RES_0603, F.Cu at (188.8, 67.1)
- added R_FF1: 1k, Capacitor-0603:Capacitor_0603, F.Cu at (211.2, 33.1)
- added R_PG1: 100K, Resistor-0603:RES_0603, F.Cu at (188.8, 69.6)
- added R_PG2: 100K, Resistor-0603:RES_0603, F.Cu at (188.8, 72.2)
- added R_PG3: 100K, Resistor-0603:RES_0603, F.Cu at (192.4, 62.0)
- added R_RT1: 33k2, Resistor-0603:RES_0603, F.Cu at (192.4, 64.5)
- added R_RT2: 33k2, Resistor-0603:RES_0603, F.Cu at (192.4, 67.1)
- added R_RT3: 33k2, Resistor-0603:RES_0603, F.Cu at (192.4, 69.6)
- added Rsense1: 2.5m, Resistor-0805:RES_0805, F.Cu at (199.6, 63.9)
- added Rsense2: 2.5m, Resistor-0805:RES_0805, F.Cu at (199.6, 68.2)
- added Rsense3: 20m, Resistor-2512:RES_WSLP2512, F.Cu at (200.4, 73.0)
- added S1: TL1017AABF160QG, E-Switch_Small:TL1017AABF160QG, F.Cu at (259.3, 42.4)
- added SW1: D2F-01-D, Switch D2F-01:D2F-01-D_OMR, F.Cu at (250.4, 64.5)
- added TP1: TestPoint, TestPoint:TestPoint_Pad_2.0x2.0mm, F.Cu at (221.7, 27.6)
- added TP2: TestPoint, TestPoint:TestPoint_Pad_2.0x2.0mm, F.Cu at (221.7, 31.6)
- added TP3: TestPoint, TestPoint:TestPoint_Pad_2.0x2.0mm, F.Cu at (221.7, 35.6)
- added U10: STLM20DD9F, STLM20DD9F:UDFN-4L_STM, F.Cu at (231.6, 103.3)
- added U11: MAX31856MUD+T, Thermocouple:21-0066J_14_MXM, F.Cu at (230.2, 89.1)
- added U12: THVD2410VDRCR, THVD2410VDRCR:VSON10_DRC_TEX, F.Cu at (258.3, 48.6)
- added U13: LM61460AASQRJRRQ1, DCDC_LM61460:VQFN-HR14_RJR_TEX, F.Cu at (172.5, 67.6)
- added U14: LM61460AASQRJRRQ1, DCDC_LM61460:VQFN-HR14_RJR_TEX, F.Cu at (172.5, 73.3)
- added U2: MAX31856MUD+T, Thermocouple:21-0066J_14_MXM, F.Cu at (35.2, 159.0)
- added U3: MAX31856MUD+T, Thermocouple:21-0066J_14_MXM, F.Cu at (230.2, 82.3)
- added U4: LM61460AASQRJRRQ1, DCDC_LM61460:VQFN-HR14_RJR_TEX, F.Cu at (172.5, 61.8)
- added U5: SQJA36EP-T1_GE3, SQJA36EP-T1-GE3:PowerPAK_SO-8L_3_VIS, F.Cu at (250.6, 55.6)
- added U6: THVD2410VDRCR, THVD2410VDRCR:VSON10_DRC_TEX, F.Cu at (214.5, 85.6)
- added U8: max11614eee+, MAX11616EEE+T:SOP64P602X175-16N, F.Cu at (108.5, 169.4)
- added U9: SQJA36EP-T1_GE3, SQJA36EP-T1-GE3:PowerPAK_SO-8L_3_VIS, F.Cu at (257.3, 55.6)
Connections:
- U1 pad 10: unconnected-(U1-GP7-Pad10) -> /1~{DRDY} THERMO
- U1 pad 11: unconnected-(U1-GP8-Pad11) -> /SCK SPI
- U1 pad 12: unconnected-(U1-GP9-Pad12) -> /~{CS} THERMO1 SPI
- U1 pad 13: Net-(U1-GND-Pad13) -> GND
- U1 pad 14: unconnected-(U1-GP10-Pad14) -> /MISO SPI
- U1 pad 15: unconnected-(U1-GP11-Pad15) -> /MOSI SPI
- U1 pad 16: unconnected-(U1-GP12-Pad16) -> /1~{FAULT} THERMO
- U1 pad 17: unconnected-(U1-GP13-Pad17) -> /~{CS} THERMO2 SPI
- U1 pad 18: Net-(U1-GND-Pad13) -> GND
- U1 pad 19: unconnected-(U1-GP14-Pad19) -> /Sensor Unit/SCL I2C
- U1 pad 2: unconnected-(U1-GP1-Pad2) -> /~{CS} THERMO3 SPI
- U1 pad 20: unconnected-(U1-GP15-Pad20) -> /Sensor Unit/SDA I2C
- U1 pad 21: unconnected-(U1-GP16-Pad21) -> /2~{DRDY} THERMO
- U1 pad 22: unconnected-(U1-GP17-Pad22) -> /2~{FAULT} THERMO
- U1 pad 23: Net-(U1-GND-Pad13) -> GND
- U1 pad 24: unconnected-(U1-GP18-Pad24) -> /3~{DRDY} THERMO
- U1 pad 25: unconnected-(U1-GP19-Pad25) -> /3~{FAULT} THERMO
- U1 pad 26: unconnected-(U1-GP20-Pad26) -> /Purge Valve Enable
- U1 pad 27: unconnected-(U1-GP21-Pad27) -> /Solenoid Valve Enable
- U1 pad 28: Net-(U1-GND-Pad13) -> GND
- U1 pad 3: Net-(U1-GND-Pad13) -> GND
- U1 pad 30: unconnected-(U1-~{RUN}-Pad30) -> Net-(U1-~{RUN})
- U1 pad 32: unconnected-(U1-GP27-Pad32) -> /Sensor Unit/Temp_Sense
- U1 pad 33: unconnected-(U1-AGND-Pad33) -> GND
- U1 pad 36: unconnected-(U1-3V3_OUT-Pad36) -> +3.3V
- U1 pad 38: Net-(U1-GND-Pad13) -> GND
- U1 pad 4: unconnected-(U1-GP2-Pad4) -> /Servo_IN1 PWM
- U1 pad 40: unconnected-(U1-VBUS-Pad40) -> +5V
- U1 pad 5: unconnected-(U1-GP3-Pad5) -> /Servo_IN2 PWM
- U1 pad 6: unconnected-(U1-GP4-Pad6) -> /READ_RS
- U1 pad 7: unconnected-(U1-GP5-Pad7) -> /WRITE_RS
- U1 pad 8: Net-(U1-GND-Pad13) -> GND
- U1 pad 9: unconnected-(U1-GP6-Pad9) -> /ENABLE_RS
- U1 pad A: Net-(U1-USB_SHIELD-PadA) -> unconnected-(U1-USB_SHIELD-PadA)_3
- U1 pad B: Net-(U1-USB_SHIELD-PadA) -> unconnected-(U1-USB_SHIELD-PadA)
- U1 pad C: Net-(U1-USB_SHIELD-PadA) -> unconnected-(U1-USB_SHIELD-PadA)_1
- U1 pad D: Net-(U1-USB_SHIELD-PadA) -> unconnected-(U1-USB_SHIELD-PadA)_2
- U1 pad D1: unconnected-(U1-SWCLK-PadD1) -> Net-(U1-SWCLK)
- U1 pad D2: Net-(U1-GND-Pad13) -> GND
- U1 pad D3: unconnected-(U1-SWDIO-PadD3) -> Net-(U1-SWDIO)
Routing:
- net +5V: track 0.00 -> 30.5 mm, vias 0 -> 1
- net GND: track 0.00 -> 14.6 mm, vias 0 -> 2
- net GNDA: track 0.00 -> 13.4 mm, vias 0 -> 1
- net +3.3V: track 0.00 -> 13.1 mm
- net /Sensor Unit/Clock I2C: track 0.00 -> 10.9 mm
- net /Sensor Unit/Data I2C: track 0.00 -> 9.88 mm
- net Net-(IC8-EN): track 0.00 -> 9.63 mm, vias 0 -> 2
- net Net-(U2-T+): track 0.00 -> 7.18 mm
- net /Sensor Unit/ADC8 Sense: track 0.00 -> 7.14 mm
- net /Sensor Unit/ADC6 Sense: track 0.00 -> 7.13 mm
- net Net-(U2-T-): track 0.00 -> 7.01 mm
- net /Sensor Unit/ADC7 Sense: track 0.00 -> 6.71 mm
- net /Sensor Unit/SDA I2C: track 0.00 -> 6.27 mm
- net /Sensor Unit/SCL I2C: track 0.00 -> 5.35 mm
- net /THERMO1 DN: track 0.00 -> 4.67 mm
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Other:
- board size 85.4 x 92.2 mm -> 85.4 x 131.4 mm

Commit message: Design da Hydra Breakout (Part 2)
Parts:
- moved C_BT3 298.2 mm to (512.7, 23.4)
- moved C_FF1 298.2 mm to (512.7, 25.6)
- moved C_IN_HFI5 298.2 mm to (516.1, 25.6)
- moved C_IN_HFI6 298.2 mm to (516.1, 27.8)
- moved C_OUT11 298.2 mm to (514.7, 59.1)
- moved C_OUT12 298.2 mm to (514.7, 62.2)
- moved C_OUT13 298.2 mm to (514.7, 65.2)
- moved C_OUT14 298.2 mm to (514.7, 68.3)
- moved C_OUT15 298.2 mm to (487.7, 37.4)
- moved R_BIAS2 298.2 mm to (505.9, 21.3)
- moved R_BT3 298.2 mm to (505.9, 27.7)
- moved R_FBB5 298.2 mm to (483.2, 64.7)
- moved U13 298.2 mm to (470.6, 60.1)
- moved C_BIAS2 298.2 mm to (519.0, 61.4)
- moved C_IN-BLK3 298.2 mm to (499.0, 50.5)
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Routing:
- net +5V: track 30.5 -> 47.0 mm
- net /Power Unit/V3 DP: track 0.00 -> 12.2 mm
- net /Sensor Unit/ADC2 Sense: track 3.44 -> 11.3 mm
- net +8.4V: track 0.00 -> 5.82 mm
- net +12V: track 0.00 -> 5.69 mm
- net /Power Unit/V2 DP: track 0.00 -> 5.08 mm
- net /Sensor Unit/5V_Sense: track 0.00 -> 5.06 mm, vias 0 -> 2
- net /Power Unit/V1 DP: track 0.00 -> 5.01 mm
- net /Sensor Unit/8.4V_Sense: track 0.00 -> 2.84 mm
- net /Sensor Unit/12V_Sense: track 0.00 -> 2.35 mm
- net /Sensor Unit/ADC1 Sense: track 4.09 -> 5.81 mm
Other:
- board size 85.4 x 131.4 mm -> 93.7 x 131.1 mm
- board text added: "ADC to I2C"
- board text added: "Buck Converter 12V"
- board text added: "Buck Converter 5V"
- board text added: "Buck Converter 8.4V"
- board text added: "Current Sensors"
- board text added: "EMI"
- board text added: "RS Transciever"
- board text added: "Temperature Sensor"
- board text added: "Thermo 1"
- board text added: "Thermo 2"
- board text added: "Thermo 3"
- board text added: "Valve Drivers"

Commit message: Design da Hydra Breakout (Part 3)
Parts:
- removed C14: 100n, Capacitor-0603:Capacitor_0603
- removed C39: 10n, Capacitor-0603:Capacitor_0603
- removed LS1: PKLCS1212E20A0-R1, PKLCS1212E20A0-R1:PKLCS1212E20A0-R1
- removed the R19 at (210.2, 161.0)
- removed R34: 100, Capacitor-0603:Capacitor_0603
- removed SW1: D2F-01-D, Switch D2F-01:D2F-01-D_OMR
- removed U11: MAX31856MUD+T, Thermocouple:21-0066J_14_MXM
- removed U12: THVD2410VDRCR, THVD2410VDRCR:VSON10_DRC_TEX
- added C34: 10n, Capacitor-0603:Capacitor_0603, F.Cu at (47.1, 179.1)
- added C7: 100n, Capacitor-0603:Capacitor_0603, F.Cu at (104.1, 169.5)
- added CR4: VLMY1300-GS08, LED-Yellow_VLMY1300-GS08:LEDC1608X100N, F.Cu at (321.4, 56.7)
- added U7: MAX31856MUD+T, Thermocouple:21-0066J_14_MXM, F.Cu at (57.7, 177.3)
- C11: value 100n -> 10n
- C12: value 10n -> 100n
- R18: value 1k -> 10k; footprint Resistor-0402:RES_0402 -> Capacitor-0603:Capacitor_0603
- R30: value 10k -> 100; footprint Resistor-0402:RES_0402 -> Capacitor-0603:Capacitor_0603
- moved R30 167.7 mm to (106.4, 166.1)
- moved C9 52.8 mm to (52.1, 177.5), turned to 180 degrees
- moved Q7 52.1 mm to (63.3, 175.6), turned to 90 degrees
- moved TP1 50.1 mm to (306.8, 51.1)
- moved LED2 48.3 mm to (109.5, 166.1)
- moved LED3 48.2 mm to (68.8, 175.9)
- moved C_VCC1 44.6 mm to (307.9, 44.3), turned to 180 degrees
- moved R42 43.6 mm to (207.1, 76.6)
- moved Q6 40.7 mm to (104.0, 165.7), turned to 90 degrees
- moved C_IN_HFI2 36.9 mm to (310.3, 36.7), turned to 90 degrees
- moved C_IN_HFI1 36.2 mm to (312.1, 51.9), turned to -90 degrees
- moved C_BT1 35.5 mm to (310.3, 39.8), turned to 180 degrees
- moved C_OUT6 33.8 mm to (334.6, 44.7)
- moved D6 32.6 mm to (334.2, 56.2), turned to 180 degrees
- moved C_OUT5 32.0 mm to (338.4, 37.7), turned to 90 degrees
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Connections:
- C11 pad 1: Net-(U11-T+) -> Net-(U7-T-)
- C11 pad 2: Net-(U11-T-) -> GND
- C12 pad 1: Net-(U11-T-) -> GND
- C12 pad 2: GND -> +3.3V
- C9 pad 1: GND -> Net-(U7-T+)
- C9 pad 2: +3.3V -> Net-(U7-T-)
- R10 pad 1: Net-(U11-T+) -> Net-(U7-T+)
- R10 pad 2: /THERMO2 DP -> /THERMO3 DP
- R11 pad 1: Net-(U11-T-) -> Net-(U7-T-)
- R11 pad 2: /THERMO2 DN -> /THERMO3 DN
- R18 pad 1: Net-(IC1-B) -> +3.3V
- R18 pad 2: /Power Unit/Buzzer -> /READ_RS
- R30 pad 1: /ENABLE_RS -> Net-(Q6-Pad2)
- R30 pad 2: GND -> Net-(LED2-Pad1)
- R32 pad 1: Net-(Q6-Pad2) -> Net-(Q7-Pad2)
- R32 pad 2: Net-(LED2-Pad1) -> Net-(LED3-Pad1)
- R4 pad 2: /THERMO3 DN -> /THERMO2 DP
- R5 pad 2: /THERMO3 DP -> /THERMO2 DN
- REF** pad 1: (no net) -> GND
- U3 pad 13: /3~{FAULT} THERMO -> /2~{FAULT} THERMO
- U3 pad 2: /THERMO3 DP -> /THERMO2 DN
- U3 pad 7: /3~{DRDY} THERMO -> /2~{DRDY} THERMO
- U3 pad 9: /~{CS} THERMO3 SPI -> /~{CS} THERMO2 SPI
Routing:
- net Net-(C_OUT1-Pad1): track 0.00 -> 46.3 mm
- net +3.3V: track 13.1 -> 48.2 mm
- net GND: track 14.6 -> 34.3 mm, vias 2 -> 3
- net Net-(U3-T+): track 0.00 -> 14.4 mm
- net Net-(U14-FB): track 0.00 -> 14.2 mm
- net Net-(U3-T-): track 0.00 -> 14.0 mm
- net /Power Unit/DC.DC1 VCC: track 0.00 -> 11.6 mm
- net Net-(U14-SW): track 0.00 -> 9.51 mm
- net /THERMO2 DN: track 0.00 -> 9.33 mm
- net /Power Unit/V1 DP: track 5.01 -> 12.5 mm
- net Net-(U7-T+): track 0.00 -> 7.18 mm
- net VBUS: track 0.00 -> 7.01 mm
- net Net-(U7-T-): track 0.00 -> 7.01 mm
- net GNDA: track 13.4 -> 18.9 mm, vias 1 -> 2
- net Net-(U14-EN/SYNC): track 0.00 -> 5.20 mm
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
Commit message: Design da Hydra Breakout (Part 4)
Parts:
- removed IC1: BC846BLT1G, BJT NPN:SOT96P237X111-3N
- removed the R18 at (218.7, 158.2)
- added ?: , , F.Cu at (56.3, 189.4)
- added ?: , , F.Cu at (98.4, 184.0)
- added CR1: VLMY1300-GS08, LED-Yellow_VLMY1300-GS08:LEDC1608X100N, F.Cu at (126.0, 77.4)
- added CR2: VLMY1300-GS08, LED-Yellow_VLMY1300-GS08:LEDC1608X100N, F.Cu at (475.3, 51.0)
- added CR3: VLMY1300-GS08, LED-Yellow_VLMY1300-GS08:LEDC1608X100N, F.Cu at (390.3, 43.7)
- added REF**: Pico_01pin, Pico_Conn1x1:Pico_01pin, F.Cu at (62.5, 187.8)
- added REF**: Pico_01pin, Pico_Conn1x1:Pico_01pin, F.Cu at (108.8, 182.4)
- added REF**: Pico_01pin, Pico_Conn1x1:Pico_01pin, F.Cu at (51.9, 163.4)
- added REF**: Pico_01pin, Pico_Conn1x1:Pico_01pin, F.Cu at (217.3, 156.8)
- added REF**: Pico_01pin, Pico_Conn1x1:Pico_01pin, F.Cu at (71.8, 187.8)
- added REF**: Pico_01pin, Pico_Conn1x1:Pico_01pin, F.Cu at (85.5, 181.4)
- added REF**: Pico_01pin, Pico_Conn1x1:Pico_01pin, F.Cu at (66.7, 187.8)
- added REF**: Pico_01pin, Pico_Conn1x1:Pico_01pin, F.Cu at (226.8, 151.8)
- added REF**: Pico_01pin, Pico_Conn1x1:Pico_01pin, F.Cu at (49.3, 163.4)
- added REF**: Pico_01pin, Pico_Conn1x1:Pico_01pin, F.Cu at (116.8, 176.6)
- added REF**: Pico_01pin, Pico_Conn1x1:Pico_01pin, F.Cu at (74.7, 182.0)
- added REF**: Pico_01pin, Pico_Conn1x1:Pico_01pin, F.Cu at (116.5, 182.4)
- added REF**: Pico_01pin, Pico_Conn1x1:Pico_01pin, F.Cu at (20.9, 157.6)
- added REF**: Pico_01pin, Pico_Conn1x1:Pico_01pin, F.Cu at (69.3, 187.8)
- added REF**: Pico_01pin, Pico_Conn1x1:Pico_01pin, F.Cu at (231.3, 153.8)
- added REF**: Pico_01pin, Pico_Conn1x1:Pico_01pin, F.Cu at (224.4, 151.8)
- added REF**: Pico_01pin, Pico_Conn1x1:Pico_01pin, F.Cu at (40.8, 155.2)
- added REF**: Pico_01pin, Pico_Conn1x1:Pico_01pin, F.Cu at (95.9, 174.2)
- added REF**: Pico_01pin, Pico_Conn1x1:Pico_01pin, F.Cu at (20.9, 162.4)
- added REF**: Pico_01pin, Pico_Conn1x1:Pico_01pin, F.Cu at (46.8, 163.4)
- added REF**: Pico_01pin, Pico_Conn1x1:Pico_01pin, F.Cu at (40.0, 163.4)
- added REF**: Pico_01pin, Pico_Conn1x1:Pico_01pin, F.Cu at (74.4, 187.8)
- added REF**: Pico_01pin, Pico_Conn1x1:Pico_01pin, F.Cu at (85.5, 176.6)
- added REF**: Pico_01pin, Pico_Conn1x1:Pico_01pin, F.Cu at (104.6, 182.4)
- added REF**: Pico_01pin, Pico_Conn1x1:Pico_01pin, F.Cu at (217.3, 154.6)
- added REF**: Pico_01pin, Pico_Conn1x1:Pico_01pin, F.Cu at (44.2, 163.4)
- added REF**: Pico_01pin, Pico_Conn1x1:Pico_01pin, F.Cu at (217.3, 158.9)
- added REF**: Pico_01pin, Pico_Conn1x1:Pico_01pin, F.Cu at (53.8, 179.6)
- added REF**: Pico_01pin, Pico_Conn1x1:Pico_01pin, F.Cu at (111.4, 182.4)
- added REF**: Pico_01pin, Pico_Conn1x1:Pico_01pin, F.Cu at (52.2, 157.6)
- added REF**: Pico_01pin, Pico_Conn1x1:Pico_01pin, F.Cu at (43.4, 186.8)
- added REF**: Pico_01pin, Pico_Conn1x1:Pico_01pin, F.Cu at (43.4, 182.0)
- added REF**: Pico_01pin, Pico_Conn1x1:Pico_01pin, F.Cu at (231.3, 159.5)
- added REF**: Pico_01pin, Pico_Conn1x1:Pico_01pin, F.Cu at (158.3, 171.2)
- added REF**: Pico_01pin, Pico_Conn1x1:Pico_01pin, F.Cu at (33.8, 163.4)
- added REF**: Pico_01pin, Pico_Conn1x1:Pico_01pin, F.Cu at (113.9, 182.4)
- added REF**: Pico_01pin, Pico_Conn1x1:Pico_01pin, F.Cu at (63.3, 179.6)
- added REF**: Pico_01pin, Pico_Conn1x1:Pico_01pin, F.Cu at (98.4, 182.4)
- added REF**: Pico_01pin, Pico_Conn1x1:Pico_01pin, F.Cu at (56.3, 187.8)
- added REF**: Pico_01pin, Pico_Conn1x1:Pico_01pin, B.Cu at (222.0, 151.8)
- added REF**: Pico_01pin, Pico_Conn1x1:Pico_01pin, F.Cu at (105.4, 174.2)
- added REF**: Pico_01pin, Pico_Conn1x1:Pico_01pin, F.Cu at (31.3, 155.2)
- moved Q3 174.8 mm to (343.5, 114.8)
- moved Q2 168.7 mm to (338.1, 114.8)
- moved R57 168.4 mm to (343.4, 111.0), turned to -90 degrees
- moved R58 168.0 mm to (343.5, 117.8)
- moved R35 166.8 mm to (338.1, 111.1), turned to -90 degrees
- moved R43 166.2 mm to (338.1, 117.8)
- moved R68 150.6 mm to (326.7, 127.5), turned to 180 degrees
- moved R17 145.3 mm to (314.7, 127.7), turned to 180 degrees
- moved D7 142.4 mm to (325.2, 109.8)
- moved D4 140.2 mm to (313.3, 109.8)
- moved U9 133.2 mm to (325.2, 121.7)
- moved U5 128.0 mm to (313.3, 121.7)
- moved R42 77.4 mm to (129.7, 77.4), turned to 180 degrees
- moved C_VCC2 74.9 mm to (376.5, 27.5), turned to 180 degrees
- moved C_VCC3 69.1 mm to (460.5, 34.7), turned to 180 degrees
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Routing:
- net GNDA: track 18.9 -> 72.4 mm, vias 2 -> 15
- net /MOSI SPI: track 0.00 -> 50.6 mm
- net Net-(C_OUT10-Pad1): track 0.00 -> 44.1 mm
- net /MISO SPI: track 0.00 -> 42.1 mm
- net GND: track 34.3 -> 70.7 mm, vias 3 -> 23
- net /SCK SPI: track 0.00 -> 33.6 mm
- net +5V: track 47.0 -> 79.6 mm, vias 1 -> 2
- net Net-(U4-BIAS): track 0.00 -> 15.2 mm
- net VDC: track 0.00 -> 14.9 mm
- net Net-(U13-FB): track 0.00 -> 14.5 mm
- net /Power Unit/DC.DC2 VCC: track 0.00 -> 12.0 mm
- net Net-(U4-FB): track 0.00 -> 11.8 mm
- net Net-(U4-SW): track 0.00 -> 10.8 mm
- net /~{CS} THERMO2 SPI: track 0.00 -> 8.51 mm
- net /~{CS} THERMO1 SPI: track 0.00 -> 8.51 mm
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- added copper zone on F.Cu, net +3.3V
- added copper zone on B.Cu, net GND
- added copper zone on F.Cu, net GND
- added copper zone on F.Cu, net GNDA
Other:
- board size 93.7 x 131.1 mm -> 480.7 x 176.7 mm
