File: Boards/Rocket Systems/Elytra/Elytra.kicad_sch (KiCad schematic)
At the start: 115 parts, among them J1 2200981271, J2 XT60PW-F, J3 XT60PW-M, J4 XT60PW-F, J5 XT60PW-M, J6 XT60PW-F, J7 XT60PW-M, J8 XT60PW-F, J9 XT60PW-M, K1 G3VM-31DR_TR05_, K2 G3VM-31DR_TR05_, K3 G3VM-31DR_TR05_, Q1 FJB102TM, Q2 FJB102TM, Q3 FJB102TM, Q4 FJB102TM, U13 LM61460AASQRJRRQ1, U4 MPQ3431AGL-AEC1-Z

Commit message: update pcb elytra
update a pcb elytra + modificacao footprint conversor
Parts:
- removed J3, J5, J7, J9: XT60PW-M, Connector_AMASS:AMASS_XT60-M_1x02_P7.20mm_Vertical, symbol XT60PW-M:XT60PW-M
Connections:
- net VBAT1 is gone; now on net VBAT: J2.1
- net KEY_OUT: now also J8.2
- net VDC: now also J8.1
Other:
- moved on the sheet: J2, J4, J8

Commit message: mudancas pcb elytra
elytr
Parts:
- DSUB1: footprint (none) -> HDL15-SL-B:HDL15-SL-B
Changed lines of the file:
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@@
 		(fields_autoplaced yes)
 		(property "Reference" "R10"
-			(at 422.275 258.4449 0)
+			(at 842.01 518.1599 0)
 			(effects
 				(font
@@
 		)
 		(property "Value" "1.2"
-			(at 422.275 260.9849 0)
+			(at 842.01 520.6999 0)
 			(effects
 				(font
@@
 		)
 		(property "Footprint" "RES_SM_7W_TEC"
-			(at 417.957 259.715 90)
+			(at 837.692 519.43 90)
 			(effects
 				(font
@@
 		)
 		(property "Datasheet" "~"
-			(at 419.735 259.715 0)
+			(at 839.47 519.43 0)
 			(effects
 				(font
@@
 		)
 		(property "Description" "Resistor"
-			(at 419.735 259.715 0)
+			(at 839.47 519.43 0)
 			(effects
 				(font
@@
 			)
 		)
-		(property "Footprint" ""
+		(property "Footprint" "HDL15-SL-B:HDL15-SL-B"
 			(at 49.53 184.15 0)
 			(effects
