File: Boards/Rocket Systems/HYDRA/IO Connectors.kicad_sch (KiCad schematic)
At the start: 14 parts, among them J3 XT30UPB-F, J4 XT30UPB-F, J5 5024430270, J6 5024430570, J7 5024430270, J8 XT30UPB-F, U31 ThermoConnector, U32 ThermoConnector, U33 ThermoConnector

Commit message: Elytra Update and HYDRA Update
Connections:
- net QuickDisco N2 OUT: no longer DSUB1.6
- net QuickDisco N2 PWR: no longer DSUB1.7
- net QuickDisco N2O OUT: no longer DSUB1.4
- net QuickDisco N2O PWR: no longer DSUB1.5
- net ACT_N2 OUT: no longer names the net of DSUB1.14
- net ACT_N2 PWR: no longer names the net of DSUB1.15
- net ACT_N2O OUT: no longer names the net of DSUB1.10
- net ACT_N2O PWR: no longer names the net of DSUB1.11
- net Extra Valve OUT: no longer names the net of DSUB1.2
- net Extra Valve PWR: no longer names the net of DSUB1.3
- net VENT_N2 OUT: no longer names the net of DSUB1.12
- net VENT_N2 PWR: no longer names the net of DSUB1.13
- net VENT_N2O OUT: no longer names the net of DSUB1.8
- net VENT_N2O PWR: no longer names the net of DSUB1.9
Other:
- moved on the sheet: H1, H2, H3, H4
Changed lines of the file:
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@@
 	(text "Thermocouples - 3 Differential Connections (6) - INPUTs -> To Type-K probes\nRS485 Transceiver - 1 Differential Connection (2) - INPUT/OUTPUT \nPurge Valve Drive - 1 Connection - INPUT\nMain Valve PWM Signal Control - 1 Connection - OUTPUT\nPressure Sensor Signal Input - 1 Connection - INPUT\n8.4V Power Line - 1 Connection - Power Input -> Servo Motors\n12V Power Line - 1 Connection - Power Input -> Pressure Sensor & Valve Driver\nBattery Power Supply - 1 Connection - Power Input\nBattery Ground - 1 Connection - Power Output"
 		(exclude_from_sim no)
-		(at 137.795 83.185 0)
+		(at 43.18 142.24 0)
 		(effects
 			(font
@@
 		)
 	)
+	(hierarchical_label "QuickDisco N2O PWR"
+		(shape input)
+		(at 42.545 27.305 0)
+		(effects
+			(font
+				(size 1.27 1.27)
+			)
+			(justify left)
+		)
+	)
 	(hierarchical_label "THERMO3 DN"
 		(shape output)
@@
 		)
 	)
-	(hierarchical_label "QuickDisco N2O PWR"
-		(shape input)
-		(at 55.245 67.31 0)
-		(effects
-			(font
-				(size 1.27 1.27)
-			)
-			(justify left)
-		)
-	)
 	(hierarchical_label "PRESSURE2 Sense"
 		(shape output)
@@
 		)
 	)
-	(hierarchical_label "QuickDisco N2O OUT"
-		(shape output)
-		(at 55.245 69.85 0)
-		(effects
-			(font
-				(size 1.27 1.27)
-			)
-			(justify left)
-		)
-	)
 	(hierarchical_label "SERVO OUT"
 		(shape input)
@@
 		)
 	)
-	(hierarchical_label "Extra Valve PWR"
+	(hierarchical_label "QuickDisco N2 PWR"
 		(shape input)
-		(at 55.245 72.39 0)
-		(effects
-			(font
-				(size 1.27 1.27)
-			)
-			(justify left)
-		)
-	)
-	(hierarchical_label "ACT_N2O PWR"
-		(shape input)
-		(at 55.245 52.07 0)
-		(effects
-			(font
-				(size 1.27 1.27)
-			)
-			(justify left)
-		)
-	)
-	(hierarchical_label "ACT_N2 OUT"
+		(at 42.545 22.225 0)
+		(effects
+			(font
+				(size 1.27 1.27)
+			)
+			(justify left)
+		)
+	)
+	(hierarchical_label "QuickDisco N2O OUT"
 		(shape output)
-		(at 55.245 44.45 0)
-		(effects
-			(font
-				(size 1.27 1.27)
-			)
-			(justify left)
-		)
-	)
-	(hierarchical_label "QuickDisco N2 OUT"
-		(shape output)
-		(at 55.245 64.77 0)
+		(at 42.545 29.845 0)
 		(effects
 			(font
@@
 		)
 	)
+	(hierarchical_label "QuickDisco N2 OUT"
+		(shape output)
+		(at 42.545 24.765 0)
+		(effects
+			(font
+				(size 1.27 1.27)
+			)
+			(justify left)
+		)
+	)
 	(hierarchical_label "SERVO PWR"
 		(shape input)
@@
 		)
 	)
-	(hierarchical_label "VENT_N2O PWR"
-		(shape input)
-		(at 55.245 57.15 0)
-		(effects
-			(font
-				(size 1.27 1.27)
-			)
-			(justify left)
-		)
-	)
 	(hierarchical_label "THERMO3 DP"
 		(shape output)
@@
 		)
 	)
-	(hierarchical_label "VENT_N2 PWR"
-		(shape input)
-		(at 55.245 46.99 0)
-		(effects
-			(font
-				(size 1.27 1.27)
-			)
-			(justify left)
-		)
-	)
-	(hierarchical_label "Extra Valve OUT"
-		(shape output)
-		(at 55.245 74.93 0)
-		(effects
-			(font
-				(size 1.27 1.27)
-			)
-			(justify left)
-		)
-	)
-	(hierarchical_label "VENT_N2 OUT"
-		(shape output)
-		(at 55.245 49.53 0)
-		(effects
-			(font
-				(size 1.27 1.27)
-			)
-			(justify left)
-		)
-	)
 	(hierarchical_label "CAM IN"
 		(shape input)
@@
 		)
 	)
-	(hierarchical_label "ACT_N2O OUT"
-		(shape output)
-		(at 55.245 54.61 0)
-		(effects
-			(font
-				(size 1.27 1.27)
-			)
-			(justify left)
-		)
-	)
-	(hierarchical_label "VENT_N2O OUT"
-		(shape output)
-		(at 55.245 59.69 0)
-		(effects
-			(font
-				(size 1.27 1.27)
-			)
-			(justify left)
-		)
-	)
-	(hierarchical_label "ACT_N2 PWR"
-		(shape input)
-		(at 55.245 41.91 0)
-		(effects
-			(font
-				(size 1.27 1.27)
-			)
-			(justify left)
-		)
-	)
-	(hierarchical_label "QuickDisco N2 PWR"
-		(shape input)
-		(at 55.245 62.23 0)
-		(effects
-			(font
-				(size 1.27 1.27)
-			)
-			(justify left)
-		)
-	)
 	(hierarchical_label "THERMO1 DN"
 		(shape output)
@@
 	(symbol
 		(lib_id "Mechanical:MountingHole")
-		(at 46.99 111.125 0)
+		(at 46.355 107.315 0)
 		(unit 1)
 		(exclude_from_sim no)
@@
 		(fields_autoplaced yes)
 		(property "Reference" "H1"
-			(at 49.53 109.8549 0)
+			(at 48.895 106.0449 0)
 			(effects
 				(font
@@
 		)
 		(property "Value" "MountingHole"
-			(at 49.53 112.3949 0)
+			(at 48.895 108.5849 0)
 			(effects
 				(font
@@
 		)
 		(property "Footprint" "MountingHole:MountingHole_3.2mm_M3_ISO7380"
-			(at 46.99 111.125 0)
+			(at 46.355 107.315 0)
 			(effects
 				(font
@@
 		)
 		(property "Datasheet" "~"
-			(at 46.99 111.125 0)
+			(at 46.355 107.315 0)
 			(effects
 				(font
@@
 		)
 		(property "Description" "Mounting Hole without connection"
-			(at 46.99 111.125 0)
+			(at 46.355 107.315 0)
 			(effects
 				(font
@@
 	(symbol
 		(lib_id "Mechanical:MountingHole")
-		(at 68.58 125.095 0)
+		(at 67.945 121.285 0)
 		(unit 1)
 		(exclude_from_sim no)
@@
 		(fields_autoplaced yes)
 		(property "Reference" "H4"
-			(at 71.12 123.8249 0)
+			(at 70.485 120.0149 0)
 			(effects
 				(font
@@
 		)
 		(property "Value" "MountingHole"
-			(at 71.12 126.3649 0)
+			(at 70.485 122.5549 0)
 			(effects
 				(font
@@
 		)
 		(property "Footprint" "MountingHole:MountingHole_3.2mm_M3_ISO7380"
-			(at 68.58 125.095 0)
+			(at 67.945 121.285 0)
 			(effects
 				(font
@@
 		)
 		(property "Datasheet" "~"
-			(at 68.58 125.095 0)
+			(at 67.945 121.285 0)
 			(effects
 				(font
@@
 		)
 		(property "Description" "Mounting Hole without connection"
-			(at 68.58 125.095 0)
+			(at 67.945 121.285 0)
 			(effects
 				(font
@@
 	(symbol
 		(lib_id "power:Earth")
-		(at 68.58 114.935 0)
+		(at 67.945 111.125 0)
 		(unit 1)
 		(exclude_from_sim no)
@@
 		(dnp no)
 		(property "Reference" "#PWR079"
-			(at 68.58 121.285 0)
+			(at 67.945 117.475 0)
 			(effects
 				(font
@@
 		)
 		(property "Value" "AGND"
-			(at 68.58 118.745 0)
+			(at 67.945 114.935 0)
 			(effects
 				(font
@@
 		)
 		(property "Footprint" ""
-			(at 68.58 114.935 0)
+			(at 67.945 111.125 0)
 			(effects
 				(font
@@
 		)
 		(property "Datasheet" "~"
-			(at 68.58 114.935 0)
+			(at 67.945 111.125 0)
 			(effects
 				(font
@@
 		)
 		(property "Description" "Power symbol creates a global label with name \"Earth\""
-			(at 68.58 114.935 0)
+			(at 67.945 111.125 0)
 			(effects
 				(font
@@
 	(symbol
 		(lib_id "Mechanical:MountingHole_Pad")
-		(at 68.58 112.395 0)
+		(at 67.945 108.585 0)
 		(unit 1)
 		(exclude_from_sim no)
@@
 		(fields_autoplaced yes)
 		(property "Reference" "H2"
-			(at 71.755 109.8549 0)
+			(at 71.12 106.0449 0)
 			(effects
 				(font
@@
 		)
 		(property "Value" "MountingHole_Pad"
-			(at 71.755 112.3949 0)
+			(at 71.12 108.5849 0)
 			(effects
 				(font
@@
 		)
 		(property "Footprint" "MountingHole:MountingHole_3.2mm_M3_ISO7380_Pad"
-			(at 68.58 112.395 0)
+			(at 67.945 108.585 0)
 			(effects
 				(font
@@
 		)
 		(property "Datasheet" "~"
-			(at 68.58 112.395 0)
+			(at 67.945 108.585 0)
 			(effects
 				(font
@@
 		)
 		(property "Description" "Mounting Hole with connection"
-			(at 68.58 112.395 0)
+			(at 67.945 108.585 0)
 			(effects
 				(font
@@
 	(symbol
 		(lib_id "Mechanical:MountingHole")
-		(at 46.99 124.46 0)
+		(at 46.355 120.65 0)
 		(unit 1)
 		(exclude_from_sim no)
@@
 		(fields_autoplaced yes)
 		(property "Reference" "H3"
-			(at 49.53 123.1899 0)
+			(at 48.895 119.3799 0)
 			(effects
 				(font
@@
 		)
 		(property "Value" "MountingHole"
-			(at 49.53 125.7299 0)
+			(at 48.895 121.9199 0)
 			(effects
 				(font
@@
 		)
 		(property "Footprint" "MountingHole:MountingHole_3.2mm_M3_ISO7380"
-			(at 46.99 124.46 0)
+			(at 46.355 120.65 0)
 			(effects
 				(font
@@
 		)
 		(property "Datasheet" "~"
-			(at 46.99 124.46 0)
+			(at 46.355 120.65 0)
 			(effects
 				(font
@@
 		)
 		(property "Description" "Mounting Hole without connection"
-			(at 46.99 124.46 0)
-			(effects
-				(font
+			(at 46.355 120.65 0)
+			(effects
+				(font

Commit message: HYDRA Update - footprints and schematics
Parts:
- removed DSUB1: ~, HDL15-SL-B:HDL15-SL-B, symbol HDL15-SL-B:HDL15-SL-B
- removed J4: XT30UPB-F, XT30UPB-F:XT30UPBF, symbol XT30UPB-F:XT30UPB-F
- removed J7: 5024430270, CONN_502443-02xx_MOL, symbol 5024430270:5024430270
Other:
- moved on the sheet: H1, H2, H3, H4, J3, J5, J6, J8, U31, U32, U33

Commit message: HYDRA placemenent
Parts:
- removed J3: XT30UPB-F, XT30UPB-F:XT30UPBF, symbol XT30UPB-F:XT30UPB-F
- added J10: 1723103103, 1723103103:MOLEX_1723103103, symbol 1723103103:1723103103
- added J3, J4: 26013116, 26013116:MOLEX_26013116, symbol 26013116:26013116
- added J7: 1723163206, 1723163206:MOLEX_1723163206, symbol 1723163206:1723163206
- added J8: 1723163304, 1723163304:MOLEX_1723163304, symbol 1723163304:1723163304
- added J9: 1723103102, 1723103102:CONN02_1723103102_MOL, symbol 1723103102:1723103102
- J11: renamed from J6; footprint CONN_502443-05xx_MOL -> 5024430570:CONN_502443-05xx_MOL
- J6: renamed from J5; footprint CONN_502443-02xx_MOL -> 5024430270:CONN_502443-02xx_MOL
- renumbered H3 to H2, H2 to H3, J8 to J5
Connections:
- net AGND: now also J6.3 (MP1), J6.4 (MP2)
- net CAM IN: now also J9.1
- net CAM OUT: now also J9.2
- net GND: now also J11.6, J11.7, J10.S1 (SHIELD1), J10.S2 (SHIELD2), J7.S1 (SHIELD1), J7.S2 (SHIELD2), J8.S1 (SHIELD1), J8.S2 (SHIELD2), J9.3 (SHIELD1), J9.4 (SHIELD2)
- net PWM HV: now also J10.2
- net QuickDisco N2 OUT: now also J8.1
- net QuickDisco N2 PWR: now also J8.3
- net QuickDisco N2O OUT: now also J8.2
- net QuickDisco N2O PWR: now also J8.4
- net RS_DN: now also J6.2; no longer J6.1
- net RS_DP: now also J6.1; no longer J6.2
- net SBVALVE_1_COM: now also J4.4
- net SBVALVE_1_T2: now also J4.6
- net SBVALVE_1_T3: now also J4.5
- net SBVALVE_2_COM: now also J3.4
- net SBVALVE_2_T2: now also J3.6
- net SBVALVE_2_T3: now also J3.5
- net SOL_VALVE_1 OUT: now also J7.1
- net SOL_VALVE_1 PWR: now also J7.4
- net SOL_VALVE_2 OUT: now also J7.2
- net SOL_VALVE_2 PWR: now also J7.5
- net SOL_VALVE_3 OUT: now also J7.3
- net SOL_VALVE_3 PWR: now also J7.6
- net STVALVE_1_CLOSED: now also J4.2
- net STVALVE_1_GND: now also J4.1
- net STVALVE_1_OPEN: now also J4.3
- net STVALVE_2_CLOSED: now also J3.2
- net STVALVE_2_GND: now also J3.1
- net STVALVE_2_OPEN: now also J3.3
- new net SERVOGND: J10.3
- new net SERVOPWR: J10.1
Other:
- note added: "CAN-BUS 1x2x0.22m² 24AWG"
- note added: "Igus Chainflex CFTHERMO 2x0.23mm² 24AWG"
- note added: "Igus Chainflex M12x1 4x0.34m² 22AWG"
- note added: "JZ-500 2x1.5mm² 16AWG"
- note added: "TRONIC-CY (LiY-CY) 3x0.5mm² 20AWG"
- note removed: "Thermocouples - 3 Differential Connections (6) - INPUTs -> To Type-K probes RS485 Transceiver - 1 Differential Connection (2) - INPUT/OUTPUT Purge Valve Drive - 1 Connection - INPUT Main Valve PWM Signal Control - 1 Connection - OUTPUT Pressure Sensor Signal Input - 1 Connection - INPUT 8.4V Power Line - 1 Connection - Power Input -> Servo Motors 12V Power Line - 1 Connection - Power Input -> Pre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"
- company: (none) -> Porto Space Team
- title: (none) -> Hydraulic Regulation & Actuation system
- moved on the sheet: H1, H2, H3, H4, J5, U31, U32, U33
