File: Boards/Rocket Systems/HYDRA/HYDRA.kicad_sch (KiCad schematic)
At the start: 22 parts, among them IC1 NSVT30010MXV6T1G, IC2 BC846BLT1G, U1 VLMKG3400-GS08

Commit message: HYDRA schematic pinout update pt1
Other:
- sheet IO Connectors ports: added ACT_N2 OUT, ACT_N2 PWR, ACT_N2O OUT, ACT_N2O PWR, CAM IN, CAM OUT, Extra Valve OUT, Extra Valve PWR, PRESSURE1 Sense, PRESSURE2 Sense, PRESSURE3 Sense, QuickDisco N2 OUT, QuickDisco N2 PWR, QuickDisco N2O OUT, QuickDisco N2O PWR, RS_DN, RS_DP, SERVO OUT, SERVO PWR, Servo_OUT1 PWM, Servo_OUT2 PWM, THERMO1 DN, THERMO1 DP, THERMO2 DN, THERMO2 DP, THERMO3 DN, THERMO3 DP, VENT_N2 OUT, VENT_N2 PWR, VENT_N2O OUT, VENT_N2O PWR; removed none

Commit message: HYDRA schematic update, ELYTRA FULL REWORK
Other:
- note removed: "TODO: Escolher connectores ADC FAULT DESIGN ATUALIZAR PROJECT SYMBOLS LIB ADICIONAR FOOTPRINTS CORRER ERC -- LAYOUT"
- moved on the sheet: CR1, CR2, CR3, CR4, CR5, CR6, IC1, IC2, LS1, R1, R10, R11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

Commit message: Elytra Update and HYDRA Update
Other:
- sheet Actuation Unit ports: added SOL_VALVE_1, SOL_VALVE_1 DUTY, SOL_VALVE_1 OUT, SOL_VALVE_1 PWR, SOL_VALVE_1 ~{FAULT}, SOL_VALVE_2, SOL_VALVE_2 DUTY, SOL_VALVE_2 OUT, SOL_VALVE_2 PWR, SOL_VALVE_2 ~{FAULT}, SOL_VALVE_3, SOL_VALVE_3 DUTY, SOL_VALVE_3 OUT, SOL_VALVE_3 PWR, SOL_VALVE_3 ~{FAULT}, STVALVE_1, STVALVE_1_CLOSED, STVALVE_1_GND, STVALVE_1_OPEN, STVALVE_1_PWR, STVALVE_2, STVALVE_2_CLOSED, STVALVE_2_GND, STVALVE_2_OPEN, STVALVE_2_PWR; removed ACT_N2 DUTY, ACT_N2 OUT, ACT_N2 PWR, ACT_N2 Valve, ACT_N2O DUTY, ACT_N2O OUT, ACT_N2O PWR, ACT_N2O Valve, Extra Valve, Servo_IN1 PWM, Servo_IN2 PWM, Servo_OUT1 PWM, Servo_OUT2 PWM, VENT_N2 DUTY, VENT_N2 OUT, VENT_N2 PWR, VENT_N2 Valve, VENT_N2O DUTY, VENT_N2O OUT, VENT_N2O PWR, VENT_N2O Valve, ~{ACT_N2 FAULT}, ~{ACT_N2O FAULT}, ~{VENT_N2 FAULT}, ~{VENT_N2O FAULT}
- sheet IO Connectors ports: added none; removed ACT_N2 OUT, ACT_N2 PWR, ACT_N2O OUT, ACT_N2O PWR, Servo_OUT1 PWM, Servo_OUT2 PWM, VENT_N2 OUT, VENT_N2 PWR, VENT_N2O OUT, VENT_N2O PWR
- sheet RP2040 Standard ports: added none; removed GP2/PWM1 A, GP3/PWM1 B
- sheet Sensor Unit ports: added SBVALVE_1_COM, SBVALVE_1_T2, SBVALVE_1_T3, SBVALVE_2_COM, SBVALVE_2_T2, SBVALVE_2_T3, SOL_VALVE_1 ~{FAULT}, SOL_VALVE_2 ~{FAULT}, SOL_VALVE_3 ~{FAULT}; removed DAC_OUT4, ~{ACT_N2 FAULT}, ~{ACT_N2O FAULT}, ~{VENT_N2 FAULT}, ~{VENT_N2O FAULT}
- note added: "TODO: REVER ACTUATION UNIT - VALVE ACTUATER DRIVERS REVER FOOTPRINTS E COMPONENTES DAS PCBs TODAS CORRIGIR ERC"

Commit message: HYDRA Update - footprints and schematics
Parts:
- removed CR2: VLMY1300-GS08, LED-Yellow_VLMY1300-GS08:LED_VISHAY_VLMX1300_VIS, symbol VLMY1300-GS08:VLMY1300-GS08
- removed IC2: BC846BLT1G, BJT NPN:SOT96P237X111-3N, symbol BC846BLT1G:BC846BLT1G
- removed LS1: PKMCS0909E4000-R1, PKMCS0909E4000-R1:SPKR_PKMCS0909E4000-R1, symbol PKMCS0909E4000-R1:PKMCS0909E4000-R1
- removed R11, R12: 1k, Resistor-0402:RES_0402, symbol Device:R
- removed R2: 65, Resistor-0402:RES_0402, symbol Device:R
Other:
- sheet Actuation Unit ports: added PWM HV, PWM LV; removed Extra Valve OUT, Extra Valve PWR, STVALVE_1_PWR, STVALVE_2_PWR
- sheet IO Connectors ports: added PWM HV, SBVALVE_1_COM, SBVALVE_1_T2, SBVALVE_1_T3, SBVALVE_2_COM, SBVALVE_2_T2, SBVALVE_2_T3, SOL_VALVE_1 OUT, SOL_VALVE_1 PWR, SOL_VALVE_2 OUT, SOL_VALVE_2 PWR, SOL_VALVE_3 OUT, SOL_VALVE_3 PWR, STVALVE_1_CLOSED, STVALVE_1_GND, STVALVE_1_OPEN, STVALVE_2_CLOSED, STVALVE_2_GND, STVALVE_2_OPEN; removed Extra Valve OUT, Extra Valve PWR, SERVO OUT, SERVO PWR
- sheet Power Unit ports: added none; removed SERVO OUT, SERVO PWR
- sheet RP2040 Standard ports: added GP28/PWM6 A; removed GPIO28
- note added: "FALTA PWR DO SERVO (CONECTORES)"
- moved on the sheet: CR1, CR3, CR4, CR5, CR6, IC1, R1, R10, R3, R4, R5, R6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

Commit message: HYDRA placemenent
Parts:
- added LS1: PKMCS0909E4000-R1, PKMCS0909E4000-R1:SPKR_PKMCS0909E4000-R1, symbol PKMCS0909E4000-R1:PKMCS0909E4000-R1
- added R10, R11: 1k, Resistor-0603:RES_0603, symbol Device:R
- added U2: BC846BLT1G, BC846BLT1G:SOT-23_ONS, symbol BC846BLT1G:BC846BLT1G
- CR1: footprint LED-Yellow_VLMY1300-GS08:LED_VISHAY_VLMX1300_VIS -> LED-Yellow_VLMY1300-GS08:LEDC1608X100N
- CR2: renamed from CR3; footprint LED-Yellow_VLMY1300-GS08:LED_VISHAY_VLMX1300_VIS -> LED-Yellow_VLMY1300-GS08:LEDC1608X100N
- CR3: renamed from CR4; footprint LED-Yellow_VLMY1300-GS08:LED_VISHAY_VLMX1300_VIS -> LED-Yellow_VLMY1300-GS08:LEDC1608X100N
- CR4: renamed from CR5; footprint LED-Yellow_VLMY1300-GS08:LED_VISHAY_VLMX1300_VIS -> LED-Yellow_VLMY1300-GS08:LEDC1608X100N
- CR5: renamed from CR6; footprint LED-Yellow_VLMY1300-GS08:LED_VISHAY_VLMX1300_VIS -> LED-Yellow_VLMY1300-GS08:LEDC1608X100N
- IC1: footprint 2 PNP:SOT-563_1P3X1P7_ONS -> NSVT30010MXV6T1G:SOTFL50P160X60-6N
- R1: value 65 -> 62; footprint Resistor-0402:RES_0402 -> Resistor-0603:RES_0603
- R2: renamed from R3; footprint Resistor-0402:RES_0402 -> Resistor-0603:RES_0603
- R3: renamed from R4; footprint Resistor-0402:RES_0402 -> Resistor-0603:RES_0603
- R4: renamed from R5; footprint Resistor-0402:RES_0402 -> Resistor-0603:RES_0603
- R5: renamed from R6; footprint Resistor-0402:RES_0402 -> Resistor-0603:RES_0603
- R7: renamed from R8; footprint Resistor-0402:RES_0402 -> Resistor-0603:RES_0603
- R8: renamed from R9; footprint Resistor-0402:RES_0402 -> Resistor-0603:RES_0603
- renumbered R7 to R6, R10 to R9
Connections:
- net +5V: now also LS1.1, R11.1
- net GND: now also U2.2 (E); no longer R2.1
- net +3.3VA renamed +3.3V
- new net: R10.1, U2.1 (B)
- new net: LS1.2, R11.2, U2.3 (C)
- new net AGND: R2.1
- new net Buzzer: R10.2
- no-connect marks 0 -> 1
Other:
- sheet IO Connectors ports: added GNDBAT, SERVOGND, SERVOPWR, VBAT; removed none
- sheet Power Unit ports: added SERVOGND, SERVOPWR; removed none
- sheet RP2040 Standard ports: added GP3/PWM1 B, GPIO2, GPIO28; removed GP28/PWM6 A
- note removed: "FALTA PWR DO SERVO (CONECTORES)"
- note removed: "TODO: REVER ACTUATION UNIT - VALVE ACTUATER DRIVERS REVER FOOTPRINTS E COMPONENTES DAS PCBs TODAS CORRIGIR ERC"
- title: Temperature & Valve Control System -> Hydraulic Regulation & Actuation system
- moved on the sheet: CR1, CR2, CR3, CR4, CR5, IC1, R1, R2, R3, R4, R5, R6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

Commit message: HYDRA full design for manufacturing
Changed lines of the file:
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@@
 	(generator "eeschema")
 	(generator_version "9.0")
-	(paper "User" 469.9 431.8)
+	(paper "User" 330.2 355.6)
 	(title_block
 		(title "Hydraulic Regulation & Actuation system")
@@
 	(wire
 		(pts
-			(xy 134.62 158.75) (xy 118.11 158.75)
+			(xy 177.8 189.865) (xy 219.075 189.865)
 		)
 		(stroke
@@
 	(wire
 		(pts
-			(xy 177.8 189.865) (xy 219.075 189.865)
+			(xy 114.3 161.29) (xy 134.62 161.29)
 		)
 		(stroke
@@
 	(wire
 		(pts
+			(xy 177.8 33.02) (xy 219.075 33.02)
+		)
+		(stroke
+			(width 0)
+			(type default)
+		)
+	)
+	(wire
+		(pts
 			(xy 177.8 201.295) (xy 219.075 201.295)
 		)
@@
 	(wire
 		(pts
-			(xy 177.8 33.02) (xy 219.075 33.02)
-		)
-		(stroke
-			(width 0)
-			(type default)
-		)
-	)
-	(wire
-		(pts
 			(xy 101.6 307.34) (xy 101.6 313.055)
 		)
@@
 	(wire
 		(pts
-			(xy 177.8 35.56) (xy 219.075 35.56)
-		)
-		(stroke
-			(width 0)
-			(type default)
-		)
-	)
-	(wire
-		(pts
 			(xy 80.645 123.825) (xy 134.62 123.825)
 		)
@@
 	(wire
 		(pts
+			(xy 118.11 158.75) (xy 134.62 158.75)
+		)
+		(stroke
+			(width 0)
+			(type default)
+		)
+	)
+	(wire
+		(pts
 			(xy 26.67 303.53) (xy 26.67 306.07)
 		)
@@
 	(wire
 		(pts
-			(xy 134.62 161.29) (xy 114.3 161.29)
-		)
-		(stroke
-			(width 0)
-			(type default)
-		)
-	)
-	(wire
-		(pts
 			(xy 177.8 226.695) (xy 219.075 226.695)
 		)
@@
 	(wire
 		(pts
+			(xy 177.8 35.56) (xy 219.075 35.56)
+		)
+		(stroke
+			(width 0)
+			(type default)
+		)
+	)
+	(wire
+		(pts
 			(xy 65.405 303.53) (xy 65.405 306.07)
 		)
@@
 	(wire
 		(pts
-			(xy 134.62 163.83) (xy 110.49 163.83)
-		)
-		(stroke
-			(width 0)
-			(type default)
-		)
-	)
-	(wire
-		(pts
 			(xy 177.8 76.2) (xy 219.075 76.2)
 		)
@@
 		)
 	)
+	(wire
+		(pts
+			(xy 110.49 163.83) (xy 134.62 163.83)
+		)
+		(stroke
+			(width 0)
+			(type default)
+		)
+	)
 	(label "3~{DRDY} THERMO"
 		(at 186.69 81.28 0)
@@
 		)
 	)
-	(label "MOSI SPI"
-		(at 185.42 38.1 0)
-		(effects
-			(font
-				(size 1.27 1.27)
-			)
-			(justify left bottom)
-		)
-	)
-	(label "~{CS} THERMO3 SPI"
-		(at 185.42 30.48 0)
+	(label "MISO SPI"
+		(at 185.42 33.02 0)
 		(effects
 			(font
@@
 		)
 	)
-	(label "MISO SPI"
-		(at 185.42 35.56 0)
+	(label "MOSI SPI"
+		(at 185.42 38.1 0)
 		(effects
 			(font
@@
 		)
 	)
-	(label "SCK SPI"
-		(at 185.42 33.02 0)
+	(label "~{CS} THERMO3 SPI"
+		(at 185.42 30.48 0)
 		(effects
 			(font
@@
 		)
 	)
+	(label "SCK SPI"
+		(at 185.42 35.56 0)
+		(effects
+			(font
+				(size 1.27 1.27)
+			)
+			(justify left bottom)
+		)
+	)
 	(symbol
 		(lib_id "power:Earth")
@@
 		)
 		(pin "SCK SPI" output
-			(at 177.8 33.02 0)
+			(at 177.8 35.56 0)
 			(effects
 				(font
@@
 		)
 		(pin "MISO SPI" input
-			(at 177.8 35.56 0)
+			(at 177.8 33.02 0)
 			(effects
 				(font
@@
 		)
 		(pin "SOL_VALVE_1 DUTY" input
-			(at 134.62 158.75 180)
+			(at 134.62 163.83 180)
 			(effects
 				(font
@@
 		)
 		(pin "SOL_VALVE_3 DUTY" input
-			(at 134.62 163.83 180)
+			(at 134.62 158.75 180)
 			(effects
 				(font
