File: Boards/MissionControl/mission.control/mission.control.kicad_pcb (KiCad board)
At the start: 2 copper layers, 10 parts

Commit message: Algumas mudancas nas PCBs
 Algumas mudancas nas PCBs
Parts:
- added U2: ~, DCDCModule:DCDC_Module, F.Cu at (88.8, 112.5)
- added U2: MAX485_MODULE_5V_LOGIC_TLL_TO_RS-485_CONVERTER, MAX485Module:MODULE_MAX485_MODULE_5V_LOGIC_TLL_TO_RS-485_CONVERTER, F.Cu at (211.9, 132.2)
- added U3: ~, CANController:CANController, F.Cu at (100.7, 146.5)
- A1: renamed from RASPBERRYPI PICO
- Button1: renamed from FIRE BUTTON 
- FireButton1: renamed from ABORT BUTTON
- moved U1 51.0 mm to (147.5, 143.0), turned to 180 degrees
- renumbered ARMKEY to ArmKey1, RÁDIO to U1
Connections:
- net Net-(A1-GPIO16) renamed /RADIO_MISO
- net Net-(A1-GPIO17) renamed /RADIO_CS
- net Net-(A1-GPIO18) renamed /RADIO_SCK
- net Net-(A1-GPIO19) renamed /RADIO_MOSI
- A1 pad 14: Net-(A1-GPIO10) -> unconnected-(A1-GPIO10-Pad14)
- A1 pad 15: Net-(A1-GPIO11) -> unconnected-(A1-GPIO11-Pad15)
- A1 pad 16: unconnected-(A1-GPIO12-Pad16) -> /BUZZER_SIGNAL
- A1 pad 17: unconnected-(A1-GPIO13-Pad17) -> /RADIO_NRESET
- A1 pad 19: Net-(A1-GPIO14) -> /RADIO_BUSY
- A1 pad 20: Net-(A1-GPIO15) -> /RADIO_DIO1
- A1 pad 26: Net-(A1-GPIO20) -> unconnected-(A1-GPIO20-Pad26)
- A1 pad 27: Net-(A1-GPIO21) -> unconnected-(A1-GPIO21-Pad27)
- A1 pad 29: Net-(A1-GPIO22) -> unconnected-(A1-GPIO22-Pad29)
- A1 pad 36: Net-(A1-3V3) -> unconnected-(A1-3V3-Pad36)
- A1 pad 4: Net-(A1-GPIO2) -> unconnected-(A1-GPIO2-Pad4)
- A1 pad 40: unconnected-(A1-VBUS-Pad40) -> +5V
- ArmKey1 pad 1: Net-(A1-3V3) -> +3.3V
- ArmKey1 pad 2: Net-(A1-GPIO2) -> /ARM_SIGNAL
- Button1 pad 1: Net-(A1-3V3) -> Net-(ARMKEY1-Pin_1)
- Button1 pad 2: Net-(A1-GPIO14) -> Net-(Button1-Pin_2)
- C1 pad 1: Net-(A1-3V3) -> +3.3V
- C2 pad 1: Net-(A1-3V3) -> +3.3V
- FireButton1 pad 1: Net-(A1-3V3) -> +3.3V
- FireButton1 pad 2: Net-(A1-GPIO15) -> /FIRE_SIGNAL
- R1 pad 1: Net-(A1-GPIO2) -> Net-(ARMKEY1-Pin_2)
- R2 pad 1: Net-(A1-GPIO14) -> Net-(Button1-Pin_2)
- R3 pad 1: Net-(A1-GPIO15) -> Net-(Button2-Pin_2)
- U1 pad 1: Net-(A1-3V3) -> +3.3V
- U1 pad 11: Net-(A1-GPIO22) -> /RADIO_NRESET
- U1 pad 12: Net-(A1-GPIO20) -> /RADIO_BUSY
- U1 pad 13: Net-(A1-GPIO21) -> /RADIO_DIO1
- U1 pad 8: Net-(A1-GPIO10) -> /RADIO_RX_EN
- U1 pad 9: Net-(A1-GPIO11) -> /RADIO_TX_EN
Other:
- board outline added: 41.6 x 31.6 mm
- copper layers 2 -> 4

Commit message: Atualização
Parts:
- removed Button1: ., CONN_SD-39357-001_02P_MOL:CONN_SD-39357-001_02P_MOL
- removed the U2 at (88.8, 112.5)
- removed the U2 at (211.9, 132.2)
- added AbortButton1: ., TerminalBlock:TerminalBlock_Xinya_XY308-2.54-2P_1x02_P2.54mm_Horizontal, F.Cu at (110.0, 71.2)
- added BZ1: Buzzer, Buzzer_Beeper:Buzzer_TDK_PS1240P02BT_D12.2mm_H6.5mm, F.Cu at (169.6, 76.0)
- added Led1: ., TerminalBlock:TerminalBlock_Xinya_XY308-2.54-2P_1x02_P2.54mm_Horizontal, F.Cu at (110.2, 92.5)
- added R4: 10KΩ, Resistor_SMD:R_0402_1005Metric, F.Cu at (120.5, 78.5)
- added R5: 10KΩ, Resistor_SMD:R_0402_1005Metric, F.Cu at (120.5, 80.5)
- added R6: 1KΩ, Resistor_SMD:R_0402_1005Metric, F.Cu at (107.5, 103.0)
- added U2: MAX485_MODULE_5V_LOGIC_TLL_TO_RS-485_CONVERTER, MAX485Module:MODULE_MAX485_MODULE_5V_LOGIC_TLL_TO_RS-485_CONVERTER, F.Cu at (116.5, 120.0)
- ArmKey1, FireButton1: footprint CONN_SD-39357-001_02P_MOL:CONN_SD-39357-001_02P_MOL -> TerminalBlock:TerminalBlock_Xinya_XY308-2.54-2P_1x02_P2.54mm_Horizontal
- R1: value 10k -> 220Ω
- R2: value 10k -> 100Ω
- R3: value 10k -> 10KΩ
- moved U3 80.2 mm to (170.5, 107.0), turned to 90 degrees
- moved C2 58.8 mm to (148.6, 139.0)
- moved R2 55.9 mm to (160.5, 71.5)
- moved C1 52.4 mm to (148.6, 137.7)
- moved R3 49.7 mm to (119.5, 74.0)
- moved FireButton1 33.6 mm to (110.0, 85.2), turned to -90 degrees
- moved ArmKey1 19.0 mm to (110.0, 78.2), turned to -90 degrees
- moved U1 15.0 mm to (137.6, 131.7)
- moved A1 14.8 mm to (137.2, 94.0)
- moved R1 6.10 mm to (122.5, 94.5)
Connections:
- A1 pad 1: unconnected-(A1-GPIO0-Pad1) -> /CAN_INT
- A1 pad 10: unconnected-(A1-GPIO7-Pad10) -> /BUZZER_SIGNAL
- A1 pad 11: unconnected-(A1-GPIO8-Pad11) -> /LED_SIGNAL
- A1 pad 12: unconnected-(A1-GPIO9-Pad12) -> /ARM_SIGNAL
- A1 pad 14: unconnected-(A1-GPIO10-Pad14) -> /ABORT_SIGNAL
- A1 pad 15: unconnected-(A1-GPIO11-Pad15) -> /FIRE_SIGNAL
- A1 pad 16: /BUZZER_SIGNAL -> /RS_DI
- A1 pad 17: /RADIO_NRESET -> /RS_RO
- A1 pad 19: /RADIO_BUSY -> /RADIO_DIO1
- A1 pad 2: unconnected-(A1-GPIO1-Pad2) -> /CAN_CS
- A1 pad 20: /RADIO_DIO1 -> /RADIO_BUSY
- A1 pad 21: /RADIO_MISO -> /SPI0_MISO
- A1 pad 24: /RADIO_SCK -> /SPI0_SCK
- A1 pad 25: /RADIO_MOSI -> /SPI0_MOSI
- A1 pad 29: unconnected-(A1-GPIO22-Pad29) -> /RS_DE
- A1 pad 4: unconnected-(A1-GPIO2-Pad4) -> /BUZZER_SIGNAL
- A1 pad 5: unconnected-(A1-GPIO3-Pad5) -> /RADIO_NRESET
- A1 pad 7: unconnected-(A1-GPIO5-Pad7) -> /RADIO_TX_EN
- A1 pad 9: unconnected-(A1-GPIO6-Pad9) -> /RADIO_RX_EN
- R1 pad 2: GND -> /LED_SIGNAL
- R2 pad 1: Net-(Button1-Pin_2) -> /BUZZER_SIGNAL
- R2 pad 2: GND -> Net-(BZ1-+)
- R3 pad 1: Net-(Button2-Pin_2) -> GND
- R3 pad 2: GND -> /FIRE_SIGNAL
- U1 pad 3: /RADIO_MISO -> /SPI0_MISO
- U1 pad 4: /RADIO_MOSI -> /SPI0_MOSI
- U1 pad 5: /RADIO_SCK -> /SPI0_SCK
- U3 pad 2: /CAN_SCK -> /SPI0_SCK
- U3 pad 3: unconnected-(U3-SI-Pad3) -> /SPI0_MOSI
- U3 pad 4: unconnected-(U3-SO-Pad4) -> /SPI0_MISO
- U3 pad 5: unconnected-(U3-CS-Pad5) -> /CAN_CS
Routing:
- net +5V: track 0.00 -> 143.1 mm
- net /CAN_CS: track 0.00 -> 90.6 mm, vias 0 -> 1
- net /SPI0_MOSI: track 0.00 -> 61.9 mm
- net /RADIO_NRESET: track 0.00 -> 60.3 mm, vias 0 -> 1
- net /SPI0_SCK: track 0.00 -> 52.8 mm
- net /SPI0_MISO: track 0.00 -> 52.6 mm
- net /RADIO_RX_EN: track 0.00 -> 52.0 mm, vias 0 -> 1
- net /RADIO_TX_EN: track 0.00 -> 50.8 mm, vias 0 -> 1
- net /RADIO_DIO1: track 0.00 -> 24.0 mm
- net /RS_DI: track 0.00 -> 23.6 mm
- net /RADIO_CS: track 0.31 -> 20.9 mm
- net /RADIO_BUSY: track 0.00 -> 16.9 mm
- net /RS_TXEN: track 0.00 -> 14.3 mm
- net /RS_RO: track 0.00 -> 14.2 mm
- net GND: track 0.00 -> 6.81 mm
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Other:
- board size 41.6 x 31.6 mm -> 85.5 x 79 mm

Commit message: Atualização
Parts:
- moved R1 23.0 mm to (121.2, 71.5)
- moved Led 22.5 mm to (113.0, 70.2)
- moved R3 19.6 mm to (121.2, 93.5)
- moved AbortBtn 14.5 mm to (113.0, 85.4)
- moved FireBtn 8.33 mm to (113.0, 93.0)
- moved R4 7.74 mm to (121.2, 86.2)
- moved BZ1 3.06 mm to (172.6, 76.7)
- moved C2 3.06 mm to (151.6, 139.7)
- moved A1 3.06 mm to (140.2, 94.7)
- moved R6 3.06 mm to (110.5, 103.7)
- moved RS485 3.06 mm to (119.5, 120.7)
- moved C1 3.06 mm to (151.6, 138.4)
- moved U1 3.06 mm to (140.6, 132.4)
- moved ArmKey 3.03 mm to (113.0, 77.8)
- moved R2 2.76 mm to (162.8, 73.0), turned to -90 degrees
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- renumbered AbortButton1 to AbortBtn, ArmKey1 to ArmKey, U3 to CAN, FireButton1 to FireBtn, Led1 to Led, U2 to RS485
Connections:
- A1 pad 36: unconnected-(A1-3V3-Pad36) -> +3.3V
Routing:
- net /CAN_INT: track 0.00 -> 76.2 mm
- net /BUZZER_SIGNAL: track 0.00 -> 37.1 mm
- net /ARM_SIGNAL: track 0.00 -> 35.4 mm
- net /ABORT_SIGNAL: track 0.00 -> 33.2 mm
- net /FIRE_SIGNAL: track 0.00 -> 29.2 mm
- net /LED_SIGNAL: track 0.00 -> 28.1 mm
- net Net-(BZ1-+): track 0.00 -> 11.1 mm
- net Net-(Led1-Pin_1): track 0.00 -> 8.27 mm
- net GND: track 6.81 -> 14.8 mm, vias 0 -> 9
- net /CAN_CS: track 90.6 -> 98.3 mm
- net +5V: track 143.1 -> 140.1 mm
- net /SPI0_MISO: track 52.6 -> 50.7 mm
- net /RADIO_RX_EN: track 52.0 -> 50.6 mm
- net /RADIO_NRESET: track 60.3 -> 61.4 mm, vias 1 -> 0
- net /RS_DI: track 23.6 -> 22.8 mm
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- added copper zone on F.Cu, net +3.3V
- added copper zone on B.Cu, net GND
Other:
- board size 85.5 x 79 mm -> 81.2 x 77.5 mm
- copper layers 4 -> 2

Commit message: para o alex arranjar ;)
Parts:
- renumbered AbortBtn to AbortButton1, ArmKey to ArmKey1, FireBtn to FireButton1, Led to Led1, RS485 to U2, CAN to U3
Connections:
- A1 pad 10: /BUZZER_SIGNAL -> unconnected-(A1-GPIO7-Pad10)
Routing:
- net /CAN_CS: track 98.3 -> 86.7 mm, vias 1 -> 0
- net /BUZZER_SIGNAL: track 37.1 -> 48.0 mm
- net +5V: track 140.1 -> 133.6 mm
- net /RADIO_NRESET: track 61.4 -> 57.4 mm
- net /RADIO_TX_EN: track 50.8 -> 47.4 mm
- net /CAN_INT: track 76.2 -> 78.0 mm
- net /RADIO_BUSY: track 16.9 -> 17.6 mm
Changed lines of the file:
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@@
 	(net 39 "/CAN_CS")
 	(net 40 "/CAN_INT")
+	(net 41 "unconnected-(A1-GPIO7-Pad10)")
 	(footprint "CANController:CANController"
 		(layer "F.Cu")
 		(at 169.98 107.66 90)
-		(property "Reference" "CAN"
+		(property "Reference" "U3"
 			(at 0 -0.5 90)
 			(unlocked yes)
@@
 		(layer "F.Cu")
 		(at 119.52 120.66 90)
-		(property "Reference" "RS485"
+		(property "Reference" "U2"
 			(at 0 0 90)
 			(layer "F.SilkS")
@@
 		(descr "Terminal Block Xinya XY308-2.54-2P, 2 pins, pitch 2.54mm, size 5.58x6.5mm, drill diameter 1.2mm, pad diameter 2mm, http://www.xinyaelectronic.com/product/xy308-254, script-generated using https://gitlab.com/kicad/libraries/kicad-footprint-generator/-/tree/master/scripts/TerminalBlock_Xinya")
 		(tags "THT Terminal Block Xinya XY308-2.54-2P pitch 2.54mm size 5.58x6.5mm drill 1.2mm pad 2mm")
-		(property "Reference" "Led"
+		(property "Reference" "Led1"
 			(at 1.79 -5 90)
 			(layer "F.SilkS")
@@
 		(descr "Terminal Block Xinya XY308-2.54-2P, 2 pins, pitch 2.54mm, size 5.58x6.5mm, drill diameter 1.2mm, pad diameter 2mm, http://www.xinyaelectronic.com/product/xy308-254, script-generated using https://gitlab.com/kicad/libraries/kicad-footprint-generator/-/tree/master/scripts/TerminalBlock_Xinya")
 		(tags "THT Terminal Block Xinya XY308-2.54-2P pitch 2.54mm size 5.58x6.5mm drill 1.2mm pad 2mm")
-		(property "Reference" "AbortBtn"
+		(property "Reference" "AbortButton1"
 			(at 1.123333 -4.75 90)
 			(layer "F.SilkS")
@@
 		(descr "Terminal Block Xinya XY308-2.54-2P, 2 pins, pitch 2.54mm, size 5.58x6.5mm, drill diameter 1.2mm, pad diameter 2mm, http://www.xinyaelectronic.com/product/xy308-254, script-generated using https://gitlab.com/kicad/libraries/kicad-footprint-generator/-/tree/master/scripts/TerminalBlock_Xinya")
 		(tags "THT Terminal Block Xinya XY308-2.54-2P pitch 2.54mm size 5.58x6.5mm drill 1.2mm pad 2mm")
-		(property "Reference" "ArmKey"
+		(property "Reference" "ArmKey1"
 			(at 1.206667 -4.75 90)
 			(layer "F.SilkS")
@@
 			(layers "F.Cu" "F.Mask")
 			(roundrect_rratio 0.5)
-			(net 1 "/BUZZER_SIGNAL")
+			(net 41 "unconnected-(A1-GPIO7-Pad10)")
 			(pinfunction "GPIO7")
 			(pintype "bidirectional")
@@
 			(layers "*.Cu" "*.Mask")
 			(remove_unused_layers no)
-			(net 1 "/BUZZER_SIGNAL")
+			(net 41 "unconnected-(A1-GPIO7-Pad10)")
 			(pinfunction "GPIO7")
 			(pintype "bidirectional")
@@
 		(descr "Terminal Block Xinya XY308-2.54-2P, 2 pins, pitch 2.54mm, size 5.58x6.5mm, drill diameter 1.2mm, pad diameter 2mm, http://www.xinyaelectronic.com/product/xy308-254, script-generated using https://gitlab.com/kicad/libraries/kicad-footprint-generator/-/tree/master/scripts/TerminalBlock_Xinya")
 		(tags "THT Terminal Block Xinya XY308-2.54-2P pitch 2.54mm size 5.58x6.5mm drill 1.2mm pad 2mm")
-		(property "Reference" "FireBtn"
+		(property "Reference" "FireButton1"
 			(at 1.04 -4.75 90)
 			(layer "F.SilkS")
@@
 	)
 	(segment
-		(start 162.75 72.49)
-		(end 158.76 68.5)
+		(start 127.35 69)
+		(end 127.35 75.5)
+		(width 0.5)
+		(layer "F.Cu")
+		(net 1)
+	)
+	(segment
+		(start 127.85 68.5)
+		(end 127.35 69)
 		(width 0.5)
 		(layer "F.Cu")
@@
 	(segment
 		(start 158.76 68.5)
-		(end 141.03 68.5)
+		(end 127.85 68.5)
+		(width 0.5)
+		(layer "F.Cu")
+		(net 1)
+	)
+	(segment
+		(start 130.07 78.22)
+		(end 130.51 78.22)
 		(width 0.5)
 		(layer "F.Cu")
@@
 	)
 	(segment
-		(start 141.03 68.5)
-		(end 131.31 78.22)
+		(start 127.35 75.5)
+		(end 130.07 78.22)
+		(width 0.5)
+		(layer "F.Cu")
+		(net 1)
+	)
+	(segment
+		(start 162.75 72.49)
+		(end 158.76 68.5)
 		(width 0.5)
 		(layer "F.Cu")
@@
 	)
 	(segment
+		(start 130.51 133.21)
+		(end 131.9281 134.6281)
+		(width 0.5)
+		(layer "F.Cu")
+		(net 5)
+	)
+	(segment
 		(start 132.9319 134.6281)
 		(end 132.6652 134.6281)
@@
 	)
 	(segment
-		(start 130.51 132.4729)
-		(end 130.51 118.86)
+		(start 131.9281 134.6281)
+		(end 132.9319 134.6281)
 		(width 0.5)
 		(layer "F.Cu")
@@
 	)
 	(segment
-		(start 132.6652 134.6281)
-		(end 130.51 132.4729)
+		(start 130.51 118.86)
+		(end 130.51 133.21)
 		(width 0.5)
 		(layer "F.Cu")
@@
 	)
 	(segment
-		(start 141.25 125.5)
-		(end 141.25 89)
+		(start 133.3919 133.3581)
+		(end 136.4 130.35)
 		(width 0.5)
 		(layer "F.Cu")
@@
 	)
 	(segment
-		(start 133 80.75)
-		(end 132.99 80.76)
+		(start 136.4 84.15)
+		(end 133 80.75)
 		(width 0.5)
 		(layer "F.Cu")
@@
 	)
 	(segment
-		(start 133.3919 133.3581)
-		(end 141.25 125.5)
+		(start 136.4 130.35)
+		(end 136.4 84.15)
 		(width 0.5)
 		(layer "F.Cu")
@@
 	)
 	(segment
-		(start 141.25 89)
-		(end 133 80.75)
+		(start 133 80.75)
+		(end 132.99 80.76)
 		(width 0.5)
 		(layer "F.Cu")
@@
 	)
 	(segment
-		(start 137 123.729024)
-		(end 137 95)
+		(start 133.65 91.65)
+		(end 132.92 90.92)
 		(width 0.5)
 		(layer "B.Cu")
@@
 	(segment
 		(start 142.430976 129.16)
-		(end 137 123.729024)
+		(end 133.65 120.379024)
 		(width 0.5)
 		(layer "B.Cu")
@@
 	)
 	(segment
-		(start 137 95)
-		(end 132.92 90.92)
+		(start 133.65 120.379024)
+		(end 133.65 91.65)
 		(width 0.5)
 		(layer "B.Cu")
@@
 	)
 	(segment
-		(start 132.92 90.92)
-		(end 131.31 90.92)
+		(start 147.09 129.16)
+		(end 142.430976 129.16)
 		(width 0.5)
 		(layer "B.Cu")
@@
 	)
 	(segment
-		(start 147.09 129.16)
-		(end 142.430976 129.16)
+		(start 132.92 90.92)
+		(end 131.31 90.92)
 		(width 0.5)
 		(layer "B.Cu")
@@
 	)
 	(segment
-		(start 139.09 93.62)
-		(end 131.31 85.84)
+		(start 132.9319 130.8181)
+		(end 135 128.75)
 		(width 0.5)
 		(layer "F.Cu")
@@
 	)
 	(segment
-		(start 139.09 124.66)
-		(end 139.09 93.62)
+		(start 135 89.53)
+		(end 131.31 85.84)
 		(width 0.5)
 		(layer "F.Cu")
@@
 	)
 	(segment
-		(start 132.9319 130.8181)
-		(end 139.09 124.66)
+		(start 135 128.75)
+		(end 135 89.53)
 		(width 0.5)
 		(layer "F.Cu")
@@
 	)
 	(segment
-		(start 176.88 93.2)
-		(end 154.28 70.6)
-		(width 0.5)
+		(start 162.205197 142.6)
+		(end 176.88 127.925197)
+		(width 1.5)
 		(layer "F.Cu")
 		(net 37)
 	)
 	(segment
-		(start 176.88 137.8)
-		(end 176.88 127.81)
-		(width 0.5)
+		(start 123.33 141.26)
+		(end 124.67 142.6)
+		(width 1.5)
 		(layer "F.Cu")
 		(net 37)
 	)
 	(segment
-		(start 123.33 141.26)
-		(end 125.27 143.2)
-		(width 0.5)
+		(start 176.88 127.81)
+		(end 179.48 127.81)
+		(width 2)
 		(layer "F.Cu")
 		(net 37)
 	)
 	(segment
-		(start 179.48 127.81)
-		(end 176.88 127.81)
-		(width 0.75)
+		(start 176.88 93.63)
+		(end 153.85 70.6)
+		(width 1.25)
 		(layer "F.Cu")
 		(net 37)
 	)
 	(segment
-		(start 176.88 127.81)
-		(end 176.88 93.2)
-		(width 0.5)
+		(start 176.88 127.925197)
+		(end 176.88 127.81)
+		(width 1.5)
 		(layer "F.Cu")
 		(net 37)
 	)
 	(segment
-		(start 171.48 143.2)
-		(end 176.88 137.8)
-		(width 0.5)
+		(start 153.85 70.6)
+		(end 149.89 70.6)
+		(width 1.25)
 		(layer "F.Cu")
 		(net 37)
 	)
 	(segment
-		(start 154.28 70.6)
-		(end 149.89 70.6)
-		(width 0.5)
+		(start 124.67 142.6)
+		(end 162.205197 142.6)
+		(width 1.5)
 		(layer "F.Cu")
 		(net 37)
 	)
 	(segment
-		(start 125.27 143.2)
-		(end 171.48 143.2)
-		(width 0.5)
+		(start 176.88 127.81)
+		(end 176.88 93.63)
+		(width 1.25)
 		(layer "F.Cu")
 		(net 37)
@@
 	)
 	(segment
-		(start 171.48 127.81)
-		(end 171.48 94.7)
-		(width 0.5)
-		(layer "F.Cu")
-		(net 39)
-	)
-	(segment
-		(start 171.48 94.7)
-		(end 153.44 76.66)
-		(width 0.5)
-		(layer "F.Cu")
-		(net 39)
-	)
-	(via
-		(at 153.44 76.66)
-		(size 0.5)
-		(drill 0.2)
-		(layers "F.Cu" "B.Cu")
-		(net 39)
-	)
-	(segment
-		(start 126.98 72.7)
-		(end 127.42 73.14)
-		(width 0.5)
-		(layer "B.Cu")
-		(net 39)
-	)
-	(segment
-		(start 153.44 76.66)
-		(end 153.44 71.66)
-		(width 0.5)
+		(start 137.75 79.58)
+		(end 131.31 73.14)
+		(width 0.25)
 		(layer "B.Cu")
 		(net 39)
 	)
 	(segment
-		(start 150.94 69.16)
-		(end 128.52 69.16)
-		(width 0.5)
+		(start 151.482 130.4)
+		(end 137.75 116.668)
+		(width 0.25)
 		(layer "B.Cu")
 		(net 39)
 	)
 	(segment
-		(start 128.52 69.16)
-		(end 126.98 70.7)
-		(width 0.5)
+		(start 168.89 130.4)
+		(end 151.482 130.4)
+		(width 0.25)
 		(layer "B.Cu")
 		(net 39)
 	)
 	(segment
-		(start 126.98 70.7)
-		(end 126.98 72.7)
-		(width 0.5)
+		(start 171.48 127.81)
+		(end 168.89 130.4)
+		(width 0.25)
 		(layer "B.Cu")
 		(net 39)
 	)
 	(segment
-		(start 127.42 73.14)
-		(end 131.31 73.14)
-		(width 0.5)
+		(start 137.75 116.668)
+		(end 137.75 79.58)
+		(width 0.25)
 		(layer "B.Cu")
 		(net 39)
 	)
 	(segment
-		(start 153.44 71.66)
-		(end 150.94 69.16)
+		(start 160.83 85.53)
+		(end 152.25 76.95)
 		(width 0.5)
 		(layer "B.Cu")
-		(net 39)
+		(net 40)
 	)
 	(segment
-		(start 149.007841 76.701)
-		(end 137.411 76.701)
+		(start 152.25 76.95)
+		(end 137.66 76.95)
 		(width 0.5)
 		(layer "B.Cu")
@@
 	)
 	(segment
-		(start 160.83 88.523159)
-		(end 149.007841 76.701)
+		(start 137.66 76.95)
+		(end 137.411 76.701)
 		(width 0.5)
 		(layer "B.Cu")
@@
 	)
 	(segment
-		(start 160.83 111.2)
-		(end 160.83 88.523159)
-		(width 0.5)
-		(layer "B.Cu")
-		(net 40)
-	)
-	(segment
 		(start 160.83 127.81)
-		(end 160.83 111.2)
+		(end 160.83 85.53)
 		(width 0.5)
 		(layer "B.Cu")
