File: Boards/MissionControl/mission.control/mission.control.kicad_pcb (KiCad board)
At the start: 2 copper layers, 81.2 x 77.5 mm, 17 parts, among them U1 E28-2G4M27SX, U2 MAX485_MODULE_5V_LOGIC_TLL_TO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

Commit message: resolvido :)
Parts:
- renumbered AbortButton1 to AbortBtn, ArmKey1 to ArmKey, FireButton1 to FireBtn, Led1 to Led
Routing:
- net /CAN_CS: track 86.7 -> 83.5 mm
Changed lines of the file:
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@@
 				"o3Zqoy9RNtiAhZtX9p5c1EF6/ErIk7DVitXd+eA+/GqIVXTu6zzsHkNZD/32P2KQfbD97z9+f18P"
 				"9VFy/UVe8z/XZNNbqqf6fCgbffr5y294FNwBrgsJpk4tPUeSg+XfvxOz5cJe+QvvXhvAP+dAPASx"
-				"/h+ykqUlQ9FDwQAAAABJRU5ErkJggg=="
+				"/h+ykqUlQ9FDwQAAAABJRU5ErkJgggAAAAAAAAAAAAAAAAAAAAAAAAAAAAAAAAAAAAAAAAAAAAAA"
+				"AAAAAAAAAAAAAAAAAAAAAAAAAAAAAAAAAAAAAAAAAAAAAAAAAAAAAAAAAAAAAAAAAAAAAAAAAAAA"
+				"AAAAAAAAAAAAAAAAAAAAAAAAAAAAAAAAAAAAAAAAAAAAAAAAAAAAAAAAAAAAAAAAAAAAAAAAAAAA"
+				"AAAAAAAAAAAAAAAAAAAAAAAAAAAAAAAAAAAAAAAAAAAAAAAAAAAAAAAAAAAAAAAAAAAAAAAAAAAA"
+				"AAAAAAAAAAAAAAAAAAAAAAAAAAAAAAAAAAAAAAAAAAAAAAAAAAAAAAAAAAAAAAAAAAAAAAAAAAAA"
+				"AAAAAAAAAAAAAAAAAAAAAAAAAAAAAAAAAAAAAAAAAAAAAAAAAAAAAAAAAAAAAAAAAAAAAAAAAAAA"
+				"AAAAAAAAAAAAAAAAAAAAAAAAAAAAAAAAAAAAAAAAAAAAAAAAAAAAAAAAAAAAAAAAAAAAAAAAAAAA"
+				"AAAAAAAAAAAAAAAAAAAAAAAAAAAAAAAAAAAAAAAAAAAAAAAAAAAAAAAAAAAAAAAAAAAAAAAAAAAA"
+				"AAAAAAAAAAAAAAAAAAAAAAAAAAAAAAAAAAAAAAAAAAAAAAAAAAAAAAAAAAAAAAAAAAAAAAAAAAAA"
+				"AAAAAAAAAAAAAAAAAAAAAAAAAAAAAAAAAAAAAAAAAAAAAAAAAAAAAAAAAAAAAAAAAAAAAAAAAAAA"
+				"AAAAAAAAAAAAAAAAAAAAAAAAAAAAAAAAAAAAAAAAAAAAAAAAAAAAAAAAAAAAAAAAAAAAAAAAAAAA"
+				"AAAAAAAAAAAAAAAAAAAAAAAAAAAAAAAAAAAAAAAAAAAAAAAAAAAAAAAAAAAAAAAAAAAAAAAAAAAA"
+				"AAAAAAAAAAAAAAAAAAAAAAAAAAAAAAAAAAAAAAAAAAAAAAAAAAAAAAAAAAAAAAAAAAAAAAAAAAAA"
+				"AAAAAAAAAAAAAAAAAAAAAAAAAAAAAAAAAAAAAAAAAAAAAAAAAAAAAAAAAAAAAAAAAAAAAAAAAAAA"
+				"AAAAAAAAAAAAAAAAAAAAAAAAAAAAAAAAAAAAAAAAAAAAAAAAAAAAAAAAAAAAAAAAAAAAAAAAAAAA"
+				"AAAAAAAAAAAAAAAAAAAAAAAAAAAAAAAAAAAAAAAAAAAAAAAAAAAAAAAAAAAAAAAAAAAAAAAAAAAA"
+				"AAAAAAAAAAAAAAAAAAAAAAAAAAAAAAAAAAAAAAAAAAAAAAAAAAAAAAAAAAAAAAAAAAAAAAAAAAAA"
+				"AAAAAAAAAAAAAAAAAAAAAAAAAAAAAAAAAAAAAAAAAAAAAAAAAAAAAAAAAAAAAAAAAAAAAAAAAAAA"
+				"AAAAAAAAAAAAAAAAAAAAAAAAAAAAAAAAAAAAAAAAAAAAAAAAAAAAAAAAAAAAAAAAAAAAAAAAAAAA"
+				"AAAAAAAAAAAAAAAAAAAAAAAAAAAAAAAAAAAAAAAAAAAAAAAAAAAAAAAAAAAAAAAAAAAAAAAAAAAA"
+				"AAAAAAAAAAAAAAAAAAAAAAAAAAAAAAAAAAAAAAAAAAAAAAAAAAAAAAAAAAAAAAAAAAAAAAAAAAAA"
+				"AAAAAAAAAAAAAAAAAAAAAAAAAAAAAAAAAAAAAAAAAAAAAAAAAAAAAAAAAAAAAAAAAAAAAAAAAAAA"
+				"AAAAAAAAAAAAAAAAAAAAAAAAAAAAAAAAAAAAAAAAAAAAAAAAAAAAAAAAAAAAAAAAAAAAAAAAAAAA"
+				"AAAAAAAAAAAAAAAAAAAAAAAAAAAAAAAAAAAAAAAAAAAAAAAAAAAAAAAAAAAAAAAAAAAAAAAAAAAA"
+				"AAAAAAAAAAAAAAAAAAAAAAAAAAAAAAAAAAAAAAAAAAAAAAAAAAAAAAAAAAAAAAAAAAAAAAAAAAAA"
+				"AAAAAAAAAAAAAAAAAAAAAAAAAAAAAAAAAAAAAAAAAAAAAAAAAAAAAAAAAAAAAAAAAAAAAAAAAAAA"
+				"AAAAAAAAAAAAAAAAAAAAAAAAAAAAAAAAAAAAAAAAAAAAAAAAAAAAAAAAAAAAAAAAAAAAAAAAAAAA"
+				"AAAAAAAAAAAAAAAAAAAAAAAAAAAAAAAAAAAAAAAAAAAAAAAAAAAAAAAAAAAAAAAAAAAAAAAAAAAA"
+				"AAAAAAAAAAAAAAAAAAAAAAAAAAAAAAAAAAAAAAAAAAAAAAAAAAAAAAAAAAAAAAAAAAAAAAAAAAAA"
+				"AAAAAAAAAAAAAAAAAAAAAAAAAAAAAAAAAAAAAAAAAAAAAAAAAAAAAAAAAAAAAAAAAAAAAAAAAAAA"
+				"AAAAAAAAAAAAAAAAAAAAAAAAAAAAAAAAAAAAAAAAAAAAAAAAAAAAAAAAAAAAAAAAAAAAAAAAAAAA"
+				"AAAAAAAAAAAAAAAAAAAAAAAAAAAAAAAAAAAAAAAAAAAAAAAAAAAAAAAAAAAAAAAAAAAAAAAAAAAA"
+				"AAAAAAAAAAAAAAAAAAAAAAAAAAAAAAAAAAAAAAAAAAAAAAAAAAAAAAAAAAAAAAAAAAAAAAAAAAAA"
+				"AAAAAAAAAAAAAAAAAAAAAAAAAAAAAAAAAAAAAAAAAAAAAAAAAAAAAAAAAAAAAAAAAAAAAAAAAAAA"
+				"AAAAAAAAAAAAAAAAAAAAAAAAAAAAAAAAAAAAAAAAAAAAAAAAAAAAAAAAAAAAAAAAAAAAAAAAAAAA"
+				"AAAAAAAAAAAAAAAAAAAAAAAAAAAAAAAAAAAAAAAAAAAAAAAAAAAAAAAAAAAAAAAAAAAAAAAAAAAA"
+				"AAAAAAAAAAAAAAAAAAAAAAAAAAAAAA=="
 			)
 		)
@@
 		(descr "Terminal Block Xinya XY308-2.54-2P, 2 pins, pitch 2.54mm, size 5.58x6.5mm, drill diameter 1.2mm, pad diameter 2mm, http://www.xinyaelectronic.com/product/xy308-254, script-generated using https://gitlab.com/kicad/libraries/kicad-footprint-generator/-/tree/master/scripts/TerminalBlock_Xinya")
 		(tags "THT Terminal Block Xinya XY308-2.54-2P pitch 2.54mm size 5.58x6.5mm drill 1.2mm pad 2mm")
-		(property "Reference" "Led1"
+		(property "Reference" "Led"
 			(at 1.79 -5 90)
 			(layer "F.SilkS")
@@
 			(layer "F.Fab")
 		)
-		(fp_text user "*"
-			(at -9.67 -7.45 180)
-			(unlocked yes)
-			(layer "F.SilkS")
-			(effects
-				(font
-					(size 1 1)
-					(thickness 0.15)
-				)
-			)
-		)
-		(fp_text user "*"
-			(at -9.67 -7.45 0)
-			(layer "F.SilkS")
-			(effects
-				(font
-					(size 1 1)
-					(thickness 0.15)
-				)
-			)
-		)
-		(fp_text user "*"
-			(at -9.67 -7.45 180)
-			(unlocked yes)
-			(layer "B.SilkS")
-			(effects
-				(font
-					(size 1 1)
-					(thickness 0.15)
-				)
-			)
-		)
 		(fp_text user "${REFERENCE}"
 			(at 0 0 180)
@@
 		(tags "resistor")
 		(property "Reference" "R6"
-			(at 0 -1.17 90)
+			(at -0.153641 0.98 90)
 			(layer "F.SilkS")
 			(effects
@@
 		(descr "Terminal Block Xinya XY308-2.54-2P, 2 pins, pitch 2.54mm, size 5.58x6.5mm, drill diameter 1.2mm, pad diameter 2mm, http://www.xinyaelectronic.com/product/xy308-254, script-generated using https://gitlab.com/kicad/libraries/kicad-footprint-generator/-/tree/master/scripts/TerminalBlock_Xinya")
 		(tags "THT Terminal Block Xinya XY308-2.54-2P pitch 2.54mm size 5.58x6.5mm drill 1.2mm pad 2mm")
-		(property "Reference" "AbortButton1"
+		(property "Reference" "AbortBtn"
 			(at 1.123333 -4.75 90)
 			(layer "F.SilkS")
@@
 		(descr "Terminal Block Xinya XY308-2.54-2P, 2 pins, pitch 2.54mm, size 5.58x6.5mm, drill diameter 1.2mm, pad diameter 2mm, http://www.xinyaelectronic.com/product/xy308-254, script-generated using https://gitlab.com/kicad/libraries/kicad-footprint-generator/-/tree/master/scripts/TerminalBlock_Xinya")
 		(tags "THT Terminal Block Xinya XY308-2.54-2P pitch 2.54mm size 5.58x6.5mm drill 1.2mm pad 2mm")
-		(property "Reference" "ArmKey1"
+		(property "Reference" "ArmKey"
 			(at 1.206667 -4.75 90)
 			(layer "F.SilkS")
@@
 		(descr "Terminal Block Xinya XY308-2.54-2P, 2 pins, pitch 2.54mm, size 5.58x6.5mm, drill diameter 1.2mm, pad diameter 2mm, http://www.xinyaelectronic.com/product/xy308-254, script-generated using https://gitlab.com/kicad/libraries/kicad-footprint-generator/-/tree/master/scripts/TerminalBlock_Xinya")
 		(tags "THT Terminal Block Xinya XY308-2.54-2P pitch 2.54mm size 5.58x6.5mm drill 1.2mm pad 2mm")
-		(property "Reference" "FireButton1"
+		(property "Reference" "FireBtn"
 			(at 1.04 -4.75 90)
 			(layer "F.SilkS")
@@
 	)
 	(segment
-		(start 137.75 79.58)
-		(end 131.31 73.14)
-		(width 0.25)
-		(layer "B.Cu")
+		(start 131.31 73.14)
+		(end 132.67 74.5)
+		(width 0.5)
+		(layer "F.Cu")
 		(net 39)
 	)
 	(segment
-		(start 151.482 130.4)
-		(end 137.75 116.668)
-		(width 0.25)
-		(layer "B.Cu")
+		(start 153.48 74.5)
+		(end 171.49 92.51)
+		(width 0.5)
+		(layer "F.Cu")
 		(net 39)
 	)
 	(segment
-		(start 168.89 130.4)
-		(end 151.482 130.4)
-		(width 0.25)
-		(layer "B.Cu")
+		(start 171.49 92.51)
+		(end 171.48 92.52)
+		(width 0.5)
+		(layer "F.Cu")
 		(net 39)
 	)
 	(segment
-		(start 171.48 127.81)
-		(end 168.89 130.4)
-		(width 0.25)
-		(layer "B.Cu")
+		(start 132.67 74.5)
+		(end 153.48 74.5)
+		(width 0.5)
+		(layer "F.Cu")
 		(net 39)
 	)
 	(segment
-		(start 137.75 116.668)
-		(end 137.75 79.58)
-		(width 0.25)
-		(layer "B.Cu")
+		(start 171.48 92.52)
+		(end 171.48 127.81)
+		(width 0.5)
+		(layer "F.Cu")
+		(net 39)
+	)
+	(segment
+		(start 171.49 92.51)
+		(end 171.5 92.52)
+		(width 0.5)
+		(layer "F.Cu")
 		(net 39)
 	)

Commit message: PCBs acabadas e modulo de radio feito
Parts:
- removed C1: 100uF, Resistor_SMD:R_0402_1005Metric
- removed C2: 0.1uF, Resistor_SMD:R_0402_1005Metric
- added G***: LOGO, Eurocircuits:LogoEurocircuits, F.Cu at (172.4, 138.4)
- added G***: LOGO, LogoPST:LogoPST, B.Cu at (171.6, 104.2)
- U1: footprint Rádio:E28-2G4M27SX_CGD -> Radio_Module_PST:Radio_Module_PST
- moved R2 12.9 mm to (175.3, 70.0), turned to 0 degrees
- moved BZ1 7.21 mm to (179.7, 75.6)
- moved U3 3.82 mm to (171.6, 104.2)
- moved U1 3.02 mm to (140.8, 135.4)
Connections:
- A1 pad 29: /RS_DE -> /RS_TXEN
Routing:
- net /RS_TXEN: track 14.3 -> 53.3 mm
- net +5V: track 133.6 -> 147.1 mm
- net /BUZZER_SIGNAL: track 48.0 -> 59.1 mm
- net GND: track 14.8 -> 5.13 mm, vias 9 -> 4
- net /RADIO_RX_EN: track 50.6 -> 45.0 mm, vias 1 -> 0
- net +3.3V: track 4.67 -> 0.00 mm
- net Net-(BZ1-+): track 11.1 -> 7.19 mm
- net /SPI0_MOSI: track 61.7 -> 58.6 mm
- net /RADIO_CS: track 20.9 -> 17.8 mm
- net /RADIO_TX_EN: track 47.4 -> 44.4 mm
- net /SPI0_SCK: track 52.5 -> 49.9 mm
- net /CAN_CS: track 83.5 -> 82.0 mm
- net /SPI0_MISO: track 50.7 -> 49.4 mm
- net /CAN_INT: track 78.0 -> 76.9 mm
- net /RADIO_DIO1: track 24.3 -> 23.6 mm
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Other:
- board size 81.2 x 77.5 mm -> 81.2 x 82.6 mm
