File: Boards/Rocket Systems/GNC/GNC_Board/GNC_Board.kicad_sch (KiCad schematic)
At the start: 0 parts

Commit message: Add files via upload
Parts:
- added C1, C10, C6, C7, C8: 100n, symbol Device:C
- added C2: 120n, symbol Device:C
- added C3, C4: 22p, symbol Device:C
- added C5, C9: 1u, symbol Device:C
- added R1, R2, R3, R4, R5: 10k, symbol Device:R
- added SW1: SW_SPDT, symbol Switch:SW_SPDT
- added U1: BNO055, Package_LGA:LGA-28_5.2x3.8mm_P0.5mm, symbol Sensor_Motion:BNO055
- added U2: BMP280, Package_LGA:Bosch_LGA-8_2x2.5mm_P0.65mm_ClockwisePinNumbering, symbol Sensor_Pressure:BMP280
- added U3: LIS3MDL, Package_LGA:LGA-12_2x2mm_P0.5mm, symbol Sensor_Magnetic:LIS3MDL
- added U4: BMP388, QFN_BMP388_BOS, symbol BMP388:BMP388
- added U5: LIS3MDL, LGA-12_2X2X1_STM, symbol LIS3MDL:LIS3MDL
- added Y1: 32.768KHz, symbol Device:Crystal
Connections:
- new net: C4.1, U1.26 (XOUT32), Y1.2
- new net: C3.1, U1.27 (XIN32), Y1.1
- new net: C5.2, U1.9 (CAP)
- new net: C10.1, U3.4 (C1)
- new net: R5.2, SW1.1 (A)
- new net +3.3V: C1.1, C2.1, C6.1, C7.1, C8.1, C9.1, R1.1, R2.1, R3.1, R4.1, R5.1, U1.28 (VDDIO), U2.2 (CSB), U2.5 (SDO), U2.6 (VDDIO), U2.8 (VDD), U3.10 (~{CS}), U3.5 (Vdd), U3.6 (Vdd_IO), U3.9 (SDO/SA1)
- new net GND: C1.2, C10.2, C2.2, C3.2, C4.2, C5.1, C6.2, C7.2, C8.2, C9.2, SW1.3 (C), U1.18 (COM2), U1.2 (GND), U1.25 (GNDIO), U1.5 (PS1), U1.6 (PS0), U2.1 (GND), U2.7 (GND), U3.12 (GND), U3.2 (GND), U3.3 (GND)
- new net Interrupt output: U1.14 (INT)
- new net I²C_ADDR_SEL: U1.17 (COM3)
- new net NReset: R1.2, U1.11 (~{RESET})
- new net SCL: R4.2, U1.19 (COM1), U2.4 (SCK), U3.1 (SCL/SPC)
- new net SDA: R3.2, U1.20 (COM0), U2.3 (SDI), U3.11 (SDA/SDI/SDO)
- new net bootloader indicator: U1.10 (BL_IND)
- new net nBoot_load: R2.2, SW1.2 (B), U1.4 (~{BOOT_LOAD_PIN})
- no-connect marks 0 -> 4
Other:
- note added: "BMP280 1st Barometer"
- note added: "BMP280 2nd Barometer"
- note added: "GNC Board"
- note added: "LIS3MDL 3rd Barometer"
- note added: "LIS3MDL Magnometer"
- note added: "Nbootloader"
- note added: "Porto Space Team"
- note added: "Rafael Netto"
