File: Boards/Breakout Boards/STM32G4 Breakout Board/stm32g474ce_mcu/stm32g474ce_mcu.kicad_pcb (KiCad board)
At the start: 2 copper layers, 39 parts, among them J2 Conn_01x04_Pin, J3 DX07S016JA1R1500, SW1 RESET, SW2 SW_SPDT, U1 STM32G473CEUx, U2 MCP2562FDT, U3 MCP2562FDT, U4 AMS1117-3.3, U5 AMS1117-5.0, Y1 8MHz, Y2 3.768k

Commit message: j
Parts:
- removed Y1: 8MHz, KiCad:ABLS
- added Y3: 8Mhz, Crystal:Crystal_SMD_0603-2Pin_6.0x3.5mm_HandSoldering, F.Cu at (110.7, 64.6)
- C11, C12: value 9u -> 9p
- moved SW1 153.8 mm to (103.3, 80.0), turned to -90 degrees
- moved C15 147.6 mm to (98.5, 82.2), turned to -90 degrees
- moved C17 67.3 mm to (102.6, 23.6), turned to 90 degrees
- moved U1 64.4 mm to (104.7, 51.6), turned to 90 degrees
- moved C16 59.7 mm to (97.4, 23.4), turned to 90 degrees
- moved C5 58.0 mm to (98.8, 55.4), turned to -90 degrees
- moved C18 56.5 mm to (109.1, 73.5), turned to -90 degrees
- moved C1 52.6 mm to (98.4, 45.3)
- moved C4 51.8 mm to (98.8, 50.1), turned to -90 degrees
- moved U2 50.9 mm to (103.8, 73.5), turned to 180 degrees
- moved U3 48.3 mm to (100.6, 18.2), turned to 180 degrees
- moved C19 48.1 mm to (98.5, 76.9), turned to 90 degrees
- moved C2 46.4 mm to (104.3, 45.1)
- moved C3 41.5 mm to (110.1, 54.0), turned to 90 degrees
- moved R2 38.9 mm to (100.0, 23.6), turned to 90 degrees
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Connections:
- net /LSE clock renamed /OSC32_IN
- net Net-(U1-PC15) renamed /OSC32_OUT
- net Net-(U1-PF0) renamed /OSC_IN
- net Net-(U1-PF1) renamed /OSC_OUT
Routing:
- net GND: track 10.2 -> 0.00 mm, vias 7 -> 0
- net +5V: track 6.41 -> 0.00 mm
- net +3.3V: track 3.82 -> 0.00 mm
- net VBUS: track 2.75 -> 0.00 mm
Other:
- board text added: "BOOT0"
- board text added: "RESET"
