File: Boards/Breakout Boards/E28-2G4M27SX DEV BOARD/Radio_dev_board/Radio_dev_board.kicad_pcb (KiCad board)
At the start: 2 copper layers, 27 x 28.3 mm, 5 parts, among them J1 Conn_01x08_Pin, J2 Conn_01x08_Pin, U1 E28-2G4M27SX

Commit message: changes
Other:
- board text added: "BUSY"
- board text added: "DIO1"
- board text added: "DIO2"
- board text added: "DIO3"
- board text added: "GND"
- board text added: "MISO"
- board text added: "MOSI"
- board text added: "NRESET"
- board text added: "NSS"
- board text added: "RX_EN"
- board text added: "SCK"
- board text added: "TX_EN"
- board text added: "VCC"
