File: Boards/GSat/GSat board/GSat board.kicad_pcb (KiCad board)
At the start: 2 copper layers, 110 x 70 mm, 23 parts, among them IC1 NEO-M8Q-0, J2 PCB.RPSMAFRA.HT, U1 TMC2209_SILENTSTEPSTICK, U12 MMBT3906-7-F, U2 TMC2209_SILENTSTEPSTICK

Commit message: small update GSat
Parts:
- added U3: E28-2G4M27SX, Radio_Module_PST:Radio_Module_PST, F.Cu at (124.2, 76.8)
- added U4: E28-2G4M27SX, Radio_Module_PST:Radio_Module_PST, F.Cu at (124.2, 108.5)
Connections:
- A1 pad 11: unconnected-(A1-GPIO8-Pad11) -> /LimitSwitch1
- A1 pad 12: unconnected-(A1-GPIO9-Pad12) -> /LimitSwitch2
- A1 pad 14: unconnected-(A1-GPIO10-Pad14) -> /LimitSwitch3
- U1 pad 14: unconnected-(U1-MS2-Pad14) -> +3.3V
- U1 pad 15: unconnected-(U1-MS1-Pad15) -> +3.3V
- U2 pad 14: unconnected-(U2-MS2-Pad14) -> +3.3V
- U2 pad 15: unconnected-(U2-MS1-Pad15) -> +3.3V

Commit message: GSAT (Squematic update)
Parts:
- removed BT1: BAT-HLD-012-SMT-TR, BAT_HLD_012:BAT_BAT-HLD-012-SMT-TR
- removed C1: 4.7u, Capacitor-0402:Capacitor_0402
- removed C2, C3: 100n, Capacitor-0402:Capacitor_0402
- removed CR3: VLMC3100-GS08, LED-Green_VLMC3100-GS08:LED_PLCC_VSMB
- removed D2: PMEG2010ER, Diode-Schottky_PMEG2010ER:SODFL3517X110N
- removed FL1: FTCap0603, FTCap_0603:FTCap_0603
- removed J2: PCB.RPSMAFRA.HT, PCB.RPSMAFRA.HT:PCBRPSMAFRAHT
- removed JP1, JP2: Jumper_2_Open, Jumper:SolderJumper-2_P1.3mm_Open_RoundedPad1.0x1.5mm
- removed L1: 27n, Inductor-0402:Inductor_0402
- removed R10: 10k, Resistor-0402:RES_0402
- removed R5: 10, Resistor-0402:RES_0402
- removed R7: 150, Resistor-0603:RES_0603
- removed U12: MMBT3906-7-F, MMBT3906-7-F:SOT103P240X110-3N
- added C37: 4.7uF, Capacitor-0402:Capacitor_0402, F.Cu at (116.1, 84.2)
- added C39: 4.7uF, Capacitor-0402:Capacitor_0402, F.Cu at (116.1, 86.3)
- added C40: 1uF, Capacitor-0402:Capacitor_0402, F.Cu at (116.1, 88.5)
- added IC2: MCP23017-E_SP, MCP23017:DIP794W56P254L3486H508Q28N, F.Cu at (70.1, 97.3)
- added J10: Conn_01x05_Pin, Connector_PinSocket_2.54mm:PinSocket_1x05_P2.54mm_Vertical, F.Cu at (112.0, 102.9)
- added J11: Conn_01x06_Pin, Connector_PinSocket_2.54mm:PinSocket_1x06_P2.54mm_Vertical, F.Cu at (107.4, 102.9)
- added R1: 1K, Resistor_SMD:R_0603_1608Metric_Pad0.98x0.95mm_HandSolder, F.Cu at (112.5, 92.2)
- added R11: 10k, Resistor-0402:RES_0402, F.Cu at (115.9, 106.0)
- added R12: 10k, Resistor-0402:RES_0402, F.Cu at (115.9, 108.2)
- added R13: 10k, Resistor-0402:RES_0402, F.Cu at (115.9, 110.3)
- added R14: 10k, Resistor-0402:RES_0402, F.Cu at (115.9, 112.5)
- added R2: 10K, Resistor_SMD:R_0603_1608Metric_Pad0.98x0.95mm_HandSolder, F.Cu at (112.5, 94.7)
- added R3: 10K, Resistor_SMD:R_0603_1608Metric_Pad0.98x0.95mm_HandSolder, F.Cu at (112.5, 97.2)
- added TP1: TestPoint, TestPoint:TestPoint_Pad_2.0x2.0mm, F.Cu at (112.4, 80.8)
- added TP2: TestPoint, TestPoint:TestPoint_Pad_2.0x2.0mm, F.Cu at (112.4, 84.8)
- added TP7: TestPoint, TestPoint:TestPoint_Pad_2.0x2.0mm, F.Cu at (112.4, 88.9)
- added U10: ST1L05APU33R, LDO ST1L05A:DFN_5APU33R_STM, F.Cu at (117.4, 93.3)
- added U5: MAX485_MODULE_5V_LOGIC_TLL_TO_RS-485_CONVERTER, MAX485Module:MODULE_MAX485_MODULE_5V_LOGIC_TLL_TO_RS-485_CONVERTER, F.Cu at (87.9, 71.0)
- added U6: ~, DCDCModule:DCDC_Module, F.Cu at (90.9, 110.8)
- IC1: value NEO-M8Q-0 -> LTC4418IUF#PBF; footprint NEO-M8Q-0:NEO-M8_UBL -> LTC4418:QFN50P400X400X80-21N-D
- moved U4 62.7 mm to (106.6, 48.4)
- moved U3 53.8 mm to (78.6, 48.4)
- moved C4 38.8 mm to (116.1, 79.8)
- moved C5 38.8 mm to (116.1, 82.0)
- moved IC1 33.0 mm to (112.8, 118.5)
- moved U2 29.9 mm to (101.9, 89.7), turned to 0 degrees
- moved R6 22.5 mm to (115.9, 101.7)
- moved R8 22.5 mm to (115.9, 103.9)
- moved U1 21.5 mm to (84.6, 89.7), turned to 0 degrees
- moved A1 9.25 mm to (52.5, 82.0)
Connections:
- A1 pad 1: unconnected-(A1-GPIO0-Pad1) -> /GPS RX UART
- A1 pad 10: unconnected-(A1-GPIO7-Pad10) -> /I2C#2 SCL
- A1 pad 11: /LimitSwitch1 -> /RS_TX
- A1 pad 12: /LimitSwitch2 -> /RS_RX
- A1 pad 14: /LimitSwitch3 -> /UNI_BUSY
- A1 pad 15: unconnected-(A1-GPIO11-Pad15) -> /UNI_DIO1
- A1 pad 16: unconnected-(A1-GPIO12-Pad16) -> /MSD MISO
- A1 pad 17: unconnected-(A1-GPIO13-Pad17) -> /CS_MSD
- A1 pad 19: unconnected-(A1-GPIO14-Pad19) -> /MSD CLK
- A1 pad 2: unconnected-(A1-GPIO1-Pad2) -> /GPS TX UART
- A1 pad 20: unconnected-(A1-GPIO15-Pad20) -> /MSD MOSI
- A1 pad 21: unconnected-(A1-GPIO16-Pad21) -> /RADIO MISO
- A1 pad 22: /Driver1 Dir -> /CS_OMNI
- A1 pad 24: /Driver1 Step -> /RADIO CLK
- A1 pad 25: /Driver2 Dir -> /RADIO MOSI
- A1 pad 26: /Driver2 Step -> /CS_UNI
- A1 pad 27: unconnected-(A1-GPIO21-Pad27) -> /OMNI_BUSY
- A1 pad 29: unconnected-(A1-GPIO22-Pad29) -> /OMNI_DIO1
- A1 pad 34: unconnected-(A1-GPIO28_ADC2-Pad34) -> /GPS PPS
- A1 pad 35: unconnected-(A1-ADC_VREF-Pad35) -> GND
- A1 pad 4: unconnected-(A1-GPIO2-Pad4) -> /Driver1 Step
- A1 pad 5: unconnected-(A1-GPIO3-Pad5) -> /Driver2 Step
- A1 pad 6: /GPS TX UART -> /I2C#1 SDA
- A1 pad 7: /GPS RX UART -> /I2C#1 SCL
- A1 pad 9: /GPS ~{BOOT} -> /I2C#2 SDA
- IC1 pad 10: GND -> unconnected-(IC1-INTVCC-Pad10)
- IC1 pad 11: /RF -> unconnected-(IC1-G2-Pad11)
- IC1 pad 12: GND -> unconnected-(IC1-VS2-Pad12)
- IC1 pad 13: GND -> unconnected-(IC1-G1-Pad13)
- IC1 pad 20: /GPS TX UART -> unconnected-(IC1-HYS-Pad20)
- IC1 pad 21: /GPS RX UART -> unconnected-(IC1-GND_2-Pad21)
- IC1 pad 3: Net-(IC1-TIMEPULSE) -> unconnected-(IC1-OV1-Pad3)
- IC1 pad 4: /INT GPS -> unconnected-(IC1-UV2-Pad4)
- IC1 pad 7: GND -> unconnected-(IC1-~{VALID2}-Pad7)
- IC1 pad 8: /GPS ~{BOOT} -> unconnected-(IC1-GND_1-Pad8)
- IC1 pad 9: Net-(IC1-VCC_RF) -> unconnected-(IC1-CAS-Pad9)
- U1 pad 14: +3.3V -> /Driver1 MS2
- U1 pad 15: +3.3V -> /Driver1 MS1
- U2 pad 14: +3.3V -> /Driver2 MS2
- U2 pad 15: +3.3V -> /Driver2 MS1
- U3 pad 10: unconnected-(U3-GND-Pad10) -> GND
- U3 pad 11: unconnected-(U3-NRESET-Pad11) -> /UNI_NRESET
- U3 pad 12: unconnected-(U3-BUSY-Pad12) -> /UNI_BUSY
- U3 pad 13: unconnected-(U3-DIO1-Pad13) -> /UNI_DIO1
- U3 pad 16: unconnected-(U3-GND-Pad16) -> GND
- U3 pad 3: /MISO -> /RADIO MISO
- U3 pad 4: /MOSI -> /RADIO MOSI
- U3 pad 5: /CLK -> /RADIO CLK
- U3 pad 6: /CS -> /CS_UNI
- U3 pad 8: /ANT_RX_EN -> /UNI_RX_EN
- U3 pad 9: unconnected-(U3-TX_EN-Pad9) -> /UNI_TX_EN
- U4 pad 10: unconnected-(U4-GND-Pad10) -> GND
- U4 pad 11: unconnected-(U4-NRESET-Pad11) -> /OMNI_NRESET
- U4 pad 12: unconnected-(U4-BUSY-Pad12) -> /OMNI_BUSY
- U4 pad 13: unconnected-(U4-DIO1-Pad13) -> /OMNI_DIO1
- U4 pad 16: unconnected-(U4-GND-Pad16) -> GND
- U4 pad 3: /MISO -> /RADIO MISO
- U4 pad 4: /MOSI -> /RADIO MOSI
- U4 pad 5: /CLK -> /RADIO CLK
- U4 pad 6: /CS -> /CS_OMNI
- U4 pad 8: /ANT_RX_EN -> /OMNI_RX_EN
- U4 pad 9: unconnected-(U4-TX_EN-Pad9) -> /OMNI_TX_EN
Other:
- board outline removed

Commit message: GSAT update
Parts:
- removed TP1, TP7: TestPoint, TestPoint:TestPoint_Pad_2.0x2.0mm
- added C41: 1nF, Capacitor-0402:Capacitor_0402, F.Cu at (224.0, 90.7)
- added C42: 100nF, Capacitor-0402:Capacitor_0402, F.Cu at (232.0, 87.7)
- added C43: 100nF, Capacitor-0402:Capacitor_0402, F.Cu at (223.5, 87.1)
- added C44: 100nF, Capacitor-0402:Capacitor_0402, F.Cu at (223.5, 88.4)
- added C45: 100nF, Capacitor-0402:Capacitor_0402, F.Cu at (229.3, 85.1)
- added C46: 100nF, Capacitor-0402:Capacitor_0402, F.Cu at (226.8, 85.1)
- added C47: 220uF, Capacitor-0402:Capacitor_0402, F.Cu at (224.2, 85.1)
- added D1: SMBJ24CA, SMBJ24CA:DIOM5436X244N, F.Cu at (214.1, 87.4)
- added D2: SMBJ24CA, SMBJ24CA:DIOM5436X244N, F.Cu at (231.8, 100.5)
- added F1: 0ABB-6000-TM, 0ABB-6000-TM:0ABB6000TM, F.Cu at (213.7, 92.8)
- added F2: 0ABB-6000-TM, 0ABB-6000-TM:0ABB6000TM, F.Cu at (226.9, 98.5)
- added J12: XT30UPB-F, XT30UPB-F:XT30UPBF, F.Cu at (216.2, 98.5)
- added J2: XT30UPB-F, XT30UPB-F:XT30UPBF, F.Cu at (202.8, 92.8)
- added Q1: PMOS, Package_TO_SOT_SMD:TO-252-3_TabPin2, F.Cu at (221.5, 80.6)
- added Q2: PMOS, Package_TO_SOT_SMD:TO-252-3_TabPin2, F.Cu at (223.2, 72.6)
- added Q3: PMOS, Package_TO_SOT_SMD:TO-252-3_TabPin2, F.Cu at (235.4, 80.6)
- added Q4: PMOS, Package_TO_SOT_SMD:TO-252-3_TabPin2, F.Cu at (233.8, 72.6)
- added R10: 9.31K, Resistor_SMD:R_0603_1608Metric_Pad0.98x0.95mm_HandSolder, F.Cu at (230.3, 94.3)
- added R15: 39.6K, Resistor_SMD:R_0603_1608Metric_Pad0.98x0.95mm_HandSolder, F.Cu at (233.0, 93.4)
- added R4: 1M, Resistor_SMD:R_0603_1608Metric_Pad0.98x0.95mm_HandSolder, F.Cu at (223.3, 92.5)
- added R5: 9.31K, Resistor_SMD:R_0603_1608Metric_Pad0.98x0.95mm_HandSolder, F.Cu at (226.8, 92.5)
- added R7: 39.6K, Resistor_SMD:R_0603_1608Metric_Pad0.98x0.95mm_HandSolder, F.Cu at (230.3, 92.5)
- added R9: 1M, Resistor_SMD:R_0603_1608Metric_Pad0.98x0.95mm_HandSolder, F.Cu at (227.8, 95.2)
- added TP3: TestPoint, TestPoint:TestPoint_Pad_2.0x2.0mm, F.Cu at (219.5, 87.2)
- added TP4: TestPoint, TestPoint:TestPoint_Pad_2.0x2.0mm, F.Cu at (236.8, 93.0)
- added TP5: TestPoint, TestPoint:TestPoint_Pad_2.0x2.0mm, F.Cu at (228.5, 67.5)
- moved A1 170.3 mm to (215.1, 132.4), turned to 180 degrees
- moved J11 144.3 mm to (251.5, 109.9)
- moved J10 143.8 mm to (252.0, 135.6)
- moved U5 119.7 mm to (194.0, 126.2), turned to -90 degrees
- moved IC1 119.1 mm to (228.0, 88.6), turned to 90 degrees
- moved TP2 89.7 mm to (29.2, 118.6)
- moved U10 81.5 mm to (44.9, 130.6)
- moved C37 47.0 mm to (105.0, 129.8)
- moved C39 47.0 mm to (105.0, 132.0)
- moved C4 47.0 mm to (105.0, 125.5)
- moved C5 47.0 mm to (105.0, 127.7)
- moved R1 44.3 mm to (115.7, 48.0)
- moved R2 44.3 mm to (115.7, 50.5)
- moved R3 44.3 mm to (115.7, 53.0)
- moved C40 37.8 mm to (108.3, 125.5)
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Connections:
- IC1 pad 1: unconnected-(IC1-TMR-Pad1) -> Net-(IC1-TMR)
- IC1 pad 10: unconnected-(IC1-INTVCC-Pad10) -> /LTC441_EN
- IC1 pad 11: unconnected-(IC1-G2-Pad11) -> Net-(IC1-G2)
- IC1 pad 12: unconnected-(IC1-VS2-Pad12) -> Net-(IC1-VS2)
- IC1 pad 13: unconnected-(IC1-G1-Pad13) -> Net-(IC1-G1)
- IC1 pad 14: unconnected-(IC1-VS1-Pad14) -> Net-(IC1-VS1)
- IC1 pad 15: unconnected-(IC1-VOUT-Pad15) -> +24V
- IC1 pad 16: unconnected-(IC1-V2-Pad16) -> /VBAT
- IC1 pad 17: unconnected-(IC1-V1-Pad17) -> /VMAIN
- IC1 pad 18: unconnected-(IC1-EN-Pad18) -> /LTC441_EN
- IC1 pad 19: unconnected-(IC1-~{SHDN}-Pad19) -> /LTC441_EN
- IC1 pad 2: unconnected-(IC1-UV1-Pad2) -> Net-(IC1-UV1)
- IC1 pad 20: unconnected-(IC1-HYS-Pad20) -> GND
- IC1 pad 21: unconnected-(IC1-GND_2-Pad21) -> GND
- IC1 pad 3: unconnected-(IC1-OV1-Pad3) -> Net-(IC1-OV1)
- IC1 pad 4: unconnected-(IC1-UV2-Pad4) -> Net-(IC1-UV2)
- IC1 pad 5: unconnected-(IC1-OV2-Pad5) -> Net-(IC1-OV2)
- IC1 pad 8: unconnected-(IC1-GND_1-Pad8) -> GND
- U1 pad 8: VExt -> +24V
- U2 pad 8: VExt -> +24V
Routing:
- net /GPS PPS: track 0.00 -> 58.4 mm
- net /VBAT: track 0.00 -> 44.6 mm, vias 0 -> 3
- net /VMAIN: track 0.00 -> 41.4 mm, vias 0 -> 2
- net /CS_MSD: track 0.00 -> 40.7 mm
- net +24V: track 0.00 -> 37.2 mm, vias 0 -> 4
- net /GPS TX UART: track 0.00 -> 33.5 mm
- net /GPS RX UART: track 0.00 -> 32.7 mm
- net /MSD MOSI: track 0.00 -> 30.3 mm
- net /MSD CLK: track 0.00 -> 29.5 mm
- net /MSD MISO: track 0.00 -> 27.4 mm
- net Net-(IC1-VS2): track 0.00 -> 26.0 mm
- net Net-(IC1-G1): track 0.00 -> 25.3 mm
- net Net-(IC1-G2): track 0.00 -> 20.9 mm
- net Net-(IC1-VS1): track 0.00 -> 20.5 mm
- net Net-(IC1-OV2): track 0.00 -> 10.5 mm
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Other:
- board outline added: 100 x 140 mm
- board text added: "100x140 Limite"
- board text added: "Con MOTORES, para cima preferencial"
- board text added: "DOIS LIMIT SWITCHES"
- board text added: "Power e Comms no meio preferencialmente"
- board text added: "SD e GPS"
- board text added: "UM LIMIT Encoder Magnet coder"

Commit message: GSPOT update
mais algum routing feito
Parts:
- added J13: B4B-XH-A_LF__SN_, B4B-XH-A_LF__SN_:B4BXHALFSN, F.Cu at (170.2, 82.2)
- added J14: B4B-XH-A_LF__SN_, B4B-XH-A_LF__SN_:B4BXHALFSN, F.Cu at (170.3, 59.1)
- added J15: B4B-XH-A_LF__SN_, B4B-XH-A_LF__SN_:B4BXHALFSN, F.Cu at (176.2, 147.8)
- added J16: B4B-XH-A_LF__SN_, B4B-XH-A_LF__SN_:B4BXHALFSN, F.Cu at (176.2, 132.0)
- moved TP2 215.9 mm to (231.5, 43.3), turned to 90 degrees
- moved U10 208.7 mm to (232.0, 38.0), turned to 90 degrees
- moved U6 184.3 mm to (243.3, 54.3), turned to 90 degrees
- moved C37 158.5 mm to (234.8, 38.9), turned to -90 degrees
- moved C39 155.6 mm to (231.2, 41.1)
- moved C40 154.6 mm to (236.3, 38.8), turned to -90 degrees
- moved U3 147.2 mm to (213.8, 76.7)
- moved R1 146.0 mm to (220.8, 149.5), turned to -90 degrees
- moved IC2 139.8 mm to (235.0, 136.4)
- moved U1 120.9 mm to (185.8, 83.8)
- moved U4 115.1 mm to (213.8, 47.4)
- moved U2 110.3 mm to (185.7, 60.6)
- moved C5 104.4 mm to (193.4, 72.2)
- moved C4 89.1 mm to (190.0, 98.9), turned to -90 degrees
- moved R8 77.0 mm to (190.7, 72.2)
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Connections:
- U6 pad 1: VDC -> +24V
Routing:
- net /Driver2 Step: track 0.00 -> 110.2 mm, vias 0 -> 3
- net /I2C#1 SDA: track 0.00 -> 93.6 mm, vias 0 -> 3
- net /I2C#1 SCL: track 0.00 -> 93.5 mm, vias 0 -> 2
- net /Driver1 Step: track 0.00 -> 89.4 mm, vias 0 -> 2
- net /UNI_DIO1: track 0.00 -> 61.0 mm, vias 0 -> 2
- net /UNI_BUSY: track 0.00 -> 60.9 mm, vias 0 -> 2
- net /Driver2 Dir: track 0.00 -> 44.0 mm, vias 0 -> 1
- net /I2C#2 SDA: track 0.00 -> 36.9 mm
- net /I2C#2 SCL: track 0.00 -> 36.9 mm
- net /RS_ENABLE: track 0.00 -> 34.5 mm, vias 0 -> 1
- net /Driver2 MS2: track 0.00 -> 32.0 mm, vias 0 -> 1
- net /Driver2 MS1: track 0.00 -> 29.8 mm, vias 0 -> 1
- net /RS_TX: track 0.00 -> 29.7 mm, vias 0 -> 1
- net /RS_RX: track 0.00 -> 23.6 mm, vias 0 -> 1
- net /Driver1 Dir: track 0.00 -> 22.2 mm, vias 0 -> 1
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
Commit message: GSPOT
Parts:
- removed TP5: TestPoint, TestPoint:TestPoint_Pad_2.0x2.0mm
- added J1: B3B-XH-A_LF__SN_, B3B-XH-A_LF__SN:B3BXHALFSN, F.Cu at (176.2, 115.8)
- added J3: B3B-XH-A_LF__SN_, B3B-XH-A_LF__SN:B3BXHALFSN, F.Cu at (175.8, 39.8)
- added J4: B3B-XH-A_LF__SN_, B3B-XH-A_LF__SN:B3BXHALFSN, F.Cu at (189.2, 39.8)
- moved R14 145.5 mm to (241.7, 145.2), turned to 180 degrees
- moved R2 93.8 mm to (228.2, 74.8), turned to 90 degrees
- moved R3 89.8 mm to (229.2, 48.2), turned to 90 degrees
- moved R11 87.0 mm to (181.5, 114.2), turned to -90 degrees
- moved R13 57.9 mm to (190.7, 44.0), turned to 180 degrees
- moved R12 44.1 mm to (177.0, 44.0), turned to 180 degrees
- moved C39 2.70 mm to (232.4, 43.5), turned to 180 degrees
- moved U10 2.58 mm to (232.7, 40.5)
- moved U6 2.58 mm to (244.0, 56.8)
- moved C37 2.58 mm to (235.4, 41.4)
- moved C40 2.58 mm to (236.9, 41.3)
- moved TP2 2.58 mm to (232.2, 45.8)
- moved R1 2.03 mm to (220.8, 151.5)
- moved U5 2.03 mm to (220.8, 127.4)
- moved J13 1.50 mm to (171.8, 82.2)
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Connections:
- A1 pad 33: unconnected-(A1-AGND-Pad33) -> GND
- C39 pad 2: +3.3V -> +3.3V IC
- TP2 pad 1: +3.3V -> +3.3V IC
- U1 pad 16: +3.3V -> +3.3V IC
- U1 pad 2: +3.3V -> +3.3V IC
- U10 pad 2: +3.3V -> +3.3V IC
- U2 pad 16: +3.3V -> +3.3V IC
- U2 pad 2: +3.3V -> +3.3V IC
Routing:
- net /CS_MSD: track 51.3 -> 43.5 mm
- net +24V: track 37.2 -> 30.6 mm
- net /RS_TX: track 29.7 -> 31.7 mm
- net /RS_RX: track 23.6 -> 25.6 mm
- net Net-(U1-M1B): track 12.2 -> 10.3 mm
- net Net-(U2-M1B): track 12.1 -> 10.3 mm
- net Net-(U1-M2B): track 10.0 -> 8.55 mm
- net Net-(U1-M2A): track 9.27 -> 7.77 mm
- net Net-(U1-M1A): track 9.25 -> 7.75 mm
- net Net-(U2-M2A): track 9.17 -> 7.75 mm
- net Net-(U2-M2B): track 9.95 -> 8.53 mm
- net Net-(U2-M1A): track 9.15 -> 7.73 mm
- net /RS_ENABLE: track 34.5 -> 34.0 mm

Commit message: gsat
Parts:
- added IC3: SP3485CN-L_TR, SP3485CN-L_TR:SOIC127P600X175-8N, F.Cu at (309.9, 84.7)
- added R16: 4.7k, Resistor_SMD:R_0603_1608Metric_Pad0.98x0.95mm_HandSolder, F.Cu at (303.5, 82.8)
- added R17: 120, Resistor_SMD:R_0603_1608Metric_Pad0.98x0.95mm_HandSolder, F.Cu at (303.5, 85.3)
- added R18: 4.7k, Resistor_SMD:R_0603_1608Metric_Pad0.98x0.95mm_HandSolder, F.Cu at (303.5, 87.8)
