File: Boards/GSat/GSat board/GSat board.kicad_sch (KiCad schematic)
At the start: 30 parts, among them IC1 NEO-M8Q-0, J1 Conn_01x04_Pin, J2 PCB.RPSMAFRA.HT, J3 Conn_01x04_Pin, J4 Conn_01x04_Pin, J5 Conn_01x04_Pin, J6 Conn_01x03_Pin, J7 Conn_01x03_Pin, J8 Conn_01x03_Pin, U1 TMC2209_SILENTSTEPSTICK, U12 MMBT3906-7-F, U2 TMC2209_SILENTSTEPSTICK

Commit message: small update GSat
Parts:
- added R11, R12, R13: 10k, Resistor-0402:RES_0402, symbol Device:R
- added R2, R3: 10K, Resistor_SMD:R_0603_1608Metric_Pad0.98x0.95mm_HandSolder, symbol Device:R
- added U3, U4: E28-2G4M27SX, Radio_Module_PST:Radio_Module_PST, symbol E28-2G4M27S:E28-2G4M27SX
Connections:
- net +3.3V: now also J6.3 (Pin_3), J7.3 (Pin_3), J8.3 (Pin_3), U1.14 (MS2), U1.15 (MS1), U2.14 (MS2), U2.15 (MS1), R11.2, R12.2, R13.2, U3.1 (VCC), U4.1 (VCC)
- net Driver1 Dir: now also A1.27 (GPIO21); no longer A1.22 (GPIO17)
- net Driver1 Step: now also A1.29 (GPIO22); no longer A1.24 (GPIO18)
- net GND: now also A1.35 (ADC_VREF), R2.2, R3.2, U3.10 (GND), U3.16 (GND), U3.2 (GND), U3.7 (GND), U4.10 (GND), U4.16 (GND), U4.2 (GND), U4.7 (GND)
- net GPS ~{BOOT}: no longer A1.9 (GPIO6)
- net INT GPS: now also A1.9 (GPIO6)
- net LimitSwitch1: now also A1.1 (GPIO0), R11.1
- net LimitSwitch2: now also A1.2 (GPIO1), R12.1
- net LimitSwitch3: now also A1.4 (GPIO2), R13.1
- net OMNI_RX_EN: now reaches A1.10 (GPIO7)
- net OMNI_RX_EN: now also U4.8 (RX_EN)
- net OMNI_TX_EN: now reaches A1.11 (GPIO8)
- net OMNI_TX_EN: now also U4.9 (TX_EN)
- net CS_OMNI: now reaches A1.12 (GPIO9)
- net CS_OMNI: now also U4.6 (NSS_CTS)
- net CLK: now reaches A1.14 (GPIO10)
- net CLK: now also U3.5 (SCK_RTSN), U4.5 (SCK_RTSN)
- net MOSI: now reaches A1.15 (GPIO11)
- net MOSI: now also U3.4 (MOSI_RX), U4.4 (MOSI_RX)
- net MISO: now reaches A1.16 (GPIO12)
- net MISO: now also U3.3 (MISO_TX), U4.3 (MISO_TX)
- net CS_UNI: now reaches A1.17 (GPIO13)
- net CS_UNI: now also U3.6 (NSS_CTS)
- net OMNI_BUSY: now reaches A1.19 (GPIO14)
- net OMNI_BUSY: now also U4.12 (BUSY)
- net OMNI_DIO1: now reaches A1.20 (GPIO15)
- net OMNI_DIO1: now also R3.1, U4.13 (DIO1)
- net UNI_RX_EN: now reaches A1.21 (GPIO16)
- net UNI_RX_EN: now also U3.8 (RX_EN)
- net UNI_DIO1: now reaches A1.34 (GPIO28_ADC2)
- net UNI_DIO1: now also R2.1, U3.13 (DIO1)
- net NRESET: now reaches A1.5 (GPIO3)
- net NRESET: now also U3.11 (NRESET), U4.11 (NRESET)
- new net UNI_BUSY: A1.24 (GPIO18), U3.12 (BUSY)
- new net UNI_TX_EN: A1.22 (GPIO17), U3.9 (TX_EN)
Other:
- moved on the sheet: C4, J1, J4, J5, J6, J7, J8, R6, U1

Commit message: GSAT (Squematic update)
Parts:
- removed BT1: BAT-HLD-012-SMT-TR, BAT_HLD_012:BAT_BAT-HLD-012-SMT-TR, symbol BAT-HLD-012-SMT-TR:BAT-HLD-012-SMT-TR
- removed C1: 4.7u, Capacitor-0402:Capacitor_0402, symbol Device:C_Small
- removed C2, C3: 100n, Capacitor-0402:Capacitor_0402, symbol Device:C_Small
- removed CR3: VLMC3100-GS08, LED-Green_VLMC3100-GS08:LED_PLCC_VSMB, symbol GreenLED__VLMC3100-GS08:VLMC3100-GS08
- removed D2: PMEG2010ER, Diode-Schottky_PMEG2010ER:SODFL3517X110N, symbol PMEG2010ER:PMEG2010ER
- removed FL1: FTCap0603, FTCap_0603:FTCap_0603, symbol FTCap0603:FTCap0603
- removed IC1: NEO-M8Q-0, NEO-M8Q-0:NEO-M8_UBL, symbol NEO-M8Q-0:NEO-M8Q-0
- removed J2: PCB.RPSMAFRA.HT, PCB.RPSMAFRA.HT:PCBRPSMAFRAHT, symbol PCB_RPSMAFRA_HT:PCB.RPSMAFRA.HT
- removed JP1, JP2: Jumper_2_Open, Jumper:SolderJumper-2_P1.3mm_Open_RoundedPad1.0x1.5mm, symbol Jumper:Jumper_2_Open
- removed L1: 27n, Inductor-0402:Inductor_0402, symbol Device:L
- removed R10: 10k, Resistor-0402:RES_0402, symbol Device:R
- removed R5: 10, Resistor-0402:RES_0402, symbol Device:R
- removed R7: 150, Resistor-0603:RES_0603, symbol Device:R
- removed U12: MMBT3906-7-F, MMBT3906-7-F:SOT103P240X110-3N, symbol MMBT3906-7-F:MMBT3906-7-F
- added C37, C39: 4.7uF, Capacitor-0402:Capacitor_0402, symbol Device:C
- added C40: 1uF, Capacitor-0402:Capacitor_0402, symbol Device:C
- added IC1: LTC4418IUF#PBF, LTC4418:QFN50P400X400X80-21N-D, symbol LTC4418IUF#PBF:LTC4418IUF#PBF
- added IC2: MCP23017-E_SP, MCP23017:DIP794W56P254L3486H508Q28N, symbol MCP23017-E_SP:MCP23017-E_SP
- added J10: Conn_01x05_Pin, Connector_PinSocket_2.54mm:PinSocket_1x05_P2.54mm_Vertical, symbol Connector:Conn_01x05_Pin
- added J11: Conn_01x06_Pin, Connector_PinSocket_2.54mm:PinSocket_1x06_P2.54mm_Vertical, symbol Connector:Conn_01x06_Pin
- added J9: Conn_01x02_Pin, symbol Connector:Conn_01x02_Pin
- added R1: 1K, Resistor_SMD:R_0603_1608Metric_Pad0.98x0.95mm_HandSolder, symbol Device:R
- added R14: 10k, Resistor-0402:RES_0402, symbol Device:R
- added TP1, TP2, TP7: TestPoint, TestPoint:TestPoint_Pad_2.0x2.0mm, symbol Connector:TestPoint
- added U10: ST1L05APU33R, LDO ST1L05A:DFN_5APU33R_STM, symbol LDO_ST1L05A:ST1L05APU33R
- added U5: MAX485_MODULE_5V_LOGIC_TLL_TO_RS-485_CONVERTER, MAX485Module:MODULE_MAX485_MODULE_5V_LOGIC_TLL_TO_RS-485_CONVERTER, symbol MAX485_MODULE_5V_LOGIC_TLL_TO_RS-485_CONVERTER:MAX485_MODULE_5V_LOGIC_TLL_TO_RS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
- added U6: ~, DCDCModule:DCDC_Module, symbol Mini Dc-Dc:MiniDCDCBoost
Connections:
- net +3.3V: now also C39.2, IC2.9 (VDD), J10.1 (Pin_1), J11.1 (Pin_1), R14.1, TP2.1, U10.2 (V0); no longer U1.14 (MS2), U1.15 (MS1), U2.14 (MS2), U2.15 (MS1)
- net +5V: now also C37.2, C40.2, TP1.1, U10.3 (V1), U5.4 (VCC), U6.3 (OUT+)
- net CS_OMNI: now also A1.22 (GPIO17); no longer A1.12 (GPIO9)
- net CS_UNI: now also A1.26 (GPIO20); no longer A1.17 (GPIO13)
- net Driver1 Dir: now also IC2.24 (GPA3); no longer A1.27 (GPIO21)
- net Driver1 Step: now also A1.4 (GPIO2); no longer A1.29 (GPIO22)
- net Driver2 Dir: now also IC2.25 (GPA4); no longer A1.25 (GPIO19)
- net Driver2 Step: now also A1.5 (GPIO3); no longer A1.26 (GPIO20)
- net GND: now also C37.1, C39.1, C40.1, IC2.10 (VSS), IC2.15 (A0), IC2.16 (A1), IC2.17 (A2), J10.2 (Pin_2), J11.6 (Pin_6), R1.2, TP7.1, U10.6 (GND), U10.7 (GND), U5.1 (GND), U6.2 (IN-), U6.4 (OUT-)
- net GPS RX UART: now also A1.1 (GPIO0), J10.4 (Pin_4); no longer A1.7 (GPIO5)
- net GPS TX UART: now also A1.2 (GPIO1), J10.3 (Pin_3); no longer A1.6 (GPIO4)
- net LimitSwitch1: now also IC2.21 (GPA0); no longer A1.1 (GPIO0)
- net LimitSwitch2: now also IC2.22 (GPA1); no longer A1.2 (GPIO1)
- net LimitSwitch3: now also IC2.23 (GPA2); no longer A1.4 (GPIO2)
- net OMNI_BUSY: now also A1.27 (GPIO21); no longer A1.19 (GPIO14)
- net OMNI_DIO1: now also A1.29 (GPIO22); no longer A1.20 (GPIO15)
- net OMNI_RX_EN: now also IC2.27 (GPA6); no longer A1.10 (GPIO7)
- net OMNI_TX_EN: now also IC2.28 (GPA7); no longer A1.11 (GPIO8)
- net UNI_BUSY: now also A1.14 (GPIO10); no longer A1.24 (GPIO18)
- net UNI_DIO1: now also A1.15 (GPIO11); no longer A1.34 (GPIO28_ADC2)
- net UNI_RX_EN: now also IC2.2 (GPB1); no longer A1.21 (GPIO16)
- net UNI_TX_EN: now also IC2.3 (GPB2); no longer A1.22 (GPIO17)
- net CLK renamed RADIO CLK
- net RADIO CLK: now also A1.24 (GPIO18); no longer A1.14 (GPIO10)
- net I2C SCL renamed I2C#1 SCL
- net I2C#1 SCL: now also A1.7 (GPIO5), IC2.12 (SCL); no longer J5.2 (Pin_2)
- net I2C SDA renamed I2C#1 SDA
- net I2C#1 SDA: now also A1.6 (GPIO4), IC2.13 (SDA); no longer J5.3 (Pin_3)
- net INT GPS renamed I2C#2 SDA
- net I2C#2 SDA: now also J5.3 (Pin_3)
- net MISO renamed RADIO MISO
- net RADIO MISO: now also A1.21 (GPIO16); no longer A1.16 (GPIO12)
- net MOSI renamed RADIO MOSI
- net RADIO MOSI: now also A1.25 (GPIO19); no longer A1.15 (GPIO11)
- removed net NRESET: A1.5 (GPIO3), U3.11 (NRESET), U4.11 (NRESET)
- new net: J9.2 (Pin_2), U5.2 (A)
- new net: J9.1 (Pin_1), U5.3 (B)
- new net: IC2.18 (~{RESET}), R14.2
- new net CS_MSD: A1.17 (GPIO13), J11.2 (Pin_2)
- new net Driver1 MS1: IC2.5 (GPB4), U1.15 (MS1)
- new net Driver1 MS2: IC2.6 (GPB5), U1.14 (MS2)
- new net Driver2 MS1: IC2.7 (GPB6), U2.15 (MS1)
- new net Driver2 MS2: IC2.8 (GPB7), U2.14 (MS2)
- new net EXP INTERRUPT: IC2.20 (INTA)
- new net GPS PPS: A1.34 (GPIO28_ADC2), J10.5 (Pin_5)
- new net I2C#2 SCL: A1.10 (GPIO7), J5.2 (Pin_2)
- new net MSD CLK: A1.19 (GPIO14), J11.4 (Pin_4)
- new net MSD MISO: A1.16 (GPIO12), J11.5 (Pin_5)
- new net MSD MOSI: A1.20 (GPIO15), J11.3 (Pin_3)
- new net OMNI_NRESET: IC2.26 (GPA5), U4.11 (NRESET)
- new net RS_ENABLE: IC2.4 (GPB3), R1.1, U5.6 (RE), U5.7 (DE)
- new net RS_RX: A1.12 (GPIO9), U5.5 (RO)
- new net RS_TX: A1.11 (GPIO8), U5.8 (DI)
- new net UNI_NRESET: IC2.1 (GPB0), U3.11 (NRESET)
- new net VDC: U6.1 (IN+)
- no-connect marks 23 -> 14
Other:
- moved on the sheet: A1, C4, C5, J1, J3, J4, J5, R2, R3, R6, R8, U1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

Commit message: GSAT update
Parts:
- removed TP1, TP7: TestPoint, TestPoint:TestPoint_Pad_2.0x2.0mm, symbol Connector:TestPoint
- added C41: 1nF, Capacitor-0402:Capacitor_0402, symbol Device:C
- added C42, C43, C44, C45, C46: 100nF, Capacitor-0402:Capacitor_0402, symbol Device:C
- added C47: 220uF, Capacitor-0402:Capacitor_0402, symbol Device:C
- added D1, D2: SMBJ24CA, SMBJ24CA:DIOM5436X244N, symbol SMBJ24CA:SMBJ24CA
- added F1, F2: 0ABB-6000-TM, 0ABB-6000-TM:0ABB6000TM, symbol 0ABB-6000-TM:0ABB-6000-TM
- added J12, J2: XT30UPB-F, XT30UPB-F:XT30UPBF, symbol XT30UPB-F:XT30UPB-F
- added Q1, Q2, Q3, Q4: PMOS, Package_TO_SOT_SMD:TO-252-3_TabPin2, symbol Simulation_SPICE:PMOS
- added R10, R5: 9.31K, Resistor_SMD:R_0603_1608Metric_Pad0.98x0.95mm_HandSolder, symbol Device:R
- added R15, R7: 39.6K, Resistor_SMD:R_0603_1608Metric_Pad0.98x0.95mm_HandSolder, symbol Device:R
- added R4, R9: 1M, Resistor_SMD:R_0603_1608Metric_Pad0.98x0.95mm_HandSolder, symbol Device:R
- added TP3, TP4, TP5: TestPoint, TestPoint:TestPoint_Pad_2.0x2.0mm, symbol Connector:TestPoint
Connections:
- net VExt is gone; now on net +24V: U1.8 (VM), U2.8 (VM)
- net GND: now also IC1.20 (HYS), IC1.21 (GND_2), IC1.8 (GND_1), C41.1, C42.1, C43.2, C44.2, C45.1, C46.1, C47.1, D1.2, D2.2, J12.1, J2.1, R15.2, R7.2
- net at IC1.1 (TMR): now also C41.2
- net LTC441_EN: now reaches IC1.10 (INTVCC)
- net LTC441_EN: now also IC1.18 (EN), IC1.19 (~{SHDN}), C42.2
- net at IC1.11 (G2): now also Q3.1 (G), Q4.1 (G)
- net at IC1.12 (VS2): now also C45.2, Q3.3 (S), Q4.3 (S)
- net at IC1.13 (G1): now also Q1.1 (G), Q2.1 (G)
- net at IC1.14 (VS1): now also C46.2, Q1.3 (S), Q2.3 (S)
- net +24V: now reaches IC1.15 (VOUT)
- net +24V: now also C47.2, Q2.2 (D), Q4.2 (D), TP5.1
- net VBAT: now reaches IC1.16 (V2)
- net VBAT: now also C43.1, D2.1, F2.1, Q3.2 (D), R9.1, TP4.1
- net VMAIN: now reaches IC1.17 (V1)
- net VMAIN: now also C44.1, D1.1, F1.1, Q1.2 (D), R4.1, TP3.1
- net at IC1.2 (UV1): now also R4.2, R5.1
- net at IC1.3 (OV1): now also R5.2, R7.1
- net at IC1.4 (UV2): now also R10.1, R9.2
- net at IC1.5 (OV2): now also R10.2, R15.1
- new net: F2.2, J12.2
- new net: F1.2, J2.2
- no-connect marks 14 -> 17
Other:
- note added: "Conectores TODOS"
- note removed: "Power Options (Possibilidade dos 24V) Power Por Bateria ou Tomada Radio GSat-Rocket Com GSat-MissionControl (RS & Radio ???)"
- moved on the sheet: C37, C39, C40, J10, J11, J9, R1, R2, R3, TP2, U10, U3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

Commit message: GSPOT update
mais algum routing feito
Parts:
- removed J1, J3, J4, J5: Conn_01x04_Pin, symbol Connector:Conn_01x04_Pin
- added J13, J14, J15, J16: B4B-XH-A_LF__SN_, B4BXHALFSN, symbol B4B-XH-A_LF__SN_:B4B-XH-A_LF__SN_
Connections:
- net VDC is gone; now on net +24V: U6.1 (IN+)
- net +3.3V: now also J15.1, J16.1
- net GND: now also J15.4, J16.4
- net I2C#1 SCL: now also J15.3
- net I2C#1 SDA: now also J15.2
- net I2C#2 SCL: now also J16.3
- net I2C#2 SDA: now also J16.2
- net at U2.6 (M2B): now also J14.4
- net at U2.3 (M1B): now also J14.3
- net at U2.5 (M2A): now also J14.2
- net at U2.4 (M1A): now also J14.1
- net at U1.6 (M2B): now also J13.4
- net at U1.3 (M1B): now also J13.3
- net at U1.5 (M2A): now also J13.2
- net at U1.4 (M1A): now also J13.1
Other:
- moved on the sheet: C4, C5

Commit message: GSPOT
Parts:
- removed J6, J7, J8: Conn_01x03_Pin, symbol Connector:Conn_01x03_Pin
- removed TP5: TestPoint, TestPoint:TestPoint_Pad_2.0x2.0mm, symbol Connector:TestPoint
- added J1, J3, J4: B3B-XH-A_LF__SN_, B3BXHALFSN, symbol B3B-XH-A_LF__SN_:B3B-XH-A_LF__SN_
Connections:
- net +3.3V: now also J1.1, J3.1, J4.1; no longer C39.2, TP2.1, U1.16 (~{EN}), U1.2 (VIO), U10.2 (V0), U2.16 (~{EN}), U2.2 (VIO)
- net GND: now also A1.33 (AGND), J1.3, J3.3, J4.3
- net LimitSwitch1: now also J1.2
- net LimitSwitch2: now also J3.2
- net LimitSwitch3: now also J4.2
- new net +3.3V IC: C39.2, TP2.1, U1.16 (~{EN}), U1.2 (VIO), U10.2 (V0), U2.16 (~{EN}), U2.2 (VIO)
- no-connect marks 17 -> 22

Commit message: gsat
Parts:
- added IC3: SP3485CN-L_TR, SOIC127P600X175-8N, symbol SP3485CN-L_TR:SP3485CN-L_TR
- added R16, R18: 4.7k, Resistor_SMD:R_0603_1608Metric_Pad0.98x0.95mm_HandSolder, symbol Device:R_Small
- added R17: 120, Resistor_SMD:R_0603_1608Metric_Pad0.98x0.95mm_HandSolder, symbol Device:R_Small
- U6: value ~ -> (none)
Connections:
- net +3.3V: now also IC3.8 (VCC), R18.2
- net GND: now also IC3.5 (GND), R16.1
- net RS_ENABLE: now also IC3.2 (~{RE}), IC3.3 (DE)
- net RS_RX: now also IC3.1 (RO)
- net RS_TX: now also IC3.4 (DI)
- new net RS_A: IC3.6 (A), R17.2, R18.1
- new net RS_B: IC3.7 (B), R16.2, R17.1
Other:
- note added: "Lista de melhoramentos: -retirar o conectores todos -trocar footprints 0402 e 0603 para algo maior -separar o radio em dois canais de spi -mudar do max485 para o sp3485 -mudar ldo para o https://mauser.pt/001-9136/regulador-de-tensao-ld1117v33-3-3v-0-8a"
- moved on the sheet: J9, R1, U5
